File: HYDRA_VMM3_Adapter/TPC_Adapter.kicad_sch (KiCad schematic)
At the start: 1 part

Commit message: .
Connections:
- net Col_2-Row_1: now reaches U1.17 (Col_2-Row_1)
- net Col_2-Row_2: now reaches U1.18 (Col_2-Row_2)
- net Col_2-Row_3: now reaches U1.19 (Col_2-Row_3)
- net Col_3-Row_1: now reaches U1.33 (Col_3-Row_1)
- net Col_3-Row_2: now reaches U1.34 (Col_3-Row_2)
- net Col_3-Row_3: now reaches U1.35 (Col_3-Row_3)
- net Col_4-Row_1: now reaches U1.49 (Col_4-Row_1)
- net Col_4-Row_2: now reaches U1.50 (Col_4-Row_2)
- net Col_4-Row_3: now reaches U1.51 (Col_4-Row_3)
- net Col_5-Row_1: now reaches U1.65 (Col_5-Row_1)
- net Col_5-Row_2: now reaches U1.66 (Col_5-Row_2)
- net Col_5-Row_3: now reaches U1.67 (Col_5-Row_3)
- net Col_6-Row_1: now reaches U1.81 (Col_6-Row_1)
- net Col_6-Row_2: now reaches U1.82 (Col_6-Row_2)
- net Col_6-Row_3: now reaches U1.83 (Col_6-Row_3)
- net Col_7-Row_1: now reaches U1.97 (Col_7-Row_1)
- net Col_7-Row_2: now reaches U1.98 (Col_7-Row_2)
- net Col_7-Row_3: now reaches U1.99 (Col_7-Row_3)

Commit message: .
Connections:
- net Col_8-Row_1: now reaches U1.113 (Col_8-Row_1)
- net Col_8-Row_2: now reaches U1.114 (Col_8-Row_2)
- net Col_8-Row_3: now reaches U1.115 (Col_8-Row_3)
- net Col_9-Row_1: now reaches U1.129 (Col_9-Row_1)
- net Col_9-Row_2: now reaches U1.130 (Col_9-Row_2)
- net Col_9-Row_3: now reaches U1.131 (Col_9-Row_3)
- net Col_10-Row_1: now reaches U1.145 (Col_10-Row_1)
- net Col_10-Row_2: now reaches U1.146 (Col_10-Row_2)
- net Col_10-Row_3: now reaches U1.147 (Col_10-Row_3)
- net Col_11-Row_1: now reaches U1.161 (Col_11-Row_1)
- net Col_11-Row_2: now reaches U1.162 (Col_11-Row_2)
- net Col_11-Row_3: now reaches U1.163 (Col_11-Row_3)
- net Col_12-Row_1: now reaches U1.177 (Col_12-Row_1)
- net Col_12-Row_2: now reaches U1.178 (Col_12-Row_2)
- net Col_12-Row_3: now reaches U1.179 (Col_12-Row_3)
- net Col_13-Row_1: now reaches U1.193 (Col_13-Row_1)
- net Col_13-Row_2: now reaches U1.194 (Col_13-Row_2)
- net Col_13-Row_3: now reaches U1.195 (Col_13-Row_3)
- net Col_14-Row_1: now reaches U1.209 (Col_14-Row_1)
- net Col_14-Row_2: now reaches U1.210 (Col_14-Row_2)
- net Col_14-Row_3: now reaches U1.211 (Col_14-Row_3)
- net Col_15-Row_1: now reaches U1.225 (Col_15-Row_1)
- net Col_15-Row_2: now reaches U1.226 (Col_15-Row_2)
- net Col_15-Row_3: now reaches U1.227 (Col_15-Row_3)
- net Col_16-Row_1: now reaches U1.241 (Col_16-Row_1)
- net Col_16-Row_2: now reaches U1.242 (Col_16-Row_2)
- net Col_16-Row_3: now reaches U1.243 (Col_16-Row_3)
- net Col_17-Row_1: now reaches U1.257 (Col_17-Row_1)
- net Col_17-Row_2: now reaches U1.258 (Col_17-Row_2)
- net Col_17-Row_3: now reaches U1.259 (Col_17-Row_3)
- net Col_18-Row_1: now reaches U1.273 (Col_18-Row_1)
- net Col_18-Row_2: now reaches U1.274 (Col_18-Row_2)
- net Col_18-Row_3: now reaches U1.275 (Col_18-Row_3)
- net Col_19-Row_3: now reaches U1.289 (Col_19-Row_1)
- net Col_19-Row_2: now reaches U1.290 (Col_19-Row_2)
- net Col_19-Row_1: now reaches U1.291 (Col_19-Row_3)
- net Col_20-Row_1: now reaches U1.305 (Col_20-Row_1)
- net Col_20-Row_2: now reaches U1.306 (Col_20-Row_2)
- net Col_20-Row_3: now reaches U1.307 (Col_20-Row_3)
- net Col_21-Row_1: now reaches U1.321 (Col_21-Row_1)
- net Col_21-Row_2: now reaches U1.322 (Col_21-Row_2)
- net Col_21-Row_3: now reaches U1.323 (Col_21-Row_3)
- net Col_22-Row_1: now reaches U1.337 (Col_22-Row_1)
- net Col_22-Row_2: now reaches U1.338 (Col_22-Row_2)
- net Col_22-Row_3: now reaches U1.339 (Col_22-Row_3)
