File: HYDRA_VMM3_Adapter/_autosave-HYDRA_VMM3_Adapter.kicad_pcb (KiCad board)
At the start: 8 copper layers, 121.5 x 31.5 mm, 7 parts, among them J1 ME1014010101011, J2 ME1014010101011, J3 ME1014010101011, J4 ME1014010101011, J5 ME1014010101011, J6 ME1014010101011

Commit message: .
Connections:
- J4 pad B10: unconnected-(J4-PadB10) -> Col_2-Row_3
- J4 pad B11: unconnected-(J4-PadB11) -> Col_3-Row_1
- J4 pad B12: unconnected-(J4-PadB12) -> Col_3-Row_2
- J4 pad B13: unconnected-(J4-PadB13) -> Col_3-Row_3
- J4 pad B14: unconnected-(J4-PadB14) -> Col_4-Row_1
- J4 pad B15: Col_2-Row_1 -> Col_4-Row_2
- J4 pad B16: Col_2-Row_2 -> Col_4-Row_3
- J4 pad B17: Col_2-Row_3 -> Col_5-Row_1
- J4 pad B18: Col_3-Row_1 -> Col_5-Row_2
- J4 pad B19: Col_3-Row_2 -> Col_5-Row_3
- J4 pad B20: Col_3-Row_3 -> Col_6-Row_1
- J4 pad B21: Col_4-Row_1 -> Col_6-Row_2
- J4 pad B22: Col_4-Row_2 -> Col_6-Row_3
- J4 pad B23: Col_4-Row_3 -> Col_7-Row_1
- J4 pad B24: Col_5-Row_1 -> Col_7-Row_2
- J4 pad B25: Col_5-Row_2 -> Col_7-Row_3
- J4 pad B26: Col_5-Row_3 -> Col_8-Row_1
- J4 pad B27: Col_6-Row_1 -> Col_8-Row_2
- J4 pad B28: Col_6-Row_2 -> Col_8-Row_3
- J4 pad B29: Col_6-Row_3 -> Col_9-Row_1
- J4 pad B30: Col_7-Row_1 -> Col_9-Row_2
- J4 pad B31: Col_7-Row_2 -> Col_9-Row_3
- J4 pad B32: Col_7-Row_3 -> Col_10-Row_1
- J4 pad B33: Col_8-Row_1 -> Col_10-Row_2
- J4 pad B34: Col_8-Row_2 -> Col_10-Row_3
- J4 pad B35: Col_8-Row_3 -> Col_11-Row_1
- J4 pad B36: Col_9-Row_1 -> Col_11-Row_2
- J4 pad B37: Col_9-Row_2 -> Col_11-Row_3
- J4 pad B38: Col_9-Row_3 -> Col_12-Row_1
- J4 pad B39: unconnected-(J4-PadB39) -> Col_12-Row_2
- J4 pad B40: unconnected-(J4-PadB40) -> Col_12-Row_3
- J4 pad B41: unconnected-(J4-PadB41) -> Col_13-Row_1
- J4 pad B42: unconnected-(J4-PadB42) -> Col_13-Row_2
- J4 pad B43: unconnected-(J4-PadB43) -> Col_13-Row_3
- J4 pad B44: unconnected-(J4-PadB44) -> Col_14-Row_1
- J4 pad B45: unconnected-(J4-PadB45) -> Col_14-Row_2
- J4 pad B46: unconnected-(J4-PadB46) -> Col_14-Row_3
- J4 pad B47: unconnected-(J4-PadB47) -> Col_15-Row_1
- J4 pad B48: unconnected-(J4-PadB48) -> Col_15-Row_2
- J4 pad B49: unconnected-(J4-PadB49) -> Col_15-Row_3
- J4 pad B50: unconnected-(J4-PadB50) -> Col_16-Row_1
- J4 pad B51: unconnected-(J4-PadB51) -> Col_16-Row_2
- J4 pad B52: unconnected-(J4-PadB52) -> Col_16-Row_3
- J4 pad B53: unconnected-(J4-PadB53) -> Col_17-Row_1
- J4 pad B54: unconnected-(J4-PadB54) -> Col_17-Row_2
- J4 pad B55: unconnected-(J4-PadB55) -> Col_17-Row_3
- J4 pad B56: unconnected-(J4-PadB56) -> Col_18-Row_1
- J4 pad B57: unconnected-(J4-PadB57) -> Col_18-Row_2
- J4 pad B58: unconnected-(J4-PadB58) -> Col_18-Row_3
- J4 pad B59: unconnected-(J4-PadB59) -> Col_19-Row_1
- J4 pad B60: unconnected-(J4-PadB60) -> Col_19-Row_2
- J4 pad B61: unconnected-(J4-PadB61) -> Col_19-Row_3
- J4 pad B62: unconnected-(J4-PadB62) -> Col_20-Row_1
- J4 pad B63: unconnected-(J4-PadB63) -> Col_20-Row_2
- J4 pad B64: unconnected-(J4-PadB64) -> Col_20-Row_3
- J4 pad B65: unconnected-(J4-PadB65) -> Col_21-Row_1
- J4 pad B66: unconnected-(J4-PadB66) -> Col_21-Row_2
- J4 pad B67: unconnected-(J4-PadB67) -> Col_21-Row_3
- J4 pad B68: unconnected-(J4-PadB68) -> Col_22-Row_1
- J4 pad B69: unconnected-(J4-PadB69) -> Col_22-Row_2
- J4 pad B70: unconnected-(J4-PadB70) -> Col_22-Row_3
- J4 pad B8: unconnected-(J4-PadB8) -> Col_2-Row_1
- J4 pad B9: unconnected-(J4-PadB9) -> Col_2-Row_2
- U1 pad 145: unconnected-(U1-Col_10-Row_1-Pad145) -> Col_10-Row_1
- U1 pad 146: unconnected-(U1-Col_10-Row_2-Pad146) -> Col_10-Row_2
- U1 pad 147: unconnected-(U1-Col_10-Row_3-Pad147) -> Col_10-Row_3
- U1 pad 161: unconnected-(U1-Col_11-Row_1-Pad161) -> Col_11-Row_1
- U1 pad 162: unconnected-(U1-Col_11-Row_2-Pad162) -> Col_11-Row_2
- U1 pad 163: unconnected-(U1-Col_11-Row_3-Pad163) -> Col_11-Row_3
- U1 pad 177: unconnected-(U1-Col_12-Row_1-Pad177) -> Col_12-Row_1
- U1 pad 178: unconnected-(U1-Col_12-Row_2-Pad178) -> Col_12-Row_2
- U1 pad 179: unconnected-(U1-Col_12-Row_3-Pad179) -> Col_12-Row_3
- U1 pad 193: unconnected-(U1-Col_13-Row_1-Pad193) -> Col_13-Row_1
- U1 pad 194: unconnected-(U1-Col_13-Row_2-Pad194) -> Col_13-Row_2
- U1 pad 195: unconnected-(U1-Col_13-Row_3-Pad195) -> Col_13-Row_3
- U1 pad 209: unconnected-(U1-Col_14-Row_1-Pad209) -> Col_14-Row_1
- U1 pad 210: unconnected-(U1-Col_14-Row_2-Pad210) -> Col_14-Row_2
- U1 pad 211: unconnected-(U1-Col_14-Row_3-Pad211) -> Col_14-Row_3
- U1 pad 225: unconnected-(U1-Col_15-Row_1-Pad225) -> Col_15-Row_1
- U1 pad 226: unconnected-(U1-Col_15-Row_2-Pad226) -> Col_15-Row_2
- U1 pad 227: unconnected-(U1-Col_15-Row_3-Pad227) -> Col_15-Row_3
- U1 pad 241: unconnected-(U1-Col_16-Row_1-Pad241) -> Col_16-Row_1
- U1 pad 242: unconnected-(U1-Col_16-Row_2-Pad242) -> Col_16-Row_2
- U1 pad 243: unconnected-(U1-Col_16-Row_3-Pad243) -> Col_16-Row_3
- U1 pad 257: unconnected-(U1-Col_17-Row_1-Pad257) -> Col_17-Row_1
- U1 pad 258: unconnected-(U1-Col_17-Row_2-Pad258) -> Col_17-Row_2
- U1 pad 259: unconnected-(U1-Col_17-Row_3-Pad259) -> Col_17-Row_3
- U1 pad 273: unconnected-(U1-Col_18-Row_1-Pad273) -> Col_18-Row_1
- U1 pad 274: unconnected-(U1-Col_18-Row_2-Pad274) -> Col_18-Row_2
- U1 pad 275: unconnected-(U1-Col_18-Row_3-Pad275) -> Col_18-Row_3
- U1 pad 289: unconnected-(U1-Col_19-Row_1-Pad289) -> Col_19-Row_3
- U1 pad 290: unconnected-(U1-Col_19-Row_2-Pad290) -> Col_19-Row_2
- U1 pad 291: unconnected-(U1-Col_19-Row_3-Pad291) -> Col_19-Row_1
- U1 pad 305: unconnected-(U1-Col_20-Row_1-Pad305) -> Col_20-Row_1
- U1 pad 306: unconnected-(U1-Col_20-Row_2-Pad306) -> Col_20-Row_2
- U1 pad 307: unconnected-(U1-Col_20-Row_3-Pad307) -> Col_20-Row_3
- U1 pad 321: unconnected-(U1-Col_21-Row_1-Pad321) -> Col_21-Row_1
- U1 pad 322: unconnected-(U1-Col_21-Row_2-Pad322) -> Col_21-Row_2
- U1 pad 323: unconnected-(U1-Col_21-Row_3-Pad323) -> Col_21-Row_3
- U1 pad 337: unconnected-(U1-Col_22-Row_1-Pad337) -> Col_22-Row_1
- U1 pad 338: unconnected-(U1-Col_22-Row_2-Pad338) -> Col_22-Row_2
- U1 pad 339: unconnected-(U1-Col_22-Row_3-Pad339) -> Col_22-Row_3
Routing:
- net Col_5-Row_1: track 9.20 -> 0.00 mm, vias 2 -> 0
- net Col_6-Row_1: track 9.06 -> 0.00 mm, vias 2 -> 0
- net Col_3-Row_1: track 7.46 -> 0.00 mm, vias 1 -> 0
- net Col_4-Row_1: track 7.33 -> 0.00 mm, vias 2 -> 0
- net Col_2-Row_1: track 7.28 -> 0.00 mm, vias 1 -> 0
- net Col_4-Row_2: track 7.23 -> 0.03 mm, vias 1 -> 0
- net Col_5-Row_3: track 7.07 -> 0.00 mm, vias 1 -> 0
- net Col_4-Row_3: track 6.95 -> 0.00 mm, vias 2 -> 0
- net Col_3-Row_3: track 6.91 -> 0.00 mm, vias 2 -> 0
- net Col_3-Row_2: track 6.74 -> 0.00 mm, vias 2 -> 0
- net Col_5-Row_2: track 6.69 -> 0.00 mm, vias 2 -> 0
- net Col_6-Row_2: track 6.68 -> 0.00 mm, vias 2 -> 0
- net Col_2-Row_2: track 6.10 -> 0.00 mm, vias 2 -> 0
- net Col_2-Row_3: track 5.92 -> 0.00 mm, vias 2 -> 0
- net Col_9-Row_1: track 5.27 -> 0.00 mm, vias 1 -> 0
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