File: HYDRA_VMM3_Adapter/_autosave-HYDRA_VMM3_Adapter.kicad_sch (KiCad schematic)
At the start: 12 parts, among them J1 ME1014010101011, J10 Conn_01x01_Socket, J2 ME1014010101011, J3 ME1014010101011, J4 ME1014010101011, J5 ME1014010101011, J6 ME1014010101011, J7 Conn_01x01_Socket, J8 Conn_01x01_Socket, J9 Conn_01x01_Socket

Commit message: .
Other:
- moved on the sheet: J2A, J2B, J3A, J3B, J5A, J5B
Changed lines of the file:
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@@
 		(lib_name "ME1014010101011_1")
 		(lib_id "HYDRA_Amphenol_card:ME1014010101011")
-		(at 327.66 190.5 0)
+		(at 317.5 190.5 0)
 		(unit 2)
 		(exclude_from_sim no)
@@
 		(fields_autoplaced yes)
 		(property "Reference" "J5"
-			(at 327.66 139.7 0)
+			(at 317.5 139.7 0)
 			(effects
 				(font
@@
 		)
 		(property "Value" "ME1014010101011"
-			(at 327.66 142.24 0)
+			(at 317.5 142.24 0)
 			(effects
 				(font
@@
 		)
 		(property "Footprint" "HYDRA_Amphenol_card_footprint:AMPHENOL_ME1014010101011"
-			(at 327.66 190.5 0)
+			(at 317.5 190.5 0)
 			(effects
 				(font
@@
 		)
 		(property "Datasheet" ""
-			(at 327.66 190.5 0)
+			(at 317.5 190.5 0)
 			(effects
 				(font
@@
 		)
 		(property "Description" ""
-			(at 327.66 190.5 0)
+			(at 317.5 190.5 0)
 			(effects
 				(font
@@
 		)
 		(property "PARTREV" "11"
-			(at 327.66 190.5 0)
+			(at 317.5 190.5 0)
 			(effects
 				(font
@@
 		)
 		(property "STANDARD" "Manufacturer Recommendations"
-			(at 327.66 190.5 0)
+			(at 317.5 190.5 0)
 			(effects
 				(font
@@
 		)
 		(property "SNAPEDA_PN" "ME1014010101011"
-			(at 327.66 190.5 0)
+			(at 317.5 190.5 0)
 			(effects
 				(font
@@
 		)
 		(property "MAXIMUM_PACKAGE_HEIGHT" "9.1mm"
-			(at 327.66 190.5 0)
+			(at 317.5 190.5 0)
 			(effects
 				(font
@@
 		)
 		(property "MANUFACTURER" "Amphenol"
-			(at 327.66 190.5 0)
+			(at 317.5 190.5 0)
 			(effects
 				(font
@@
 	(symbol
 		(lib_id "HYDRA_Amphenol_card:ME1014010101011")
-		(at 328.93 83.82 0)
+		(at 318.77 83.82 0)
 		(unit 1)
 		(exclude_from_sim no)
@@
 		(fields_autoplaced yes)
 		(property "Reference" "J5"
-			(at 328.93 33.02 0)
+			(at 318.77 33.02 0)
 			(effects
 				(font
@@
 		)
 		(property "Value" "ME1014010101011"
-			(at 328.93 35.56 0)
+			(at 318.77 35.56 0)
 			(effects
 				(font
@@
 		)
 		(property "Footprint" "HYDRA_Amphenol_card_footprint:AMPHENOL_ME1014010101011"
-			(at 328.93 83.82 0)
+			(at 318.77 83.82 0)
 			(effects
 				(font
@@
 		)
 		(property "Datasheet" ""
-			(at 328.93 83.82 0)
+			(at 318.77 83.82 0)
 			(effects
 				(font
@@
 		)
 		(property "Description" ""
-			(at 328.93 83.82 0)
+			(at 318.77 83.82 0)
 			(effects
 				(font
@@
 		)
 		(property "PARTREV" "11"
-			(at 328.93 83.82 0)
+			(at 318.77 83.82 0)
 			(effects
 				(font
@@
 		)
 		(property "STANDARD" "Manufacturer Recommendations"
-			(at 328.93 83.82 0)
+			(at 318.77 83.82 0)
 			(effects
 				(font
@@
 		)
 		(property "SNAPEDA_PN" "ME1014010101011"
-			(at 328.93 83.82 0)
+			(at 318.77 83.82 0)
 			(effects
 				(font
@@
 		)
 		(property "MAXIMUM_PACKAGE_HEIGHT" "9.1mm"
-			(at 328.93 83.82 0)
+			(at 318.77 83.82 0)
 			(effects
 				(font
@@
 		)
 		(property "MANUFACTURER" "Amphenol"
-			(at 328.93 83.82 0)
+			(at 318.77 83.82 0)
 			(effects
 				(font
@@
 		(lib_name "ME1014010101011_1")
 		(lib_id "HYDRA_Amphenol_card:ME1014010101011")
-		(at 264.16 185.42 0)
+		(at 254 185.42 0)
 		(unit 2)
 		(exclude_from_sim no)
@@
 		(fields_autoplaced yes)
 		(property "Reference" "J2"
-			(at 264.16 134.62 0)
+			(at 254 134.62 0)
 			(effects
 				(font
@@
 		)
 		(property "Value" "ME1014010101011"
-			(at 264.16 137.16 0)
+			(at 254 137.16 0)
 			(effects
 				(font
@@
 		)
 		(property "Footprint" "HYDRA_Amphenol_card_footprint:AMPHENOL_ME1014010101011"
-			(at 264.16 185.42 0)
+			(at 254 185.42 0)
 			(effects
 				(font
@@
 		)
 		(property "Datasheet" ""
-			(at 264.16 185.42 0)
+			(at 254 185.42 0)
 			(effects
 				(font
@@
 		)
 		(property "Description" ""
-			(at 264.16 185.42 0)
+			(at 254 185.42 0)
 			(effects
 				(font
@@
 		)
 		(property "PARTREV" "11"
-			(at 264.16 185.42 0)
+			(at 254 185.42 0)
 			(effects
 				(font
@@
 		)
 		(property "STANDARD" "Manufacturer Recommendations"
-			(at 264.16 185.42 0)
+			(at 254 185.42 0)
 			(effects
 				(font
@@
 		)
 		(property "SNAPEDA_PN" "ME1014010101011"
-			(at 264.16 185.42 0)
+			(at 254 185.42 0)
 			(effects
 				(font
@@
 		)
 		(property "MAXIMUM_PACKAGE_HEIGHT" "9.1mm"
-			(at 264.16 185.42 0)
+			(at 254 185.42 0)
 			(effects
 				(font
@@
 		)
 		(property "MANUFACTURER" "Amphenol"
-			(at 264.16 185.42 0)
+			(at 254 185.42 0)
 			(effects
 				(font
@@
 	(symbol
 		(lib_id "HYDRA_Amphenol_card:ME1014010101011")
-		(at 391.16 85.09 0)
+		(at 375.92 83.82 0)
 		(unit 1)
 		(exclude_from_sim no)
@@
 		(fields_autoplaced yes)
 		(property "Reference" "J3"
-			(at 391.16 34.29 0)
+			(at 375.92 33.02 0)
 			(effects
 				(font
@@
 		)
 		(property "Value" "ME1014010101011"
-			(at 391.16 36.83 0)
+			(at 375.92 35.56 0)
 			(effects
 				(font
@@
 		)
 		(property "Footprint" "HYDRA_Amphenol_card_footprint:AMPHENOL_ME1014010101011"
-			(at 391.16 85.09 0)
+			(at 375.92 83.82 0)
 			(effects
 				(font
@@
 		)
 		(property "Datasheet" ""
-			(at 391.16 85.09 0)
+			(at 375.92 83.82 0)
 			(effects
 				(font
@@
 		)
 		(property "Description" ""
-			(at 391.16 85.09 0)
+			(at 375.92 83.82 0)
 			(effects
 				(font
@@
 		)
 		(property "PARTREV" "11"
-			(at 391.16 85.09 0)
+			(at 375.92 83.82 0)
 			(effects
 				(font
@@
 		)
 		(property "STANDARD" "Manufacturer Recommendations"
-			(at 391.16 85.09 0)
+			(at 375.92 83.82 0)
 			(effects
 				(font
@@
 		)
 		(property "SNAPEDA_PN" "ME1014010101011"
-			(at 391.16 85.09 0)
+			(at 375.92 83.82 0)
 			(effects
 				(font
@@
 		)
 		(property "MAXIMUM_PACKAGE_HEIGHT" "9.1mm"
-			(at 391.16 85.09 0)
+			(at 375.92 83.82 0)
 			(effects
 				(font
@@
 		)
 		(property "MANUFACTURER" "Amphenol"
-			(at 391.16 85.09 0)
+			(at 375.92 83.82 0)
 			(effects
 				(font
@@
 		(lib_name "ME1014010101011_1")
 		(lib_id "HYDRA_Amphenol_card:ME1014010101011")
-		(at 391.16 187.96 0)
+		(at 375.92 186.69 0)
 		(unit 2)
 		(exclude_from_sim no)
@@
 		(fields_autoplaced yes)
 		(property "Reference" "J3"
-			(at 391.16 137.16 0)
+			(at 375.92 135.89 0)
 			(effects
 				(font
@@
 		)
 		(property "Value" "ME1014010101011"
-			(at 391.16 139.7 0)
+			(at 375.92 138.43 0)
 			(effects
 				(font
@@
 		)
 		(property "Footprint" "HYDRA_Amphenol_card_footprint:AMPHENOL_ME1014010101011"
-			(at 391.16 187.96 0)
+			(at 375.92 186.69 0)
 			(effects
 				(font
@@
 		)
 		(property "Datasheet" ""
-			(at 391.16 187.96 0)
+			(at 375.92 186.69 0)
 			(effects
 				(font
@@
 		)
 		(property "Description" ""
-			(at 391.16 187.96 0)
+			(at 375.92 186.69 0)
 			(effects
 				(font
@@
 		)
 		(property "PARTREV" "11"
-			(at 391.16 187.96 0)
+			(at 375.92 186.69 0)
 			(effects
 				(font
@@
 		)
 		(property "STANDARD" "Manufacturer Recommendations"
-			(at 391.16 187.96 0)
+			(at 375.92 186.69 0)
 			(effects
 				(font
@@
 		)
 		(property "SNAPEDA_PN" "ME1014010101011"
-			(at 391.16 187.96 0)
+			(at 375.92 186.69 0)
 			(effects
 				(font
@@
 		)
 		(property "MAXIMUM_PACKAGE_HEIGHT" "9.1mm"
-			(at 391.16 187.96 0)
+			(at 375.92 186.69 0)
 			(effects
 				(font
@@
 		)
 		(property "MANUFACTURER" "Amphenol"
-			(at 391.16 187.96 0)
+			(at 375.92 186.69 0)
 			(effects
 				(font
@@
 	(symbol
 		(lib_id "HYDRA_Amphenol_card:ME1014010101011")
-		(at 264.16 85.09 0)
+		(at 254 85.09 0)
 		(unit 1)
 		(exclude_from_sim no)
@@
 		(fields_autoplaced yes)
 		(property "Reference" "J2"
-			(at 264.16 34.29 0)
+			(at 254 34.29 0)
 			(effects
 				(font
@@
 		)
 		(property "Value" "ME1014010101011"
-			(at 264.16 36.83 0)
+			(at 254 36.83 0)
 			(effects
 				(font
@@
 		)
 		(property "Footprint" "HYDRA_Amphenol_card_footprint:AMPHENOL_ME1014010101011"
-			(at 264.16 85.09 0)
+			(at 254 85.09 0)
 			(effects
 				(font
@@
 		)
 		(property "Datasheet" ""
-			(at 264.16 85.09 0)
+			(at 254 85.09 0)
 			(effects
 				(font
@@
 		)
 		(property "Description" ""
-			(at 264.16 85.09 0)
+			(at 254 85.09 0)
 			(effects
 				(font
@@
 		)
 		(property "PARTREV" "11"
-			(at 264.16 85.09 0)
+			(at 254 85.09 0)
 			(effects
 				(font
@@
 		)
 		(property "STANDARD" "Manufacturer Recommendations"
-			(at 264.16 85.09 0)
+			(at 254 85.09 0)
 			(effects
 				(font
@@
 		)
 		(property "SNAPEDA_PN" "ME1014010101011"
-			(at 264.16 85.09 0)
+			(at 254 85.09 0)
 			(effects
 				(font
@@
 		)
 		(property "MAXIMUM_PACKAGE_HEIGHT" "9.1mm"
-			(at 264.16 85.09 0)
+			(at 254 85.09 0)
 			(effects
 				(font
@@
 		)
 		(property "MANUFACTURER" "Amphenol"
-			(at 264.16 85.09 0)
+			(at 254 85.09 0)
 			(effects
 				(font
