File: HYDRA_VMM3_Adapter/HYDRA_VMM3_Adapter.kicad_pcb (KiCad board)
At the start: 8 copper layers, 121.5 x 31.5 mm, 7 parts, among them J1 ME1014010101011, J2 ME1014010101011, J3 ME1014010101011, J4 ME1014010101011, J5 ME1014010101011, J6 ME1014010101011

Commit message: .
Parts:
- moved J4 38.3 mm to (75.7, 55.3)
- moved J5 38.3 mm to (75.7, 66.3)
- moved J6 38.3 mm to (75.7, 77.3)
- moved U1 38.3 mm to (63.7, 49.8)
- moved J1 38.3 mm to (137.7, 55.3)
- moved J2 38.3 mm to (137.7, 66.3)
- moved J3 38.3 mm to (137.7, 77.3)
Connections:
- J4 pad A15: unconnected-(J4-PadA15) -> Col_2-Row_4
- J4 pad A16: unconnected-(J4-PadA16) -> Col_2-Row_5
- J4 pad A17: unconnected-(J4-PadA17) -> Col_2-Row_6
- J4 pad A18: unconnected-(J4-PadA18) -> Col_3-Row_4
- J4 pad A19: unconnected-(J4-PadA19) -> Col_3-Row_5
- J4 pad A20: unconnected-(J4-PadA20) -> Col_3-Row_6
- J4 pad A21: unconnected-(J4-PadA21) -> Col_4-Row_4
- J4 pad A22: unconnected-(J4-PadA22) -> Col_4-Row_5
- J4 pad A23: unconnected-(J4-PadA23) -> Col_4-Row_6
- J4 pad A24: unconnected-(J4-PadA24) -> Col_5-Row_4
- J4 pad A25: unconnected-(J4-PadA25) -> Col_5-Row_5
- J4 pad A26: unconnected-(J4-PadA26) -> Col_5-Row_6
- J4 pad A27: unconnected-(J4-PadA27) -> Col_6-Row_4
- J4 pad A28: unconnected-(J4-PadA28) -> Col_6-Row_5
- J4 pad A29: unconnected-(J4-PadA29) -> Col_6-Row_6
- J4 pad A30: unconnected-(J4-PadA30) -> Col_7-Row_4
- J4 pad A31: unconnected-(J4-PadA31) -> Col_7-Row_5
- J4 pad A32: unconnected-(J4-PadA32) -> Col_7-Row_6
- J4 pad A33: unconnected-(J4-PadA33) -> Col_8-Row_4
- J4 pad A34: unconnected-(J4-PadA34) -> Col_8-Row_5
- J4 pad A35: unconnected-(J4-PadA35) -> Col_8-Row_6
- J4 pad A36: unconnected-(J4-PadA36) -> Col_9-Row_4
- J4 pad A37: unconnected-(J4-PadA37) -> Col_9-Row_5
- J4 pad A38: unconnected-(J4-PadA38) -> Col_10-Row_4
- J4 pad A39: unconnected-(J4-PadA39) -> Col_10-Row_5
- J4 pad A40: unconnected-(J4-PadA40) -> Col_11-Row_4
- J4 pad A41: unconnected-(J4-PadA41) -> Col_11-Row_5
- J4 pad A42: unconnected-(J4-PadA42) -> Col_12-Row_4
- J4 pad A43: unconnected-(J4-PadA43) -> Col_12-Row_5
- J4 pad A44: unconnected-(J4-PadA44) -> Col_13-Row_4
- J4 pad A45: unconnected-(J4-PadA45) -> Col_13-Row_5
- J4 pad A46: unconnected-(J4-PadA46) -> Col_14-Row_4
- J4 pad A47: unconnected-(J4-PadA47) -> Col_14-Row_5
- J4 pad A48: unconnected-(J4-PadA48) -> Col_15-Row_4
- J4 pad A49: unconnected-(J4-PadA49) -> Col_15-Row_5
- J4 pad A50: unconnected-(J4-PadA50) -> Col_16-Row_4
- J4 pad A51: unconnected-(J4-PadA51) -> Col_16-Row_5
- J4 pad A52: unconnected-(J4-PadA52) -> Col_17-Row_4
- J4 pad A53: unconnected-(J4-PadA53) -> Col_17-Row_5
- J4 pad A54: unconnected-(J4-PadA54) -> Col_18-Row_4
- J4 pad A55: unconnected-(J4-PadA55) -> Col_18-Row_5
- J4 pad A56: unconnected-(J4-PadA56) -> Col_19-Row_4
- J4 pad A57: unconnected-(J4-PadA57) -> Col_19-Row_5
- J4 pad A58: unconnected-(J4-PadA58) -> Col_20-Row_4
- J4 pad A59: unconnected-(J4-PadA59) -> Col_20-Row_5
- J4 pad A60: unconnected-(J4-PadA60) -> Col_21-Row_4
- J4 pad A61: unconnected-(J4-PadA61) -> Col_21-Row_5
- J4 pad A62: unconnected-(J4-PadA62) -> Col_22-Row_4
- J4 pad A63: unconnected-(J4-PadA63) -> Col_22-Row_5
- J4 pad A64: unconnected-(J4-PadA64) -> Col_20-Row_3
- J4 pad A65: unconnected-(J4-PadA65) -> Col_21-Row_1
- J4 pad A66: unconnected-(J4-PadA66) -> Col_21-Row_2
- J4 pad A67: unconnected-(J4-PadA67) -> Col_21-Row_3
- J4 pad A68: unconnected-(J4-PadA68) -> Col_22-Row_1
- J4 pad A69: unconnected-(J4-PadA69) -> Col_22-Row_2
- J4 pad A70: unconnected-(J4-PadA70) -> Col_22-Row_3
- J4 pad B39: unconnected-(J4-PadB39) -> Col_10-Row_1
- J4 pad B40: unconnected-(J4-PadB40) -> Col_10-Row_2
- J4 pad B41: unconnected-(J4-PadB41) -> Col_10-Row_3
- J4 pad B42: unconnected-(J4-PadB42) -> Col_11-Row_1
- J4 pad B43: unconnected-(J4-PadB43) -> Col_11-Row_2
- J4 pad B44: unconnected-(J4-PadB44) -> Col_11-Row_3
- J4 pad B45: unconnected-(J4-PadB45) -> Col_12-Row_1
- J4 pad B46: unconnected-(J4-PadB46) -> Col_12-Row_2
- J4 pad B47: unconnected-(J4-PadB47) -> Col_12-Row_3
- J4 pad B48: unconnected-(J4-PadB48) -> Col_13-Row_1
- J4 pad B49: unconnected-(J4-PadB49) -> Col_13-Row_2
- J4 pad B50: unconnected-(J4-PadB50) -> Col_13-Row_3
- J4 pad B51: unconnected-(J4-PadB51) -> Col_14-Row_1
- J4 pad B52: unconnected-(J4-PadB52) -> Col_14-Row_2
- J4 pad B53: unconnected-(J4-PadB53) -> Col_14-Row_3
- J4 pad B54: unconnected-(J4-PadB54) -> Col_15-Row_1
- J4 pad B55: unconnected-(J4-PadB55) -> Col_15-Row_2
- J4 pad B56: unconnected-(J4-PadB56) -> Col_15-Row_3
- J4 pad B57: unconnected-(J4-PadB57) -> Col_16-Row_1
- J4 pad B58: unconnected-(J4-PadB58) -> Col_16-Row_2
- J4 pad B59: unconnected-(J4-PadB59) -> Col_16-Row_3
- J4 pad B60: unconnected-(J4-PadB60) -> Col_17-Row_1
- J4 pad B61: unconnected-(J4-PadB61) -> Col_17-Row_2
- J4 pad B62: unconnected-(J4-PadB62) -> Col_17-Row_3
- J4 pad B63: unconnected-(J4-PadB63) -> Col_18-Row_1
- J4 pad B64: unconnected-(J4-PadB64) -> Col_18-Row_2
- J4 pad B65: unconnected-(J4-PadB65) -> Col_18-Row_3
- J4 pad B66: unconnected-(J4-PadB66) -> Col_19-Row_1
- J4 pad B67: unconnected-(J4-PadB67) -> Col_19-Row_2
- J4 pad B68: unconnected-(J4-PadB68) -> Col_19-Row_3
- J4 pad B69: unconnected-(J4-PadB69) -> Col_20-Row_1
- J4 pad B70: unconnected-(J4-PadB70) -> Col_20-Row_2
- U1 pad 100: unconnected-(U1-Col_7-Row_4-Pad100) -> Col_7-Row_4
- U1 pad 101: unconnected-(U1-Col_7-Row_5-Pad101) -> Col_7-Row_5
- U1 pad 102: unconnected-(U1-Col_7-Row_6-Pad102) -> Col_7-Row_6
- U1 pad 116: unconnected-(U1-Col_8-Row_4-Pad116) -> Col_8-Row_4
- U1 pad 117: unconnected-(U1-Col_8-Row_5-Pad117) -> Col_8-Row_5
- U1 pad 118: unconnected-(U1-Col_8-Row_6-Pad118) -> Col_8-Row_6
- U1 pad 132: unconnected-(U1-Col_9-Row_4-Pad132) -> Col_9-Row_4
- U1 pad 133: unconnected-(U1-Col_9-Row_5-Pad133) -> Col_9-Row_5
- U1 pad 145: unconnected-(U1-Col_10-Row_1-Pad145) -> Col_10-Row_1
- U1 pad 146: unconnected-(U1-Col_10-Row_2-Pad146) -> Col_10-Row_2
- U1 pad 147: unconnected-(U1-Col_10-Row_3-Pad147) -> Col_10-Row_3
- U1 pad 148: unconnected-(U1-Col_10-Row_4-Pad148) -> Col_10-Row_4
- U1 pad 149: unconnected-(U1-Col_10-Row_5-Pad149) -> Col_10-Row_5
- U1 pad 161: unconnected-(U1-Col_11-Row_1-Pad161) -> Col_11-Row_1
- U1 pad 162: unconnected-(U1-Col_11-Row_2-Pad162) -> Col_11-Row_2
- U1 pad 163: unconnected-(U1-Col_11-Row_3-Pad163) -> Col_11-Row_3
- U1 pad 164: unconnected-(U1-Col_11-Row_4-Pad164) -> Col_11-Row_4
- U1 pad 165: unconnected-(U1-Col_11-Row_5-Pad165) -> Col_11-Row_5
- U1 pad 177: unconnected-(U1-Col_12-Row_1-Pad177) -> Col_12-Row_1
- U1 pad 178: unconnected-(U1-Col_12-Row_2-Pad178) -> Col_12-Row_2
- U1 pad 179: unconnected-(U1-Col_12-Row_3-Pad179) -> Col_12-Row_3
- U1 pad 180: unconnected-(U1-Col_12-Row_4-Pad180) -> Col_12-Row_4
- U1 pad 181: unconnected-(U1-Col_12-Row_5-Pad181) -> Col_12-Row_5
- U1 pad 193: unconnected-(U1-Col_13-Row_1-Pad193) -> Col_13-Row_1
- U1 pad 194: unconnected-(U1-Col_13-Row_2-Pad194) -> Col_13-Row_2
- U1 pad 195: unconnected-(U1-Col_13-Row_3-Pad195) -> Col_13-Row_3
- U1 pad 196: unconnected-(U1-Col_13-Row_4-Pad196) -> Col_13-Row_4
- U1 pad 197: unconnected-(U1-Col_13-Row_5-Pad197) -> Col_13-Row_5
- U1 pad 20: unconnected-(U1-Col_2-Row_4-Pad20) -> Col_2-Row_4
- U1 pad 209: unconnected-(U1-Col_14-Row_1-Pad209) -> Col_14-Row_1
- U1 pad 21: unconnected-(U1-Col_2-Row_5-Pad21) -> Col_2-Row_5
- U1 pad 210: unconnected-(U1-Col_14-Row_2-Pad210) -> Col_14-Row_2
- U1 pad 211: unconnected-(U1-Col_14-Row_3-Pad211) -> Col_14-Row_3
- U1 pad 212: unconnected-(U1-Col_14-Row_4-Pad212) -> Col_14-Row_4
- U1 pad 213: unconnected-(U1-Col_14-Row_5-Pad213) -> Col_14-Row_5
- U1 pad 22: unconnected-(U1-Col_2-Row_6-Pad22) -> Col_2-Row_6
- U1 pad 225: unconnected-(U1-Col_15-Row_1-Pad225) -> Col_15-Row_1
- U1 pad 226: unconnected-(U1-Col_15-Row_2-Pad226) -> Col_15-Row_2
- U1 pad 227: unconnected-(U1-Col_15-Row_3-Pad227) -> Col_15-Row_3
- U1 pad 228: unconnected-(U1-Col_15-Row_4-Pad228) -> Col_15-Row_4
- U1 pad 229: unconnected-(U1-Col_15-Row_5-Pad229) -> Col_15-Row_5
- U1 pad 241: unconnected-(U1-Col_16-Row_1-Pad241) -> Col_16-Row_1
- U1 pad 242: unconnected-(U1-Col_16-Row_2-Pad242) -> Col_16-Row_2
- U1 pad 243: unconnected-(U1-Col_16-Row_3-Pad243) -> Col_16-Row_3
- U1 pad 244: unconnected-(U1-Col_16-Row_4-Pad244) -> Col_16-Row_4
- U1 pad 245: unconnected-(U1-Col_16-Row_5-Pad245) -> Col_16-Row_5
- U1 pad 257: unconnected-(U1-Col_17-Row_1-Pad257) -> Col_17-Row_1
- U1 pad 258: unconnected-(U1-Col_17-Row_2-Pad258) -> Col_17-Row_2
- U1 pad 259: unconnected-(U1-Col_17-Row_3-Pad259) -> Col_17-Row_3
- U1 pad 260: unconnected-(U1-Col_17-Row_4-Pad260) -> Col_17-Row_4
- U1 pad 261: unconnected-(U1-Col_17-Row_5-Pad261) -> Col_17-Row_5
- U1 pad 273: unconnected-(U1-Col_18-Row_1-Pad273) -> Col_18-Row_1
- U1 pad 274: unconnected-(U1-Col_18-Row_2-Pad274) -> Col_18-Row_2
- U1 pad 275: unconnected-(U1-Col_18-Row_3-Pad275) -> Col_18-Row_3
- U1 pad 276: unconnected-(U1-Col_18-Row_4-Pad276) -> Col_18-Row_4
- U1 pad 277: unconnected-(U1-Col_18-Row_5-Pad277) -> Col_18-Row_5
- U1 pad 289: unconnected-(U1-Col_19-Row_1-Pad289) -> Col_19-Row_3
- U1 pad 290: unconnected-(U1-Col_19-Row_2-Pad290) -> Col_19-Row_2
- U1 pad 291: unconnected-(U1-Col_19-Row_3-Pad291) -> Col_19-Row_1
- U1 pad 292: unconnected-(U1-Col_19-Row_4-Pad292) -> Col_19-Row_4
- U1 pad 293: unconnected-(U1-Col_19-Row_5-Pad293) -> Col_19-Row_5
- U1 pad 305: unconnected-(U1-Col_20-Row_1-Pad305) -> Col_20-Row_1
- U1 pad 306: unconnected-(U1-Col_20-Row_2-Pad306) -> Col_20-Row_2
- U1 pad 307: unconnected-(U1-Col_20-Row_3-Pad307) -> Col_20-Row_3
- U1 pad 308: unconnected-(U1-Col_20-Row_4-Pad308) -> Col_20-Row_4
- U1 pad 309: unconnected-(U1-Col_20-Row_5-Pad309) -> Col_20-Row_5
- U1 pad 321: unconnected-(U1-Col_21-Row_1-Pad321) -> Col_21-Row_1
- U1 pad 322: unconnected-(U1-Col_21-Row_2-Pad322) -> Col_21-Row_2
- U1 pad 323: unconnected-(U1-Col_21-Row_3-Pad323) -> Col_21-Row_3
- U1 pad 324: unconnected-(U1-Col_21-Row_4-Pad324) -> Col_21-Row_4
- U1 pad 325: unconnected-(U1-Col_21-Row_5-Pad325) -> Col_21-Row_5
- U1 pad 337: unconnected-(U1-Col_22-Row_1-Pad337) -> Col_22-Row_1
- U1 pad 338: unconnected-(U1-Col_22-Row_2-Pad338) -> Col_22-Row_2
- U1 pad 339: unconnected-(U1-Col_22-Row_3-Pad339) -> Col_22-Row_3
- U1 pad 340: unconnected-(U1-Col_22-Row_4-Pad340) -> Col_22-Row_4
- U1 pad 341: unconnected-(U1-Col_22-Row_5-Pad341) -> Col_22-Row_5
- U1 pad 36: unconnected-(U1-Col_3-Row_4-Pad36) -> Col_3-Row_4
- U1 pad 37: unconnected-(U1-Col_3-Row_5-Pad37) -> Col_3-Row_5
- U1 pad 38: unconnected-(U1-Col_3-Row_6-Pad38) -> Col_3-Row_6
- U1 pad 52: unconnected-(U1-Col_4-Row_4-Pad52) -> Col_4-Row_4
- U1 pad 53: unconnected-(U1-Col_4-Row_5-Pad53) -> Col_4-Row_5
- U1 pad 54: unconnected-(U1-Col_4-Row_6-Pad54) -> Col_4-Row_6
- U1 pad 68: unconnected-(U1-Col_5-Row_4-Pad68) -> Col_5-Row_4
- U1 pad 69: unconnected-(U1-Col_5-Row_5-Pad69) -> Col_5-Row_5
- U1 pad 70: unconnected-(U1-Col_5-Row_6-Pad70) -> Col_5-Row_6
- U1 pad 84: unconnected-(U1-Col_6-Row_4-Pad84) -> Col_6-Row_4
- U1 pad 85: unconnected-(U1-Col_6-Row_5-Pad85) -> Col_6-Row_5
- U1 pad 86: unconnected-(U1-Col_6-Row_6-Pad86) -> Col_6-Row_6
Routing:
- net Col_22-Row_5: track 0.00 -> 11.1 mm, vias 0 -> 2
- net Col_21-Row_4: track 0.00 -> 10.8 mm, vias 0 -> 2
- net Col_22-Row_4: track 0.00 -> 10.7 mm, vias 0 -> 2
- net Col_21-Row_5: track 0.00 -> 9.84 mm, vias 0 -> 2
- net Col_22-Row_1: track 0.00 -> 9.62 mm, vias 0 -> 2
- net Col_21-Row_1: track 0.00 -> 9.54 mm, vias 0 -> 2
- net Col_5-Row_1: track 9.20 -> 0.00 mm, vias 2 -> 0
- net Col_20-Row_4: track 0.00 -> 9.20 mm, vias 0 -> 2
- net Col_6-Row_1: track 9.06 -> 0.00 mm, vias 2 -> 0
- net Col_22-Row_2: track 0.00 -> 8.86 mm, vias 0 -> 1
- net Col_21-Row_2: track 0.00 -> 8.86 mm, vias 0 -> 1
- net Col_3-Row_1: track 7.46 -> 0.00 mm, vias 1 -> 0
- net Col_4-Row_1: track 7.33 -> 0.00 mm, vias 2 -> 0
- net Col_2-Row_1: track 7.28 -> 0.00 mm, vias 1 -> 0
- net Col_4-Row_2: track 7.23 -> 0.03 mm, vias 1 -> 0
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
Commit message: .
Routing:
- net Col_21-Row_4: track 10.8 -> 0.00 mm, vias 2 -> 0
- net Col_20-Row_4: track 9.20 -> 0.00 mm, vias 2 -> 0
- added copper zone on In1.Cu, net GND
- added copper zone on In2.Cu, net GND
- added copper zone on In3.Cu, net GND
- added copper zone on In4.Cu, net GND
- added copper zone on In5.Cu, net GND
- added copper zone on In6.Cu, net GND
Changed lines of the file:
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@@
-	)
-	(via blind
-		(at 101.675 57.27)
-		(size 0.28)
-		(drill 0.1)
-		(layers "F.Cu" "In1.Cu")
-		(net 1356)
-	)
-	(segment
-		(start 100.855 58.09)
-		(end 101.675 57.27)
-		(width 0.1)
-		(layer "In1.Cu")
-		(net 1356)
-	)
-	(segment
-		(start 93.55 58.09)
-		(end 100.855 58.09)
-		(width 0.1)
-		(layer "In1.Cu")
-		(net 1356)
-	)
-	(segment
-		(start 93.03 57.57)
-		(end 93.55 58.09)
-		(width 0.1)
-		(layer "In1.Cu")
-		(net 1356)
-	)
-	(via blind
-		(at 93.03 57.57)
-		(size 0.28)
-		(drill 0.1)
-		(layers "In1.Cu" "B.Cu")
-		(net 1356)
-	)
-	(via blind
-		(at 103.675 57.27)
-		(size 0.28)
-		(drill 0.1)
-		(layers "F.Cu" "In1.Cu")
-		(net 1357)
-	)
-	(segment
-		(start 102.895 56.49)
-		(end 103.675 57.27)
-		(width 0.1)
-		(layer "In1.Cu")
-		(net 1357)
-	)
-	(segment
-		(start 94.335 56.49)
-		(end 102.895 56.49)
-		(width 0.1)
-		(layer "In1.Cu")
-		(net 1357)
-	)
-	(via blind
-		(at 94.335 56.49)
-		(size 0.28)
-		(drill 0.1)
-		(layers "In1.Cu" "B.Cu")
-		(net 1357)
-	)
-	(segment
-		(start 94.23 56.595)
-		(end 94.23 57.57)
-		(width 0.1)
-		(layer "B.Cu")
-		(net 1357)
-	)
-	(segment
-		(start 94.335 56.49)
-		(end 94.23 56.595)
-		(width 0.1)
-		(layer "B.Cu")
-		(net 1357)
 	)
 	(via blind
@@
 		(net 1352)
 		(net_name "GND")
-		(layers "F&B.Cu")
+		(layers "F.Cu" "In1.Cu" "In2.Cu" "In3.Cu" "In4.Cu" "In5.Cu" "In6.Cu" "B.Cu")
 		(hatch edge 0.5)
 		(connect_pads

Commit message: .
Parts:
- moved J1 0.34 mm to (137.7, 55.6)
- moved J4 0.34 mm to (75.7, 55.6)
- moved J3 0.34 mm to (137.7, 76.9)
- moved J6 0.34 mm to (75.7, 76.9)
Connections:
- J4 pad A36: Col_9-Row_4 -> Col_9-Row_5
- J4 pad A37: Col_9-Row_5 -> Col_9-Row_4
- J4 pad A38: Col_10-Row_4 -> Col_10-Row_5
- J4 pad A39: Col_10-Row_5 -> Col_10-Row_4
- J4 pad A40: Col_11-Row_4 -> Col_11-Row_5
- J4 pad A41: Col_11-Row_5 -> Col_11-Row_4
- J4 pad A42: Col_12-Row_4 -> Col_12-Row_5
- J4 pad A43: Col_12-Row_5 -> Col_12-Row_4
- J4 pad A44: Col_13-Row_4 -> Col_13-Row_5
- J4 pad A45: Col_13-Row_5 -> Col_13-Row_4
- J4 pad A46: Col_14-Row_4 -> Col_14-Row_5
- J4 pad A47: Col_14-Row_5 -> Col_14-Row_4
- J4 pad A48: Col_15-Row_4 -> Col_15-Row_5
- J4 pad A49: Col_15-Row_5 -> Col_15-Row_4
- J4 pad A50: Col_16-Row_4 -> Col_16-Row_5
- J4 pad A51: Col_16-Row_5 -> Col_16-Row_4
- J4 pad A52: Col_17-Row_4 -> Col_17-Row_5
- J4 pad A53: Col_17-Row_5 -> Col_17-Row_4
- J4 pad A54: Col_18-Row_4 -> Col_18-Row_5
- J4 pad A55: Col_18-Row_5 -> Col_18-Row_4
- J4 pad A56: Col_19-Row_4 -> Col_19-Row_5
- J4 pad A57: Col_19-Row_5 -> Col_19-Row_4
- J4 pad A58: Col_20-Row_4 -> Col_20-Row_5
- J4 pad A59: Col_20-Row_5 -> Col_20-Row_4
- J4 pad A60: Col_21-Row_4 -> Col_20-Row_3
- J4 pad A62: Col_22-Row_4 -> Col_21-Row_4
- J4 pad A63: Col_22-Row_5 -> Col_21-Row_1
- J4 pad A64: Col_20-Row_3 -> Col_21-Row_2
- J4 pad A65: Col_21-Row_1 -> Col_21-Row_3
- J4 pad A66: Col_21-Row_2 -> Col_22-Row_5
- J4 pad A67: Col_21-Row_3 -> Col_22-Row_4
Routing:
- net Col_22-Row_5: track 11.1 -> 0.00 mm, vias 2 -> 0
- net Col_22-Row_4: track 10.7 -> 0.00 mm, vias 2 -> 0
- net Col_21-Row_5: track 9.84 -> 0.00 mm, vias 2 -> 0
- net Col_22-Row_1: track 9.62 -> 0.00 mm, vias 2 -> 1
- net Col_21-Row_1: track 9.54 -> 0.00 mm, vias 2 -> 0
- net Col_21-Row_2: track 8.86 -> 0.02 mm, vias 1 -> 0
- net Col_21-Row_3: track 6.61 -> 0.00 mm, vias 1 -> 0
- net Col_20-Row_3: track 6.40 -> 0.00 mm, vias 1 -> 0
- net Col_19-Row_1: track 3.31 -> 0.00 mm, vias 1 -> 0
- net Col_20-Row_1: track 3.16 -> 0.00 mm, vias 1 -> 0
- net Col_18-Row_1: track 2.80 -> 0.00 mm, vias 1 -> 0
- net Col_11-Row_3: track 2.70 -> 0.00 mm, vias 1 -> 0
- net Col_12-Row_3: track 2.61 -> 0.00 mm, vias 1 -> 0
- net Col_17-Row_1: track 2.58 -> 0.00 mm, vias 1 -> 0
- net Col_13-Row_3: track 2.53 -> 0.00 mm, vias 1 -> 0
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Other:
- copper layers 8 -> 10

Commit message: .
Routing:
- net Col_22-Row_1: track 0.00 -> 11.9 mm, vias 1 -> 2
- net Col_22-Row_5: track 0.00 -> 8.43 mm, vias 0 -> 2
- net Col_22-Row_4: track 0.00 -> 8.00 mm, vias 0 -> 2
- net Col_21-Row_3: track 0.00 -> 7.65 mm, vias 0 -> 2
- net Col_18-Row_4: vias 1 -> 0
Changed lines of the file:
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@@
-	)
-	(segment
-		(start 95.675 55.22)
-		(end 95.675 55.27)
-		(width 0.1)
-		(layer "In2.Cu")
-		(net 118)
-	)
-	(segment
-		(start 93.63 55.225)
-		(end 93.675 55.27)
-		(width 0.1)
-		(layer "In2.Cu")
-		(net 126)
 	)
 	(segment
@@
 	)
 	(segment
-		(start 85.675 53.27)
+		(start 85.83 52.97)
 		(end 85.675 53.125)
 		(width 0.1)
@@
 	(segment
 		(start 85.675 53.125)
-		(end 85.83 52.97)
+		(end 85.675 53.27)
 		(width 0.1)
 		(layer "F.Cu")
@@
 	)
 	(segment
-		(start 84.03 52.97)
-		(end 83.975 52.97)
+		(start 83.975 52.97)
+		(end 84.03 52.97)
 		(width 0.1)
 		(layer "B.Cu")
@@
 	)
 	(segment
-		(start 83.975 52.97)
-		(end 83.675 53.27)
+		(start 83.675 53.27)
+		(end 83.975 52.97)
 		(width 0.1)
 		(layer "B.Cu")
 		(net 189)
 	)
+	(via blind
+		(at 103.675 55.27)
+		(size 0.28)
+		(drill 0.1)
+		(layers "F.Cu" "In7.Cu")
+		(net 246)
+	)
+	(segment
+		(start 97.23 57.725)
+		(end 98.795 56.16)
+		(width 0.1)
+		(layer "In7.Cu")
+		(net 246)
+	)
+	(segment
+		(start 98.795 56.16)
+		(end 102.785 56.16)
+		(width 0.1)
+		(layer "In7.Cu")
+		(net 246)
+	)
+	(segment
+		(start 102.785 56.16)
+		(end 103.675 55.27)
+		(width 0.1)
+		(layer "In7.Cu")
+		(net 246)
+	)
+	(segment
+		(start 97.23 57.91)
+		(end 97.23 57.725)
+		(width 0.1)
+		(layer "In7.Cu")
+		(net 246)
+	)
+	(via blind
+		(at 97.23 57.91)
+		(size 0.28)
+		(drill 0.1)
+		(layers "In7.Cu" "B.Cu")
+		(net 246)
+	)
 	(segment
 		(start 103.675 53.27)
@@
 	)
 	(segment
-		(start 101.315 56.4)
-		(end 104.555 56.4)
+		(start 104.605 56.35)
+		(end 105.675 55.28)
+		(width 0.1)
+		(layer "In2.Cu")
+		(net 1032)
+	)
+	(segment
+		(start 100.235 57.48)
+		(end 101.365 56.35)
+		(width 0.1)
+		(layer "In2.Cu")
+		(net 1032)
+	)
+	(segment
+		(start 100.235 57.91)
+		(end 100.235 57.48)
+		(width 0.1)
+		(layer "In2.Cu")
+		(net 1032)
+	)
+	(segment
+		(start 101.365 56.35)
+		(end 104.605 56.35)
 		(width 0.1)
 		(layer "In2.Cu")
@@
 		(net 1032)
 	)
-	(segment
-		(start 100.235 57.91)
-		(end 100.235 57.48)
-		(width 0.1)
-		(layer "In2.Cu")
-		(net 1032)
-	)
-	(segment
-		(start 104.555 56.4)
-		(end 105.675 55.28)
-		(width 0.1)
-		(layer "In2.Cu")
-		(net 1032)
-	)
-	(segment
-		(start 100.235 57.48)
-		(end 101.315 56.4)
-		(width 0.1)
-		(layer "In2.Cu")
-		(net 1032)
-	)
 	(via blind
 		(at 100.235 57.91)
@@
 	)
 	(via blind
+		(at 105.675 51.27)
+		(size 0.28)
+		(drill 0.1)
+		(layers "F.Cu" "In2.Cu")
+		(net 1033)
+	)
+	(segment
+		(start 99.995 55.99)
+		(end 104.235 55.99)
+		(width 0.1)
+		(layer "In2.Cu")
+		(net 1033)
+	)
+	(segment
+		(start 99.03 56.955)
+		(end 99.995 55.99)
+		(width 0.1)
+		(layer "In2.Cu")
+		(net 1033)
+	)
+	(segment
+		(start 104.545 52.4)
+		(end 105.675 51.27)
+		(width 0.1)
+		(layer "In2.Cu")
+		(net 1033)
+	)
+	(segment
+		(start 104.545 55.68)
+		(end 104.545 52.4)
+		(width 0.1)
+		(layer "In2.Cu")
+		(net 1033)
+	)
+	(segment
+		(start 99.03 57.91)
+		(end 99.03 56.955)
+		(width 0.1)
+		(layer "In2.Cu")
+		(net 1033)
+	)
+	(segment
+		(start 104.235 55.99)
+		(end 104.545 55.68)
+		(width 0.1)
+		(layer "In2.Cu")
+		(net 1033)
+	)
+	(via blind
 		(at 99.03 57.91)
 		(size 0.28)
 		(drill 0.1)
-		(layers "F.Cu" "B.Cu")
+		(layers "In2.Cu" "B.Cu")
 		(net 1033)
 	)
@@
 	)
 	(segment
-		(start 104.885 54.06)
+		(start 100.865 56)
+		(end 104.265 56)
+		(width 0.1)
+		(layer "In4.Cu")
+		(net 1035)
+	)
+	(segment
+		(start 104.695 55.57)
+		(end 104.695 54.25)
+		(width 0.1)
+		(layer "In4.Cu")
+		(net 1035)
+	)
+	(segment
+		(start 99.63 57.235)
+		(end 100.865 56)
+		(width 0.1)
+		(layer "In4.Cu")
+		(net 1035)
+	)
+	(segment
+		(start 104.265 56)
+		(end 104.695 55.57)
+		(width 0.1)
+		(layer "In4.Cu")
+		(net 1035)
+	)
+	(segment
+		(start 99.63 57.91)
+		(end 99.63 57.235)
+		(width 0.1)
+		(layer "In4.Cu")
+		(net 1035)
+	)
+	(segment
+		(start 104.695 54.25)
 		(end 105.675 53.27)
-		(width 0.1)
-		(layer "In4.Cu")
-		(net 1035)
-	)
-	(segment
-		(start 104.885 55.38)
-		(end 104.885 54.06)
-		(width 0.1)
-		(layer "In4.Cu")
-		(net 1035)
-	)
-	(segment
-		(start 104.265 56)
-		(end 104.885 55.38)
-		(width 0.1)
-		(layer "In4.Cu")
-		(net 1035)
-	)
-	(segment
-		(start 99.63 57.91)
-		(end 101.54 56)
-		(width 0.1)
-		(layer "In4.Cu")
-		(net 1035)
-	)
-	(segment
-		(start 101.54 56)
-		(end 104.265 56)
 		(width 0.1)
 		(layer "In4.Cu")
@@
 		(layers "F.Cu" "In1.Cu")
 		(net 1056)
+	)
+	(via blind
+		(at 105.675 59.27)
+		(size 0.28)
+		(drill 0.1)
+		(layers "F.Cu" "In2.Cu")
+		(net 1061)
+	)
+	(segment
+		(start 98.28 58.36)
+		(end 104.765 58.36)
+		(width 0.1)
+		(layer "In2.Cu")
+		(net 1061)
+	)
+	(segment
+		(start 97.83 57.91)
+		(end 98.28 58.36)
+		(width 0.1)
+		(layer "In2.Cu")
+		(net 1061)
+	)
+	(segment
+		(start 104.765 58.36)
+		(end 105.675 59.27)
+		(width 0.1)
+		(layer "In2.Cu")
+		(net 1061)
+	)
+	(via blind
+		(at 97.83 57.91)
+		(size 0.28)
+		(drill 0.1)
+		(layers "In2.Cu" "B.Cu")
+		(net 1061)
+	)
+	(segment
+		(start 97.835 57.91)
+		(end 97.845 57.9)
+		(width 0.1)
+		(layer "B.Cu")
+		(net 1061)
+	)
+	(segment
+		(start 97.83 57.91)
+		(end 97.835 57.91)
+		(width 0.1)
+		(layer "B.Cu")
+		(net 1061)
 	)
 	(segment
@@
 	)
 	(via blind
+		(at 105.675 57.27)
+		(size 0.28)
+		(drill 0.1)
+		(layers "F.Cu" "In4.Cu")
+		(net 1358)
+	)
+	(segment
+		(start 98.43 58.135)
+		(end 98.43 57.91)
+		(width 0.1)
+		(layer "In4.Cu")
+		(net 1358)
+	)
+	(segment
+		(start 104.605 58.34)
+		(end 98.635 58.34)
+		(width 0.1)
+		(layer "In4.Cu")
+		(net 1358)
+	)
+	(segment
+		(start 98.635 58.34)
+		(end 98.43 58.135)
+		(width 0.1)
+		(layer "In4.Cu")
+		(net 1358)
+	)
+	(segment
+		(start 105.675 57.27)
+		(end 104.605 58.34)
+		(width 0.1)
+		(layer "In4.Cu")
+		(net 1358)
+	)
+	(via blind
+		(at 98.43 57.91)
+		(size 0.28)
+		(drill 0.1)
+		(layers "In4.Cu" "B.Cu")
+		(net 1358)
+	)
+	(via blind
 		(at 99.675 59.27)
 		(size 0.28)
@@
 		(layers "F.Cu" "In1.Cu")
 		(net 1367)
-	)
-	(via blind
-		(at 97.675 57.27)
-		(size 0.28)
-		(drill 0.1)
-		(layers "F.Cu" "In1.Cu")
-		(net 1368)
 	)
 	(via blind
@@
 		)
 	)
+	(group ""
+		(members "2bd8a0f5-fa13-404f-9e23-b5e3eb3f9f1f" "5b28fafc-aa0b-4d5a-9e14-3c4fe65d1dc7"
+			"819ff71e-eaf9-433c-bcbd-f9404cb084fc" "8f8d56d9-bdc7-466a-a018-b93755e1db65"
+			"97702ce6-1448-4603-979a-5e5adac4e668" "c743d2d1-0b9b-4ecf-8e98-fe951271f9a1"
+			"dcc3714e-a2c5-4a87-bdc6-37f0cc12959e"
+		)
+	)

Commit message: .
Routing:
- net Col_22-Row_1: track 11.9 -> 0.04 mm
- net Col_22-Row_2: track 9.14 -> 0.00 mm
- net Col_22-Row_5: track 8.43 -> 0.02 mm
- net Col_22-Row_4: track 8.00 -> 0.00 mm
- net Col_21-Row_3: track 7.65 -> 0.00 mm
- net Col_22-Row_3: track 6.80 -> 0.00 mm
- net Col_3-Row_2: track 0.00 -> 0.31 mm, vias 0 -> 1
- net Col_14-Row_2: track 0.02 -> 0.28 mm, vias 0 -> 1
- net Col_13-Row_3: track 0.00 -> 0.06 mm, vias 0 -> 1
- net Col_2-Row_1: track 0.00 -> 0.05 mm, vias 0 -> 1
- net Col_10-Row_3: track 0.00 -> 0.05 mm, vias 0 -> 1
- net Col_8-Row_1: track 0.00 -> 0.05 mm, vias 0 -> 1
- net Col_19-Row_3: track 0.00 -> 0.04 mm, vias 0 -> 1
- net Col_21-Row_1: track 0.00 -> 0.04 mm, vias 0 -> 2
- net Col_16-Row_3: track 0.00 -> 0.04 mm, vias 0 -> 1
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
Commit message: .
Routing:
- net Col_21-Row_1: track 0.04 -> 12.5 mm
- net Col_22-Row_1: track 0.04 -> 11.6 mm
- net Col_21-Row_2: track 0.03 -> 10.4 mm
- net Col_21-Row_5: track 0.00 -> 9.41 mm
- net Col_22-Row_2: track 0.00 -> 9.36 mm
- net Col_20-Row_5: track 0.00 -> 9.21 mm
- net Col_20-Row_3: track 0.02 -> 8.67 mm
- net Col_21-Row_4: track 0.00 -> 8.51 mm
- net Col_19-Row_5: track 0.00 -> 8.41 mm
- net Col_22-Row_5: track 0.02 -> 8.43 mm
- net Col_20-Row_4: track 0.00 -> 8.31 mm
- net Col_21-Row_3: track 0.00 -> 8.15 mm
- net Col_22-Row_4: track 0.00 -> 7.77 mm
- net Col_18-Row_5: track 0.01 -> 7.61 mm
- net Col_19-Row_4: track 0.00 -> 7.51 mm
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- added copper zone on In7.Cu, net GND
- added copper zone on In8.Cu, net GND

Commit message: .
Routing:
- net Col_6-Row_1: track 0.03 -> 8.13 mm
- net Col_5-Row_1: track 0.01 -> 7.91 mm
- net Col_4-Row_1: track 0.01 -> 7.85 mm
- net Col_3-Row_1: track 0.02 -> 7.68 mm
- net Col_2-Row_1: track 0.05 -> 7.57 mm
- net Col_6-Row_4: track 0.02 -> 7.23 mm
- net Col_4-Row_4: track 0.00 -> 7.08 mm
- net Col_6-Row_2: track 0.00 -> 7.04 mm, vias 1 -> 2
- net Col_5-Row_4: track 0.02 -> 7.03 mm
- net Col_5-Row_6: track 0.00 -> 6.96 mm
- net Col_6-Row_5: track 0.00 -> 6.93 mm
- net Col_3-Row_4: track 0.00 -> 6.88 mm
- net Col_5-Row_3: track 0.02 -> 6.81 mm
- net Col_4-Row_6: track 0.00 -> 6.76 mm
- net Col_5-Row_5: track 0.00 -> 6.73 mm
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