File: HYDRA_VMM3_Adapter/HYDRA_VMM3_Adapter.kicad_pcb (KiCad board)
At the start: 10 copper layers, 121.5 x 31.5 mm, 7 parts, among them J1 ME1014010101011, J2 ME1014010101011, J3 ME1014010101011, J4 ME1014010101011, J5 ME1014010101011, J6 ME1014010101011

Commit message: .
Connections:
- J4 pad A59: Col_20-Row_4 -> Col_20-Row_3
- J4 pad A60: Col_20-Row_3 -> Col_20-Row_4
- J4 pad B29: Col_6-Row_3 -> Col_7-Row_1
- J4 pad B30: Col_7-Row_1 -> Col_6-Row_3
Routing:
- net Col_14-Row_2: track 0.62 -> 2.88 mm, vias 1 -> 2
- net Col_15-Row_2: track 0.46 -> 2.59 mm, vias 1 -> 2
- net Col_22-Row_1: track 11.6 -> 9.96 mm, vias 2 -> 1
- net Col_18-Row_2: track 1.06 -> 2.65 mm
- net Col_5-Row_2: track 6.35 -> 7.88 mm
- net Col_21-Row_1: track 12.5 -> 11.0 mm
- net Col_16-Row_2: track 1.16 -> 2.59 mm
- net Col_17-Row_2: track 0.90 -> 2.32 mm
- net Col_21-Row_2: track 10.4 -> 11.6 mm
- net Col_10-Row_2: track 3.98 -> 5.20 mm
- net Col_8-Row_2: track 4.08 -> 5.28 mm
- net Col_18-Row_4: track 7.05 -> 8.24 mm
- net Col_5-Row_1: track 7.91 -> 9.02 mm, vias 1 -> 2
- net Col_19-Row_4: track 7.51 -> 8.62 mm
- net Col_20-Row_3: track 8.67 -> 9.78 mm, vias 2 -> 3
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- removed copper zone on In7.Cu, net GND
- removed copper zone on In8.Cu, net GND
Other:
- copper layers 10 -> 8

Commit message: .
Parts:
- added Input_A1: 39-30-1060, Molex_PCB_Power_Connector:MOLEX_39-30-1060, B.Cu at (37.9, 66.3)
- added Input_B1: 39-30-1060, Molex_PCB_Power_Connector:MOLEX_39-30-1060, B.Cu at (175.4, 66.3)
- added J10: Conn_01x01_Socket, MountingHole:MountingHole_3.2mm_M3_DIN965_Pad, F.Cu at (26.9, 54.5)
- added J7: Conn_01x01_Socket, MountingHole:MountingHole_3.2mm_M3_DIN965_Pad, F.Cu at (26.9, 78.0)
- added J8: Conn_01x01_Socket, MountingHole:MountingHole_3.2mm_M3_DIN965_Pad, F.Cu at (186.4, 78.0)
- added J9: Conn_01x01_Socket, MountingHole:MountingHole_3.2mm_M3_DIN965_Pad, F.Cu at (186.4, 54.5)
Connections:
- J1 pad A15: unconnected-(J1-PadA15) -> Col_43-Row_1
- J1 pad A16: unconnected-(J1-PadA16) -> Col_43-Row_2
- J1 pad A17: unconnected-(J1-PadA17) -> Col_43-Row_3
- J1 pad A18: unconnected-(J1-PadA18) -> Col_42-Row_1
- J1 pad A19: unconnected-(J1-PadA19) -> Col_42-Row_2
- J1 pad A20: unconnected-(J1-PadA20) -> Col_42-Row_3
- J1 pad A21: unconnected-(J1-PadA21) -> Col_41-Row_1
- J1 pad A22: unconnected-(J1-PadA22) -> Col_41-Row_2
- J1 pad A23: unconnected-(J1-PadA23) -> Col_41-Row_3
- J1 pad A24: unconnected-(J1-PadA24) -> Col_40-Row_1
- J1 pad A25: unconnected-(J1-PadA25) -> Col_40-Row_2
- J1 pad A26: unconnected-(J1-PadA26) -> Col_40-Row_3
- J1 pad A27: unconnected-(J1-PadA27) -> Col_39-Row_1
- J1 pad A28: unconnected-(J1-PadA28) -> Col_39-Row_2
- J1 pad A29: unconnected-(J1-PadA29) -> Col_38-Row_1
- J1 pad A30: unconnected-(J1-PadA30) -> Col_39-Row_3
- J1 pad A31: unconnected-(J1-PadA31) -> Col_38-Row_2
- J1 pad A32: unconnected-(J1-PadA32) -> Col_38-Row_3
- J1 pad A33: unconnected-(J1-PadA33) -> Col_37-Row_1
- J1 pad A34: unconnected-(J1-PadA34) -> Col_37-Row_2
- J1 pad A35: unconnected-(J1-PadA35) -> Col_37-Row_3
- J1 pad A36: unconnected-(J1-PadA36) -> Col_36-Row_1
- J1 pad A37: unconnected-(J1-PadA37) -> Col_36-Row_2
- J1 pad A38: unconnected-(J1-PadA38) -> Col_36-Row_3
- J1 pad A39: unconnected-(J1-PadA39) -> Col_35-Row_1
- J1 pad A40: unconnected-(J1-PadA40) -> Col_35-Row_2
- J1 pad A41: unconnected-(J1-PadA41) -> Col_35-Row_3
- J1 pad A42: unconnected-(J1-PadA42) -> Col_34-Row_1
- J1 pad A43: unconnected-(J1-PadA43) -> Col_34-Row_2
- J1 pad A44: unconnected-(J1-PadA44) -> Col_34-Row_3
- J1 pad A45: unconnected-(J1-PadA45) -> Col_33-Row_1
- J1 pad A46: unconnected-(J1-PadA46) -> Col_33-Row_2
- J1 pad A47: unconnected-(J1-PadA47) -> Col_33-Row_3
- J1 pad A48: unconnected-(J1-PadA48) -> Col_32-Row_1
- J1 pad A49: unconnected-(J1-PadA49) -> Col_32-Row_2
- J1 pad A50: unconnected-(J1-PadA50) -> Col_32-Row_3
- J1 pad A51: unconnected-(J1-PadA51) -> Col_31-Row_1
- J1 pad A52: unconnected-(J1-PadA52) -> Col_31-Row_2
- J1 pad A53: unconnected-(J1-PadA53) -> Col_31-Row_3
- J1 pad A54: unconnected-(J1-PadA54) -> Col_30-Row_1
- J1 pad A55: unconnected-(J1-PadA55) -> Col_30-Row_2
- J1 pad A56: unconnected-(J1-PadA56) -> Col_30-Row_3
- J1 pad A57: unconnected-(J1-PadA57) -> Col_29-Row_1
- J1 pad A58: unconnected-(J1-PadA58) -> Col_29-Row_2
- J1 pad A59: unconnected-(J1-PadA59) -> Col_29-Row_3
- J1 pad A60: unconnected-(J1-PadA60) -> Col_28-Row_1
- J1 pad A61: unconnected-(J1-PadA61) -> Col_28-Row_2
- J1 pad A62: unconnected-(J1-PadA62) -> Col_28-Row_3
- J1 pad A63: unconnected-(J1-PadA63) -> Col_27-Row_1
- J1 pad A64: unconnected-(J1-PadA64) -> Col_27-Row_2
- J1 pad A65: unconnected-(J1-PadA65) -> Col_27-Row_3
- J1 pad A66: unconnected-(J1-PadA66) -> Col_26-Row_1
- J1 pad A67: unconnected-(J1-PadA67) -> Col_26-Row_2
- J1 pad A68: unconnected-(J1-PadA68) -> Col_26-Row_3
- J1 pad A69: unconnected-(J1-PadA69) -> Col_25-Row_1
- J1 pad A70: unconnected-(J1-PadA70) -> Col_25-Row_2
- J1 pad B15: unconnected-(J1-PadB15) -> Col_43-Row_4
- J1 pad B16: unconnected-(J1-PadB16) -> Col_43-Row_5
- J1 pad B17: unconnected-(J1-PadB17) -> Col_43-Row_6
- J1 pad B18: unconnected-(J1-PadB18) -> Col_42-Row_4
- J1 pad B19: unconnected-(J1-PadB19) -> Col_42-Row_5
- J1 pad B20: unconnected-(J1-PadB20) -> Col_42-Row_6
- J1 pad B21: unconnected-(J1-PadB21) -> Col_41-Row_4
- J1 pad B22: unconnected-(J1-PadB22) -> Col_41-Row_5
- J1 pad B23: unconnected-(J1-PadB23) -> Col_41-Row_6
- J1 pad B24: unconnected-(J1-PadB24) -> Col_40-Row_4
- J1 pad B25: unconnected-(J1-PadB25) -> Col_40-Row_5
- J1 pad B26: unconnected-(J1-PadB26) -> Col_40-Row_6
- J1 pad B27: unconnected-(J1-PadB27) -> Col_39-Row_4
- J1 pad B28: unconnected-(J1-PadB28) -> Col_39-Row_5
- J1 pad B29: unconnected-(J1-PadB29) -> Col_39-Row_6
- J1 pad B30: unconnected-(J1-PadB30) -> Col_38-Row_4
- J1 pad B31: unconnected-(J1-PadB31) -> Col_38-Row_5
- J1 pad B32: unconnected-(J1-PadB32) -> Col_38-Row_6
- J1 pad B33: unconnected-(J1-PadB33) -> Col_37-Row_4
- J1 pad B34: unconnected-(J1-PadB34) -> Col_37-Row_5
- J1 pad B35: unconnected-(J1-PadB35) -> Col_37-Row_6
- J1 pad B36: unconnected-(J1-PadB36) -> Col_36-Row_5
- J1 pad B37: unconnected-(J1-PadB37) -> Col_36-Row_4
- J1 pad B38: unconnected-(J1-PadB38) -> Col_35-Row_5
- J1 pad B39: unconnected-(J1-PadB39) -> Col_35-Row_4
- J1 pad B40: unconnected-(J1-PadB40) -> Col_34-Row_5
- J1 pad B41: unconnected-(J1-PadB41) -> Col_34-Row_4
- J1 pad B42: unconnected-(J1-PadB42) -> Col_33-Row_5
- J1 pad B43: unconnected-(J1-PadB43) -> Col_33-Row_4
- J1 pad B44: unconnected-(J1-PadB44) -> Col_32-Row_5
- J1 pad B45: unconnected-(J1-PadB45) -> Col_32-Row_4
- J1 pad B46: unconnected-(J1-PadB46) -> Col_31-Row_5
- J1 pad B47: unconnected-(J1-PadB47) -> Col_31-Row_4
- J1 pad B48: unconnected-(J1-PadB48) -> Col_30-Row_5
- J1 pad B49: unconnected-(J1-PadB49) -> Col_30-Row_4
- J1 pad B50: unconnected-(J1-PadB50) -> Col_29-Row_5
- J1 pad B51: unconnected-(J1-PadB51) -> Col_29-Row_4
- J1 pad B52: unconnected-(J1-PadB52) -> Col_28-Row_5
- J1 pad B53: unconnected-(J1-PadB53) -> Col_28-Row_4
- J1 pad B54: unconnected-(J1-PadB54) -> Col_27-Row_5
- J1 pad B55: unconnected-(J1-PadB55) -> Col_27-Row_4
- J1 pad B56: unconnected-(J1-PadB56) -> Col_26-Row_5
- J1 pad B57: unconnected-(J1-PadB57) -> Col_26-Row_4
- J1 pad B58: unconnected-(J1-PadB58) -> Col_25-Row_5
- J1 pad B59: unconnected-(J1-PadB59) -> Col_25-Row_3
- J1 pad B60: unconnected-(J1-PadB60) -> Col_25-Row_4
- J1 pad B61: unconnected-(J1-PadB61) -> Col_24-Row_5
- J1 pad B62: unconnected-(J1-PadB62) -> Col_24-Row_4
- J1 pad B63: unconnected-(J1-PadB63) -> Col_24-Row_1
- J1 pad B64: unconnected-(J1-PadB64) -> Col_24-Row_2
- J1 pad B65: unconnected-(J1-PadB65) -> Col_24-Row_3
- J1 pad B66: unconnected-(J1-PadB66) -> Col_23-Row_5
- J1 pad B67: unconnected-(J1-PadB67) -> Col_23-Row_4
- J1 pad B68: unconnected-(J1-PadB68) -> Col_23-Row_1
- J1 pad B69: unconnected-(J1-PadB69) -> Col_23-Row_2
- J1 pad B70: unconnected-(J1-PadB70) -> Col_23-Row_3
- U1 pad 353: unconnected-(U1-Col_23-Row_1-Pad353) -> Col_23-Row_1
- U1 pad 354: unconnected-(U1-Col_23-Row_2-Pad354) -> Col_23-Row_2
- U1 pad 355: unconnected-(U1-Col_23-Row_3-Pad355) -> Col_23-Row_3
- U1 pad 356: unconnected-(U1-Col_23-Row_4-Pad356) -> Col_23-Row_4
- U1 pad 357: unconnected-(U1-Col_23-Row_5-Pad357) -> Col_23-Row_5
- U1 pad 369: unconnected-(U1-Col_24-Row_1-Pad369) -> Col_24-Row_1
- U1 pad 370: unconnected-(U1-Col_24-Row_2-Pad370) -> Col_24-Row_2
- U1 pad 371: unconnected-(U1-Col_24-Row_3-Pad371) -> Col_24-Row_3
- U1 pad 372: unconnected-(U1-Col_24-Row_4-Pad372) -> Col_24-Row_4
- U1 pad 373: unconnected-(U1-Col_24-Row_5-Pad373) -> Col_24-Row_5
- U1 pad 385: unconnected-(U1-Col_25-Row_1-Pad385) -> Col_25-Row_1
- U1 pad 386: unconnected-(U1-Col_25-Row_2-Pad386) -> Col_25-Row_2
- U1 pad 387: unconnected-(U1-Col_25-Row_3-Pad387) -> Col_25-Row_3
- U1 pad 388: unconnected-(U1-Col_25-Row_4-Pad388) -> Col_25-Row_4
- U1 pad 389: unconnected-(U1-Col_25-Row_5-Pad389) -> Col_25-Row_5
- U1 pad 401: unconnected-(U1-Col_26-Row_1-Pad401) -> Col_26-Row_1
- U1 pad 402: unconnected-(U1-Col_26-Row_2-Pad402) -> Col_26-Row_2
- U1 pad 403: unconnected-(U1-Col_26-Row_3-Pad403) -> Col_26-Row_3
- U1 pad 404: unconnected-(U1-Col_26-Row_4-Pad404) -> Col_26-Row_4
- U1 pad 405: unconnected-(U1-Col_26-Row_5-Pad405) -> Col_26-Row_5
- U1 pad 417: unconnected-(U1-Col_27-Row_1-Pad417) -> Col_27-Row_1
- U1 pad 418: unconnected-(U1-Col_27-Row_2-Pad418) -> Col_27-Row_2
- U1 pad 419: unconnected-(U1-Col_27-Row_3-Pad419) -> Col_27-Row_3
- U1 pad 420: unconnected-(U1-Col_27-Row_4-Pad420) -> Col_27-Row_4
- U1 pad 421: unconnected-(U1-Col_27-Row_5-Pad421) -> Col_27-Row_5
- U1 pad 433: unconnected-(U1-Col_28-Row_1-Pad433) -> Col_28-Row_1
- U1 pad 434: unconnected-(U1-Col_28-Row_2-Pad434) -> Col_28-Row_2
- U1 pad 435: unconnected-(U1-Col_28-Row_3-Pad435) -> Col_28-Row_3
- U1 pad 436: unconnected-(U1-Col_28-Row_4-Pad436) -> Col_28-Row_4
- U1 pad 437: unconnected-(U1-Col_28-Row_5-Pad437) -> Col_28-Row_5
- U1 pad 449: unconnected-(U1-Col_29-Row_1-Pad449) -> Col_29-Row_1
- U1 pad 450: unconnected-(U1-Col_29-Row_2-Pad450) -> Col_29-Row_2
- U1 pad 451: unconnected-(U1-Col_29-Row_3-Pad451) -> Col_29-Row_3
- U1 pad 452: unconnected-(U1-Col_29-Row_4-Pad452) -> Col_29-Row_4
- U1 pad 453: unconnected-(U1-Col_29-Row_5-Pad453) -> Col_29-Row_5
- U1 pad 465: unconnected-(U1-Col_30-Row_1-Pad465) -> Col_30-Row_1
- U1 pad 466: unconnected-(U1-Col_30-Row_2-Pad466) -> Col_30-Row_2
- U1 pad 467: unconnected-(U1-Col_30-Row_3-Pad467) -> Col_30-Row_3
- U1 pad 468: unconnected-(U1-Col_30-Row_4-Pad468) -> Col_30-Row_4
- U1 pad 469: unconnected-(U1-Col_30-Row_5-Pad469) -> Col_30-Row_5
- U1 pad 481: unconnected-(U1-Col_31-Row_1-Pad481) -> Col_31-Row_1
- U1 pad 482: unconnected-(U1-Col_31-Row_2-Pad482) -> Col_31-Row_2
- U1 pad 483: unconnected-(U1-Col_31-Row_3-Pad483) -> Col_31-Row_3
- U1 pad 484: unconnected-(U1-Col_31-Row_4-Pad484) -> Col_31-Row_4
- U1 pad 485: unconnected-(U1-Col_31-Row_5-Pad485) -> Col_31-Row_5
- U1 pad 497: unconnected-(U1-Col_32-Row_1-Pad497) -> Col_32-Row_1
- U1 pad 498: unconnected-(U1-Col_32-Row_2-Pad498) -> Col_32-Row_2
- U1 pad 499: unconnected-(U1-Col_32-Row_3-Pad499) -> Col_32-Row_3
- U1 pad 500: unconnected-(U1-Col_32-Row_4-Pad500) -> Col_32-Row_4
- U1 pad 501: unconnected-(U1-Col_32-Row_5-Pad501) -> Col_32-Row_5
- U1 pad 513: unconnected-(U1-Col_33-Row_1-Pad513) -> Col_33-Row_1
- U1 pad 514: unconnected-(U1-Col_33-Row_2-Pad514) -> Col_33-Row_2
- U1 pad 515: unconnected-(U1-Col_33-Row_3-Pad515) -> Col_33-Row_3
- U1 pad 516: unconnected-(U1-Col_33-Row_4-Pad516) -> Col_33-Row_4
- U1 pad 517: unconnected-(U1-Col_33-Row_5-Pad517) -> Col_33-Row_5
- U1 pad 529: unconnected-(U1-Col_34-Row_1-Pad529) -> Col_34-Row_1
- U1 pad 530: unconnected-(U1-Col_34-Row_2-Pad530) -> Col_34-Row_2
- U1 pad 531: unconnected-(U1-Col_34-Row_3-Pad531) -> Col_34-Row_3
- U1 pad 532: unconnected-(U1-Col_34-Row_4-Pad532) -> Col_34-Row_4
- U1 pad 533: unconnected-(U1-Col_34-Row_5-Pad533) -> Col_34-Row_5
- U1 pad 545: unconnected-(U1-Col_35-Row_1-Pad545) -> Col_35-Row_1
- U1 pad 546: unconnected-(U1-Col_35-Row_2-Pad546) -> Col_35-Row_2
- U1 pad 547: unconnected-(U1-Col_35-Row_3-Pad547) -> Col_35-Row_3
- U1 pad 548: unconnected-(U1-Col_35-Row_4-Pad548) -> Col_35-Row_4
- U1 pad 549: unconnected-(U1-Col_35-Row_5-Pad549) -> Col_35-Row_5
- U1 pad 561: unconnected-(U1-Col_36-Row_1-Pad561) -> Col_36-Row_1
- U1 pad 562: unconnected-(U1-Col_36-Row_2-Pad562) -> Col_36-Row_2
- U1 pad 563: unconnected-(U1-Col_36-Row_3-Pad563) -> Col_36-Row_3
- U1 pad 564: unconnected-(U1-Col_36-Row_4-Pad564) -> Col_36-Row_4
- U1 pad 565: unconnected-(U1-Col_36-Row_5-Pad565) -> Col_36-Row_5
- U1 pad 577: unconnected-(U1-Col_37-Row_1-Pad577) -> Col_37-Row_1
- U1 pad 578: unconnected-(U1-Col_37-Row_2-Pad578) -> Col_37-Row_2
- U1 pad 579: unconnected-(U1-Col_37-Row_3-Pad579) -> Col_37-Row_3
- U1 pad 580: unconnected-(U1-Col_37-Row_4-Pad580) -> Col_37-Row_4
- U1 pad 581: unconnected-(U1-Col_37-Row_5-Pad581) -> Col_37-Row_5
- U1 pad 582: unconnected-(U1-Col_37-Row_6-Pad582) -> Col_37-Row_6
- U1 pad 593: unconnected-(U1-Col_38-Row_1-Pad593) -> Col_38-Row_1
- U1 pad 594: unconnected-(U1-Col_38-Row_2-Pad594) -> Col_38-Row_2
- U1 pad 595: unconnected-(U1-Col_38-Row_3-Pad595) -> Col_38-Row_3
- U1 pad 596: unconnected-(U1-Col_38-Row_4-Pad596) -> Col_38-Row_4
- U1 pad 597: unconnected-(U1-Col_38-Row_5-Pad597) -> Col_38-Row_5
- U1 pad 598: unconnected-(U1-Col_38-Row_6-Pad598) -> Col_38-Row_6
- U1 pad 609: unconnected-(U1-Col_39-Row_1-Pad609) -> Col_39-Row_1
- U1 pad 610: unconnected-(U1-Col_39-Row_2-Pad610) -> Col_39-Row_2
- U1 pad 611: unconnected-(U1-Col_39-Row_3-Pad611) -> Col_39-Row_3
- U1 pad 612: unconnected-(U1-Col_39-Row_4-Pad612) -> Col_39-Row_4
- U1 pad 613: unconnected-(U1-Col_39-Row_5-Pad613) -> Col_39-Row_5
- U1 pad 614: unconnected-(U1-Col_39-Row_6-Pad614) -> Col_39-Row_6
- U1 pad 625: unconnected-(U1-Col_40-Row_1-Pad625) -> Col_40-Row_1
- U1 pad 626: unconnected-(U1-Col_40-Row_2-Pad626) -> Col_40-Row_2
- U1 pad 627: unconnected-(U1-Col_40-Row_3-Pad627) -> Col_40-Row_3
- U1 pad 628: unconnected-(U1-Col_40-Row_4-Pad628) -> Col_40-Row_4
- U1 pad 629: unconnected-(U1-Col_40-Row_5-Pad629) -> Col_40-Row_5
- U1 pad 630: unconnected-(U1-Col_40-Row_6-Pad630) -> Col_40-Row_6
- U1 pad 641: unconnected-(U1-Col_41-Row_1-Pad641) -> Col_41-Row_1
- U1 pad 642: unconnected-(U1-Col_41-Row_2-Pad642) -> Col_41-Row_2
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Routing:
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Other:
- board size 121.5 x 31.5 mm -> 167.5 x 31.5 mm
- board text added: "G"
- board text added: "P1"
- board text added: "P2"

Commit message: .
Connections:
- J6 pad A15: unconnected-(J6-PadA15) -> Col_4-Row_15
- J6 pad A16: unconnected-(J6-PadA16) -> Col_4-Row_16
- J6 pad A17: unconnected-(J6-PadA17) -> Col_5-Row_14
- J6 pad A18: unconnected-(J6-PadA18) -> Col_5-Row_15
- J6 pad A19: unconnected-(J6-PadA19) -> Col_5-Row_16
- J6 pad A20: unconnected-(J6-PadA20) -> Col_6-Row_14
- J6 pad A21: unconnected-(J6-PadA21) -> Col_6-Row_15
- J6 pad A22: unconnected-(J6-PadA22) -> Col_6-Row_16
- J6 pad A23: unconnected-(J6-PadA23) -> Col_7-Row_14
- J6 pad A24: unconnected-(J6-PadA24) -> Col_7-Row_15
- J6 pad A25: unconnected-(J6-PadA25) -> Col_7-Row_16
- J6 pad A26: unconnected-(J6-PadA26) -> Col_8-Row_14
- J6 pad A27: unconnected-(J6-PadA27) -> Col_8-Row_15
- J6 pad A28: unconnected-(J6-PadA28) -> Col_8-Row_16
- J6 pad A29: unconnected-(J6-PadA29) -> Col_9-Row_14
- J6 pad A30: unconnected-(J6-PadA30) -> Col_9-Row_15
- J6 pad A31: unconnected-(J6-PadA31) -> Col_9-Row_16
- J6 pad A32: unconnected-(J6-PadA32) -> Col_10-Row_14
- J6 pad A33: unconnected-(J6-PadA33) -> Col_10-Row_15
- J6 pad A34: unconnected-(J6-PadA34) -> Col_10-Row_16
- J6 pad A35: unconnected-(J6-PadA35) -> Col_11-Row_14
- J6 pad A36: unconnected-(J6-PadA36) -> Col_11-Row_15
- J6 pad A37: unconnected-(J6-PadA37) -> Col_11-Row_16
- J6 pad A38: unconnected-(J6-PadA38) -> Col_12-Row_14
- J6 pad A39: unconnected-(J6-PadA39) -> Col_12-Row_15
- J6 pad A40: unconnected-(J6-PadA40) -> Col_12-Row_16
- J6 pad A41: unconnected-(J6-PadA41) -> Col_13-Row_14
- J6 pad A42: unconnected-(J6-PadA42) -> Col_13-Row_15
- J6 pad A43: unconnected-(J6-PadA43) -> Col_13-Row_16
- J6 pad A44: unconnected-(J6-PadA44) -> Col_14-Row_14
- J6 pad A45: unconnected-(J6-PadA45) -> Col_14-Row_15
- J6 pad A46: unconnected-(J6-PadA46) -> Col_14-Row_16
- J6 pad A47: unconnected-(J6-PadA47) -> Col_15-Row_14
- J6 pad A48: unconnected-(J6-PadA48) -> Col_15-Row_15
- J6 pad A49: unconnected-(J6-PadA49) -> Col_15-Row_16
- J6 pad A50: unconnected-(J6-PadA50) -> Col_16-Row_14
- J6 pad A51: unconnected-(J6-PadA51) -> Col_16-Row_15
- J6 pad A52: unconnected-(J6-PadA52) -> Col_16-Row_16
- J6 pad A53: unconnected-(J6-PadA53) -> Col_17-Row_14
- J6 pad A54: unconnected-(J6-PadA54) -> Col_17-Row_15
- J6 pad A55: unconnected-(J6-PadA55) -> Col_17-Row_16
- J6 pad A56: unconnected-(J6-PadA56) -> Col_18-Row_14
- J6 pad A57: unconnected-(J6-PadA57) -> Col_18-Row_15
- J6 pad A58: unconnected-(J6-PadA58) -> Col_18-Row_16
- J6 pad A59: unconnected-(J6-PadA59) -> Col_19-Row_14
- J6 pad A60: unconnected-(J6-PadA60) -> Col_19-Row_15
- J6 pad A61: unconnected-(J6-PadA61) -> Col_19-Row_16
- J6 pad A62: unconnected-(J6-PadA62) -> Col_20-Row_14
- J6 pad A63: unconnected-(J6-PadA63) -> Col_20-Row_15
- J6 pad A64: unconnected-(J6-PadA64) -> Col_20-Row_16
- J6 pad A65: unconnected-(J6-PadA65) -> Col_21-Row_14
- J6 pad A66: unconnected-(J6-PadA66) -> Col_21-Row_15
- J6 pad A67: unconnected-(J6-PadA67) -> Col_21-Row_16
- J6 pad A68: unconnected-(J6-PadA68) -> Col_22-Row_14
- J6 pad A69: unconnected-(J6-PadA69) -> Col_22-Row_15
- J6 pad A70: unconnected-(J6-PadA70) -> Col_22-Row_16
- J6 pad B15: unconnected-(J6-PadB15) -> Col_2-Row_14
- J6 pad B16: unconnected-(J6-PadB16) -> Col_2-Row_15
- J6 pad B17: unconnected-(J6-PadB17) -> Col_2-Row_16
- J6 pad B18: unconnected-(J6-PadB18) -> Col_3-Row_14
- J6 pad B19: unconnected-(J6-PadB19) -> Col_3-Row_15
- J6 pad B20: unconnected-(J6-PadB20) -> Col_3-Row_16
- J6 pad B21: unconnected-(J6-PadB21) -> Col_4-Row_14
- J6 pad B22: unconnected-(J6-PadB22) -> Col_2-Row_13
- J6 pad B23: unconnected-(J6-PadB23) -> Col_2-Row_12
- J6 pad B24: unconnected-(J6-PadB24) -> Col_3-Row_13
- J6 pad B25: unconnected-(J6-PadB25) -> Col_3-Row_12
- J6 pad B26: unconnected-(J6-PadB26) -> Col_4-Row_13
- J6 pad B27: unconnected-(J6-PadB27) -> Col_4-Row_12
- J6 pad B28: unconnected-(J6-PadB28) -> Col_5-Row_13
- J6 pad B29: unconnected-(J6-PadB29) -> Col_5-Row_12
- J6 pad B30: unconnected-(J6-PadB30) -> Col_6-Row_13
- J6 pad B31: unconnected-(J6-PadB31) -> Col_6-Row_12
- J6 pad B32: unconnected-(J6-PadB32) -> Col_7-Row_13
- J6 pad B33: unconnected-(J6-PadB33) -> Col_7-Row_12
- J6 pad B34: unconnected-(J6-PadB34) -> Col_8-Row_13
- J6 pad B35: unconnected-(J6-PadB35) -> Col_8-Row_12
- J6 pad B36: unconnected-(J6-PadB36) -> Col_9-Row_13
- J6 pad B37: unconnected-(J6-PadB37) -> Col_9-Row_12
- J6 pad B38: unconnected-(J6-PadB38) -> Col_10-Row_13
- J6 pad B39: unconnected-(J6-PadB39) -> Col_10-Row_12
- J6 pad B40: unconnected-(J6-PadB40) -> Col_11-Row_13
- J6 pad B41: unconnected-(J6-PadB41) -> Col_11-Row_12
- J6 pad B42: unconnected-(J6-PadB42) -> Col_12-Row_13
- J6 pad B43: unconnected-(J6-PadB43) -> Col_12-Row_12
- J6 pad B44: unconnected-(J6-PadB44) -> Col_13-Row_13
- J6 pad B45: unconnected-(J6-PadB45) -> Col_13-Row_12
- J6 pad B46: unconnected-(J6-PadB46) -> Col_14-Row_13
- J6 pad B47: unconnected-(J6-PadB47) -> Col_14-Row_12
- J6 pad B48: unconnected-(J6-PadB48) -> Col_15-Row_13
- J6 pad B49: unconnected-(J6-PadB49) -> Col_15-Row_12
- J6 pad B50: unconnected-(J6-PadB50) -> Col_16-Row_13
- J6 pad B51: unconnected-(J6-PadB51) -> Col_16-Row_12
- J6 pad B52: unconnected-(J6-PadB52) -> Col_16-Row_11
- J6 pad B53: unconnected-(J6-PadB53) -> Col_17-Row_13
- J6 pad B54: unconnected-(J6-PadB54) -> Col_17-Row_12
- J6 pad B55: unconnected-(J6-PadB55) -> Col_17-Row_11
- J6 pad B56: unconnected-(J6-PadB56) -> Col_18-Row_13
- J6 pad B57: unconnected-(J6-PadB57) -> Col_18-Row_12
- J6 pad B58: unconnected-(J6-PadB58) -> Col_18-Row_11
- J6 pad B59: unconnected-(J6-PadB59) -> Col_19-Row_13
- J6 pad B60: unconnected-(J6-PadB60) -> Col_19-Row_12
- J6 pad B61: unconnected-(J6-PadB61) -> Col_19-Row_11
- J6 pad B62: unconnected-(J6-PadB62) -> Col_20-Row_13
- J6 pad B63: unconnected-(J6-PadB63) -> Col_20-Row_12
- J6 pad B64: unconnected-(J6-PadB64) -> Col_20-Row_11
- J6 pad B65: unconnected-(J6-PadB65) -> Col_21-Row_13
- J6 pad B66: unconnected-(J6-PadB66) -> Col_21-Row_12
- J6 pad B67: unconnected-(J6-PadB67) -> Col_21-Row_11
- J6 pad B68: unconnected-(J6-PadB68) -> Col_22-Row_13
- J6 pad B69: unconnected-(J6-PadB69) -> Col_22-Row_12
- J6 pad B70: unconnected-(J6-PadB70) -> Col_22-Row_11
- U1 pad 108: unconnected-(U1-Col_7-Row_12-Pad108) -> Col_7-Row_12
- U1 pad 109: unconnected-(U1-Col_7-Row_13-Pad109) -> Col_7-Row_13
- U1 pad 110: unconnected-(U1-Col_7-Row_14-Pad110) -> Col_7-Row_14
- U1 pad 111: unconnected-(U1-Col_7-Row_15-Pad111) -> Col_7-Row_15
- U1 pad 112: unconnected-(U1-Col_7-Row_16-Pad112) -> Col_7-Row_16
- U1 pad 124: unconnected-(U1-Col_8-Row_12-Pad124) -> Col_8-Row_12
- U1 pad 125: unconnected-(U1-Col_8-Row_13-Pad125) -> Col_8-Row_13
- U1 pad 126: unconnected-(U1-Col_8-Row_14-Pad126) -> Col_8-Row_14
- U1 pad 127: unconnected-(U1-Col_8-Row_15-Pad127) -> Col_8-Row_15
- U1 pad 128: unconnected-(U1-Col_8-Row_16-Pad128) -> Col_8-Row_16
- U1 pad 140: unconnected-(U1-Col_9-Row_12-Pad140) -> Col_9-Row_12
- U1 pad 141: unconnected-(U1-Col_9-Row_13-Pad141) -> Col_9-Row_13
- U1 pad 142: unconnected-(U1-Col_9-Row_14-Pad142) -> Col_9-Row_14
- U1 pad 143: unconnected-(U1-Col_9-Row_15-Pad143) -> Col_9-Row_15
- U1 pad 144: unconnected-(U1-Col_9-Row_16-Pad144) -> Col_9-Row_16
- U1 pad 156: unconnected-(U1-Col_10-Row_12-Pad156) -> Col_10-Row_12
- U1 pad 157: unconnected-(U1-Col_10-Row_13-Pad157) -> Col_10-Row_13
- U1 pad 158: unconnected-(U1-Col_10-Row_14-Pad158) -> Col_10-Row_14
- U1 pad 159: unconnected-(U1-Col_10-Row_15-Pad159) -> Col_10-Row_15
- U1 pad 160: unconnected-(U1-Col_10-Row_16-Pad160) -> Col_10-Row_16
- U1 pad 172: unconnected-(U1-Col_11-Row_12-Pad172) -> Col_11-Row_12
- U1 pad 173: unconnected-(U1-Col_11-Row_13-Pad173) -> Col_11-Row_13
- U1 pad 174: unconnected-(U1-Col_11-Row_14-Pad174) -> Col_11-Row_14
- U1 pad 175: unconnected-(U1-Col_11-Row_15-Pad175) -> Col_11-Row_15
- U1 pad 176: unconnected-(U1-Col_11-Row_16-Pad176) -> Col_11-Row_16
- U1 pad 188: unconnected-(U1-Col_12-Row_12-Pad188) -> Col_12-Row_12
- U1 pad 189: unconnected-(U1-Col_12-Row_13-Pad189) -> Col_12-Row_13
- U1 pad 190: unconnected-(U1-Col_12-Row_14-Pad190) -> Col_12-Row_14
- U1 pad 191: unconnected-(U1-Col_12-Row_15-Pad191) -> Col_12-Row_15
- U1 pad 192: unconnected-(U1-Col_12-Row_16-Pad192) -> Col_12-Row_16
- U1 pad 204: unconnected-(U1-Col_13-Row_12-Pad204) -> Col_13-Row_12
- U1 pad 205: unconnected-(U1-Col_13-Row_13-Pad205) -> Col_13-Row_13
- U1 pad 206: unconnected-(U1-Col_13-Row_14-Pad206) -> Col_13-Row_14
- U1 pad 207: unconnected-(U1-Col_13-Row_15-Pad207) -> Col_13-Row_15
- U1 pad 208: unconnected-(U1-Col_13-Row_16-Pad208) -> Col_13-Row_16
- U1 pad 220: unconnected-(U1-Col_14-Row_12-Pad220) -> Col_14-Row_12
- U1 pad 221: unconnected-(U1-Col_14-Row_13-Pad221) -> Col_14-Row_13
- U1 pad 222: unconnected-(U1-Col_14-Row_14-Pad222) -> Col_14-Row_14
- U1 pad 223: unconnected-(U1-Col_14-Row_15-Pad223) -> Col_14-Row_15
- U1 pad 224: unconnected-(U1-Col_14-Row_16-Pad224) -> Col_14-Row_16
- U1 pad 236: unconnected-(U1-Col_15-Row_12-Pad236) -> Col_15-Row_12
- U1 pad 237: unconnected-(U1-Col_15-Row_13-Pad237) -> Col_15-Row_13
- U1 pad 238: unconnected-(U1-Col_15-Row_14-Pad238) -> Col_15-Row_14
- U1 pad 239: unconnected-(U1-Col_15-Row_15-Pad239) -> Col_15-Row_15
- U1 pad 240: unconnected-(U1-Col_15-Row_16-Pad240) -> Col_15-Row_16
- U1 pad 251: unconnected-(U1-Col_16-Row_11-Pad251) -> Col_16-Row_11
- U1 pad 252: unconnected-(U1-Col_16-Row_12-Pad252) -> Col_16-Row_12
- U1 pad 253: unconnected-(U1-Col_16-Row_13-Pad253) -> Col_16-Row_13
- U1 pad 254: unconnected-(U1-Col_16-Row_14-Pad254) -> Col_16-Row_14
- U1 pad 255: unconnected-(U1-Col_16-Row_15-Pad255) -> Col_16-Row_15
- U1 pad 256: unconnected-(U1-Col_16-Row_16-Pad256) -> Col_16-Row_16
- U1 pad 267: unconnected-(U1-Col_17-Row_11-Pad267) -> Col_17-Row_11
- U1 pad 268: unconnected-(U1-Col_17-Row_12-Pad268) -> Col_17-Row_12
- U1 pad 269: unconnected-(U1-Col_17-Row_13-Pad269) -> Col_17-Row_13
- U1 pad 270: unconnected-(U1-Col_17-Row_14-Pad270) -> Col_17-Row_14
- U1 pad 271: unconnected-(U1-Col_17-Row_15-Pad271) -> Col_17-Row_15
- U1 pad 272: unconnected-(U1-Col_17-Row_16-Pad272) -> Col_17-Row_16
- U1 pad 28: unconnected-(U1-Col_2-Row_12-Pad28) -> Col_2-Row_12
- U1 pad 283: unconnected-(U1-Col_18-Row_11-Pad283) -> Col_18-Row_11
- U1 pad 284: unconnected-(U1-Col_18-Row_12-Pad284) -> Col_18-Row_12
- U1 pad 285: unconnected-(U1-Col_18-Row_13-Pad285) -> Col_18-Row_13
- U1 pad 286: unconnected-(U1-Col_18-Row_14-Pad286) -> Col_18-Row_14
- U1 pad 287: unconnected-(U1-Col_18-Row_15-Pad287) -> Col_18-Row_15
- U1 pad 288: unconnected-(U1-Col_18-Row_16-Pad288) -> Col_18-Row_16
- U1 pad 29: unconnected-(U1-Col_2-Row_13-Pad29) -> Col_2-Row_13
- U1 pad 299: unconnected-(U1-Col_19-Row_11-Pad299) -> Col_19-Row_11
- U1 pad 30: unconnected-(U1-Col_2-Row_14-Pad30) -> Col_2-Row_14
- U1 pad 300: unconnected-(U1-Col_19-Row_12-Pad300) -> Col_19-Row_12
- U1 pad 301: unconnected-(U1-Col_19-Row_13-Pad301) -> Col_19-Row_13
- U1 pad 302: unconnected-(U1-Col_19-Row_14-Pad302) -> Col_19-Row_14
- U1 pad 303: unconnected-(U1-Col_19-Row_15-Pad303) -> Col_19-Row_15
- U1 pad 304: unconnected-(U1-Col_19-Row_16-Pad304) -> Col_19-Row_16
- U1 pad 31: unconnected-(U1-Col_2-Row_15-Pad31) -> Col_2-Row_15
- U1 pad 315: unconnected-(U1-Col_20-Row_11-Pad315) -> Col_20-Row_11
- U1 pad 316: unconnected-(U1-Col_20-Row_12-Pad316) -> Col_20-Row_12
- U1 pad 317: unconnected-(U1-Col_20-Row_13-Pad317) -> Col_20-Row_13
- U1 pad 318: unconnected-(U1-Col_20-Row_14-Pad318) -> Col_20-Row_14
- U1 pad 319: unconnected-(U1-Col_20-Row_15-Pad319) -> Col_20-Row_15
- U1 pad 32: unconnected-(U1-Col_2-Row_16-Pad32) -> Col_2-Row_16
- U1 pad 320: unconnected-(U1-Col_20-Row_16-Pad320) -> Col_20-Row_16
- U1 pad 331: unconnected-(U1-Col_21-Row_11-Pad331) -> Col_21-Row_11
- U1 pad 332: unconnected-(U1-Col_21-Row_12-Pad332) -> Col_21-Row_12
- U1 pad 333: unconnected-(U1-Col_21-Row_13-Pad333) -> Col_21-Row_13
- U1 pad 334: unconnected-(U1-Col_21-Row_14-Pad334) -> Col_21-Row_14
- U1 pad 335: unconnected-(U1-Col_21-Row_15-Pad335) -> Col_21-Row_15
- U1 pad 336: unconnected-(U1-Col_21-Row_16-Pad336) -> Col_21-Row_16
- U1 pad 347: unconnected-(U1-Col_22-Row_11-Pad347) -> Col_22-Row_11
- U1 pad 348: unconnected-(U1-Col_22-Row_12-Pad348) -> Col_22-Row_12
- U1 pad 349: unconnected-(U1-Col_22-Row_13-Pad349) -> Col_22-Row_13
- U1 pad 350: unconnected-(U1-Col_22-Row_14-Pad350) -> Col_22-Row_14
- U1 pad 351: unconnected-(U1-Col_22-Row_15-Pad351) -> Col_22-Row_15
- U1 pad 352: unconnected-(U1-Col_22-Row_16-Pad352) -> Col_22-Row_16
- U1 pad 44: unconnected-(U1-Col_3-Row_12-Pad44) -> Col_3-Row_12
- U1 pad 45: unconnected-(U1-Col_3-Row_13-Pad45) -> Col_3-Row_13
- U1 pad 46: unconnected-(U1-Col_3-Row_14-Pad46) -> Col_3-Row_14
- U1 pad 47: unconnected-(U1-Col_3-Row_15-Pad47) -> Col_3-Row_15
- U1 pad 48: unconnected-(U1-Col_3-Row_16-Pad48) -> Col_3-Row_16
- U1 pad 60: unconnected-(U1-Col_4-Row_12-Pad60) -> Col_4-Row_12
- U1 pad 61: unconnected-(U1-Col_4-Row_13-Pad61) -> Col_4-Row_13
- U1 pad 62: unconnected-(U1-Col_4-Row_14-Pad62) -> Col_4-Row_14
- U1 pad 63: unconnected-(U1-Col_4-Row_15-Pad63) -> Col_4-Row_15
- U1 pad 64: unconnected-(U1-Col_4-Row_16-Pad64) -> Col_4-Row_16
- U1 pad 76: unconnected-(U1-Col_5-Row_12-Pad76) -> Col_5-Row_12
- U1 pad 77: unconnected-(U1-Col_5-Row_13-Pad77) -> Col_5-Row_13
- U1 pad 78: unconnected-(U1-Col_5-Row_14-Pad78) -> Col_5-Row_14
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
Commit message: .
Connections:
- J3 pad A15: unconnected-(J3-PadA15) -> Col_43-Row_14
- J3 pad A16: unconnected-(J3-PadA16) -> Col_43-Row_15
- J3 pad A17: unconnected-(J3-PadA17) -> Col_43-Row_16
- J3 pad A18: unconnected-(J3-PadA18) -> Col_42-Row_14
- J3 pad A19: unconnected-(J3-PadA19) -> Col_42-Row_15
- J3 pad A20: unconnected-(J3-PadA20) -> Col_42-Row_16
- J3 pad A21: unconnected-(J3-PadA21) -> Col_41-Row_14
- J3 pad A22: unconnected-(J3-PadA22) -> Col_43-Row_13
- J3 pad A23: unconnected-(J3-PadA23) -> Col_43-Row_12
- J3 pad A24: unconnected-(J3-PadA24) -> Col_42-Row_13
- J3 pad A25: unconnected-(J3-PadA25) -> Col_42-Row_12
- J3 pad A26: unconnected-(J3-PadA26) -> Col_41-Row_13
- J3 pad A27: unconnected-(J3-PadA27) -> Col_41-Row_12
- J3 pad A28: unconnected-(J3-PadA28) -> Col_40-Row_13
- J3 pad A29: unconnected-(J3-PadA29) -> Col_40-Row_12
- J3 pad A30: unconnected-(J3-PadA30) -> Col_39-Row_13
- J3 pad A31: unconnected-(J3-PadA31) -> Col_39-Row_12
- J3 pad A32: unconnected-(J3-PadA32) -> Col_38-Row_13
- J3 pad A33: unconnected-(J3-PadA33) -> Col_38-Row_12
- J3 pad A34: unconnected-(J3-PadA34) -> Col_37-Row_13
- J3 pad A35: unconnected-(J3-PadA35) -> Col_37-Row_12
- J3 pad A36: unconnected-(J3-PadA36) -> Col_36-Row_13
- J3 pad A37: unconnected-(J3-PadA37) -> Col_36-Row_12
- J3 pad A38: unconnected-(J3-PadA38) -> Col_35-Row_13
- J3 pad A39: unconnected-(J3-PadA39) -> Col_35-Row_12
- J3 pad A40: unconnected-(J3-PadA40) -> Col_34-Row_13
- J3 pad A41: unconnected-(J3-PadA41) -> Col_34-Row_12
- J3 pad A42: unconnected-(J3-PadA42) -> Col_33-Row_13
- J3 pad A43: unconnected-(J3-PadA43) -> Col_33-Row_12
- J3 pad A44: unconnected-(J3-PadA44) -> Col_32-Row_13
- J3 pad A45: unconnected-(J3-PadA45) -> Col_32-Row_12
- J3 pad A46: unconnected-(J3-PadA46) -> Col_31-Row_13
- J3 pad A47: unconnected-(J3-PadA47) -> Col_31-Row_12
- J3 pad A48: unconnected-(J3-PadA48) -> Col_30-Row_13
- J3 pad A49: unconnected-(J3-PadA49) -> Col_30-Row_12
- J3 pad A50: unconnected-(J3-PadA50) -> Col_29-Row_13
- J3 pad A51: unconnected-(J3-PadA51) -> Col_29-Row_12
- J3 pad A52: unconnected-(J3-PadA52) -> Col_29-Row_11
- J3 pad A53: unconnected-(J3-PadA53) -> Col_28-Row_13
- J3 pad A54: unconnected-(J3-PadA54) -> Col_28-Row_12
- J3 pad A55: unconnected-(J3-PadA55) -> Col_28-Row_11
- J3 pad A56: unconnected-(J3-PadA56) -> Col_27-Row_13
- J3 pad A57: unconnected-(J3-PadA57) -> Col_27-Row_12
- J3 pad A58: unconnected-(J3-PadA58) -> Col_27-Row_11
- J3 pad A59: unconnected-(J3-PadA59) -> Col_26-Row_13
- J3 pad A60: unconnected-(J3-PadA60) -> Col_26-Row_12
- J3 pad A61: unconnected-(J3-PadA61) -> Col_26-Row_11
- J3 pad A62: unconnected-(J3-PadA62) -> Col_25-Row_13
- J3 pad A63: unconnected-(J3-PadA63) -> Col_25-Row_12
- J3 pad A64: unconnected-(J3-PadA64) -> Col_25-Row_11
- J3 pad A65: unconnected-(J3-PadA65) -> Col_24-Row_13
- J3 pad A66: unconnected-(J3-PadA66) -> Col_24-Row_12
- J3 pad A67: unconnected-(J3-PadA67) -> Col_24-Row_11
- J3 pad A68: unconnected-(J3-PadA68) -> Col_23-Row_13
- J3 pad A69: unconnected-(J3-PadA69) -> Col_23-Row_12
- J3 pad A70: unconnected-(J3-PadA70) -> Col_23-Row_11
- J3 pad B15: unconnected-(J3-PadB15) -> Col_41-Row_15
- J3 pad B16: unconnected-(J3-PadB16) -> Col_41-Row_16
- J3 pad B17: unconnected-(J3-PadB17) -> Col_40-Row_14
- J3 pad B18: unconnected-(J3-PadB18) -> Col_40-Row_15
- J3 pad B19: unconnected-(J3-PadB19) -> Col_40-Row_16
- J3 pad B20: unconnected-(J3-PadB20) -> Col_39-Row_14
- J3 pad B21: unconnected-(J3-PadB21) -> Col_39-Row_15
- J3 pad B22: unconnected-(J3-PadB22) -> Col_39-Row_16
- J3 pad B23: unconnected-(J3-PadB23) -> Col_38-Row_14
- J3 pad B24: unconnected-(J3-PadB24) -> Col_38-Row_15
- J3 pad B25: unconnected-(J3-PadB25) -> Col_38-Row_16
- J3 pad B26: unconnected-(J3-PadB26) -> Col_37-Row_14
- J3 pad B27: unconnected-(J3-PadB27) -> Col_37-Row_15
- J3 pad B28: unconnected-(J3-PadB28) -> Col_37-Row_16
- J3 pad B29: unconnected-(J3-PadB29) -> Col_36-Row_14
- J3 pad B30: unconnected-(J3-PadB30) -> Col_36-Row_15
- J3 pad B31: unconnected-(J3-PadB31) -> Col_36-Row_16
- J3 pad B32: unconnected-(J3-PadB32) -> Col_35-Row_14
- J3 pad B33: unconnected-(J3-PadB33) -> Col_35-Row_15
- J3 pad B34: unconnected-(J3-PadB34) -> Col_35-Row_16
- J3 pad B35: unconnected-(J3-PadB35) -> Col_34-Row_14
- J3 pad B36: unconnected-(J3-PadB36) -> Col_34-Row_15
- J3 pad B37: unconnected-(J3-PadB37) -> Col_34-Row_16
- J3 pad B38: unconnected-(J3-PadB38) -> Col_33-Row_14
- J3 pad B39: unconnected-(J3-PadB39) -> Col_33-Row_15
- J3 pad B40: unconnected-(J3-PadB40) -> Col_33-Row_16
- J3 pad B41: unconnected-(J3-PadB41) -> Col_32-Row_14
- J3 pad B42: unconnected-(J3-PadB42) -> Col_32-Row_15
- J3 pad B43: unconnected-(J3-PadB43) -> Col_32-Row_16
- J3 pad B44: unconnected-(J3-PadB44) -> Col_31-Row_14
- J3 pad B45: unconnected-(J3-PadB45) -> Col_31-Row_15
- J3 pad B46: unconnected-(J3-PadB46) -> Col_31-Row_16
- J3 pad B47: unconnected-(J3-PadB47) -> Col_30-Row_14
- J3 pad B48: unconnected-(J3-PadB48) -> Col_30-Row_15
- J3 pad B49: unconnected-(J3-PadB49) -> Col_30-Row_16
- J3 pad B50: unconnected-(J3-PadB50) -> Col_29-Row_14
- J3 pad B51: unconnected-(J3-PadB51) -> Col_29-Row_15
- J3 pad B52: unconnected-(J3-PadB52) -> Col_29-Row_16
- J3 pad B53: unconnected-(J3-PadB53) -> Col_28-Row_14
- J3 pad B54: unconnected-(J3-PadB54) -> Col_28-Row_15
- J3 pad B55: unconnected-(J3-PadB55) -> Col_28-Row_16
- J3 pad B56: unconnected-(J3-PadB56) -> Col_27-Row_14
- J3 pad B57: unconnected-(J3-PadB57) -> Col_27-Row_15
- J3 pad B58: unconnected-(J3-PadB58) -> Col_27-Row_16
- J3 pad B59: unconnected-(J3-PadB59) -> Col_26-Row_14
- J3 pad B60: unconnected-(J3-PadB60) -> Col_26-Row_15
- J3 pad B61: unconnected-(J3-PadB61) -> Col_26-Row_16
- J3 pad B62: unconnected-(J3-PadB62) -> Col_25-Row_14
- J3 pad B63: unconnected-(J3-PadB63) -> Col_25-Row_15
- J3 pad B64: unconnected-(J3-PadB64) -> Col_25-Row_16
- J3 pad B65: unconnected-(J3-PadB65) -> Col_24-Row_14
- J3 pad B66: unconnected-(J3-PadB66) -> Col_24-Row_15
- J3 pad B67: unconnected-(J3-PadB67) -> Col_24-Row_16
- J3 pad B68: unconnected-(J3-PadB68) -> Col_23-Row_14
- J3 pad B69: unconnected-(J3-PadB69) -> Col_23-Row_15
- J3 pad B70: unconnected-(J3-PadB70) -> Col_23-Row_16
- U1 pad 363: unconnected-(U1-Col_23-Row_11-Pad363) -> Col_23-Row_11
- U1 pad 364: unconnected-(U1-Col_23-Row_12-Pad364) -> Col_23-Row_12
- U1 pad 365: unconnected-(U1-Col_23-Row_13-Pad365) -> Col_23-Row_13
- U1 pad 366: unconnected-(U1-Col_23-Row_14-Pad366) -> Col_23-Row_14
- U1 pad 367: unconnected-(U1-Col_23-Row_15-Pad367) -> Col_23-Row_15
- U1 pad 368: unconnected-(U1-Col_23-Row_16-Pad368) -> Col_23-Row_16
- U1 pad 379: unconnected-(U1-Col_24-Row_11-Pad379) -> Col_24-Row_11
- U1 pad 380: unconnected-(U1-Col_24-Row_12-Pad380) -> Col_24-Row_12
- U1 pad 381: unconnected-(U1-Col_24-Row_13-Pad381) -> Col_24-Row_13
- U1 pad 382: unconnected-(U1-Col_24-Row_14-Pad382) -> Col_24-Row_14
- U1 pad 383: unconnected-(U1-Col_24-Row_15-Pad383) -> Col_24-Row_15
- U1 pad 384: unconnected-(U1-Col_24-Row_16-Pad384) -> Col_24-Row_16
- U1 pad 395: unconnected-(U1-Col_25-Row_11-Pad395) -> Col_25-Row_11
- U1 pad 396: unconnected-(U1-Col_25-Row_12-Pad396) -> Col_25-Row_12
- U1 pad 397: unconnected-(U1-Col_25-Row_13-Pad397) -> Col_25-Row_13
- U1 pad 398: unconnected-(U1-Col_25-Row_14-Pad398) -> Col_25-Row_14
- U1 pad 399: unconnected-(U1-Col_25-Row_15-Pad399) -> Col_25-Row_15
- U1 pad 400: unconnected-(U1-Col_25-Row_16-Pad400) -> Col_25-Row_16
- U1 pad 411: unconnected-(U1-Col_26-Row_11-Pad411) -> Col_26-Row_11
- U1 pad 412: unconnected-(U1-Col_26-Row_12-Pad412) -> Col_26-Row_12
- U1 pad 413: unconnected-(U1-Col_26-Row_13-Pad413) -> Col_26-Row_13
- U1 pad 414: unconnected-(U1-Col_26-Row_14-Pad414) -> Col_26-Row_14
- U1 pad 415: unconnected-(U1-Col_26-Row_15-Pad415) -> Col_26-Row_15
- U1 pad 416: unconnected-(U1-Col_26-Row_16-Pad416) -> Col_26-Row_16
- U1 pad 427: unconnected-(U1-Col_27-Row_11-Pad427) -> Col_27-Row_11
- U1 pad 428: unconnected-(U1-Col_27-Row_12-Pad428) -> Col_27-Row_12
- U1 pad 429: unconnected-(U1-Col_27-Row_13-Pad429) -> Col_27-Row_13
- U1 pad 430: unconnected-(U1-Col_27-Row_14-Pad430) -> Col_27-Row_14
- U1 pad 431: unconnected-(U1-Col_27-Row_15-Pad431) -> Col_27-Row_15
- U1 pad 432: unconnected-(U1-Col_27-Row_16-Pad432) -> Col_27-Row_16
- U1 pad 443: unconnected-(U1-Col_28-Row_11-Pad443) -> Col_28-Row_11
- U1 pad 444: unconnected-(U1-Col_28-Row_12-Pad444) -> Col_28-Row_12
- U1 pad 445: unconnected-(U1-Col_28-Row_13-Pad445) -> Col_28-Row_13
- U1 pad 446: unconnected-(U1-Col_28-Row_14-Pad446) -> Col_28-Row_14
- U1 pad 447: unconnected-(U1-Col_28-Row_15-Pad447) -> Col_28-Row_15
- U1 pad 448: unconnected-(U1-Col_28-Row_16-Pad448) -> Col_28-Row_16
- U1 pad 459: unconnected-(U1-Col_29-Row_11-Pad459) -> Col_29-Row_11
- U1 pad 460: unconnected-(U1-Col_29-Row_12-Pad460) -> Col_29-Row_12
- U1 pad 461: unconnected-(U1-Col_29-Row_13-Pad461) -> Col_29-Row_13
- U1 pad 462: unconnected-(U1-Col_29-Row_14-Pad462) -> Col_29-Row_14
- U1 pad 463: unconnected-(U1-Col_29-Row_15-Pad463) -> Col_29-Row_15
- U1 pad 464: unconnected-(U1-Col_29-Row_16-Pad464) -> Col_29-Row_16
- U1 pad 476: unconnected-(U1-Col_30-Row_12-Pad476) -> Col_30-Row_12
- U1 pad 477: unconnected-(U1-Col_30-Row_13-Pad477) -> Col_30-Row_13
- U1 pad 478: unconnected-(U1-Col_30-Row_14-Pad478) -> Col_30-Row_14
- U1 pad 479: unconnected-(U1-Col_30-Row_15-Pad479) -> Col_30-Row_15
- U1 pad 480: unconnected-(U1-Col_30-Row_16-Pad480) -> Col_30-Row_16
- U1 pad 492: unconnected-(U1-Col_31-Row_12-Pad492) -> Col_31-Row_12
- U1 pad 493: unconnected-(U1-Col_31-Row_13-Pad493) -> Col_31-Row_13
- U1 pad 494: unconnected-(U1-Col_31-Row_14-Pad494) -> Col_31-Row_14
- U1 pad 495: unconnected-(U1-Col_31-Row_15-Pad495) -> Col_31-Row_15
- U1 pad 496: unconnected-(U1-Col_31-Row_16-Pad496) -> Col_31-Row_16
- U1 pad 508: unconnected-(U1-Col_32-Row_12-Pad508) -> Col_32-Row_12
- U1 pad 509: unconnected-(U1-Col_32-Row_13-Pad509) -> Col_32-Row_13
- U1 pad 510: unconnected-(U1-Col_32-Row_14-Pad510) -> Col_32-Row_14
- U1 pad 511: unconnected-(U1-Col_32-Row_15-Pad511) -> Col_32-Row_15
- U1 pad 512: unconnected-(U1-Col_32-Row_16-Pad512) -> Col_32-Row_16
- U1 pad 524: unconnected-(U1-Col_33-Row_12-Pad524) -> Col_33-Row_12
- U1 pad 525: unconnected-(U1-Col_33-Row_13-Pad525) -> Col_33-Row_13
- U1 pad 526: unconnected-(U1-Col_33-Row_14-Pad526) -> Col_33-Row_14
- U1 pad 527: unconnected-(U1-Col_33-Row_15-Pad527) -> Col_33-Row_15
- U1 pad 528: unconnected-(U1-Col_33-Row_16-Pad528) -> Col_33-Row_16
- U1 pad 540: unconnected-(U1-Col_34-Row_12-Pad540) -> Col_34-Row_12
- U1 pad 541: unconnected-(U1-Col_34-Row_13-Pad541) -> Col_34-Row_13
- U1 pad 542: unconnected-(U1-Col_34-Row_14-Pad542) -> Col_34-Row_14
- U1 pad 543: unconnected-(U1-Col_34-Row_15-Pad543) -> Col_34-Row_15
- U1 pad 544: unconnected-(U1-Col_34-Row_16-Pad544) -> Col_34-Row_16
- U1 pad 556: unconnected-(U1-Col_35-Row_12-Pad556) -> Col_35-Row_12
- U1 pad 557: unconnected-(U1-Col_35-Row_13-Pad557) -> Col_35-Row_13
- U1 pad 558: unconnected-(U1-Col_35-Row_14-Pad558) -> Col_35-Row_14
- U1 pad 559: unconnected-(U1-Col_35-Row_15-Pad559) -> Col_35-Row_15
- U1 pad 560: unconnected-(U1-Col_35-Row_16-Pad560) -> Col_35-Row_16
- U1 pad 572: unconnected-(U1-Col_36-Row_12-Pad572) -> Col_36-Row_12
- U1 pad 573: unconnected-(U1-Col_36-Row_13-Pad573) -> Col_36-Row_13
- U1 pad 574: unconnected-(U1-Col_36-Row_14-Pad574) -> Col_36-Row_14
- U1 pad 575: unconnected-(U1-Col_36-Row_15-Pad575) -> Col_36-Row_15
- U1 pad 576: unconnected-(U1-Col_36-Row_16-Pad576) -> Col_36-Row_16
- U1 pad 588: unconnected-(U1-Col_37-Row_12-Pad588) -> Col_37-Row_12
- U1 pad 589: unconnected-(U1-Col_37-Row_13-Pad589) -> Col_37-Row_13
- U1 pad 590: unconnected-(U1-Col_37-Row_14-Pad590) -> Col_37-Row_14
- U1 pad 591: unconnected-(U1-Col_37-Row_15-Pad591) -> Col_37-Row_15
- U1 pad 592: unconnected-(U1-Col_37-Row_16-Pad592) -> Col_37-Row_16
- U1 pad 604: unconnected-(U1-Col_38-Row_12-Pad604) -> Col_38-Row_12
- U1 pad 605: unconnected-(U1-Col_38-Row_13-Pad605) -> Col_38-Row_13
- U1 pad 606: unconnected-(U1-Col_38-Row_14-Pad606) -> Col_38-Row_14
- U1 pad 607: unconnected-(U1-Col_38-Row_15-Pad607) -> Col_38-Row_15
- U1 pad 608: unconnected-(U1-Col_38-Row_16-Pad608) -> Col_38-Row_16
- U1 pad 620: unconnected-(U1-Col_39-Row_12-Pad620) -> Col_39-Row_12
- U1 pad 621: unconnected-(U1-Col_39-Row_13-Pad621) -> Col_39-Row_13
- U1 pad 622: unconnected-(U1-Col_39-Row_14-Pad622) -> Col_39-Row_14
- U1 pad 623: unconnected-(U1-Col_39-Row_15-Pad623) -> Col_39-Row_15
- U1 pad 624: unconnected-(U1-Col_39-Row_16-Pad624) -> Col_39-Row_16
- U1 pad 636: unconnected-(U1-Col_40-Row_12-Pad636) -> Col_40-Row_12
- U1 pad 637: unconnected-(U1-Col_40-Row_13-Pad637) -> Col_40-Row_13
- U1 pad 638: unconnected-(U1-Col_40-Row_14-Pad638) -> Col_40-Row_14
- U1 pad 639: unconnected-(U1-Col_40-Row_15-Pad639) -> Col_40-Row_15
- U1 pad 640: unconnected-(U1-Col_40-Row_16-Pad640) -> Col_40-Row_16
- U1 pad 652: unconnected-(U1-Col_41-Row_12-Pad652) -> Col_41-Row_12
- U1 pad 653: unconnected-(U1-Col_41-Row_13-Pad653) -> Col_41-Row_13
- U1 pad 654: unconnected-(U1-Col_41-Row_14-Pad654) -> Col_41-Row_14
- U1 pad 655: unconnected-(U1-Col_41-Row_15-Pad655) -> Col_41-Row_15
- U1 pad 656: unconnected-(U1-Col_41-Row_16-Pad656) -> Col_41-Row_16
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Routing:
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