File: HYDRA_VMM3_Adapter/HYDRA_VMM3_Adapter.kicad_sch (KiCad schematic)
At the start: 12 parts, among them J1 ME1014010101011, J10 Conn_01x01_Socket, J2 ME1014010101011, J3 ME1014010101011, J4 ME1014010101011, J5 ME1014010101011, J6 ME1014010101011, J7 Conn_01x01_Socket, J8 Conn_01x01_Socket, J9 Conn_01x01_Socket

Commit message: .
Connections:
- net Col_43-Row_14: now reaches J3.A15
- net Col_43-Row_15: now reaches J3.A16
- net Col_43-Row_16: now reaches J3.A17
- net Col_42-Row_14: now reaches J3.A18
- net Col_42-Row_15: now reaches J3.A19
- net Col_42-Row_16: now reaches J3.A20
- net Col_41-Row_14: now reaches J3.A21
- net Col_43-Row_13: now reaches J3.A22
- net Col_43-Row_12: now reaches J3.A23
- net Col_42-Row_13: now reaches J3.A24
- net Col_42-Row_12: now reaches J3.A25
- net Col_41-Row_13: now reaches J3.A26
- net Col_41-Row_12: now reaches J3.A27
- net Col_40-Row_13: now reaches J3.A28
- net Col_40-Row_12: now reaches J3.A29
- net Col_39-Row_13: now reaches J3.A30
- net Col_39-Row_12: now reaches J3.A31
- net Col_38-Row_13: now reaches J3.A32
- net Col_38-Row_12: now reaches J3.A33
- net Col_37-Row_13: now reaches J3.A34
- net Col_37-Row_12: now reaches J3.A35
- net Col_41-Row_15: now reaches J3.B15
- net Col_41-Row_16: now reaches J3.B16
- net Col_40-Row_14: now reaches J3.B17
- net Col_40-Row_15: now reaches J3.B18
- net Col_40-Row_16: now reaches J3.B19
- net Col_39-Row_14: now reaches J3.B20
- net Col_39-Row_15: now reaches J3.B21
- net Col_39-Row_16: now reaches J3.B22
- net Col_38-Row_14: now reaches J3.B23
- net Col_38-Row_15: now reaches J3.B24
- net Col_38-Row_16: now reaches J3.B25
- net Col_37-Row_14: now reaches J3.B26
- net Col_37-Row_15: now reaches J3.B27
- net Col_37-Row_16: now reaches J3.B28
- net Col_36-Row_14: now reaches J3.B29
- net Col_36-Row_15: now reaches J3.B30
- net Col_36-Row_16: now reaches J3.B31
- net Col_35-Row_14: now reaches J3.B32
- net Col_35-Row_15: now reaches J3.B33
- net Col_35-Row_16: now reaches J3.B34
- net Col_34-Row_14: now reaches J3.B35
- net Col_36-Row_13: now reaches J3.A36
- net Col_36-Row_12: now reaches J3.A37
- net Col_35-Row_13: now reaches J3.A38
- net Col_35-Row_12: now reaches J3.A39
- net Col_34-Row_13: now reaches J3.A40
- net Col_34-Row_12: now reaches J3.A41
- net Col_33-Row_13: now reaches J3.A42
- net Col_33-Row_12: now reaches J3.A43
- net Col_32-Row_13: now reaches J3.A44
- net Col_32-Row_12: now reaches J3.A45
- net Col_31-Row_13: now reaches J3.A46
- net Col_31-Row_12: now reaches J3.A47
- net Col_30-Row_13: now reaches J3.A48
- net Col_30-Row_12: now reaches J3.A49
- net Col_29-Row_13: now reaches J3.A50
- net Col_29-Row_12: now reaches J3.A51
- net Col_29-Row_11: now reaches J3.A52
- net Col_28-Row_13: now reaches J3.A53
- net Col_28-Row_12: now reaches J3.A54
- net Col_28-Row_11: now reaches J3.A55
- net Col_27-Row_13: now reaches J3.A56
- net Col_27-Row_12: now reaches J3.A57
- net Col_27-Row_11: now reaches J3.A58
- net Col_26-Row_13: now reaches J3.A59
- net Col_26-Row_12: now reaches J3.A60
- net Col_26-Row_11: now reaches J3.A61
- net Col_25-Row_13: now reaches J3.A62
- net Col_25-Row_12: now reaches J3.A63
- net Col_25-Row_11: now reaches J3.A64
- net Col_24-Row_13: now reaches J3.A65
- net Col_24-Row_12: now reaches J3.A66
- net Col_24-Row_11: now reaches J3.A67
- net Col_23-Row_13: now reaches J3.A68
- net Col_23-Row_12: now reaches J3.A69
- net Col_23-Row_11: now reaches J3.A70
- net Col_34-Row_15: now reaches J3.B36
- net Col_34-Row_16: now reaches J3.B37
- net Col_33-Row_14: now reaches J3.B38
- net Col_33-Row_15: now reaches J3.B39
- net Col_33-Row_16: now reaches J3.B40
- net Col_32-Row_14: now reaches J3.B41
- net Col_32-Row_15: now reaches J3.B42
- net Col_32-Row_16: now reaches J3.B43
- net Col_31-Row_14: now reaches J3.B44
- net Col_31-Row_15: now reaches J3.B45
- net Col_31-Row_16: now reaches J3.B46
- net Col_30-Row_14: now reaches J3.B47
- net Col_30-Row_15: now reaches J3.B48
- net Col_30-Row_16: now reaches J3.B49
- net Col_29-Row_14: now reaches J3.B50
- net Col_29-Row_15: now reaches J3.B51
- net Col_29-Row_16: now reaches J3.B52
- net Col_28-Row_14: now reaches J3.B53
- net Col_28-Row_15: now reaches J3.B54
- net Col_28-Row_16: now reaches J3.B55
- net Col_27-Row_14: now reaches J3.B56
- net Col_27-Row_15: now reaches J3.B57
- net Col_27-Row_16: now reaches J3.B58
- net Col_26-Row_14: now reaches J3.B59
- net Col_26-Row_15: now reaches J3.B60
- net Col_26-Row_16: now reaches J3.B61
- net Col_25-Row_14: now reaches J3.B62
- net Col_25-Row_15: now reaches J3.B63
- net Col_25-Row_16: now reaches J3.B64
- net Col_24-Row_14: now reaches J3.B65
- net Col_24-Row_15: now reaches J3.B66
- net Col_24-Row_16: now reaches J3.B67
- net Col_23-Row_14: now reaches J3.B68
- net Col_23-Row_15: now reaches J3.B69
- net Col_23-Row_16: now reaches J3.B70
Other:
- company: (none) -> TU Darmstadt
- title: (none) -> HYDRA TPC to VMM3 adapter
- moved on the sheet: J2A, J2B, J3A, J3B, J5A, J5B
