File: HYDRA_VMM3_Adapter/HYDRA_VMM3_Adapter.kicad_sch (KiCad schematic)
At the start: 12 parts, among them J1 ME1014010101011, J10 Conn_01x01_Socket, J2 ME1014010101011, J3 ME1014010101011, J4 ME1014010101011, J5 ME1014010101011, J6 ME1014010101011, J7 Conn_01x01_Socket, J8 Conn_01x01_Socket, J9 Conn_01x01_Socket

Commit message: .
Connections:
- net GND: now also J1.A11, J1.A12, J1.A13, J1.A14, J1.B10, J1.B11, J1.B12, J1.B13, J1.B14, J1.B5, J1.B6, J1.B7, J1.B8, J1.B9, J2.A11, J2.A12, J2.A13, J2.A14, J2.B10, J2.B11, J2.B12, J2.B13, J2.B14, J2.B5, J2.B6, J2.B7, J2.B8, J2.B9, J3.A11, J3.A12, J3.A13, J3.A14, J3.B10, J3.B11, J3.B12, J3.B13, J3.B14, J3.B5, J3.B6, J3.B7, J3.B8, J3.B9, J4.A11, J4.A12, J4.A13, J4.A14, J4.B10, J4.B11, J4.B12, J4.B13, J4.B14, J4.B5, J4.B6, J4.B7, J4.B8, J4.B9, J5.A11, J5.A12, J5.A13, J5.A14, J5.B10, J5.B11, J5.B12, J5.B13, J5.B14, J5.B5, J5.B6, J5.B7, J5.B8, J5.B9, J6.A11, J6.A12, J6.A13, J6.A14, J6.B10, J6.B11, J6.B12, J6.B13, J6.B14, J6.B5, J6.B6, J6.B7, J6.B8, J6.B9
- net P1A: now also J4.B1, J4.B2, J4.B3, J4.B4, J5.B1, J5.B2, J5.B3, J5.B4, J6.B1, J6.B2, J6.B3, J6.B4
- net P1B: now also J1.B1, J1.B2, J1.B3, J1.B4, J2.B1, J2.B2, J2.B3, J2.B4, J3.B1, J3.B2, J3.B3, J3.B4
- net P2A: now also J4.A1, J4.A10, J4.A2, J4.A3, J4.A4, J4.A5, J4.A6, J4.A7, J4.A8, J4.A9, J5.A1, J5.A10, J5.A2, J5.A3, J5.A4, J5.A5, J5.A6, J5.A7, J5.A8, J5.A9, J6.A1, J6.A10, J6.A2, J6.A3, J6.A4, J6.A5, J6.A6, J6.A7, J6.A8, J6.A9
- net P2B: now also J1.A1, J1.A10, J1.A2, J1.A3, J1.A4, J1.A5, J1.A6, J1.A7, J1.A8, J1.A9, J2.A1, J2.A10, J2.A2, J2.A3, J2.A4, J2.A5, J2.A6, J2.A7, J2.A8, J2.A9, J3.A1, J3.A10, J3.A2, J3.A3, J3.A4, J3.A5, J3.A6, J3.A7, J3.A8, J3.A9
