File: HYDRA_VMM3_card/HYDRA_VMM3_CARD/HYDRA_VMM3_CARD.kicad_sch (KiCad schematic)
At the start: 1 part, among them J1 ME1014010101011

Commit message: .
Parts:
- added U1: ~, Card_Edge_Connector_FCI:Hirose-FX10, symbol FX10:FX10-140
Connections:
- new net GND: U1.141 (GND)
Other:
- moved on the sheet: J1A, J1B

Commit message: .
Parts:
- added 1.8V: 1.8V, TestPoint:TestPoint_Pad_D2.5mm, symbol Connector:TestPoint
- added 3.3V: 3.3V, TestPoint:TestPoint_Pad_D2.5mm, symbol Connector:TestPoint
- added GND: GND, TestPoint:TestPoint_Pad_2.5x2.5mm, symbol Connector:TestPoint
Connections:
- net GND: now also GND.1
- new net +1V8: 1.8V.1
- new net +3V3: 3.3V.1

Commit message: .
Parts:
- added Ch_1, Ch_10, Ch_11, Ch_12, Ch_13, Ch_14, Ch_15, Ch_16, Ch_2, Ch_3, Ch_4, Ch_5, Ch_6, Ch_7, Ch_8, Ch_9, I2C_VCC1, SCL1, SDA1, Sig_GND1, Sig_in1, Sig_out1: 20449-001E-03, IPEX:IPEX_20449-001E-03, symbol IPEX:20449-001E-03
- renumbered 1.8V to 1.8V1, 3.3V to 3.3V1, GND to GND1
Connections:
- net +1V8: now also J1.A1, J1.A10, J1.A2, J1.A3, J1.A4, J1.A5, J1.A6, J1.A7, J1.A8, J1.A9
- net +3V3: now also J1.B1, J1.B2, J1.B3, J1.B4
- net GND: now also J1.A11, J1.A12, J1.A13, J1.A14, J1.B10, J1.B11, J1.B12, J1.B13, J1.B14, J1.B5, J1.B6, J1.B7, J1.B8, J1.B9, Ch_1.2, Ch_1.3, Ch_1.4, Ch_10.2, Ch_10.3, Ch_10.4, Ch_11.2, Ch_11.3, Ch_11.4, Ch_12.2, Ch_12.3, Ch_12.4, Ch_13.2, Ch_13.3, Ch_13.4, Ch_14.2, Ch_14.3, Ch_14.4, Ch_15.2, Ch_15.3, Ch_15.4, Ch_16.2, Ch_16.3, Ch_16.4, Ch_2.2, Ch_2.3, Ch_2.4, Ch_3.2, Ch_3.3, Ch_3.4, Ch_4.2, Ch_4.3, Ch_4.4, Ch_5.2, Ch_5.3, Ch_5.4, Ch_6.2, Ch_6.3, Ch_6.4, Ch_7.2, Ch_7.3, Ch_7.4, Ch_8.2, Ch_8.3, Ch_8.4, Ch_9.2, Ch_9.3, Ch_9.4, I2C_VCC1.2, I2C_VCC1.3, I2C_VCC1.4, SCL1.2, SCL1.3, SCL1.4, SDA1.2, SDA1.3, SDA1.4, Sig_GND1.2, Sig_GND1.3, Sig_GND1.4, Sig_in1.2, Sig_in1.3, Sig_in1.4, Sig_out1.2, Sig_out1.3, Sig_out1.4
- net Ch_4: now reaches U1.10
- net Ch_4: now also Ch_4.1
- net Ch_94: now reaches U1.100
- net Ch_94: now also J1.B53
- net Ch_95: now reaches U1.101
- net Ch_95: now also J1.A54
- net Ch_96: now reaches U1.102
- net Ch_96: now also J1.B54
- net Ch_97: now reaches U1.103
- net Ch_97: now also J1.A55
- net Ch_98: now reaches U1.104
- net Ch_98: now also J1.B55
- net Ch_99: now reaches U1.105
- net Ch_99: now also J1.A56
- net Ch_100: now reaches U1.106
- net Ch_100: now also J1.B56
- net Ch_101: now reaches U1.107
- net Ch_101: now also J1.A57
- net Ch_102: now reaches U1.108
- net Ch_102: now also J1.B57
- net Ch_103: now reaches U1.109
- net Ch_103: now also J1.A58
- net Ch_5: now reaches U1.11
- net Ch_5: now also Ch_5.1
- net Ch_104: now reaches U1.110
- net Ch_104: now also J1.B58
- net Ch_105: now reaches U1.111
- net Ch_105: now also J1.A59
- net Ch_106: now reaches U1.112
- net Ch_106: now also J1.B59
- net Ch_107: now reaches U1.113
- net Ch_107: now also J1.A60
- net Ch_108: now reaches U1.114
- net Ch_108: now also J1.B70
- net Ch_109: now reaches U1.115
- net Ch_109: now also J1.A61
- net Ch_110: now reaches U1.116
- net Ch_110: now also J1.B69
- net Ch_111: now reaches U1.117
- net Ch_111: now also J1.A62
- net Ch_112: now reaches U1.118
- net Ch_112: now also J1.B68
- net Ch_113: now reaches U1.119
- net Ch_113: now also J1.A63
- net Ch_6: now reaches U1.12
- net Ch_6: now also Ch_6.1
- net Ch_114: now reaches U1.120
- net Ch_114: now also J1.B67
- net Ch_115: now reaches U1.121
- net Ch_115: now also J1.A64
- net Ch_116: now reaches U1.122
- net Ch_116: now also J1.B66
- net Ch_117: now reaches U1.123
- net Ch_117: now also J1.A65
- net Ch_118: now reaches U1.124
- net Ch_118: now also J1.B65
- net Ch_119: now reaches U1.125
- net Ch_119: now also J1.A66
- net Ch_120: now reaches U1.126
- net Ch_120: now also J1.B64
- net Ch_121: now reaches U1.127
- net Ch_121: now also J1.A67
- net Ch_122: now reaches U1.128
- net Ch_122: now also J1.B63
- net Ch_123: now reaches U1.129
- net Ch_123: now also J1.A68
- net Ch_7: now reaches U1.13
- net Ch_7: now also Ch_7.1
- net Ch_124: now reaches U1.130
- net Ch_124: now also J1.B62
- net Ch_125: now reaches U1.131
- net Ch_125: now also J1.A69
- net Ch_126: now reaches U1.132
- net Ch_126: now also J1.B61
- net Ch_127: now reaches U1.133
- net Ch_127: now also J1.A70
- net Ch_128: now reaches U1.134
- net Ch_128: now also J1.B60
- net Signal_GND: now reaches U1.135
- net Signal_GND: now also Sig_GND1.1
- net I2C_VCC: now reaches U1.136
- net I2C_VCC: now also I2C_VCC1.1
- net Signal_In: now reaches U1.137
- net Signal_In: now also Sig_in1.1
- net Signal_Out: now reaches U1.138
- net Signal_Out: now also Sig_out1.1
- net SDA: now reaches U1.139
- net SDA: now also SDA1.1
- net Ch_8: now reaches U1.14
- net Ch_8: now also Ch_8.1
- net SCL: now reaches U1.140
- net SCL: now also SCL1.1
- net Ch_9: now reaches U1.15
- net Ch_9: now also Ch_9.1
- net Ch_10: now reaches U1.16
- net Ch_10: now also Ch_10.1
- net Ch_11: now reaches U1.17
- net Ch_11: now also Ch_11.1
- net Ch_12: now reaches U1.18
- net Ch_12: now also Ch_12.1
- net Ch_13: now reaches U1.19
- net Ch_13: now also Ch_13.1
- net Ch_14: now reaches U1.20
- net Ch_14: now also Ch_14.1
- net Ch_15: now reaches U1.21
- net Ch_15: now also Ch_15.1
- net Ch_16: now reaches U1.22
- net Ch_16: now also Ch_16.1
- net Ch_17: now reaches U1.23
- net Ch_17: now also J1.A15
- net Ch_18: now reaches U1.24
- net Ch_18: now also J1.B15
- net Ch_19: now reaches U1.25
- net Ch_19: now also J1.A16
- net Ch_20: now reaches U1.26
- net Ch_20: now also J1.B16
- net Ch_21: now reaches U1.27
- net Ch_21: now also J1.A17
- net Ch_22: now reaches U1.28
- net Ch_22: now also J1.B17
- net Ch_23: now reaches U1.29
- net Ch_23: now also J1.A18
- net Ch_24: now reaches U1.30
- net Ch_24: now also J1.B18
- net Ch_25: now reaches U1.31
- net Ch_25: now also J1.A19
- net Ch_26: now reaches U1.32
- net Ch_26: now also J1.B19
- net Ch_27: now reaches U1.33
- net Ch_27: now also J1.A20
- net Ch_28: now reaches U1.34
- net Ch_28: now also J1.B20
- net Ch_29: now reaches U1.35
- net Ch_29: now also J1.A21
- net Ch_30: now reaches U1.36
- net Ch_30: now also J1.B21
- net Ch_31: now reaches U1.37
- net Ch_31: now also J1.A22
- net Ch_32: now reaches U1.38
- net Ch_32: now also J1.B22
- net Ch_33: now reaches U1.39
- net Ch_33: now also J1.A23
- net Ch_34: now reaches U1.40
- net Ch_34: now also J1.B23
- net Ch_35: now reaches U1.41
- net Ch_35: now also J1.A24
- net Ch_36: now reaches U1.42
- net Ch_36: now also J1.B24
- net Ch_37: now reaches U1.43
- net Ch_37: now also J1.A25
- net Ch_38: now reaches U1.44
- net Ch_38: now also J1.B25
- net Ch_39: now reaches U1.45
- net Ch_39: now also J1.A26
- net Ch_40: now reaches U1.46
- net Ch_40: now also J1.B26
- net Ch_41: now reaches U1.47
- net Ch_41: now also J1.A27
- net Ch_42: now reaches U1.48
- net Ch_42: now also J1.B27
- net Ch_43: now reaches U1.49
- net Ch_43: now also J1.A28
- net Ch_44: now reaches U1.50
- net Ch_44: now also J1.B28
- net Ch_45: now reaches U1.51
- net Ch_45: now also J1.A29
- net Ch_46: now reaches U1.52
- net Ch_46: now also J1.B29
- net Ch_47: now reaches U1.53
- net Ch_47: now also J1.A30
- net Ch_48: now reaches U1.54
- net Ch_48: now also J1.B30
- net Ch_49: now reaches U1.55
- net Ch_49: now also J1.A31
- net Ch_50: now reaches U1.56
- net Ch_50: now also J1.B31
- net Ch_51: now reaches U1.57
- net Ch_51: now also J1.A32
- net Ch_52: now reaches U1.58
- net Ch_52: now also J1.B32
- net Ch_53: now reaches U1.59
- net Ch_53: now also J1.A33
- net Ch_54: now reaches U1.60
- net Ch_54: now also J1.B33
- net Ch_55: now reaches U1.61
- net Ch_55: now also J1.A34
- net Ch_56: now reaches U1.62
- net Ch_56: now also J1.B34
- net Ch_57: now reaches U1.63
- net Ch_57: now also J1.A35
- net Ch_58: now reaches U1.64
- net Ch_58: now also J1.B35
- net Ch_59: now reaches U1.65
- net Ch_59: now also J1.A36
- net Ch_60: now reaches U1.66
- net Ch_60: now also J1.B36
- net Ch_61: now reaches U1.67
- net Ch_61: now also J1.A37
- net Ch_62: now reaches U1.68
- net Ch_62: now also J1.B37
- net Ch_63: now reaches U1.69
- net Ch_63: now also J1.A38
- net Ch_1: now reaches U1.7
- net Ch_1: now also Ch_1.1
- net Ch_64: now reaches U1.70
- net Ch_64: now also J1.B38
- net Ch_65: now reaches U1.71
- net Ch_65: now also J1.A39
- net Ch_66: now reaches U1.72
- net Ch_66: now also J1.B39
- net Ch_67: now reaches U1.73
- net Ch_67: now also J1.A40
- net Ch_68: now reaches U1.74
- net Ch_68: now also J1.B40
- net Ch_69: now reaches U1.75
- net Ch_69: now also J1.A41
- net Ch_70: now reaches U1.76
- net Ch_70: now also J1.B41
- net Ch_71: now reaches U1.77
- net Ch_71: now also J1.A42
- net Ch_72: now reaches U1.78
- net Ch_72: now also J1.B42
- net Ch_73: now reaches U1.79
- net Ch_73: now also J1.A43
- net Ch_2: now reaches U1.8
- net Ch_2: now also Ch_2.1
- net Ch_74: now reaches U1.80
- net Ch_74: now also J1.B43
- net Ch_75: now reaches U1.81
- net Ch_75: now also J1.A44
- net Ch_76: now reaches U1.82
- net Ch_76: now also J1.B44
- net Ch_77: now reaches U1.83
- net Ch_77: now also J1.A45
- net Ch_78: now reaches U1.84
- net Ch_78: now also J1.B45
- net Ch_79: now reaches U1.85
- net Ch_79: now also J1.A46
- net Ch_80: now reaches U1.86
- net Ch_80: now also J1.B46
- net Ch_81: now reaches U1.87
- net Ch_81: now also J1.A47
- net Ch_82: now reaches U1.88
- net Ch_82: now also J1.B47
- net Ch_83: now reaches U1.89
- net Ch_83: now also J1.A48
- net Ch_3: now reaches U1.9
- net Ch_3: now also Ch_3.1
- net Ch_84: now reaches U1.90
- net Ch_84: now also J1.B48
- net Ch_85: now reaches U1.91
- net Ch_85: now also J1.A49
- net Ch_86: now reaches U1.92
- net Ch_86: now also J1.B49
- net Ch_87: now reaches U1.93
- net Ch_87: now also J1.A50
- net Ch_88: now reaches U1.94
- net Ch_88: now also J1.B50
- net Ch_89: now reaches U1.95
- net Ch_89: now also J1.A51
- net Ch_90: now reaches U1.96
- net Ch_90: now also J1.B51
- net Ch_91: now reaches U1.97
- net Ch_91: now also J1.A52
- net Ch_92: now reaches U1.98
- net Ch_92: now also J1.B52
- net Ch_93: now reaches U1.99
- net Ch_93: now also J1.A53
Other:
- moved on the sheet: 1.8V1, 3.3V1, GND1, U1
