File: HYDRA_VMM3_card/HYDRA_VMM3_CARD/HYDRA_VMM3_CARD.kicad_sch (KiCad schematic)
At the start: 19 parts, among them J1 ME1014010101011

Commit message: .
Parts:
- added Temp_1, Temp_2: ~, IPEX:TMP104, symbol IPEX:TMP104
- added Temp_RX1, Temp_TX1: 20449-001E-03, IPEX:IPEX_20449-001E-03, symbol IPEX:20449-001E-03
Connections:
- net +3V3: now also Temp_1.1 (V+), Temp_2.1 (V+)
- net GND: now also Temp_1.2 (GND), Temp_2.2 (GND), Temp_RX1.2, Temp_RX1.3, Temp_RX1.4, Temp_TX1.2, Temp_TX1.3, Temp_TX1.4
- new net: Temp_1.4 (RX), Temp_2.3 (TX)
- new net RX: Temp_2.4 (RX), Temp_RX1.1
- new net TX: Temp_1.3 (TX), Temp_TX1.1
Other:
- moved on the sheet: SDA1, Sig_out1

Commit message: .
Parts:
- removed I2C_VCC1, SCL1, SDA1, Sig_GND1, Sig_in1, Sig_out1: 20449-001E-03, IPEX:IPEX_20449-001E-03, symbol IPEX:20449-001E-03
- added J2: Conn_01x06_Pin, Connector_PinHeader_1.00mm:PinHeader_1x06_P1.00mm_Horizontal, symbol Connector:Conn_01x06_Pin
Connections:
- net Signal_GND is gone; now on net GND: U1.135
- net +1V8: no longer 1.8_On1.2 (A)
- net +3V3: no longer 3.3V_On1.2 (A)
- net GND: now also J2.3 (Pin_3)
- net I2C_VCC: now also J2.1 (Pin_1)
- net SCL: now also J2.4 (Pin_4)
- net SDA: now also J2.5 (Pin_5)
- net Signal_In: now also J2.6 (Pin_6)
- net Signal_Out: now also J2.2 (Pin_2)
- net at 1.8V1.1, 1.8V_2.5A1.2: now also 1.8_On1.2 (A)
- net at 3.3V1.1, 3.3V_0.5A1.2: now also 3.3V_On1.2 (A)
Other:
- moved on the sheet: 1.8V1, 1.8_On1, 3.3V1, 3.3V_0.5A1, 3.3V_On1, R1, R2
