File: HYDRA_VMM3_card/HYDRA_VMM3_CARD/HYDRA_VMM3_CARD.kicad_pcb (KiCad board)
At the start: 4 copper layers, 59.3 x 23 mm, 1 part, among them J1 ME1014010101011

Commit message: .
Parts:
- added U1: ~, Card_Edge_Connector_FCI:Hirose-FX10, F.Cu at (134.7, 84.5)
Routing:
- net unconnected-(J1-PadB70): vias 1 -> 0
- net unconnected-(J1-PadB29): vias 1 -> 0
Other:
- board size 59.3 x 23 mm -> 80 x 61 mm

Commit message: .
Parts:
- moved U1 48.2 mm to (133.2, 36.3), turned to -90 degrees
Connections:
- U1 pad 141: unconnected-(U1-GND-Pad141) -> GND
Routing:
- added copper zone on B.Cu, net GND
- added copper zone on F.Cu, net GND
- added copper zone on In1.Cu, net GND
- added copper zone on In2.Cu, net GND
- added copper zone on In3.Cu, net GND
- added copper zone on In4.Cu, net GND
Other:
- copper layers 4 -> 6

Commit message: .
Parts:
- added 1: , , F.Cu at (109.7, 37.2)
- added 1.8V: 1.8V, TestPoint:TestPoint_Pad_D2.5mm, F.Cu at (64.5, 66.0)
- added 10: , , F.Cu at (109.7, 78.4)
- added 11: , , F.Cu at (112.3, 78.4)
- added 12: , , F.Cu at (114.8, 78.4)
- added 13: , , F.Cu at (76.1, 37.2)
- added 14: , , F.Cu at (76.1, 34.7)
- added 15: , , F.Cu at (76.1, 80.9)
- added 16: , , F.Cu at (76.1, 78.4)
- added 2: , , F.Cu at (112.3, 37.2)
- added 3: , , F.Cu at (114.8, 37.2)
- added 3.3V: 3.3V, TestPoint:TestPoint_Pad_D2.5mm, F.Cu at (64.5, 61.0)
- added 4: , , F.Cu at (109.7, 34.7)
- added 5: , , F.Cu at (112.3, 34.7)
- added 6: , , F.Cu at (114.8, 34.7)
- added 7: , , F.Cu at (109.7, 80.9)
- added 8: , , F.Cu at (112.3, 80.9)
- added 9: , , F.Cu at (114.8, 80.9)
- added ?: , , F.Cu at (138.1, 34.7)
- added ?: , , F.Cu at (73.5, 80.9)
- added ?: , , F.Cu at (135.5, 80.9)
- added ?: , , F.Cu at (135.5, 37.2)
- added ?: , , F.Cu at (107.2, 78.4)
- added ?: , , F.Cu at (68.5, 37.2)
- added ?: , , F.Cu at (133.0, 80.9)
- added ?: , , F.Cu at (107.2, 37.2)
- added ?: , , F.Cu at (73.5, 37.2)
- added ?: , , F.Cu at (107.2, 80.9)
- added ?: , , F.Cu at (71.0, 78.4)
- added ?: , , F.Cu at (135.5, 78.4)
- added ?: , , F.Cu at (138.1, 80.9)
- added ?: , , F.Cu at (73.5, 78.4)
- added ?: , , F.Cu at (107.2, 34.7)
- added ?: , , F.Cu at (68.5, 80.9)
- added ?: , , F.Cu at (73.5, 34.7)
- added ?: , , F.Cu at (133.0, 37.2)
- added ?: , , F.Cu at (138.1, 78.4)
- added ?: , , F.Cu at (71.0, 34.7)
- added ?: , , F.Cu at (71.0, 80.9)
- added ?: , , F.Cu at (68.5, 78.4)
- added ?: , , F.Cu at (135.5, 34.7)
- added ?: , , F.Cu at (68.5, 34.7)
- added ?: , , F.Cu at (133.0, 34.7)
- added ?: , , F.Cu at (71.0, 37.2)
- added ?: , , F.Cu at (138.1, 37.2)
- added ?: , , F.Cu at (133.0, 78.4)
- added GND: GND, TestPoint:TestPoint_Pad_2.5x2.5mm, F.Cu at (64.5, 63.5)
- moved U1 6.86 mm to (126.8, 33.9)

Commit message: .
Parts:
- added Ch_1: 20449-001E-03, IPEX:IPEX_20449-001E-03, B.Cu at (101.2, 54.6)
- added Ch_10: 20449-001E-03, IPEX:IPEX_20449-001E-03, B.Cu at (89.2, 42.6)
- added Ch_11: 20449-001E-03, IPEX:IPEX_20449-001E-03, B.Cu at (86.2, 57.6)
- added Ch_12: 20449-001E-03, IPEX:IPEX_20449-001E-03, B.Cu at (86.2, 45.6)
- added Ch_13: 20449-001E-03, IPEX:IPEX_20449-001E-03, B.Cu at (83.2, 54.6)
- added Ch_14: 20449-001E-03, IPEX:IPEX_20449-001E-03, B.Cu at (83.2, 42.6)
- added Ch_15: 20449-001E-03, IPEX:IPEX_20449-001E-03, B.Cu at (80.2, 57.6)
- added Ch_16: 20449-001E-03, IPEX:IPEX_20449-001E-03, B.Cu at (80.2, 45.6)
- added Ch_2: 20449-001E-03, IPEX:IPEX_20449-001E-03, B.Cu at (101.2, 42.6)
- added Ch_3: 20449-001E-03, IPEX:IPEX_20449-001E-03, B.Cu at (98.2, 57.6)
- added Ch_4: 20449-001E-03, IPEX:IPEX_20449-001E-03, B.Cu at (98.2, 45.6)
- added Ch_5: 20449-001E-03, IPEX:IPEX_20449-001E-03, B.Cu at (95.2, 54.6)
- added Ch_6: 20449-001E-03, IPEX:IPEX_20449-001E-03, B.Cu at (95.2, 42.6)
- added Ch_7: 20449-001E-03, IPEX:IPEX_20449-001E-03, B.Cu at (92.2, 57.6)
- added Ch_8: 20449-001E-03, IPEX:IPEX_20449-001E-03, B.Cu at (92.2, 45.6)
- added Ch_9: 20449-001E-03, IPEX:IPEX_20449-001E-03, B.Cu at (89.2, 54.6)
- added I2C_VCC1: 20449-001E-03, IPEX:IPEX_20449-001E-03, B.Cu at (139.2, 42.6)
- added SCL1: 20449-001E-03, IPEX:IPEX_20449-001E-03, B.Cu at (139.2, 52.6)
- added SDA1: 20449-001E-03, IPEX:IPEX_20449-001E-03, B.Cu at (136.2, 57.6)
- added Sig_GND1: 20449-001E-03, IPEX:IPEX_20449-001E-03, B.Cu at (136.2, 67.6)
- added Sig_in1: 20449-001E-03, IPEX:IPEX_20449-001E-03, B.Cu at (139.3, 62.6)
- added Sig_out1: 20449-001E-03, IPEX:IPEX_20449-001E-03, B.Cu at (136.2, 47.6)
- renumbered 1.8V to 1.8V1, 3.3V to 3.3V1, GND to GND1
Connections:
- 1.8V1 pad 1: +1V8 -> P2
- 3.3V1 pad 1: +3V3 -> P1
- J1 pad A1: unconnected-(J1-PadA1) -> P2
- J1 pad A10: unconnected-(J1-PadA10) -> P2
- J1 pad A11: unconnected-(J1-PadA11) -> GND
- J1 pad A12: unconnected-(J1-PadA12) -> GND
- J1 pad A13: unconnected-(J1-PadA13) -> GND
- J1 pad A14: unconnected-(J1-PadA14) -> GND
- J1 pad A15: unconnected-(J1-PadA15) -> Ch_17
- J1 pad A16: unconnected-(J1-PadA16) -> Ch_19
- J1 pad A17: unconnected-(J1-PadA17) -> Ch_21
- J1 pad A18: unconnected-(J1-PadA18) -> Ch_23
- J1 pad A19: unconnected-(J1-PadA19) -> Ch_25
- J1 pad A2: unconnected-(J1-PadA2) -> P2
- J1 pad A20: unconnected-(J1-PadA20) -> Ch_27
- J1 pad A21: unconnected-(J1-PadA21) -> Ch_29
- J1 pad A22: unconnected-(J1-PadA22) -> Ch_31
- J1 pad A23: unconnected-(J1-PadA23) -> Ch_33
- J1 pad A24: unconnected-(J1-PadA24) -> Ch_35
- J1 pad A25: unconnected-(J1-PadA25) -> Ch_37
- J1 pad A26: unconnected-(J1-PadA26) -> Ch_39
- J1 pad A27: unconnected-(J1-PadA27) -> Ch_41
- J1 pad A28: unconnected-(J1-PadA28) -> Ch_43
- J1 pad A29: unconnected-(J1-PadA29) -> Ch_45
- J1 pad A3: unconnected-(J1-PadA3) -> P2
- J1 pad A30: unconnected-(J1-PadA30) -> Ch_47
- J1 pad A31: unconnected-(J1-PadA31) -> Ch_49
- J1 pad A32: unconnected-(J1-PadA32) -> Ch_51
- J1 pad A33: unconnected-(J1-PadA33) -> Ch_53
- J1 pad A34: unconnected-(J1-PadA34) -> Ch_55
- J1 pad A35: unconnected-(J1-PadA35) -> Ch_57
- J1 pad A36: unconnected-(J1-PadA36) -> Ch_59
- J1 pad A37: unconnected-(J1-PadA37) -> Ch_61
- J1 pad A38: unconnected-(J1-PadA38) -> Ch_63
- J1 pad A39: unconnected-(J1-PadA39) -> Ch_65
- J1 pad A4: unconnected-(J1-PadA4) -> P2
- J1 pad A40: unconnected-(J1-PadA40) -> Ch_67
- J1 pad A41: unconnected-(J1-PadA41) -> Ch_69
- J1 pad A42: unconnected-(J1-PadA42) -> Ch_71
- J1 pad A43: unconnected-(J1-PadA43) -> Ch_73
- J1 pad A44: unconnected-(J1-PadA44) -> Ch_75
- J1 pad A45: unconnected-(J1-PadA45) -> Ch_77
- J1 pad A46: unconnected-(J1-PadA46) -> Ch_79
- J1 pad A47: unconnected-(J1-PadA47) -> Ch_81
- J1 pad A48: unconnected-(J1-PadA48) -> Ch_83
- J1 pad A49: unconnected-(J1-PadA49) -> Ch_85
- J1 pad A5: unconnected-(J1-PadA5) -> P2
- J1 pad A50: unconnected-(J1-PadA50) -> Ch_87
- J1 pad A51: unconnected-(J1-PadA51) -> Ch_89
- J1 pad A52: unconnected-(J1-PadA52) -> Ch_91
- J1 pad A53: unconnected-(J1-PadA53) -> Ch_93
- J1 pad A54: unconnected-(J1-PadA54) -> Ch_95
- J1 pad A55: unconnected-(J1-PadA55) -> Ch_97
- J1 pad A56: unconnected-(J1-PadA56) -> Ch_99
- J1 pad A57: unconnected-(J1-PadA57) -> Ch_101
- J1 pad A58: unconnected-(J1-PadA58) -> Ch_103
- J1 pad A59: unconnected-(J1-PadA59) -> Ch_105
- J1 pad A6: unconnected-(J1-PadA6) -> P2
- J1 pad A60: unconnected-(J1-PadA60) -> Ch_107
- J1 pad A61: unconnected-(J1-PadA61) -> Ch_109
- J1 pad A62: unconnected-(J1-PadA62) -> Ch_111
- J1 pad A63: unconnected-(J1-PadA63) -> Ch_113
- J1 pad A64: unconnected-(J1-PadA64) -> Ch_115
- J1 pad A65: unconnected-(J1-PadA65) -> Ch_117
- J1 pad A66: unconnected-(J1-PadA66) -> Ch_119
- J1 pad A67: unconnected-(J1-PadA67) -> Ch_121
- J1 pad A68: unconnected-(J1-PadA68) -> Ch_123
- J1 pad A69: unconnected-(J1-PadA69) -> Ch_125
- J1 pad A7: unconnected-(J1-PadA7) -> P2
- J1 pad A70: unconnected-(J1-PadA70) -> Ch_127
- J1 pad A8: unconnected-(J1-PadA8) -> P2
- J1 pad A9: unconnected-(J1-PadA9) -> P2
- J1 pad B1: unconnected-(J1-PadB1) -> P1
- J1 pad B10: unconnected-(J1-PadB10) -> GND
- J1 pad B11: unconnected-(J1-PadB11) -> GND
- J1 pad B12: unconnected-(J1-PadB12) -> GND
- J1 pad B13: unconnected-(J1-PadB13) -> GND
- J1 pad B14: unconnected-(J1-PadB14) -> GND
- J1 pad B15: unconnected-(J1-PadB15) -> Ch_18
- J1 pad B16: unconnected-(J1-PadB16) -> Ch_20
- J1 pad B17: unconnected-(J1-PadB17) -> Ch_22
- J1 pad B18: unconnected-(J1-PadB18) -> Ch_24
- J1 pad B19: unconnected-(J1-PadB19) -> Ch_26
- J1 pad B2: unconnected-(J1-PadB2) -> P1
- J1 pad B20: unconnected-(J1-PadB20) -> Ch_28
- J1 pad B21: unconnected-(J1-PadB21) -> Ch_30
- J1 pad B22: unconnected-(J1-PadB22) -> Ch_32
- J1 pad B23: unconnected-(J1-PadB23) -> Ch_34
- J1 pad B24: unconnected-(J1-PadB24) -> Ch_36
- J1 pad B25: unconnected-(J1-PadB25) -> Ch_38
- J1 pad B26: unconnected-(J1-PadB26) -> Ch_40
- J1 pad B27: unconnected-(J1-PadB27) -> Ch_42
- J1 pad B28: unconnected-(J1-PadB28) -> Ch_44
- J1 pad B29: unconnected-(J1-PadB29) -> Ch_46
- J1 pad B3: unconnected-(J1-PadB3) -> P1
- J1 pad B30: unconnected-(J1-PadB30) -> Ch_48
- J1 pad B31: unconnected-(J1-PadB31) -> Ch_50
- J1 pad B32: unconnected-(J1-PadB32) -> Ch_52
- J1 pad B33: unconnected-(J1-PadB33) -> Ch_54
- J1 pad B34: unconnected-(J1-PadB34) -> Ch_56
- J1 pad B35: unconnected-(J1-PadB35) -> Ch_58
- J1 pad B36: unconnected-(J1-PadB36) -> Ch_60
- J1 pad B37: unconnected-(J1-PadB37) -> Ch_62
- J1 pad B38: unconnected-(J1-PadB38) -> Ch_64
- J1 pad B39: unconnected-(J1-PadB39) -> Ch_66
- J1 pad B4: unconnected-(J1-PadB4) -> P1
- J1 pad B40: unconnected-(J1-PadB40) -> Ch_68
- J1 pad B41: unconnected-(J1-PadB41) -> Ch_70
- J1 pad B42: unconnected-(J1-PadB42) -> Ch_72
- J1 pad B43: unconnected-(J1-PadB43) -> Ch_74
- J1 pad B44: unconnected-(J1-PadB44) -> Ch_76
- J1 pad B45: unconnected-(J1-PadB45) -> Ch_78
- J1 pad B46: unconnected-(J1-PadB46) -> Ch_80
- J1 pad B47: unconnected-(J1-PadB47) -> Ch_82
- J1 pad B48: unconnected-(J1-PadB48) -> Ch_84
- J1 pad B49: unconnected-(J1-PadB49) -> Ch_86
- J1 pad B5: unconnected-(J1-PadB5) -> GND
- J1 pad B50: unconnected-(J1-PadB50) -> Ch_88
- J1 pad B51: unconnected-(J1-PadB51) -> Ch_90
- J1 pad B52: unconnected-(J1-PadB52) -> Ch_92
- J1 pad B53: unconnected-(J1-PadB53) -> Ch_94
- J1 pad B54: unconnected-(J1-PadB54) -> Ch_96
- J1 pad B55: unconnected-(J1-PadB55) -> Ch_98
- J1 pad B56: unconnected-(J1-PadB56) -> Ch_100
- J1 pad B57: unconnected-(J1-PadB57) -> Ch_102
- J1 pad B58: unconnected-(J1-PadB58) -> Ch_104
- J1 pad B59: unconnected-(J1-PadB59) -> Ch_106
- J1 pad B6: unconnected-(J1-PadB6) -> GND
- J1 pad B60: unconnected-(J1-PadB60) -> Ch_128
- J1 pad B61: unconnected-(J1-PadB61) -> Ch_126
- J1 pad B62: unconnected-(J1-PadB62) -> Ch_124
- J1 pad B63: unconnected-(J1-PadB63) -> Ch_122
- J1 pad B64: unconnected-(J1-PadB64) -> Ch_120
- J1 pad B65: unconnected-(J1-PadB65) -> Ch_118
- J1 pad B66: unconnected-(J1-PadB66) -> Ch_116
- J1 pad B67: unconnected-(J1-PadB67) -> Ch_114
- J1 pad B68: unconnected-(J1-PadB68) -> Ch_112
- J1 pad B69: unconnected-(J1-PadB69) -> Ch_110
- J1 pad B7: unconnected-(J1-PadB7) -> GND
- J1 pad B70: unconnected-(J1-PadB70) -> Ch_108
- J1 pad B8: unconnected-(J1-PadB8) -> GND
- J1 pad B9: unconnected-(J1-PadB9) -> GND
- U1 pad 10: unconnected-(U1-Pad10) -> Ch_4
- U1 pad 100: unconnected-(U1-Pad100) -> Ch_94
- U1 pad 101: unconnected-(U1-Pad101) -> Ch_95
- U1 pad 102: unconnected-(U1-Pad102) -> Ch_96
- U1 pad 103: unconnected-(U1-Pad103) -> Ch_97
- U1 pad 104: unconnected-(U1-Pad104) -> Ch_98
- U1 pad 105: unconnected-(U1-Pad105) -> Ch_99
- U1 pad 106: unconnected-(U1-Pad106) -> Ch_100
- U1 pad 107: unconnected-(U1-Pad107) -> Ch_101
- U1 pad 108: unconnected-(U1-Pad108) -> Ch_102
- U1 pad 109: unconnected-(U1-Pad109) -> Ch_103
- U1 pad 11: unconnected-(U1-Pad11) -> Ch_5
- U1 pad 110: unconnected-(U1-Pad110) -> Ch_104
- U1 pad 111: unconnected-(U1-Pad111) -> Ch_105
- U1 pad 112: unconnected-(U1-Pad112) -> Ch_106
- U1 pad 113: unconnected-(U1-Pad113) -> Ch_107
- U1 pad 114: unconnected-(U1-Pad114) -> Ch_108
- U1 pad 115: unconnected-(U1-Pad115) -> Ch_109
- U1 pad 116: unconnected-(U1-Pad116) -> Ch_110
- U1 pad 117: unconnected-(U1-Pad117) -> Ch_111
- U1 pad 118: unconnected-(U1-Pad118) -> Ch_112
- U1 pad 119: unconnected-(U1-Pad119) -> Ch_113
- U1 pad 12: unconnected-(U1-Pad12) -> Ch_6
- U1 pad 120: unconnected-(U1-Pad120) -> Ch_114
- U1 pad 121: unconnected-(U1-Pad121) -> Ch_115
- U1 pad 122: unconnected-(U1-Pad122) -> Ch_116
- U1 pad 123: unconnected-(U1-Pad123) -> Ch_117
- U1 pad 124: unconnected-(U1-Pad124) -> Ch_118
- U1 pad 125: unconnected-(U1-Pad125) -> Ch_119
- U1 pad 126: unconnected-(U1-Pad126) -> Ch_120
- U1 pad 127: unconnected-(U1-Pad127) -> Ch_121
- U1 pad 128: unconnected-(U1-Pad128) -> Ch_122
- U1 pad 129: unconnected-(U1-Pad129) -> Ch_123
- U1 pad 13: unconnected-(U1-Pad13) -> Ch_7
- U1 pad 130: unconnected-(U1-Pad130) -> Ch_124
- U1 pad 131: unconnected-(U1-Pad131) -> Ch_125
- U1 pad 132: unconnected-(U1-Pad132) -> Ch_126
- U1 pad 133: unconnected-(U1-Pad133) -> Ch_127
- U1 pad 134: unconnected-(U1-Pad134) -> Ch_128
- U1 pad 135: unconnected-(U1-Pad135) -> Signal_GND
- U1 pad 136: unconnected-(U1-Pad136) -> I2C_VCC
- U1 pad 137: unconnected-(U1-Pad137) -> Signal_In
- U1 pad 138: unconnected-(U1-Pad138) -> Signal_Out
- U1 pad 139: unconnected-(U1-Pad139) -> SDA
- U1 pad 14: unconnected-(U1-Pad14) -> Ch_8
- U1 pad 140: unconnected-(U1-Pad140) -> SCL
- U1 pad 15: unconnected-(U1-Pad15) -> Ch_9
- U1 pad 16: unconnected-(U1-Pad16) -> Ch_10
- U1 pad 17: unconnected-(U1-Pad17) -> Ch_11
- U1 pad 18: unconnected-(U1-Pad18) -> Ch_12
- U1 pad 19: unconnected-(U1-Pad19) -> Ch_13
- U1 pad 20: unconnected-(U1-Pad20) -> Ch_14
- U1 pad 21: unconnected-(U1-Pad21) -> Ch_15
- U1 pad 22: unconnected-(U1-Pad22) -> Ch_16
- U1 pad 23: unconnected-(U1-Pad23) -> Ch_17
- U1 pad 24: unconnected-(U1-Pad24) -> Ch_18
- U1 pad 25: unconnected-(U1-Pad25) -> Ch_19
- U1 pad 26: unconnected-(U1-Pad26) -> Ch_20
- U1 pad 27: unconnected-(U1-Pad27) -> Ch_21
- U1 pad 28: unconnected-(U1-Pad28) -> Ch_22
- U1 pad 29: unconnected-(U1-Pad29) -> Ch_23
- U1 pad 30: unconnected-(U1-Pad30) -> Ch_24
- U1 pad 31: unconnected-(U1-Pad31) -> Ch_25
- U1 pad 32: unconnected-(U1-Pad32) -> Ch_26
- U1 pad 33: unconnected-(U1-Pad33) -> Ch_27
- U1 pad 34: unconnected-(U1-Pad34) -> Ch_28
- U1 pad 35: unconnected-(U1-Pad35) -> Ch_29
- U1 pad 36: unconnected-(U1-Pad36) -> Ch_30
- U1 pad 37: unconnected-(U1-Pad37) -> Ch_31
- U1 pad 38: unconnected-(U1-Pad38) -> Ch_32
- U1 pad 39: unconnected-(U1-Pad39) -> Ch_33
- U1 pad 40: unconnected-(U1-Pad40) -> Ch_34
- U1 pad 41: unconnected-(U1-Pad41) -> Ch_35
- U1 pad 42: unconnected-(U1-Pad42) -> Ch_36
- U1 pad 43: unconnected-(U1-Pad43) -> Ch_37
- U1 pad 44: unconnected-(U1-Pad44) -> Ch_38
- U1 pad 45: unconnected-(U1-Pad45) -> Ch_39
- U1 pad 46: unconnected-(U1-Pad46) -> Ch_40
- U1 pad 47: unconnected-(U1-Pad47) -> Ch_41
- U1 pad 48: unconnected-(U1-Pad48) -> Ch_42
- U1 pad 49: unconnected-(U1-Pad49) -> Ch_43
- U1 pad 50: unconnected-(U1-Pad50) -> Ch_44
- U1 pad 51: unconnected-(U1-Pad51) -> Ch_45
- U1 pad 52: unconnected-(U1-Pad52) -> Ch_46
- U1 pad 53: unconnected-(U1-Pad53) -> Ch_47
- U1 pad 54: unconnected-(U1-Pad54) -> Ch_48
- U1 pad 55: unconnected-(U1-Pad55) -> Ch_49
- U1 pad 56: unconnected-(U1-Pad56) -> Ch_50
- U1 pad 57: unconnected-(U1-Pad57) -> Ch_51
- U1 pad 58: unconnected-(U1-Pad58) -> Ch_52
- U1 pad 59: unconnected-(U1-Pad59) -> Ch_53
- U1 pad 60: unconnected-(U1-Pad60) -> Ch_54
- U1 pad 61: unconnected-(U1-Pad61) -> Ch_55
- U1 pad 62: unconnected-(U1-Pad62) -> Ch_56
- U1 pad 63: unconnected-(U1-Pad63) -> Ch_57
- U1 pad 64: unconnected-(U1-Pad64) -> Ch_58
- U1 pad 65: unconnected-(U1-Pad65) -> Ch_59
- U1 pad 66: unconnected-(U1-Pad66) -> Ch_60
- U1 pad 67: unconnected-(U1-Pad67) -> Ch_61
- U1 pad 68: unconnected-(U1-Pad68) -> Ch_62
- U1 pad 69: unconnected-(U1-Pad69) -> Ch_63
- U1 pad 7: unconnected-(U1-Pad7) -> Ch_1
- U1 pad 70: unconnected-(U1-Pad70) -> Ch_64
- U1 pad 71: unconnected-(U1-Pad71) -> Ch_65
- U1 pad 72: unconnected-(U1-Pad72) -> Ch_66
- U1 pad 73: unconnected-(U1-Pad73) -> Ch_67
- U1 pad 74: unconnected-(U1-Pad74) -> Ch_68
- U1 pad 75: unconnected-(U1-Pad75) -> Ch_69
- U1 pad 76: unconnected-(U1-Pad76) -> Ch_70
- U1 pad 77: unconnected-(U1-Pad77) -> Ch_71
- U1 pad 78: unconnected-(U1-Pad78) -> Ch_72
- U1 pad 79: unconnected-(U1-Pad79) -> Ch_73
- U1 pad 8: unconnected-(U1-Pad8) -> Ch_2
- U1 pad 80: unconnected-(U1-Pad80) -> Ch_74
- U1 pad 81: unconnected-(U1-Pad81) -> Ch_75
- U1 pad 82: unconnected-(U1-Pad82) -> Ch_76
- U1 pad 83: unconnected-(U1-Pad83) -> Ch_77
- U1 pad 84: unconnected-(U1-Pad84) -> Ch_78
- U1 pad 85: unconnected-(U1-Pad85) -> Ch_79
- U1 pad 86: unconnected-(U1-Pad86) -> Ch_80
- U1 pad 87: unconnected-(U1-Pad87) -> Ch_81
- U1 pad 88: unconnected-(U1-Pad88) -> Ch_82
- U1 pad 89: unconnected-(U1-Pad89) -> Ch_83
- U1 pad 9: unconnected-(U1-Pad9) -> Ch_3
- U1 pad 90: unconnected-(U1-Pad90) -> Ch_84
- U1 pad 91: unconnected-(U1-Pad91) -> Ch_85
- U1 pad 92: unconnected-(U1-Pad92) -> Ch_86
- U1 pad 93: unconnected-(U1-Pad93) -> Ch_87
- U1 pad 94: unconnected-(U1-Pad94) -> Ch_88
- U1 pad 95: unconnected-(U1-Pad95) -> Ch_89
- U1 pad 96: unconnected-(U1-Pad96) -> Ch_90
- U1 pad 97: unconnected-(U1-Pad97) -> Ch_91
- U1 pad 98: unconnected-(U1-Pad98) -> Ch_92
- U1 pad 99: unconnected-(U1-Pad99) -> Ch_93
Routing:
- net GND: track 0.00 -> 66.1 mm
- net Ch_19: track 0.00 -> 64.0 mm, vias 0 -> 1
- net Ch_17: track 0.00 -> 63.3 mm, vias 0 -> 1
- net Ch_15: track 0.00 -> 62.7 mm, vias 0 -> 2
- net Ch_23: track 0.00 -> 62.0 mm, vias 0 -> 1
- net Ch_21: track 0.00 -> 61.7 mm, vias 0 -> 1
- net Ch_18: track 0.00 -> 61.3 mm
- net Ch_20: track 0.00 -> 60.6 mm
- net Ch_27: track 0.00 -> 59.9 mm, vias 0 -> 1
- net Ch_22: track 0.00 -> 59.9 mm
- net Ch_13: track 0.00 -> 59.7 mm, vias 0 -> 2
- net Ch_25: track 0.00 -> 59.3 mm, vias 0 -> 1
- net Ch_24: track 0.00 -> 59.2 mm
- net Ch_31: track 0.00 -> 58.5 mm, vias 0 -> 1
- net Ch_26: track 0.00 -> 58.1 mm
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
Commit message: .
Parts:
- removed Ch_1, Ch_10, Ch_11, Ch_12, Ch_13, Ch_14, Ch_15, Ch_16, Ch_2, Ch_3, Ch_4, Ch_5, Ch_6, Ch_7, Ch_8, Ch_9: 20449-001E-03, IPEX:IPEX_20449-001E-03
- added 1.8V_2.5A1: 2.5A, Fuse:Fuse_0603_1608Metric_Pad1.05x0.95mm_HandSolder, B.Cu at (67.5, 69.0)
- added 1.8_On1: LED, LED_SMD:LED_0603_1608Metric_Pad1.05x0.95mm_HandSolder, B.Cu at (64.7, 74.8)
- added 3.3V_0.5A1: 0.5A, Fuse:Fuse_0603_1608Metric_Pad1.05x0.95mm_HandSolder, B.Cu at (72.8, 65.3)
- added 3.3V_On1: LED, LED_SMD:LED_0603_1608Metric_Pad1.05x0.95mm_HandSolder, B.Cu at (64.7, 56.4)
- added Ch1: TestPoint, TestPoint:TestPoint_Pad_D1.0mm, B.Cu at (74.2, 44.0)
- added Ch10: TestPoint, TestPoint:TestPoint_Pad_D1.0mm, B.Cu at (70.7, 55.1)
- added Ch11: TestPoint, TestPoint:TestPoint_Pad_D1.0mm, B.Cu at (71.2, 45.3)
- added Ch12: TestPoint, TestPoint:TestPoint_Pad_D1.0mm, B.Cu at (71.1, 53.8)
- added Ch13: TestPoint, TestPoint:TestPoint_Pad_D1.0mm, B.Cu at (72.5, 45.8)
- added Ch14: TestPoint, TestPoint:TestPoint_Pad_D1.0mm, B.Cu at (72.4, 53.2)
- added Ch15: TestPoint, TestPoint:TestPoint_Pad_D1.0mm, B.Cu at (73.8, 45.3)
- added Ch16: TestPoint, TestPoint:TestPoint_Pad_D1.0mm, B.Cu at (73.7, 53.7)
- added Ch2: TestPoint, TestPoint:TestPoint_Pad_D1.0mm, B.Cu at (74.2, 55.0)
- added Ch3: TestPoint, TestPoint:TestPoint_Pad_D1.0mm, B.Cu at (73.7, 42.7)
- added Ch4: TestPoint, TestPoint:TestPoint_Pad_D1.0mm, B.Cu at (73.8, 56.3)
- added Ch5: TestPoint, TestPoint:TestPoint_Pad_D1.0mm, B.Cu at (72.4, 42.2)
- added Ch6: TestPoint, TestPoint:TestPoint_Pad_D1.0mm, B.Cu at (72.5, 56.8)
- added Ch7: TestPoint, TestPoint:TestPoint_Pad_D1.0mm, B.Cu at (71.1, 42.8)
- added Ch8: TestPoint, TestPoint:TestPoint_Pad_D1.0mm, B.Cu at (71.2, 56.3)
- added Ch9: TestPoint, TestPoint:TestPoint_Pad_D1.0mm, B.Cu at (70.7, 44.1)
- added R1: 1k, Resistor_SMD:R_0603_1608Metric_Pad0.98x0.95mm_HandSolder, B.Cu at (66.3, 56.3)
- added R2: 1k, Resistor_SMD:R_0603_1608Metric_Pad0.98x0.95mm_HandSolder, B.Cu at (66.3, 74.8)
- added Sig1: 20449-001E-03, IPEX:IPEX_20449-001E-03, B.Cu at (65.0, 44.0)
- added Sig1_selector: TestPoint, TestPoint:TestPoint_Pad_D1.0mm, B.Cu at (72.5, 44.0)
- added Sig2: 20449-001E-03, IPEX:IPEX_20449-001E-03, B.Cu at (65.0, 50.0)
- added Sig2_selector: TestPoint, TestPoint:TestPoint_Pad_D1.0mm, B.Cu at (72.5, 55.0)
Connections:
- 1.8V1 pad 1: P2 -> Net-(1.8V1-Pad1)
- 3.3V1 pad 1: P1 -> Net-(3.3V1-Pad1)
Routing:
- net Ch_2: track 24.6 -> 56.3 mm
- net Ch_4: track 28.6 -> 57.1 mm
- net Ch_8: track 34.8 -> 59.7 mm
- net Ch_6: track 34.1 -> 58.0 mm
- net Ch_12: track 41.4 -> 64.1 mm
- net Ch_1: track 38.4 -> 60.6 mm
- net Ch_16: track 48.1 -> 69.8 mm
- net Ch_10: track 40.8 -> 61.7 mm
- net Ch_14: track 47.6 -> 66.8 mm
- net Ch_3: track 43.9 -> 62.8 mm
- net Ch_7: track 49.9 -> 66.4 mm
- net Ch_5: track 47.6 -> 63.2 mm
- net Ch_11: track 56.3 -> 71.0 mm
- net Ch_15: track 62.7 -> 76.9 mm
- net Ch_9: track 53.3 -> 67.1 mm
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Other:
- board text added: "Heim time"
- board text added: "Heim time CH selector"
- board text added: "Master trigger"
- board text added: "Master trigger CH selector"

Commit message: .
Parts:
- removed the ? at (73.5, 80.9)
- removed the ? at (107.2, 78.4)
- removed the ? at (107.2, 80.9)
- removed the ? at (71.0, 78.4)
- removed the ? at (73.5, 78.4)
- removed the ? at (68.5, 80.9)
- removed the ? at (71.0, 80.9)
- removed the ? at (68.5, 78.4)
- added 17: , , F.Cu at (114.0, 80.9)
- added 18: , , F.Cu at (116.5, 80.9)
- added 19: , , F.Cu at (119.0, 80.9)
- added 20: , , F.Cu at (114.0, 78.4)
- added 21: , , F.Cu at (116.5, 78.4)
- added 22: , , F.Cu at (119.0, 78.4)
- added 23: , , F.Cu at (80.3, 80.9)
- added 24: , , F.Cu at (80.3, 78.4)
- added Temp_1: ~, IPEX:TMP104, B.Cu at (95.2, 40.2)
- added Temp_2: ~, IPEX:TMP104, B.Cu at (95.2, 75.4)
- added Temp_RX1: 20449-001E-03, IPEX:IPEX_20449-001E-03, B.Cu at (99.3, 36.8)
- added Temp_TX1: 20449-001E-03, IPEX:IPEX_20449-001E-03, B.Cu at (92.3, 36.8)
- moved 11 39.6 mm to (72.7, 78.4)
- moved 12 39.6 mm to (75.2, 78.4)
- moved 8 37.1 mm to (75.2, 80.9)
- moved 7 37.1 mm to (72.7, 80.9)
- moved 9 37.1 mm to (77.7, 80.9)
- moved 16 35.4 mm to (111.4, 78.4)
- moved ? 4.22 mm to (72.7, 37.2)
- moved ? 4.22 mm to (72.7, 34.7)
- moved 1 4.22 mm to (114.0, 37.2)
- moved 13 4.22 mm to (80.3, 37.2)
- moved 14 4.22 mm to (80.3, 34.7)
- moved 4 4.22 mm to (114.0, 34.7)
- moved ? 4.22 mm to (111.4, 37.2)
- moved ? 4.22 mm to (77.7, 37.2)
- moved ? 4.22 mm to (111.4, 34.7)
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Routing:
- net P1: track 48.9 -> 97.7 mm, vias 15 -> 17
- net RX: track 0.00 -> 39.3 mm
- net Net-(Temp_1-RX): track 0.00 -> 34.9 mm
- net Ch_92: track 33.1 -> 50.7 mm
- net Ch_90: track 33.5 -> 51.1 mm
- net Ch_88: track 34.0 -> 51.6 mm
- net Ch_86: track 34.6 -> 52.0 mm
- net Ch_84: track 36.0 -> 52.9 mm
- net Ch_82: track 36.7 -> 53.4 mm
- net Ch_80: track 37.1 -> 53.8 mm
- net Ch_78: track 37.6 -> 54.3 mm
- net Ch_76: track 38.0 -> 54.7 mm
- net Ch_74: track 38.6 -> 55.2 mm
- net Ch_63: track 43.6 -> 51.1 mm
- net Ch_61: track 43.3 -> 50.1 mm
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
Commit message: .
Parts:
- removed I2C_VCC1, SCL1, SDA1, Sig_GND1, Sig_in1, Sig_out1: 20449-001E-03, IPEX:IPEX_20449-001E-03
- added 25: , , F.Cu at (39.6, 79.4)
- added ?: , , F.Cu at (53.0, 79.4)
- added ?: , , F.Cu at (139.4, 57.6)
- added J2: Conn_01x06_Pin, Connector_PinHeader_1.00mm:PinHeader_1x06_P1.00mm_Horizontal, F.Cu at (137.8, 44.3)
- added REF**: TestPoint_Pad_1.0x1.0mm, TestPoint:TestPoint_Pad_1.0x1.0mm, F.Cu at (46.6, 57.8)
- added REF**: MountingHole_2.2mm_M2_DIN965_Pad, MountingHole:MountingHole_2.2mm_M2_DIN965_Pad, F.Cu at (39.6, 35.8)
- added REF**: TestPoint_Pad_1.0x1.0mm, TestPoint:TestPoint_Pad_1.0x1.0mm, B.Cu at (46.6, 57.8)
- added REF**1: MountingHole_2.2mm_M2_DIN965_Pad, MountingHole:MountingHole_2.2mm_M2_DIN965_Pad, F.Cu at (53.0, 35.8)
- added REF**2: MountingHole_2.2mm_M2_DIN965_Pad, MountingHole:MountingHole_2.2mm_M2_DIN965_Pad, F.Cu at (39.6, 57.6)
- added REF**3: MountingHole_2.2mm_M2_DIN965_Pad, MountingHole:MountingHole_2.2mm_M2_DIN965_Pad, F.Cu at (53.0, 57.6)
Connections:
- 1.8V1 pad 1: Net-(1.8V1-Pad1) -> Net-(1.8_On1-A)
- 1.8V_2.5A1 pad 2: Net-(1.8V1-Pad1) -> Net-(1.8_On1-A)
- 1.8_On1 pad 2: P2 -> Net-(1.8_On1-A)
- 3.3V1 pad 1: Net-(3.3V1-Pad1) -> Net-(3.3V_On1-A)
- 3.3V_0.5A1 pad 2: Net-(3.3V1-Pad1) -> Net-(3.3V_On1-A)
- 3.3V_On1 pad 2: P1 -> Net-(3.3V_On1-A)
- U1 pad 135: Signal_GND -> GND
Routing:
- net P1: track 97.7 -> 80.3 mm
- net Signal_GND: track 14.3 -> 0.00 mm, vias 1 -> 0
- net Net-(3.3V_On1-A): track 0.00 -> 12.5 mm
- net Net-(1.8_On1-A): track 0.00 -> 9.73 mm
- net Signal_In: track 25.9 -> 35.1 mm, vias 2 -> 1
- net Net-(3.3V1-Pad1): track 8.77 -> 0.00 mm
- net P2: track 35.1 -> 28.4 mm
- net Signal_Out: track 38.3 -> 43.8 mm, vias 2 -> 1
- net SDA: track 37.4 -> 42.2 mm, vias 2 -> 1
- net SCL: track 38.2 -> 42.2 mm, vias 2 -> 1
- net GND: track 68.1 -> 71.6 mm, vias 66 -> 806
- net I2C_VCC: track 47.1 -> 43.9 mm, vias 2 -> 1
- net Net-(1.8V1-Pad1): track 2.85 -> 0.00 mm
- net Ch_101: track 29.2 -> 30.4 mm
Other:
- board size 80 x 61 mm -> 105.3 x 61 mm
- board text added: "Project: VMM3a-Hybrid Card Adapter Version: V_0.1 11.07.2024 Author: Alexandru Enciu Institution: TU Darmstadt"
- board text added: "Technische Universität Darmstadt"
