File: TMP104_DemoBoard/TMP104_Development board/TMP104_Development board.kicad_pcb (KiCad board)
At the start: 4 copper layers, 25 x 20 mm, 28 parts, among them J1 Conn_02x03_Counter_Clockwise

Commit message: .
Parts:
- moved C5 0.50 mm to (128.9, 104.5)
- moved C6 0.50 mm to (128.9, 102.9)
Routing:
- net Net-(U13-TX): track 3.13 -> 4.60 mm
- net VCC_3.3V: vias 4 -> 5

Commit message: .
Parts:
- removed C10, C9: 0.1 uF, Capacitor_SMD:C_0603_1608Metric
- removed J1: Conn_02x03_Counter_Clockwise, Connector_PinHeader_2.54mm:PinHeader_2x03_P2.54mm_Vertical_SMD
- removed U1: ~, Molex_PCB_Power_Connector:TMP104
- added J2: 95278-801A04LF, Connector_PinHeader_2.54mm:PinHeader_2x02_P2.54mm_Vertical_SMD, F.Cu at (121.7, 103.7)
- added REF**: MountingHole_2.2mm_M2_DIN965_Pad, MountingHole:MountingHole_2.2mm_M2_DIN965_Pad, F.Cu at (140.8, 96.2)
- added REF**: MountingHole_2.2mm_M2_DIN965_Pad, MountingHole:MountingHole_2.2mm_M2_DIN965_Pad, F.Cu at (140.8, 111.2)
- U10, U11, U12, U13, U14, U15, U16, U17, U2, U3, U4, U5, U6, U7, U8, U9: value ~ -> TMP104YFFR
Routing:
- net TX_1: track 8.99 -> 0.00 mm, vias 1 -> 0
- net GND: track 38.3 -> 30.6 mm, vias 26 -> 21
- net RX_1: track 7.00 -> 0.00 mm, vias 1 -> 0
- net TX_2: track 6.81 -> 10.3 mm
- net RX_2: track 6.81 -> 9.38 mm
Other:
- board text added: "Title: TMP104 Demo Version: V1 September 2024 Author: Dr. Alexandru Enciu"
- board text removed: "RX Matrix"
- board text removed: "TX Matrix"
- board text removed: "Title: TMP104 Demo Version: V0 August 2024 Author: Dr. Alexandru Enciu"
