File: TMP104_DemoBoard/TMP104_Development board/TMP104_Development board.kicad_sch (KiCad schematic)
At the start: 28 parts, among them J1 Conn_02x03_Counter_Clockwise

Commit message: .
Parts:
- removed C10, C9: 0.1 uF, Capacitor_SMD:C_0603_1608Metric, symbol Device:C
- removed J1: Conn_02x03_Counter_Clockwise, Connector_PinHeader_2.54mm:PinHeader_2x03_P2.54mm_Vertical_SMD, symbol Connector_Generic:Conn_02x03_Counter_Clockwise
- removed U1: ~, Molex_PCB_Power_Connector:TMP104, symbol HYDRA_Symbol:TMP104
- added J2: Conn_02x02_Odd_Even, symbol Connector_Generic:Conn_02x02_Odd_Even
Connections:
- net GND: now also U10.3 (GND), U11.3 (GND), U12.3 (GND), U13.3 (GND), U14.3 (GND), U15.3 (GND), U16.3 (GND), U17.3 (GND), U2.3 (GND), U3.3 (GND), U4.3 (GND), U5.3 (GND), U6.3 (GND), U7.3 (GND), U8.3 (GND), U9.3 (GND), J2.3 (Pin_3); no longer U10.2 (GND), U11.2 (GND), U12.2 (GND), U13.2 (GND), U14.2 (GND), U15.2 (GND), U16.2 (GND), U17.2 (GND), U2.2 (GND), U3.2 (GND), U4.2 (GND), U5.2 (GND), U6.2 (GND), U7.2 (GND), U8.2 (GND), U9.2 (GND)
- net RX_2: now also U2.2 (TX), J2.2 (Pin_2); no longer U2.3 (TX)
- net TX_2: now also U14.1 (RX), J2.4 (Pin_4); no longer U14.4 (RX)
- net VCC_3.3V: now also U10.4 (VCC), U11.4 (VCC), U12.4 (VCC), U13.4 (VCC), U14.4 (VCC), U15.4 (VCC), U16.4 (VCC), U17.4 (VCC), U2.4 (VCC), U3.4 (VCC), U4.4 (VCC), U5.4 (VCC), U6.4 (VCC), U7.4 (VCC), U8.4 (VCC), U9.4 (VCC), J2.1 (Pin_1); no longer U10.1 (VCC), U11.1 (VCC), U12.1 (VCC), U13.1 (VCC), U14.1 (VCC), U15.1 (VCC), U16.1 (VCC), U17.1 (VCC), U2.1 (VCC), U3.1 (VCC), U4.1 (VCC), U5.1 (VCC), U6.1 (VCC), U7.1 (VCC), U8.1 (VCC), U9.1 (VCC)
- new net: U2.1 (RX), U3.2 (TX)
- new net: U6.1 (RX), U7.2 (TX)
- new net: U5.1 (RX), U6.2 (TX)
- new net: U10.1 (RX), U17.2 (TX)
- new net: U10.2 (TX), U11.1 (RX)
- new net: U4.1 (RX), U5.2 (TX)
- new net: U11.2 (TX), U12.1 (RX)
- new net: U12.2 (TX), U13.1 (RX)
- new net: U13.2 (TX), U9.1 (RX)
- new net: U16.2 (TX), U17.1 (RX)
- new net: U15.2 (TX), U16.1 (RX)
- new net: U14.2 (TX), U15.1 (RX)
- new net: U3.1 (RX), U4.2 (TX)
- new net: U7.1 (RX), U8.2 (TX)
- new net: U8.1 (RX), U9.2 (TX)
