File: HYDRA_VMM3_Adapter_V2/HYDRA_VMM3_Adapter_V2.kicad_sch (KiCad schematic)
At the start: 32 parts, among them J1 ME1014010101011, J10 MCX-J-P-X-RA-SM1, J12 MCX-J-P-X-RA-SM1, J13 Conn_01x01_Socket, J14 Conn_01x01_Socket, J15 Conn_01x01_Socket, J16 Conn_01x01_Socket, J2 ME1014010101011, J3 ME1014010101011, J4 ME1014010101011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

Commit message: .
Connections:
- net Master_Trigg_B_In: now reaches J12.1
- net Heimtime_B_In: now reaches J10.1
Changed lines of the file:
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@@
 	(global_label "Col_40-Row_15"
 		(shape input)
-		(at 260.35 67.31 0)
+		(at 260.35 67.31 180)
 		(fields_autoplaced yes)
 		(effects
@@
 				(size 1.27 1.27)
 			)
-			(justify left)
+			(justify right)
 		)
 		(property "Intersheetrefs" "${INTERSHEET_REFS}"
-			(at 278.5145 67.31 0)
+			(at 242.1855 67.31 0)
 			(effects
 				(font
 					(size 1.27 1.27)
 				)
-				(justify left)
+				(justify right)
 				(hide yes)
 			)
@@
 		)
 	)
+	(global_label "Heimtime_B_In"
+		(shape input)
+		(at 171.45 241.3 0)
+		(fields_autoplaced yes)
+		(effects
+			(font
+				(size 1.27 1.27)
+			)
+			(justify left)
+		)
+		(property "Intersheetrefs" "${INTERSHEET_REFS}"
+			(at 188.2238 241.3 0)
+			(effects
+				(font
+					(size 1.27 1.27)
+				)
+				(justify left)
+				(hide yes)
+			)
+		)
+	)
 	(global_label "Col_2-Row_9"
 		(shape input)
@@
 				(hide yes)
 			)
+		)
+	)
+	(global_label "Master_Trigg_B_In"
+		(shape input)
+		(at 215.9 241.3 0)
+		(fields_autoplaced yes)
+		(effects
+			(font
+				(size 1.27 1.27)
+			)
+			(justify left)
+		)
+		(property "Intersheetrefs" "${INTERSHEET_REFS}"
+			(at 235.6974 241.3 0)
+			(effects
+				(font
+					(size 1.27 1.27)
+				)
+				(justify left)
+				(hide yes)
+			)
