File: HYDRA_VMM3_card/HYDRA_VMM3_CARD_V2/HYDRA_VMM3_CARD_V2.kicad_pcb (KiCad board)
At the start: 6 copper layers, 105.3 x 61 mm, 88 parts, among them J1 ME1014010101011

Commit message: .
Parts:
- added J2: Conn_01x06_Pin, Connector_PinHeader_1.00mm:PinHeader_1x06_P1.00mm_Horizontal, F.Cu at (137.8, 44.3)
Connections:
- U1 pad 135: unconnected-(U1-Pad135) -> GND
- U1 pad 136: unconnected-(U1-Pad136) -> I2C_VCC
- U1 pad 137: unconnected-(U1-Pad137) -> Signal_In
- U1 pad 138: unconnected-(U1-Pad138) -> Signal_Out
- U1 pad 139: unconnected-(U1-Pad139) -> SDA
- U1 pad 140: unconnected-(U1-Pad140) -> SCL
Routing:
- net I2C_VCC: track 0.00 -> 43.9 mm, vias 0 -> 1
- net Signal_Out: track 0.00 -> 43.8 mm, vias 0 -> 1
- net SDA: track 0.00 -> 42.2 mm, vias 0 -> 1
- net SCL: track 0.00 -> 42.2 mm, vias 0 -> 1
- net Signal_In: track 0.00 -> 35.1 mm, vias 0 -> 1
Other:
- board text added: "Project: VMM3a-Hybrid Card Adapter Version: V_0.1 11.07.2024 Author: Alexandru Enciu Institution: TU Darmstadt"
- board text removed: "Project: VMM3a-Hybrid Card Adapter Version: V_2 23.09.2024 Author: Dr. Alexandru Enciu Institution: TU Darmstadt"

Commit message: .
Parts:
- removed 25: , 
- removed the ? at (53.0, 79.4)
- removed the ? at (139.4, 57.6)
- removed Ch1, Ch10, Ch11, Ch12, Ch13, Ch14, Ch15, Ch16, Ch2, Ch3, Ch4, Ch5, Ch6, Ch7, Ch8, Ch9, Sig1_selector, Sig2_selector: TestPoint, TestPoint:TestPoint_Pad_D1.0mm
- removed J2: Conn_01x06_Pin, Connector_PinHeader_1.00mm:PinHeader_1x06_P1.00mm_Horizontal
- removed REF** (x2): TestPoint_Pad_1.0x1.0mm, TestPoint:TestPoint_Pad_1.0x1.0mm
- removed REF**, REF**1, REF**2, REF**3: MountingHole_2.2mm_M2_DIN965_Pad, MountingHole:MountingHole_2.2mm_M2_DIN965_Pad
- removed Sig1, Sig2: 20449-001E-03, IPEX:IPEX_20449-001E-03
- removed Temp_2: ~, IPEX:TMP104
- moved Temp_1 17.9 mm to (95.2, 58.1)
Routing:
- net P1: track 80.3 -> 0.00 mm, vias 17 -> 0
- net Ch_15: track 75.6 -> 0.00 mm, vias 2 -> 0
- net GND: track 71.6 -> 0.05 mm, vias 806 -> 874
- net Ch_13: track 71.2 -> 0.00 mm, vias 2 -> 0
- net Ch_11: track 69.9 -> 0.00 mm, vias 2 -> 0
- net Ch_16: track 69.8 -> 0.00 mm, vias 1 -> 0
- net Ch_14: track 66.8 -> 0.00 mm, vias 1 -> 0
- net Ch_9: track 66.0 -> 0.00 mm, vias 2 -> 0
- net Ch_7: track 65.4 -> 0.00 mm, vias 2 -> 0
- net Ch_12: track 64.1 -> 0.00 mm, vias 1 -> 0
- net Ch_3: track 62.8 -> 0.00 mm, vias 2 -> 0
- net Ch_5: track 62.3 -> 0.00 mm, vias 2 -> 0
- net Ch_10: track 61.7 -> 0.00 mm, vias 1 -> 0
- net Ch_1: track 60.6 -> 0.00 mm, vias 2 -> 0
- net Ch_8: track 59.7 -> 0.00 mm, vias 1 -> 0
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Other:
- board text added: "Project: VMM3a-Hybrid Card Adapter Version: V_2 13.12.2024 Author: Alexandru Enciu Institution: TU Darmstadt"
- board text removed: "Heim time"
- board text removed: "Heim time CH selector"
- board text removed: "Master trigger"
- board text removed: "Master trigger CH selector"
- board text removed: "Project: VMM3a-Hybrid Card Adapter Version: V_0.1 11.07.2024 Author: Alexandru Enciu Institution: TU Darmstadt"

Commit message: .
Parts:
- removed the ? at (138.1, 34.7)
- removed the ? at (138.1, 37.2)
- added C1: 100nF, Capacitor_SMD:C_0402_1005Metric, B.Cu at (95.2, 59.3)
- added R3: 10k, Resistor_SMD:R_0201_0603Metric, F.Cu at (60.2, 84.9)
- added R4: 10k, Resistor_SMD:R_0201_0603Metric, F.Cu at (60.2, 86.7)
- added R5: 10k, Resistor_SMD:R_0201_0603Metric, F.Cu at (60.2, 88.4)
- added R6: 10k, Resistor_SMD:R_0201_0603Metric, F.Cu at (60.2, 90.2)
- added R7: 10k, Resistor_SMD:R_0201_0603Metric, F.Cu at (60.2, 91.9)
- added R8: 10k, Resistor_SMD:R_0201_0603Metric, F.Cu at (60.2, 93.7)
- moved 1.8V_2.5A1 5.32 mm to (71.9, 66.0), turned to 180 degrees
- moved 1.8_On1 5.27 mm to (64.5, 69.5)
- moved R2 5.27 mm to (66.5, 69.6)
- moved 3.3V_0.5A1 4.45 mm to (71.9, 61.0), turned to 180 degrees
- moved Temp_TX1 2.10 mm to (90.2, 36.6)
- moved 3.3V_On1 1.13 mm to (64.5, 57.5)
- moved R1 1.13 mm to (66.5, 57.4)
- moved Temp_RX1 0.92 mm to (100.2, 36.6)
- turned Temp_1 to 180 degrees
Connections:
- net Net-(1.8_On1-A) renamed P2_Out
- net Net-(3.3V_On1-A) renamed P1_Out
- J1 pad A10: P2 -> Heimtime
- J1 pad A5: P2 -> GND
- J1 pad A6: P2 -> Master_Trigg
- J1 pad A7: P2 -> GND
- J1 pad A8: P2 -> GND
- J1 pad A9: P2 -> GND
- J1 pad B1: P1 -> P2
- J1 pad B10: GND -> P1
- J1 pad B2: P1 -> P2
- J1 pad B3: P1 -> P2
- J1 pad B4: P1 -> P2
- J1 pad B8: GND -> P1
- J1 pad B9: GND -> P1
- Temp_1 pad 4: Net-(Temp_1-RX) -> RX
- U1 pad 1: unconnected-(U1-Pad1) -> bit_0
- U1 pad 135: GND -> unconnected-(U1-Pad135)
- U1 pad 136: I2C_VCC -> unconnected-(U1-Pad136)
- U1 pad 137: Signal_In -> unconnected-(U1-Pad137)
- U1 pad 138: Signal_Out -> unconnected-(U1-Pad138)
- U1 pad 139: SDA -> unconnected-(U1-Pad139)
- U1 pad 140: SCL -> unconnected-(U1-Pad140)
- U1 pad 2: unconnected-(U1-Pad2) -> bit_1
- U1 pad 3: unconnected-(U1-Pad3) -> bit_2
- U1 pad 4: unconnected-(U1-Pad4) -> bit_3
- U1 pad 5: unconnected-(U1-Pad5) -> bit_4
- U1 pad 6: unconnected-(U1-Pad6) -> bit_5
Routing:
- net Ch_19: track 64.0 -> 0.00 mm, vias 1 -> 0
- net Ch_17: track 63.3 -> 0.00 mm, vias 1 -> 0
- net Ch_23: track 62.6 -> 0.00 mm, vias 1 -> 0
- net Ch_21: track 61.9 -> 0.00 mm, vias 1 -> 0
- net Ch_18: track 61.3 -> 0.00 mm
- net Ch_27: track 60.7 -> 0.00 mm, vias 1 -> 0
- net Ch_20: track 60.6 -> 0.00 mm
- net Ch_25: track 60.0 -> 0.00 mm, vias 1 -> 0
- net Ch_22: track 59.9 -> 0.00 mm
- net Ch_31: track 59.3 -> 0.00 mm, vias 1 -> 0
- net Ch_24: track 59.2 -> 0.00 mm
- net Ch_29: track 58.6 -> 0.00 mm, vias 1 -> 0
- net Ch_26: track 58.1 -> 0.00 mm
- net Ch_35: track 57.9 -> 0.00 mm, vias 1 -> 0
- net Ch_28: track 57.3 -> 0.00 mm
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- added copper zone on B.Cu, net P1
- added copper zone on F.Cu, net P1
- added copper zone on B.Cu, net P1_Out
- added copper zone on B.Cu, net P2
- added copper zone on B.Cu, net P2_Out
