File: HYDRA_VMM3_card/HYDRA_VMM3_CARD_V2/HYDRA_VMM3_CARD_V2.kicad_pcb (KiCad board)
At the start: 6 copper layers, 105.3 x 61 mm, 63 parts, among them J1 ME1014010101011

Commit message: .
Parts:
- added C10: TCJB475M025R0100, Capacitor_Tantalum_SMD:CP_EIA-3528-12_Kemet-T, F.Cu at (59.7, 66.6)
- added C11: TCJB475M025R0100, Capacitor_Tantalum_SMD:CP_EIA-3528-12_Kemet-T, F.Cu at (59.7, 57.1)
- added C2: 10nF, Capacitor_SMD:C_0402_1005Metric, F.Cu at (139.1, 43.3)
- added C3: 10nF, Capacitor_SMD:C_0402_1005Metric, F.Cu at (139.8, 52.8)
- added C4: 10nF, Capacitor_SMD:C_0402_1005Metric, F.Cu at (142.3, 50.4)
- added C5: 10nF, Capacitor_SMD:C_0402_1005Metric, F.Cu at (138.1, 60.9)
- added C6: 10nF, Capacitor_SMD:C_0402_1005Metric, F.Cu at (138.1, 62.9)
- added C7: 10nF, Capacitor_SMD:C_0402_1005Metric, F.Cu at (138.1, 64.9)
- added C8: TCJB475M025R0100, Capacitor_Tantalum_SMD:CP_EIA-3528-12_Kemet-T, F.Cu at (59.7, 60.6)
- added C9: TCJB475M025R0100, Capacitor_Tantalum_SMD:CP_EIA-3528-12_Kemet-T, F.Cu at (59.7, 70.1)
- added R10: 0, Resistor_SMD:R_0201_0603Metric, F.Cu at (136.4, 45.0)
- added R11: 0, Resistor_SMD:R_0201_0603Metric, F.Cu at (136.4, 46.7)
- added R12: 0, Resistor_SMD:R_0201_0603Metric, F.Cu at (136.4, 48.5)
- added R13: 0, Resistor_SMD:R_0201_0603Metric, F.Cu at (136.4, 50.2)
- added R14: 10k, Resistor_SMD:R_0201_0603Metric, F.Cu at (135.5, 60.8)
- added R15: 0, Resistor_SMD:R_0201_0603Metric, F.Cu at (135.5, 62.6)
- added R16: 0, Resistor_SMD:R_0201_0603Metric, F.Cu at (135.5, 64.3)
- added R17: 0, Resistor_SMD:R_0201_0603Metric, F.Cu at (135.5, 66.1)
- added R18: 0, Resistor_SMD:R_0201_0603Metric, F.Cu at (135.5, 67.8)
- added R19: 33, Resistor_SMD:R_0201_0603Metric, F.Cu at (136.4, 52.0)
- added R20: 33, Resistor_SMD:R_0201_0603Metric, F.Cu at (135.5, 69.6)
- added R21: 33, Resistor_SMD:R_0201_0603Metric, F.Cu at (145.8, 49.3)
- added R22: 33, Resistor_SMD:R_0201_0603Metric, F.Cu at (150.2, 49.3)
- added R23: 33, Resistor_SMD:R_0201_0603Metric, F.Cu at (145.8, 51.1)
- added R24: 33, Resistor_SMD:R_0201_0603Metric, F.Cu at (150.2, 51.1)
- added R25: 33, Resistor_SMD:R_0201_0603Metric, F.Cu at (145.8, 52.8)
- added R26: 33, Resistor_SMD:R_0201_0603Metric, F.Cu at (150.2, 52.8)
- added R9: 10k, Resistor_SMD:R_0201_0603Metric, F.Cu at (136.4, 43.2)
- added U2: ~, Custom_Footprints:5PB1214CMGK8, F.Cu at (139.8, 50.4)
- added U3: ~, Custom_Footprints:5PB1214CMGK8, F.Cu at (138.9, 68.0)
- R1: renamed from R3; moved to B.Cu
- R2: renamed from R4; moved to B.Cu
- R3: renamed from R5; moved to B.Cu
- R4: renamed from R8; moved to B.Cu
- R5: renamed from R7; moved to B.Cu
- R6: moved to B.Cu
- moved R4 86.0 mm to (126.0, 38.3), turned to 180 degrees
- moved R5 85.4 mm to (127.7, 39.5), turned to 180 degrees
- moved R3 84.0 mm to (127.7, 38.3), turned to 180 degrees
- moved R6 83.0 mm to (126.0, 39.5), turned to 180 degrees
- moved R1 82.7 mm to (127.7, 37.1), turned to 180 degrees
- moved R2 82.4 mm to (126.0, 37.1), turned to 180 degrees
- renumbered R1 to R7, R2 to R8
Routing:
- net P1: track 0.32 -> 2.21 mm, vias 108 -> 86
- net GND: track 0.44 -> 1.51 mm
- net P2_Out: vias 0 -> 54
- net P1_Out: vias 0 -> 54
- added copper zone on In3.Cu, net P1
- added copper zone on F.Cu, net P1_Out
- added copper zone on F.Cu, net P2_Out
Other:
- board text added: "Geographical code"

Commit message: .
Parts:
- 3.3V_2A1: renamed from 3.3V_0.5A1; value 0.5A -> 2A
- C2, C3, C4, C5, C6, C7: footprint Capacitor_SMD:C_0402_1005Metric -> Capacitor_SMD:C_0201_0603Metric
- U2, U3: value ~ -> 5PB1214CMGK8
- renumbered 1.8V_2.5A1 to 1.8V_3.5A1
Connections:
- net Net-(U2-OE_1) renamed /Master_trigg/Enable_1
- net Net-(U2-OE_2) renamed /Master_trigg/Enable_2
- net Net-(U2-OE_3) renamed /Master_trigg/Enable_3
- net Net-(U2-OE_4) renamed /Master_trigg/Enable_4
- net Net-(U3-OE_1) renamed /Heimtime/Enable_1
- net Net-(U3-OE_2) renamed /Heimtime/Enable_2
- net Net-(U3-OE_3) renamed /Heimtime/Enable_3
- net Net-(U3-OE_4) renamed /Heimtime/Enable_4
Routing:
- net GND: track 1.51 -> 0.44 mm
- net P1: track 2.21 -> 1.14 mm, vias 86 -> 85
