File: HYDRA_VMM3_card/HYDRA_VMM3_CARD_V2/HYDRA_VMM3_CARD_V2.kicad_pcb (KiCad board)
At the start: 6 copper layers, 105.3 x 61 mm, 93 parts, among them J1 ME1014010101011, U2 5PB1214CMGK8, U3 5PB1214CMGK8

Commit message: .
Parts:
- removed 10, 16, 18, 19, 21, 22, 3, 6: , 
- removed the ? at (111.4, 37.2)
- removed the ? at (138.1, 80.9)
- removed the ? at (111.4, 34.7)
- removed the ? at (138.1, 78.4)
- removed R14, R9: 10k, Resistor_SMD:R_0201_0603Metric
- C5, C6, C7, R15, R16, R17, R18, R20, R22, R24, R26, U3: moved to B.Cu
- moved R22 17.8 mm to (134.4, 57.4), turned to 180 degrees
- moved R24 17.4 mm to (134.4, 58.3), turned to 180 degrees
- moved R26 17.0 mm to (134.8, 59.8), turned to -135 degrees
- moved R10 15.2 mm to (137.4, 60.2), turned to 90 degrees
- moved R21 14.5 mm to (134.4, 58.3), turned to 180 degrees
- moved C2 14.5 mm to (138.8, 57.8), turned to -90 degrees
- moved R20 14.2 mm to (136.2, 55.4), turned to 90 degrees
- moved R23 13.0 mm to (134.4, 57.4), turned to 180 degrees
- moved R11 12.5 mm to (139.1, 59.0), turned to 180 degrees
- moved C4 12.0 mm to (134.8, 59.8), turned to 45 degrees
- moved R25 11.4 mm to (134.8, 55.8), turned to 135 degrees
- moved U3 10.4 mm to (136.8, 57.8), turned to 180 degrees
- moved R12 8.60 mm to (139.1, 56.7), turned to 180 degrees
- moved R16 8.48 mm to (139.1, 56.7), turned to 180 degrees
- moved R19 8.22 mm to (136.2, 60.2), turned to -90 degrees
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Connections:
- 1.8_On1 pad 1: Net-(1.8_On1-K) -> GND
- 1.8_On1 pad 2: P2_Out -> Net-(1.8_On1-A)
- 3.3V_On1 pad 1: Net-(3.3V_On1-K) -> GND
- 3.3V_On1 pad 2: P1_Out -> Net-(3.3V_On1-A)
- J1 pad A15: Ch_17 -> Ch_1
- J1 pad A16: Ch_19 -> Ch_3
- J1 pad A17: Ch_21 -> Ch_5
- J1 pad A18: Ch_23 -> Ch_7
- J1 pad A19: Ch_25 -> Ch_9
- J1 pad A20: Ch_27 -> Ch_11
- J1 pad A21: Ch_29 -> Ch_13
- J1 pad A22: Ch_31 -> Ch_15
- J1 pad A23: Ch_33 -> Ch_17
- J1 pad A24: Ch_35 -> Ch_19
- J1 pad A25: Ch_37 -> Ch_21
- J1 pad A26: Ch_39 -> Ch_23
- J1 pad A27: Ch_41 -> Ch_25
- J1 pad A28: Ch_43 -> Ch_27
- J1 pad A29: Ch_45 -> Ch_29
- J1 pad A30: Ch_47 -> Ch_31
- J1 pad A31: Ch_49 -> Ch_33
- J1 pad A32: Ch_51 -> Ch_35
- J1 pad A33: Ch_53 -> Ch_37
- J1 pad A34: Ch_55 -> Ch_39
- J1 pad A35: Ch_57 -> Ch_41
- J1 pad A36: Ch_59 -> Ch_43
- J1 pad A37: Ch_61 -> Ch_45
- J1 pad A38: Ch_63 -> Ch_47
- J1 pad A39: Ch_65 -> Ch_49
- J1 pad A40: Ch_67 -> Ch_51
- J1 pad A41: Ch_69 -> Ch_53
- J1 pad A42: Ch_71 -> Ch_55
- J1 pad B15: Ch_18 -> Ch_4
- J1 pad B16: Ch_20 -> Ch_6
- J1 pad B17: Ch_22 -> Ch_8
- J1 pad B18: Ch_24 -> Ch_10
- J1 pad B19: Ch_26 -> Ch_12
- J1 pad B20: Ch_28 -> Ch_14
- J1 pad B21: Ch_30 -> Ch_16
- J1 pad B22: Ch_32 -> Ch_18
- J1 pad B23: Ch_34 -> Ch_20
- J1 pad B24: Ch_36 -> Ch_22
- J1 pad B25: Ch_38 -> Ch_24
- J1 pad B26: Ch_40 -> Ch_26
- J1 pad B27: Ch_42 -> Ch_28
- J1 pad B28: Ch_44 -> Ch_30
- J1 pad B29: Ch_46 -> Ch_32
- J1 pad B30: Ch_48 -> Ch_34
- J1 pad B31: Ch_50 -> Ch_36
- J1 pad B32: Ch_52 -> Ch_38
- J1 pad B33: Ch_54 -> Ch_40
- J1 pad B34: Ch_56 -> Ch_42
- J1 pad B35: Ch_58 -> Ch_44
- J1 pad B36: Ch_60 -> Ch_46
- J1 pad B37: Ch_62 -> Ch_48
- J1 pad B38: Ch_64 -> Ch_50
- J1 pad B39: Ch_66 -> Ch_52
- J1 pad B40: Ch_68 -> Ch_54
- J1 pad B41: Ch_70 -> Ch_56
- J1 pad B42: Ch_72 -> Ch_58
- J1 pad B43: Ch_74 -> Ch_60
- J1 pad B44: Ch_76 -> Ch_62
- J1 pad B45: Ch_78 -> Ch_64
- J1 pad B46: Ch_80 -> Ch_66
- J1 pad B47: Ch_82 -> Ch_68
- J1 pad B48: Ch_84 -> Ch_70
- J1 pad B49: Ch_86 -> Ch_72
- J1 pad B50: Ch_88 -> Ch_74
- J1 pad B51: Ch_90 -> Ch_76
- J1 pad B52: Ch_92 -> Ch_78
- J1 pad B53: Ch_94 -> Ch_80
- J1 pad B54: Ch_96 -> Ch_82
- J1 pad B55: Ch_98 -> Ch_84
- J1 pad B56: Ch_100 -> Ch_86
- J1 pad B57: Ch_102 -> Ch_88
- J1 pad B58: Ch_104 -> Ch_90
- J1 pad B59: Ch_106 -> Ch_92
- J1 pad B60: Ch_128 -> Ch_94
- J1 pad B61: Ch_126 -> Ch_96
- J1 pad B62: Ch_124 -> Ch_98
- J1 pad B63: Ch_122 -> Ch_100
- J1 pad B64: Ch_120 -> Ch_102
- J1 pad B65: Ch_118 -> Ch_104
- J1 pad B66: Ch_116 -> Ch_106
- J1 pad B67: Ch_114 -> Ch_108
- J1 pad B68: Ch_112 -> Ch_110
- J1 pad B69: Ch_110 -> Ch_112
- J1 pad B70: Ch_108 -> Ch_114
- R19 pad 2: Ch_61 -> Ch_67
- R21 pad 2: Ch_63 -> Ch_65
- R23 pad 2: Ch_65 -> Ch_63
- R25 pad 2: Ch_67 -> Ch_61
- R7 pad 1: Net-(3.3V_On1-K) -> P1_Out
- R7 pad 2: GND -> Net-(3.3V_On1-A)
- R8 pad 1: Net-(1.8_On1-K) -> P2_Out
- R8 pad 2: GND -> Net-(1.8_On1-A)
- U2 pad 6: Net-(U2-OE_OSC) -> unconnected-(U2-OE_OSC-Pad6)
- U3 pad 6: Net-(U3-OE_OSC) -> unconnected-(U3-OE_OSC-Pad6)
Routing:
- net Ch_4: track 0.00 -> 75.9 mm
- net Ch_6: track 0.00 -> 73.9 mm
- net Ch_8: track 0.00 -> 72.4 mm
- net Master_Trigg: track 0.00 -> 72.2 mm, vias 0 -> 2
- net Ch_10: track 0.00 -> 71.0 mm
- net Heimtime: track 0.00 -> 70.5 mm, vias 0 -> 2
- net Ch_12: track 0.00 -> 69.7 mm
- net Ch_14: track 0.00 -> 68.3 mm
- net Ch_16: track 0.00 -> 67.0 mm
- net Ch_18: track 0.00 -> 65.7 mm
- net Ch_20: track 0.00 -> 64.4 mm
- net Ch_22: track 0.00 -> 63.1 mm
- net Ch_24: track 0.00 -> 61.6 mm
- net Ch_26: track 0.00 -> 59.6 mm
- net Ch_28: track 0.00 -> 58.4 mm
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- added copper zone on In5.Cu, net GND
- added copper zone on In6.Cu, net GND
- removed copper zone on In3.Cu, net GND
Other:
- copper layers 6 -> 8

Commit message: .
Parts:
- moved R6 5.16 mm to (122.6, 35.7), turned to 90 degrees
- moved R5 3.99 mm to (128.7, 35.7), turned to 90 degrees
- moved R1 3.70 mm to (131.1, 35.7), turned to 90 degrees
- moved R4 3.45 mm to (123.8, 35.7), turned to 90 degrees
- moved R3 3.45 mm to (129.9, 35.7), turned to 90 degrees
- moved R2 1.75 mm to (125.0, 35.7), turned to 90 degrees
Routing:
- net Ch_14: track 68.3 -> 0.00 mm
- net Ch_18: track 65.7 -> 0.00 mm
- net Ch_22: track 63.1 -> 0.00 mm
- net Ch_28: track 58.4 -> 0.00 mm
- net Ch_32: track 57.4 -> 0.00 mm
- net Ch_36: track 55.0 -> 0.00 mm
- net Ch_40: track 52.7 -> 0.00 mm
- net Ch_44: track 50.4 -> 0.00 mm
- net Ch_48: track 47.9 -> 0.00 mm
- net Ch_52: track 44.2 -> 0.00 mm
- net Ch_60: track 43.0 -> 0.00 mm
- net Ch_56: track 42.7 -> 0.00 mm
- net Ch_64: track 41.7 -> 0.00 mm
- net Ch_68: track 40.0 -> 0.00 mm
- net Ch_72: track 38.3 -> 0.00 mm
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Other:
- board text removed: "Geographical code"

Commit message: .
Connections:
- J1 pad A60: Ch_107 -> Ch_127
- J1 pad A61: Ch_109 -> Ch_125
- J1 pad A62: Ch_111 -> Ch_123
- J1 pad A63: Ch_113 -> Ch_121
- J1 pad A64: Ch_115 -> Ch_119
- J1 pad A66: Ch_119 -> Ch_115
- J1 pad A67: Ch_121 -> Ch_113
- J1 pad A68: Ch_123 -> Ch_111
- J1 pad A69: Ch_125 -> Ch_109
- J1 pad A70: Ch_127 -> Ch_107
Routing:
- net Ch_1: track 0.00 -> 79.7 mm, vias 0 -> 1
- net Ch_3: track 0.00 -> 77.7 mm, vias 0 -> 1
- net Ch_5: track 0.00 -> 77.1 mm, vias 0 -> 1
- net Ch_9: track 0.00 -> 75.5 mm, vias 0 -> 1
- net Ch_7: track 0.00 -> 74.9 mm, vias 0 -> 1
- net Ch_11: track 0.00 -> 72.5 mm, vias 0 -> 1
- net Ch_13: track 0.00 -> 72.2 mm, vias 0 -> 1
- net Ch_17: track 0.00 -> 71.0 mm, vias 0 -> 1
- net Ch_15: track 0.00 -> 70.0 mm, vias 0 -> 1
- net Ch_19: track 0.00 -> 67.7 mm, vias 0 -> 1
- net Ch_21: track 0.00 -> 67.3 mm, vias 0 -> 1
- net Ch_23: track 0.00 -> 65.0 mm, vias 0 -> 1
- net Ch_25: track 0.00 -> 64.0 mm, vias 0 -> 1
- net Ch_29: track 0.00 -> 62.4 mm, vias 0 -> 1
- net Ch_27: track 0.00 -> 61.8 mm, vias 0 -> 1
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