File: FIFO/FIFO_prototype/FIFO_prototype.kicad_sch (KiCad schematic)
At the start: 32 parts, among them J1 Input_clock, J10 Output_C_1, J11 Output_C_3, J12 Output_C_2, J13 Output_C_4, J14 Output_B_1, J15 Output_B_3, J16 Power Connector, J17 Output_B_2, J18 Output_B_4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

Commit message: .
Parts:
- L1: footprint (none) -> Clock_Buffers:WE-TPC_4828; PartNumber (none) -> 7440430018
Connections:
- net +3.3V: now also J16.3 (Pin_3), J16.4 (Pin_4); no longer J16.1 (Pin_1), J16.2 (Pin_2)
- net EN_Group_A: now also SW1.4; no longer SW1.1
- net EN_Group_B: now also SW1.3; no longer SW1.2
- net EN_Group_C: now also SW1.2; no longer SW1.3
- net EN_Group_D: now also SW1.1; no longer SW1.4
- net GND: now also J16.1 (Pin_1), J16.2 (Pin_2); no longer J16.3 (Pin_3), J16.4 (Pin_4)
Other:
- moved on the sheet: J16, SW1
Changed lines of the file:
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@@
 	)
 	(junction
-		(at 72.39 46.99)
+		(at 72.39 44.45)
 		(diameter 0)
 		(color 0 0 0 0)
@@
 	)
 	(junction
-		(at 73.66 46.99)
+		(at 71.12 44.45)
 		(diameter 0)
 		(color 0 0 0 0)
@@
 	)
 	(junction
-		(at 71.12 46.99)
+		(at 73.66 44.45)
 		(diameter 0)
 		(color 0 0 0 0)
@@
 	(wire
 		(pts
-			(xy 73.66 46.99) (xy 76.2 46.99)
+			(xy 71.12 44.45) (xy 68.58 44.45)
 		)
 		(stroke
@@
 	(wire
 		(pts
-			(xy 73.66 62.23) (xy 73.66 74.93)
-		)
-		(stroke
-			(width 0)
-			(type default)
-		)
-	)
-	(wire
-		(pts
-			(xy 76.2 62.23) (xy 76.2 74.93)
-		)
-		(stroke
-			(width 0)
-			(type default)
-		)
-	)
-	(wire
-		(pts
 			(xy 236.22 33.02) (xy 236.22 34.29)
 		)
@@
 	(wire
 		(pts
-			(xy 71.12 46.99) (xy 72.39 46.99)
+			(xy 73.66 44.45) (xy 72.39 44.45)
 		)
 		(stroke
@@
 	(wire
 		(pts
+			(xy 68.58 59.69) (xy 68.58 74.93)
+		)
+		(stroke
+			(width 0)
+			(type default)
+		)
+	)
+	(wire
+		(pts
 			(xy 109.22 173.99) (xy 127 173.99)
 		)
@@
 	(wire
 		(pts
+			(xy 71.12 59.69) (xy 71.12 74.93)
+		)
+		(stroke
+			(width 0)
+			(type default)
+		)
+	)
+	(wire
+		(pts
 			(xy 154.94 81.28) (xy 154.94 99.06)
 		)
@@
 	(wire
 		(pts
-			(xy 72.39 45.72) (xy 72.39 46.99)
+			(xy 73.66 59.69) (xy 73.66 74.93)
+		)
+		(stroke
+			(width 0)
+			(type default)
+		)
+	)
+	(wire
+		(pts
+			(xy 72.39 43.18) (xy 72.39 44.45)
 		)
 		(stroke
@@
 	(wire
 		(pts
-			(xy 72.39 46.99) (xy 73.66 46.99)
+			(xy 72.39 44.45) (xy 71.12 44.45)
 		)
 		(stroke
@@
 	(wire
 		(pts
-			(xy 68.58 62.23) (xy 68.58 74.93)
-		)
-		(stroke
-			(width 0)
-			(type default)
-		)
-	)
-	(wire
-		(pts
 			(xy 64.77 102.87) (xy 64.77 107.95)
 		)
@@
 	(wire
 		(pts
-			(xy 149.86 105.41) (xy 149.86 114.3)
+			(xy 76.2 59.69) (xy 76.2 74.93)
 		)
 		(stroke
@@
 	(wire
 		(pts
-			(xy 100.33 53.34) (xy 101.6 53.34)
+			(xy 149.86 105.41) (xy 149.86 114.3)
 		)
 		(stroke
@@
 	(wire
 		(pts
-			(xy 71.12 62.23) (xy 71.12 74.93)
+			(xy 100.33 53.34) (xy 101.6 53.34)
 		)
 		(stroke
@@
 	(wire
 		(pts
-			(xy 68.58 46.99) (xy 71.12 46.99)
+			(xy 76.2 44.45) (xy 73.66 44.45)
 		)
 		(stroke
@@
 	(symbol
 		(lib_id "power:VCC")
-		(at 72.39 45.72 0)
+		(at 72.39 43.18 0)
+		(mirror y)
 		(unit 1)
 		(exclude_from_sim no)
@@
 		(dnp no)
 		(property "Reference" "#PWR06"
-			(at 72.39 49.53 0)
+			(at 72.39 46.99 0)
 			(effects
 				(font
@@
 		)
 		(property "Value" "+3.3V_Filtered"
-			(at 72.39 42.164 0)
+			(at 72.39 39.624 0)
 			(effects
 				(font
@@
 		)
 		(property "Footprint" ""
-			(at 72.39 45.72 0)
+			(at 72.39 43.18 0)
 			(effects
 				(font
@@
 		)
 		(property "Datasheet" ""
-			(at 72.39 45.72 0)
+			(at 72.39 43.18 0)
 			(effects
 				(font
@@
 		)
 		(property "Description" "Power symbol creates a global label with name \"VCC\""
-			(at 72.39 45.72 0)
+			(at 72.39 43.18 0)
 			(effects
 				(font
@@
 	(symbol
 		(lib_id "Connector_Generic:Conn_02x02_Counter_Clockwise")
-		(at 228.6 33.02 0)
+		(at 231.14 35.56 180)
 		(unit 1)
 		(exclude_from_sim no)
@@
 		)
 		(property "Value" "Power Connector"
-			(at 226.568 38.1 0)
+			(at 234.95 30.226 0)
 			(effects
 				(font
@@
 		)
 		(property "Footprint" "Clock_Buffers:SAMTEC_IPL1-102-01-X-D-RA-K"
-			(at 228.6 33.02 0)
+			(at 231.14 35.56 0)
 			(effects
 				(font
@@
 		)
 		(property "Datasheet" "~"
-			(at 228.6 33.02 0)
+			(at 231.14 35.56 0)
 			(effects
 				(font
@@
 		)
 		(property "Description" "Generic connector, double row, 02x02, counter clockwise pin numbering scheme (similar to DIP package numbering), script generated (kicad-library-utils/schlib/autogen/connector/)"
-			(at 228.6 33.02 0)
+			(at 231.14 35.56 0)
 			(effects
 				(font
@@
 			)
 		)
-		(property "Footprint" ""
+		(property "Footprint" "Clock_Buffers:WE-TPC_4828"
 			(at 238.76 48.26 0)
 			(effects
@@
 			)
 		)
+		(property "PartNumber" "7440430018"
+			(at 238.76 48.26 90)
+			(effects
+				(font
+					(size 1.27 1.27)
+				)
+				(hide yes)
+			)
+		)
 		(pin "1"
 		)
@@
 	(symbol
 		(lib_id "Switch:SW_DIP_x04")
-		(at 73.66 54.61 90)
+		(at 71.12 52.07 270)
+		(mirror x)
 		(unit 1)
 		(exclude_from_sim no)
@@
 		(dnp no)
 		(property "Reference" "SW1"
-			(at 61.468 51.816 90)
+			(at 83.312 49.276 90)
 			(effects
 				(font
@@
 		)
 		(property "Value" "SW_DIP_x04"
-			(at 53.34 54.61 90)
+			(at 91.44 52.07 90)
 			(effects
 				(font
@@
 		)
 		(property "Footprint" "Button_Switch_SMD:SW_DIP_SPSTx04_Slide_6.7x11.72mm_W6.73mm_P2.54mm_LowProfile_JPin"
-			(at 73.66 54.61 0)
+			(at 71.12 52.07 0)
 			(effects
 				(font
@@
 		)
 		(property "Datasheet" "~"
-			(at 73.66 54.61 0)
+			(at 71.12 52.07 0)
 			(effects
 				(font
@@
 		)
 		(property "Description" "4x DIP Switch, Single Pole Single Throw (SPST) switch, small symbol"
-			(at 73.66 54.61 0)
+			(at 71.12 52.07 0)
 			(effects
 				(font

Commit message: .
Connections:
- net EN_A_1: now also SW3.4; no longer SW3.1
- net EN_A_2: now also SW3.3; no longer SW3.2
- net EN_A_3: now also SW3.2; no longer SW3.3
- net EN_A_4: now also SW3.1; no longer SW3.4
- net EN_B_1: now also SW5.4; no longer SW5.1
- net EN_B_2: now also SW5.3; no longer SW5.2
- net EN_B_3: now also SW5.2; no longer SW5.3
- net EN_B_4: now also SW5.1; no longer SW5.4
- net EN_C_1: now also SW4.4; no longer SW4.1
- net EN_C_2: now also SW4.3; no longer SW4.2
- net EN_C_3: now also SW4.2; no longer SW4.3
- net EN_C_4: now also SW4.1; no longer SW4.4
- net EN_D_1: now also SW2.4; no longer SW2.1
- net EN_D_2: now also SW2.3; no longer SW2.2
- net EN_D_3: now also SW2.2; no longer SW2.3
- net EN_D_4: now also SW2.1; no longer SW2.4
Other:
- title: 16 Channels FIFO -> 16 Channels Clock Buffer
- moved on the sheet: SW2, SW3, SW4, SW5
