File: FIFO/FIFO_prototype/clock_buffer.kicad_sch (KiCad schematic)
At the start: 8 parts, among them U2 5PB1214CMGK8

Commit message: .
Other:
- title: 16 Channels FIFO -> 16 Channels Clock Buffer
Changed lines of the file:
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@@
 	(paper "A4")
 	(title_block
-		(title "16 Channels FIFO")
+		(title "16 Channels Clock Buffer")
 		(date "2025-01-07")
 		(rev "REV 0")
