File: FIFO/FIFO_prototype/FIFO_prototype.kicad_pcb (KiCad board)
At the start: 2 copper layers, 183 x 114.5 mm, 72 parts, among them J1 Input_clock, J10 Output_C_1, J11 Output_C_3, J12 Output_C_2, J13 Output_C_4, J14 Output_B_1, J15 Output_B_3, J16 Power Connector, J17 Output_B_2, J18 Output_B_4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

Commit message: .
Parts:
- moved C17 184.5 mm to (-15.6, 24.1)
- moved C18 184.5 mm to (-15.6, 25.9)
- moved C19 184.5 mm to (-15.6, 27.6)
- moved R19 184.5 mm to (-15.6, 29.4)
- moved R20 184.5 mm to (-15.6, 31.1)
- moved R21 184.5 mm to (-15.6, 32.9)
- moved R22 184.5 mm to (-15.6, 34.6)
- moved U5 184.5 mm to (-12.5, 25.2)
- moved SW2 156.5 mm to (-22.8, 29.5)
- moved C1 117.3 mm to (55.7, 93.4), turned to 180 degrees
- moved C2 104.0 mm to (67.7, 93.4)
- moved L1 101.6 mm to (61.7, 88.4), turned to 180 degrees
- moved J6 100.9 mm to (45.8, 29.0)
- moved C14 100.7 mm to (240.0, 121.8)
- moved C15 100.7 mm to (240.0, 123.5)
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Connections:
- J16 pad 1: +3.3V -> GND
- J16 pad 2: +3.3V -> GND
- J16 pad 3: GND -> +3.3V
- J16 pad 4: GND -> +3.3V
- SW1 pad 1: /EN_Group_A -> /EN_Group_D
- SW1 pad 2: /EN_Group_B -> /EN_Group_C
- SW1 pad 3: /EN_Group_C -> /EN_Group_B
- SW1 pad 4: /EN_Group_D -> /EN_Group_A
Routing:
- net /Input_Buffer/ClK_IN: track 0.00 -> 16.1 mm
- net /EN_Group_D: track 0.00 -> 10.2 mm
- net /EN_Group_A: track 0.00 -> 9.60 mm
- net /EN_Group_C: track 0.00 -> 9.20 mm
- net /EN_Group_B: track 0.00 -> 8.29 mm
- net GND: track 0.00 -> 3.99 mm, vias 0 -> 45
- net Net-(JP1-A): track 0.00 -> 2.25 mm
- net +3.3V_Filtered: track 0.00 -> 1.59 mm, vias 0 -> 56
- net Net-(D1-A): track 0.00 -> 1.39 mm
- added copper zone on F.Cu, net +3.3V
- added copper zone on B.Cu, net +3.3V_Filtered
- added copper zone on F.Cu, net +3.3V_Filtered
- added copper zone on F.Cu, net GND
- added copper zone on In1.Cu, net GND
- added copper zone on In2.Cu, net GND
Other:
- board size 183 x 114.5 mm -> 138.7 x 80 mm
- copper layers 2 -> 4
- board text added: "Power 3V3"

Commit message: .
Parts:
- C10, C5, C7, C9: moved to B.Cu
- moved R7 156.6 mm to (56.6, 43.8), turned to 180 degrees
- moved U2 156.6 mm to (58.9, 44.9), turned to 90 degrees
- moved R8 155.5 mm to (58.4, 42.4), turned to 90 degrees
- moved R9 155.0 mm to (59.3, 42.4), turned to 90 degrees
- moved C10 153.9 mm to (58.9, 44.9)
- moved C9 153.8 mm to (58.9, 43.8), turned to 180 degrees
- moved R10 153.2 mm to (61.2, 43.8)
- moved C8 153.1 mm to (58.9, 46.9), turned to 180 degrees
- moved SW3 142.9 mm to (58.9, 64.9), turned to -90 degrees
- moved U3 136.0 mm to (93.7, 44.9), turned to 90 degrees
- moved C11 122.2 mm to (102.5, 50.8)
- moved C12 122.2 mm to (102.5, 52.6)
- moved C13 122.2 mm to (102.5, 54.3)
- moved R11 122.2 mm to (102.5, 56.1)
- moved R12 122.2 mm to (102.5, 57.8)
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Connections:
- SW2 pad 1: /EN_D_1 -> /EN_D_4
- SW2 pad 2: /EN_D_2 -> /EN_D_3
- SW2 pad 3: /EN_D_3 -> /EN_D_2
- SW2 pad 4: /EN_D_4 -> /EN_D_1
- SW3 pad 1: /EN_A_1 -> /EN_A_4
- SW3 pad 2: /EN_A_2 -> /EN_A_3
- SW3 pad 3: /EN_A_3 -> /EN_A_2
- SW3 pad 4: /EN_A_4 -> /EN_A_1
- SW4 pad 1: /EN_C_1 -> /EN_C_4
- SW4 pad 2: /EN_C_2 -> /EN_C_3
- SW4 pad 3: /EN_C_3 -> /EN_C_2
- SW4 pad 4: /EN_C_4 -> /EN_C_1
- SW5 pad 1: /EN_B_1 -> /EN_B_4
- SW5 pad 2: /EN_B_2 -> /EN_B_3
- SW5 pad 3: /EN_B_3 -> /EN_B_2
- SW5 pad 4: /EN_B_4 -> /EN_B_1
Routing:
- net /Input_Clock_Group_A: track 0.00 -> 74.6 mm, vias 0 -> 2
- net /Input_Clock_Group_B: track 0.00 -> 50.0 mm, vias 0 -> 2
- net /Output_Group_A/ClK_Out1: track 0.00 -> 21.9 mm
- net /Output_Group_A/ClK_Out4: track 0.00 -> 21.8 mm
- net /Output_Group_A/ClK_Out2: track 0.00 -> 19.3 mm
- net /Output_Group_A/ClK_Out3: track 0.00 -> 17.6 mm
- net /EN_A_4: track 0.00 -> 17.4 mm
- net /EN_B_1: track 0.00 -> 17.4 mm
- net /EN_A_1: track 0.00 -> 17.4 mm
- net /EN_B_4: track 0.00 -> 17.3 mm
- net /EN_B_2: track 0.00 -> 15.8 mm
- net /EN_A_2: track 0.00 -> 15.8 mm
- net /EN_B_3: track 0.00 -> 15.8 mm
- net /EN_A_3: track 0.00 -> 15.8 mm
- net +3.3V_Filtered: track 1.59 -> 6.81 mm, vias 56 -> 59
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
Commit message: .
Parts:
- moved C17 190.9 mm to (174.6, 40.3)
- moved C18 190.9 mm to (174.6, 42.0)
- moved C19 190.9 mm to (174.6, 43.8)
- moved R19 190.9 mm to (174.6, 45.5)
- moved R20 190.9 mm to (174.6, 47.3)
- moved R21 190.9 mm to (174.6, 49.0)
- moved R22 190.9 mm to (174.6, 50.8)
- moved SW2 189.4 mm to (163.2, 64.9), turned to -90 degrees
- moved U5 176.8 mm to (163.2, 44.9), turned to 90 degrees
- moved R17 141.9 mm to (128.9, 42.4), turned to 90 degrees
- moved R16 141.5 mm to (128.0, 42.4), turned to 90 degrees
- moved R15 140.8 mm to (126.1, 44.3), turned to 180 degrees
- moved R18 140.3 mm to (130.8, 44.3)
- moved U4 138.7 mm to (128.4, 44.9), turned to 90 degrees
- moved C16 136.3 mm to (128.4, 46.9), turned to 180 degrees
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Routing:
- net /Input_Clock_Group_C: track 0.00 -> 49.7 mm, vias 0 -> 2
- net /Output_Group_B/ClK_Out1: track 0.00 -> 22.0 mm
- net /Output_Group_B/ClK_Out4: track 0.00 -> 22.0 mm
- net /Output_Group_C/ClK_Out4: track 0.00 -> 21.9 mm
- net /Output_Group_C/ClK_Out1: track 0.00 -> 21.9 mm
- net /Output_Group_B/ClK_Out2: track 0.00 -> 21.9 mm
- net /Output_Group_B/ClK_Out3: track 0.00 -> 21.9 mm
- net /Output_Group_C/ClK_Out2: track 0.00 -> 21.9 mm
- net /Output_Group_C/ClK_Out3: track 0.00 -> 21.9 mm
- net /EN_C_4: track 0.00 -> 17.5 mm
- net /EN_C_1: track 0.00 -> 17.4 mm
- net /EN_C_2: track 0.00 -> 15.8 mm
- net /EN_C_3: track 0.00 -> 15.8 mm
- net /Output_Group_A/ClK_Out3: track 17.6 -> 21.9 mm
- net /Output_Group_A/ClK_Out2: track 19.3 -> 21.9 mm
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
Commit message: .
Parts:
- C11, C13, C14, C15, C17, C18: moved to B.Cu
- moved C9 47.7 mm to (92.6, 77.4), turned to -45 degrees
- moved C16 46.6 mm to (160.9, 80.3)
- moved C6 46.6 mm to (145.5, 119.5)
- moved J10 46.6 mm to (147.9, 62.4)
- moved J12 46.6 mm to (156.6, 62.4)
- moved J13 46.6 mm to (174.0, 62.4)
- moved J14 46.6 mm to (113.1, 62.4)
- moved J15 46.6 mm to (130.5, 62.4)
- moved J17 46.6 mm to (121.8, 62.4)
- moved J2 46.6 mm to (182.7, 62.4)
- moved J3 46.6 mm to (200.1, 62.4)
- moved J4 46.6 mm to (191.4, 62.4)
- moved J6 46.6 mm to (78.3, 62.4)
- moved R13 46.6 mm to (126.5, 75.8)
- moved R14 46.6 mm to (128.9, 77.7)
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Routing:
- net /Input_Clock_Group_D: track 0.00 -> 73.4 mm, vias 0 -> 2
- net /EN_Group_A: track 9.60 -> 37.2 mm
- net /Input_Clock_Group_C: track 49.7 -> 73.3 mm
- net /Input_Clock_Group_B: track 50.0 -> 72.3 mm
- net /Output_Group_D/ClK_Out4: track 0.00 -> 21.9 mm
- net /Output_Group_D/ClK_Out2: track 0.00 -> 21.9 mm
- net /Output_Group_D/ClK_Out1: track 0.00 -> 21.5 mm
- net /EN_Group_B: track 8.29 -> 29.6 mm
- net /Output_Group_D/ClK_Out3: track 0.00 -> 20.4 mm
- net /EN_D_4: track 0.00 -> 17.5 mm
- net /EN_D_1: track 0.00 -> 17.5 mm
- net /EN_D_2: track 0.00 -> 15.8 mm
- net /EN_D_3: track 0.00 -> 15.8 mm
- net /EN_Group_C: track 9.20 -> 21.5 mm
- net GND: track 10.6 -> 22.5 mm, vias 56 -> 839
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- added copper zone on B.Cu, net GND
Other:
- board size 138.7 x 80 mm -> 143.7 x 80 mm
- board text added: "+"
- board text added: "-"
- board text added: "1"
- board text added: "2"
- board text added: "3"
- board text added: "4"
- board text added: "50 Ohm Termination"
- board text added: "EN_A_1"
- board text added: "EN_A_2"
- board text added: "EN_A_3"
- board text added: "EN_A_4"
- board text added: "EN_B_1"
- board text added: "EN_B_2"
- board text added: "EN_B_3"
- board text added: "EN_B_4"
- board text added: "EN_C_1"
- board text added: "EN_C_2"
- board text added: "EN_C_3"
- board text added: "EN_C_4"
- board text added: "EN_D_1"
- board text added: "EN_D_2"
- board text added: "EN_D_3"
- board text added: "EN_D_4"
- board text added: "Enable_Group_A"
- board text added: "Enable_Group_B"
- board text added: "Enable_Group_C"
- board text added: "Enable_Group_D"
- board text added: "Group A"
- board text added: "Group B"
- board text added: "Group C"
- board text added: "Group D"
- board text added: "Input Power 3.3 - 3.45 V"
- board text added: "Project: 16 Channels Clock Buffer Version: REV_0 January 2025 Author: Dr. Alexandru Enciu Institution: TU Darmstadt"
- board text added: "Technische Universität Darmstadt"
- board text removed: "Power 3V3"
