File: VMM3-Hybrid_to_Coax/VMM3_Hybrid_to_MPPC/VMM3_Hybrid_to_MPPC.kicad_pcb (KiCad board)
At the start: 4 copper layers, 60 x 52.9 mm, 107 parts, among them U10 OPA357AIDBVR, U11 OPA357AIDBVR, U2 OPA357AIDBVR, U3 OPA357AIDBVR, U4 OPA357AIDBVR, U5 OPA357AIDBVR, U6 OPA357AIDBVR, U7 OPA357AIDBVR, U8 OPA357AIDBVR, U9 OPA357AIDBVR

Commit message: .
Parts:
- added C51: 100nF, Capacitor_SMD:C_0603_1608Metric, B.Cu at (74.0, 74.2)
- added C52: 100nF, Capacitor_SMD:C_0603_1608Metric, B.Cu at (79.0, 74.2)
- added C53: 100nF, Capacitor_SMD:C_0603_1608Metric, B.Cu at (84.0, 74.2)
- added C54: 100nF, Capacitor_SMD:C_0603_1608Metric, B.Cu at (89.0, 74.2)
- added C55: 100nF, Capacitor_SMD:C_0603_1608Metric, B.Cu at (94.0, 74.2)
- added C56: 100nF, Capacitor_SMD:C_0603_1608Metric, B.Cu at (100.4, 74.2)
- added C57: 100nF, Capacitor_SMD:C_0603_1608Metric, B.Cu at (104.0, 74.2)
- added C58: 100nF, Capacitor_SMD:C_0603_1608Metric, B.Cu at (109.0, 74.2)
- added C59: 100nF, Capacitor_SMD:C_0603_1608Metric, B.Cu at (114.0, 74.2)
- added C60: 100nF, Capacitor_SMD:C_0603_1608Metric, B.Cu at (119.0, 74.2)
- added J1: Conn_01x04, Connector_PinHeader_2.54mm:PinHeader_2x02_P2.54mm_Vertical_SMD, F.Cu at (73.0, 104.7)
- C10, C14, C6: value 3pF -> 100nF; footprint Capacitor_SMD:C_0402_1005Metric -> Capacitor_SMD:C_0603_1608Metric
- C11, C15, C7: value 10 nF -> 100nF; footprint Capacitor_SMD:C_0402_1005Metric -> Capacitor_SMD:C_0603_1608Metric
- C12, C8: footprint Capacitor_SMD:C_0402_1005Metric -> Capacitor_SMD:C_0603_1608Metric
- C13, C9: value 10uF -> 100nF; footprint Capacitor_SMD:C_0402_1005Metric -> Capacitor_SMD:C_0603_1608Metric
- C50: value C -> 100nF; footprint Capacitor_SMD:C_0402_1005Metric -> Capacitor_SMD:C_0603_1608Metric
Connections:
- C10 pad 1: Net-(U2--IN) -> GND
- C10 pad 2: Net-(U2-OUT) -> HV+
- C11 pad 2: +3V3 -> HV+
- C12 pad 2: +3V3 -> HV+
- C13 pad 2: +3V3 -> HV+
- C14 pad 1: Net-(U2--IN) -> GND
- C14 pad 2: Net-(U2-OUT) -> HV+
- C15 pad 2: +3V3 -> HV+
- C50 pad 2: Net-(A1-Pad3) -> HV+
- C6 pad 1: Net-(U2--IN) -> GND
- C6 pad 2: Net-(U2-OUT) -> HV+
- C7 pad 2: +3V3 -> HV+
- C8 pad 2: +3V3 -> HV+
- C9 pad 2: +3V3 -> HV+
- U1 pad 10: Ch_4 -> GND
- U1 pad 100: Ch_94 -> GND
- U1 pad 101: Ch_95 -> GND
- U1 pad 102: Ch_96 -> GND
- U1 pad 103: Ch_97 -> GND
- U1 pad 104: Ch_98 -> GND
- U1 pad 105: Ch_99 -> GND
- U1 pad 106: Ch_100 -> GND
- U1 pad 107: Ch_101 -> GND
- U1 pad 108: Ch_102 -> GND
- U1 pad 111: Ch_105 -> GND
- U1 pad 112: Ch_106 -> GND
- U1 pad 113: Ch_107 -> GND
- U1 pad 114: Ch_108 -> GND
- U1 pad 115: Ch_109 -> GND
- U1 pad 116: Ch_110 -> GND
- U1 pad 117: Ch_111 -> GND
- U1 pad 118: Ch_112 -> GND
- U1 pad 119: Ch_113 -> GND
- U1 pad 120: Ch_114 -> GND
- U1 pad 121: Ch_115 -> GND
- U1 pad 122: Ch_116 -> GND
- U1 pad 123: Ch_117 -> GND
- U1 pad 124: Ch_118 -> GND
- U1 pad 125: Ch_119 -> GND
- U1 pad 126: Ch_120 -> GND
- U1 pad 127: Ch_121 -> GND
- U1 pad 128: Ch_122 -> GND
- U1 pad 13: Ch_7 -> GND
- U1 pad 131: Ch_125 -> GND
- U1 pad 132: Ch_126 -> GND
- U1 pad 133: Ch_127 -> GND
- U1 pad 134: Ch_128 -> GND
- U1 pad 14: Ch_8 -> GND
- U1 pad 15: Ch_9 -> GND
- U1 pad 16: Ch_10 -> GND
- U1 pad 17: Ch_11 -> GND
- U1 pad 18: Ch_12 -> GND
- U1 pad 19: Ch_13 -> GND
- U1 pad 20: Ch_14 -> GND
- U1 pad 21: Ch_15 -> GND
- U1 pad 22: Ch_16 -> GND
- U1 pad 23: Ch_17 -> GND
- U1 pad 24: Ch_18 -> GND
- U1 pad 25: Ch_19 -> GND
- U1 pad 26: Ch_20 -> GND
- U1 pad 27: Ch_21 -> GND
- U1 pad 28: Ch_22 -> GND
- U1 pad 29: Ch_23 -> GND
- U1 pad 30: Ch_24 -> GND
- U1 pad 33: Ch_27 -> GND
- U1 pad 34: Ch_28 -> GND
- U1 pad 35: Ch_29 -> GND
- U1 pad 36: Ch_30 -> GND
- U1 pad 37: Ch_31 -> GND
- U1 pad 38: Ch_32 -> GND
- U1 pad 39: Ch_33 -> GND
- U1 pad 40: Ch_34 -> GND
- U1 pad 41: Ch_35 -> GND
- U1 pad 42: Ch_36 -> GND
- U1 pad 43: Ch_37 -> GND
- U1 pad 44: Ch_38 -> GND
- U1 pad 45: Ch_39 -> GND
- U1 pad 46: Ch_40 -> GND
- U1 pad 47: Ch_41 -> GND
- U1 pad 48: Ch_42 -> GND
- U1 pad 49: Ch_43 -> GND
- U1 pad 50: Ch_44 -> GND
- U1 pad 52: Ch_46 -> GND
- U1 pad 53: Ch_47 -> GND
- U1 pad 54: Ch_48 -> GND
- U1 pad 55: Ch_49 -> GND
- U1 pad 56: Ch_50 -> GND
- U1 pad 57: Ch_51 -> GND
- U1 pad 58: Ch_52 -> GND
- U1 pad 59: Ch_53 -> GND
- U1 pad 60: Ch_54 -> GND
- U1 pad 61: Ch_55 -> GND
- U1 pad 62: Ch_56 -> GND
- U1 pad 63: Ch_57 -> GND
- U1 pad 64: Ch_58 -> GND
- U1 pad 65: Ch_59 -> GND
- U1 pad 66: Ch_60 -> GND
- U1 pad 67: Ch_61 -> GND
- U1 pad 68: Ch_62 -> GND
- U1 pad 69: Ch_63 -> GND
- U1 pad 7: Ch_1 -> GND
- U1 pad 70: Ch_64 -> GND
- U1 pad 71: Ch_65 -> GND
- U1 pad 72: Ch_66 -> GND
- U1 pad 73: Ch_67 -> GND
- U1 pad 74: Ch_68 -> GND
- U1 pad 75: Ch_69 -> GND
- U1 pad 76: Ch_70 -> GND
- U1 pad 77: Ch_71 -> GND
- U1 pad 78: Ch_72 -> GND
- U1 pad 79: Ch_73 -> GND
- U1 pad 8: Ch_2 -> GND
- U1 pad 80: Ch_74 -> GND
- U1 pad 81: Ch_75 -> GND
- U1 pad 82: Ch_76 -> GND
- U1 pad 83: Ch_77 -> GND
- U1 pad 84: Ch_78 -> GND
- U1 pad 85: Ch_79 -> GND
- U1 pad 86: Ch_80 -> GND
- U1 pad 87: Ch_81 -> GND
- U1 pad 88: Ch_82 -> GND
- U1 pad 9: Ch_3 -> GND
- U1 pad 90: Ch_84 -> GND
- U1 pad 91: Ch_85 -> GND
- U1 pad 92: Ch_86 -> GND
- U1 pad 93: Ch_87 -> GND
- U1 pad 94: Ch_88 -> GND
- U1 pad 95: Ch_89 -> GND
- U1 pad 96: Ch_90 -> GND
- U1 pad 97: Ch_91 -> GND
- U1 pad 98: Ch_92 -> GND
- U1 pad 99: Ch_93 -> GND
Routing:
- net HV+: track 7.50 -> 11.4 mm, vias 10 -> 13
- net GND: vias 522 -> 533
- added copper zone on B.Cu, net HV+

Commit message: .
Parts:
- removed A10, A2, A3, A4, A5, A6, A7, A8, A9: MICROFC-10035-SMT-TR1, Onsemi:XDCR_MICROFC-10035-SMT-TR1
- removed C10, C11, C12, C13, C14, C15, C50, C6, C7, C8, C9: 100nF, Capacitor_SMD:C_0603_1608Metric
- removed C16, C20, C24, C28, C32, C36, C40: 100nF, Capacitor_SMD:C_0402_1005Metric
- removed C17, C21, C25, C29, C33, C37, C41: 10uF, Capacitor_SMD:C_0402_1005Metric
- removed C18, C22, C26, C30, C34, C38: 3pF, Capacitor_SMD:C_0402_1005Metric
- removed C19, C23, C27, C31, C35, C39: 10 nF, Capacitor_SMD:C_0402_1005Metric
- removed C42, C43, C44, C45, C46, C47, C48, C49: C, Capacitor_SMD:C_0402_1005Metric
- removed R10, R12, R14, R16, R18, R20, R4, R6, R8: 10k, Resistor_SMD:R_0402_1005Metric
- removed R22, R23, R24, R25, R26, R27, R28, R29, R30: R, Resistor_SMD:R_0402_1005Metric
- removed U10, U11, U3, U4, U5, U6, U7, U8, U9: OPA357AIDBVR, Package_TO_SOT_SMD:SOT-23-6
- added A1: MICROFC-10035-SMT-TR1, Onsemi:XDCR_MICROFC-10035-SMT-TR1, F.Cu at (84.6, 79.2)
- added A1: MICROFC-10035-SMT-TR1, Onsemi:XDCR_MICROFC-10035-SMT-TR1, F.Cu at (119.6, 79.2)
- added A1: MICROFC-10035-SMT-TR1, Onsemi:XDCR_MICROFC-10035-SMT-TR1, F.Cu at (94.6, 79.2)
- added A1: MICROFC-10035-SMT-TR1, Onsemi:XDCR_MICROFC-10035-SMT-TR1, F.Cu at (114.6, 79.2)
- added A1: MICROFC-10035-SMT-TR1, Onsemi:XDCR_MICROFC-10035-SMT-TR1, F.Cu at (79.6, 79.2)
- added A1: MICROFC-10035-SMT-TR1, Onsemi:XDCR_MICROFC-10035-SMT-TR1, F.Cu at (104.6, 79.2)
- added A1: MICROFC-10035-SMT-TR1, Onsemi:XDCR_MICROFC-10035-SMT-TR1, F.Cu at (89.6, 79.2)
- added A1: MICROFC-10035-SMT-TR1, Onsemi:XDCR_MICROFC-10035-SMT-TR1, F.Cu at (109.6, 79.2)
- added A1: MICROFC-10035-SMT-TR1, Onsemi:XDCR_MICROFC-10035-SMT-TR1, F.Cu at (99.6, 79.2)
- added C1: C, Capacitor_SMD:C_0402_1005Metric, F.Cu at (114.5, 77.4)
- added C1: C, Capacitor_SMD:C_0402_1005Metric, F.Cu at (99.5, 77.4)
- added C1: C, Capacitor_SMD:C_0402_1005Metric, F.Cu at (79.5, 77.4)
- added C1: C, Capacitor_SMD:C_0402_1005Metric, F.Cu at (89.5, 77.4)
- added C1: C, Capacitor_SMD:C_0402_1005Metric, F.Cu at (84.5, 77.4)
- added C1: C, Capacitor_SMD:C_0402_1005Metric, F.Cu at (109.5, 77.4)
- added C1: C, Capacitor_SMD:C_0402_1005Metric, F.Cu at (104.5, 77.4)
- added C1: C, Capacitor_SMD:C_0402_1005Metric, F.Cu at (94.5, 77.4)
- added C1: C, Capacitor_SMD:C_0402_1005Metric, F.Cu at (119.5, 77.4)
- added C2: 3pF, Capacitor_SMD:C_0402_1005Metric, F.Cu at (98.0, 91.8)
- added C2: 3pF, Capacitor_SMD:C_0402_1005Metric, F.Cu at (89.5, 91.8)
- added C2: 3pF, Capacitor_SMD:C_0402_1005Metric, F.Cu at (93.7, 100.3)
- added C2: 3pF, Capacitor_SMD:C_0402_1005Metric, F.Cu at (85.2, 100.3)
- added C2: 3pF, Capacitor_SMD:C_0402_1005Metric, F.Cu at (110.7, 100.3)
- added C2: 3pF, Capacitor_SMD:C_0402_1005Metric, F.Cu at (115.0, 91.8)
- added C2: 3pF, Capacitor_SMD:C_0402_1005Metric, F.Cu at (106.5, 91.8)
- added C2: 3pF, Capacitor_SMD:C_0402_1005Metric, F.Cu at (102.2, 100.3)
- added C2: 3pF, Capacitor_SMD:C_0402_1005Metric, F.Cu at (119.2, 100.3)
- added C3: 10 nF, Capacitor_SMD:C_0402_1005Metric, F.Cu at (102.9, 89.9)
- added C3: 10 nF, Capacitor_SMD:C_0402_1005Metric, F.Cu at (115.7, 98.4)
- added C3: 10 nF, Capacitor_SMD:C_0402_1005Metric, F.Cu at (90.2, 98.4)
- added C3: 10 nF, Capacitor_SMD:C_0402_1005Metric, F.Cu at (107.2, 98.4)
- added C3: 10 nF, Capacitor_SMD:C_0402_1005Metric, F.Cu at (81.7, 98.4)
- added C3: 10 nF, Capacitor_SMD:C_0402_1005Metric, F.Cu at (85.9, 89.9)
- added C3: 10 nF, Capacitor_SMD:C_0402_1005Metric, F.Cu at (94.4, 89.9)
- added C3: 10 nF, Capacitor_SMD:C_0402_1005Metric, F.Cu at (98.7, 98.4)
- added C3: 10 nF, Capacitor_SMD:C_0402_1005Metric, F.Cu at (111.4, 89.9)
- added C4: 100nF, Capacitor_SMD:C_0402_1005Metric, F.Cu at (96.7, 98.4)
- added C4: 100nF, Capacitor_SMD:C_0402_1005Metric, F.Cu at (92.5, 89.9)
- added C4: 100nF, Capacitor_SMD:C_0402_1005Metric, F.Cu at (113.7, 98.4)
- added C4: 100nF, Capacitor_SMD:C_0402_1005Metric, F.Cu at (84.0, 89.9)
- added C4: 100nF, Capacitor_SMD:C_0402_1005Metric, F.Cu at (105.2, 98.4)
- added C4: 100nF, Capacitor_SMD:C_0402_1005Metric, F.Cu at (101.0, 89.9)
- added C4: 100nF, Capacitor_SMD:C_0402_1005Metric, F.Cu at (109.5, 89.9)
- added C4: 100nF, Capacitor_SMD:C_0402_1005Metric, F.Cu at (88.2, 98.4)
- added C4: 100nF, Capacitor_SMD:C_0402_1005Metric, F.Cu at (79.7, 98.4)
- added C5: 10uF, Capacitor_SMD:C_0402_1005Metric, F.Cu at (96.7, 99.8)
- added C5: 10uF, Capacitor_SMD:C_0402_1005Metric, F.Cu at (79.7, 99.8)
- added C5: 10uF, Capacitor_SMD:C_0402_1005Metric, F.Cu at (83.9, 91.3)
- added C5: 10uF, Capacitor_SMD:C_0402_1005Metric, F.Cu at (92.4, 91.3)
- added C5: 10uF, Capacitor_SMD:C_0402_1005Metric, F.Cu at (88.2, 99.8)
- added C5: 10uF, Capacitor_SMD:C_0402_1005Metric, F.Cu at (105.2, 99.8)
- added C5: 10uF, Capacitor_SMD:C_0402_1005Metric, F.Cu at (100.9, 91.3)
- added C5: 10uF, Capacitor_SMD:C_0402_1005Metric, F.Cu at (109.4, 91.3)
- added C5: 10uF, Capacitor_SMD:C_0402_1005Metric, F.Cu at (113.7, 99.8)
- added R1: R, Resistor_SMD:R_0402_1005Metric, F.Cu at (119.5, 76.4)
- added R1: R, Resistor_SMD:R_0402_1005Metric, F.Cu at (89.5, 76.4)
- added R1: R, Resistor_SMD:R_0402_1005Metric, F.Cu at (109.5, 76.4)
- added R1: R, Resistor_SMD:R_0402_1005Metric, F.Cu at (104.5, 76.4)
- added R1: R, Resistor_SMD:R_0402_1005Metric, F.Cu at (99.5, 76.4)
- added R1: R, Resistor_SMD:R_0402_1005Metric, F.Cu at (79.5, 76.4)
- added R1: R, Resistor_SMD:R_0402_1005Metric, F.Cu at (94.5, 76.4)
- added R1: R, Resistor_SMD:R_0402_1005Metric, F.Cu at (114.5, 76.4)
- added R1: R, Resistor_SMD:R_0402_1005Metric, F.Cu at (84.5, 76.4)
- added R2: 10k, Resistor_SMD:R_0402_1005Metric, F.Cu at (105.5, 91.8)
- added R2: 10k, Resistor_SMD:R_0402_1005Metric, F.Cu at (88.5, 91.8)
- added R2: 10k, Resistor_SMD:R_0402_1005Metric, F.Cu at (101.2, 100.3)
- added R2: 10k, Resistor_SMD:R_0402_1005Metric, F.Cu at (84.2, 100.3)
- added R2: 10k, Resistor_SMD:R_0402_1005Metric, F.Cu at (109.7, 100.3)
- added R2: 10k, Resistor_SMD:R_0402_1005Metric, F.Cu at (92.7, 100.3)
- added R2: 10k, Resistor_SMD:R_0402_1005Metric, F.Cu at (97.0, 91.8)
- added R2: 10k, Resistor_SMD:R_0402_1005Metric, F.Cu at (114.0, 91.8)
- added R2: 10k, Resistor_SMD:R_0402_1005Metric, F.Cu at (118.2, 100.3)
- added U2: OPA357AIDBVR, Package_TO_SOT_SMD:SOT-23-6, F.Cu at (116.0, 101.0)
- added U2: OPA357AIDBVR, Package_TO_SOT_SMD:SOT-23-6, F.Cu at (111.7, 92.5)
- added U2: OPA357AIDBVR, Package_TO_SOT_SMD:SOT-23-6, F.Cu at (107.5, 101.0)
- added U2: OPA357AIDBVR, Package_TO_SOT_SMD:SOT-23-6, F.Cu at (99.0, 101.0)
- added U2: OPA357AIDBVR, Package_TO_SOT_SMD:SOT-23-6, F.Cu at (82.0, 101.0)
- added U2: OPA357AIDBVR, Package_TO_SOT_SMD:SOT-23-6, F.Cu at (103.2, 92.5)
- added U2: OPA357AIDBVR, Package_TO_SOT_SMD:SOT-23-6, F.Cu at (90.5, 101.0)
- added U2: OPA357AIDBVR, Package_TO_SOT_SMD:SOT-23-6, F.Cu at (86.2, 92.5)
- added U2: OPA357AIDBVR, Package_TO_SOT_SMD:SOT-23-6, F.Cu at (94.7, 92.5)
Routing:
- net Net-(U2--IN): track 187.6 -> 189.9 mm
Other:
- board text added: "Title: Onsemi MICRO-FC-10035-TR for VMM3a Hybrid Revision: Rev_0, January 2025 Author: Dr. Alexandru Enciu, TU Darmstadt, IKP"
- board text removed: "Title: Onsemi MICRO-FC-10035-TR for VMM3a Hybrid Revision: January 2025 REV_0 Author: Dr. Alexandru Enciu, TU Darmstadt, IKP"
