File: VMM3-Hybrid_to_Coax/VMM3_Hybrid_to_MPPC/VMM3_Hybrid_to_MPPC.kicad_sch (KiCad schematic)
At the start: 1 part

Commit message: .
Parts:
- added C50, C51, C52, C53, C54, C55, C56, C57, C58, C59, C60: 100nF, Capacitor_SMD:C_0603_1608Metric, symbol Device:C
- added J1: Conn_01x04, Connector_PinHeader_2.54mm:PinHeader_2x02_P2.54mm_Vertical_SMD, symbol PCM_4ms_Connector:Conn_01x04
Connections:
- net Ch_1 is gone; now on net GND: U1.7
- net Ch_10 is gone; now on net GND: U1.16
- net Ch_100 is gone; now on net GND: U1.106
- net Ch_101 is gone; now on net GND: U1.107
- net Ch_102 is gone; now on net GND: U1.108
- net Ch_105 is gone; now on net GND: U1.111
- net Ch_106 is gone; now on net GND: U1.112
- net Ch_107 is gone; now on net GND: U1.113
- net Ch_108 is gone; now on net GND: U1.114
- net Ch_109 is gone; now on net GND: U1.115
- net Ch_11 is gone; now on net GND: U1.17
- net Ch_110 is gone; now on net GND: U1.116
- net Ch_111 is gone; now on net GND: U1.117
- net Ch_112 is gone; now on net GND: U1.118
- net Ch_113 is gone; now on net GND: U1.119
- net Ch_114 is gone; now on net GND: U1.120
- net Ch_115 is gone; now on net GND: U1.121
- net Ch_116 is gone; now on net GND: U1.122
- net Ch_117 is gone; now on net GND: U1.123
- net Ch_118 is gone; now on net GND: U1.124
- net Ch_119 is gone; now on net GND: U1.125
- net Ch_12 is gone; now on net GND: U1.18
- net Ch_120 is gone; now on net GND: U1.126
- net Ch_121 is gone; now on net GND: U1.127
- net Ch_122 is gone; now on net GND: U1.128
- net Ch_125 is gone; now on net GND: U1.131
- net Ch_126 is gone; now on net GND: U1.132
- net Ch_127 is gone; now on net GND: U1.133
- net Ch_128 is gone; now on net GND: U1.134
- net Ch_13 is gone; now on net GND: U1.19
- net Ch_14 is gone; now on net GND: U1.20
- net Ch_15 is gone; now on net GND: U1.21
- net Ch_16 is gone; now on net GND: U1.22
- net Ch_17 is gone; now on net GND: U1.23
- net Ch_18 is gone; now on net GND: U1.24
- net Ch_19 is gone; now on net GND: U1.25
- net Ch_2 is gone; now on net GND: U1.8
- net Ch_20 is gone; now on net GND: U1.26
- net Ch_21 is gone; now on net GND: U1.27
- net Ch_22 is gone; now on net GND: U1.28
- net Ch_23 is gone; now on net GND: U1.29
- net Ch_24 is gone; now on net GND: U1.30
- net Ch_27 is gone; now on net GND: U1.33
- net Ch_28 is gone; now on net GND: U1.34
- net Ch_29 is gone; now on net GND: U1.35
- net Ch_3 is gone; now on net GND: U1.9
- net Ch_30 is gone; now on net GND: U1.36
- net Ch_31 is gone; now on net GND: U1.37
- net Ch_32 is gone; now on net GND: U1.38
- net Ch_33 is gone; now on net GND: U1.39
- net Ch_34 is gone; now on net GND: U1.40
- net Ch_35 is gone; now on net GND: U1.41
- net Ch_36 is gone; now on net GND: U1.42
- net Ch_37 is gone; now on net GND: U1.43
- net Ch_38 is gone; now on net GND: U1.44
- net Ch_39 is gone; now on net GND: U1.45
- net Ch_4 is gone; now on net GND: U1.10
- net Ch_40 is gone; now on net GND: U1.46
- net Ch_41 is gone; now on net GND: U1.47
- net Ch_42 is gone; now on net GND: U1.48
- net Ch_43 is gone; now on net GND: U1.49
- net Ch_44 is gone; now on net GND: U1.50
- net Ch_46 is gone; now on net GND: U1.52
- net Ch_47 is gone; now on net GND: U1.53
- net Ch_48 is gone; now on net GND: U1.54
- net Ch_49 is gone; now on net GND: U1.55
- net Ch_50 is gone; now on net GND: U1.56
- net Ch_51 is gone; now on net GND: U1.57
- net Ch_52 is gone; now on net GND: U1.58
- net Ch_53 is gone; now on net GND: U1.59
- net Ch_54 is gone; now on net GND: U1.60
- net Ch_55 is gone; now on net GND: U1.61
- net Ch_56 is gone; now on net GND: U1.62
- net Ch_57 is gone; now on net GND: U1.63
- net Ch_58 is gone; now on net GND: U1.64
- net Ch_59 is gone; now on net GND: U1.65
- net Ch_60 is gone; now on net GND: U1.66
- net Ch_61 is gone; now on net GND: U1.67
- net Ch_62 is gone; now on net GND: U1.68
- net Ch_63 is gone; now on net GND: U1.69
- net Ch_64 is gone; now on net GND: U1.70
- net Ch_65 is gone; now on net GND: U1.71
- net Ch_66 is gone; now on net GND: U1.72
- net Ch_67 is gone; now on net GND: U1.73
- net Ch_68 is gone; now on net GND: U1.74
- net Ch_69 is gone; now on net GND: U1.75
- net Ch_7 is gone; now on net GND: U1.13
- net Ch_70 is gone; now on net GND: U1.76
- net Ch_71 is gone; now on net GND: U1.77
- net Ch_72 is gone; now on net GND: U1.78
- net Ch_73 is gone; now on net GND: U1.79
- net Ch_74 is gone; now on net GND: U1.80
- net Ch_75 is gone; now on net GND: U1.81
- net Ch_76 is gone; now on net GND: U1.82
- net Ch_77 is gone; now on net GND: U1.83
- net Ch_78 is gone; now on net GND: U1.84
- net Ch_79 is gone; now on net GND: U1.85
- net Ch_8 is gone; now on net GND: U1.14
- net Ch_80 is gone; now on net GND: U1.86
- net Ch_81 is gone; now on net GND: U1.87
- net Ch_82 is gone; now on net GND: U1.88
- net Ch_84 is gone; now on net GND: U1.90
- net Ch_85 is gone; now on net GND: U1.91
- net Ch_86 is gone; now on net GND: U1.92
- net Ch_87 is gone; now on net GND: U1.93
- net Ch_88 is gone; now on net GND: U1.94
- net Ch_89 is gone; now on net GND: U1.95
- net Ch_9 is gone; now on net GND: U1.15
- net Ch_90 is gone; now on net GND: U1.96
- net Ch_91 is gone; now on net GND: U1.97
- net Ch_92 is gone; now on net GND: U1.98
- net Ch_93 is gone; now on net GND: U1.99
- net Ch_94 is gone; now on net GND: U1.100
- net Ch_95 is gone; now on net GND: U1.101
- net Ch_96 is gone; now on net GND: U1.102
- net Ch_97 is gone; now on net GND: U1.103
- net Ch_98 is gone; now on net GND: U1.104
- net Ch_99 is gone; now on net GND: U1.105
- net GND: now also C50.1, C51.1, C52.1, C53.1, C54.1, C55.1, C56.1, C57.1, C58.1, C59.1, C60.1, J1.2 (Pin_2), J1.4 (Pin_4)
- net HV+: now also C50.2, C51.2, C52.2, C53.2, C54.2, C55.2, C56.2, C57.2, C58.2, C59.2, C60.2, J1.3 (Pin_3)
- new net +3V3: J1.1 (Pin_1)
