File: HYDRA_VMM3_card/HYDRA_VMM3_CARD_V3_Flex/HYDRA_VMM3_CARD_V3_Flex.kicad_pcb (KiCad board)
At the start: 8 copper layers, 105.3 x 61 mm, 56 parts, among them J1 ME1014010101011

Commit message: .
Parts:
- removed REF**: 68711714522, Custom_Footprints:68711714522
- added J2: FPC: 68711714522, Custom_Footprints:68711714522, F.Cu at (196.8, 101.4)
- moved 1 72.2 mm to (171.5, 80.8)
- moved 1.8V1 72.2 mm to (122.0, 109.7)
- moved 1.8_On1 72.2 mm to (123.7, 113.2)
- moved 11 72.2 mm to (129.7, 122.0)
- moved 12 72.2 mm to (132.2, 122.0)
- moved 13 72.2 mm to (137.3, 80.8)
- moved 14 72.2 mm to (137.3, 78.3)
- moved 17 72.2 mm to (171.5, 124.5)
- moved 20 72.2 mm to (171.5, 122.0)
- moved 23 72.2 mm to (137.3, 124.5)
- moved 24 72.2 mm to (137.3, 122.0)
- moved 3.3V1 72.2 mm to (122.0, 104.6)
- moved 3.3V_On1 72.2 mm to (123.7, 101.0)
- moved 7 72.2 mm to (129.7, 124.5)
- moved 8 72.2 mm to (132.2, 124.5)
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Connections:
- J1 pad A36: Ch_43 -> Ch_114
- J1 pad A37: Ch_45 -> Ch_116
- J1 pad A38: Ch_47 -> Ch_118
- J1 pad A39: Ch_49 -> Ch_120
- J1 pad A40: Ch_51 -> Ch_122
- J1 pad A41: Ch_53 -> Ch_124
- J1 pad A42: Ch_55 -> Ch_126
- J1 pad A43: Ch_73 -> Ch_128
- J1 pad A44: Ch_75 -> Ch_43
- J1 pad A45: Ch_77 -> Ch_45
- J1 pad A46: Ch_79 -> Ch_47
- J1 pad A60: Ch_127 -> Ch_107
- J1 pad A61: Ch_125 -> Ch_109
- J1 pad A62: Ch_123 -> Ch_111
- J1 pad A63: Ch_121 -> Ch_113
- J1 pad A64: Ch_119 -> Ch_115
- J1 pad A66: Ch_115 -> Ch_119
- J1 pad A67: Ch_113 -> Ch_121
- J1 pad A68: Ch_111 -> Ch_123
- J1 pad A69: Ch_109 -> Ch_125
- J1 pad A70: Ch_107 -> Ch_127
- J1 pad B15: Ch_4 -> Ch_2
- J1 pad B16: Ch_6 -> Ch_4
- J1 pad B17: Ch_8 -> Ch_6
- J1 pad B18: Ch_10 -> Ch_8
- J1 pad B19: Ch_12 -> Ch_10
- J1 pad B20: Ch_14 -> Ch_12
- J1 pad B21: Ch_16 -> Ch_14
- J1 pad B22: Ch_18 -> Ch_16
- J1 pad B23: Ch_20 -> Ch_18
- J1 pad B24: Ch_22 -> Ch_20
- J1 pad B25: Ch_24 -> Ch_22
- J1 pad B26: Ch_26 -> Ch_24
- J1 pad B27: Ch_28 -> Ch_26
- J1 pad B28: Ch_30 -> Ch_28
- J1 pad B29: Ch_32 -> Ch_30
- J1 pad B30: Ch_34 -> Ch_32
- J1 pad B31: Ch_36 -> Ch_34
- J1 pad B32: Ch_38 -> Ch_36
- J1 pad B33: Ch_40 -> Ch_38
- J1 pad B34: Ch_42 -> Ch_40
- J1 pad B35: Ch_44 -> Ch_42
- J1 pad B36: Ch_46 -> Ch_44
- J1 pad B37: Ch_48 -> Ch_46
- J1 pad B38: Ch_50 -> Ch_48
- J1 pad B39: Ch_52 -> Ch_50
- J1 pad B40: Ch_54 -> Ch_52
- J1 pad B41: Ch_56 -> Ch_54
- J1 pad B42: Ch_58 -> Ch_56
- J1 pad B43: Ch_60 -> Ch_58
- J1 pad B44: Ch_62 -> Ch_60
- J1 pad B45: Ch_64 -> Ch_62
- J1 pad B46: Ch_66 -> Ch_64
- J1 pad B47: Ch_68 -> Ch_66
- J1 pad B48: Ch_70 -> Ch_68
- J1 pad B49: Ch_72 -> Ch_70
- J1 pad B50: Ch_74 -> Ch_72
- J1 pad B51: Ch_76 -> Ch_74
- J1 pad B52: Ch_78 -> Ch_76
- J1 pad B53: Ch_80 -> Ch_78
- J1 pad B54: Ch_82 -> Ch_80
- J1 pad B55: Ch_84 -> Ch_82
- J1 pad B56: Ch_86 -> Ch_84
- J1 pad B57: Ch_114 -> Ch_86
- J1 pad B58: Ch_112 -> Ch_88
- J1 pad B59: Ch_110 -> Ch_90
- J1 pad B60: Ch_108 -> Ch_92
- J1 pad B61: Ch_106 -> Ch_94
- J1 pad B62: Ch_104 -> Ch_112
- J1 pad B63: Ch_102 -> Ch_108
- J1 pad B64: Ch_100 -> Ch_102
- J1 pad B66: Ch_96 -> Ch_110
- J1 pad B67: Ch_94 -> Ch_106
- J1 pad B68: Ch_92 -> Ch_104
- J1 pad B69: Ch_90 -> Ch_100
- J1 pad B70: Ch_88 -> Ch_96
- U1 pad 55: Ch_49 -> GND
- U1 pad 57: Ch_51 -> GND
- U1 pad 59: Ch_53 -> GND
- U1 pad 61: Ch_55 -> Ch_57
- U1 pad 63: Ch_57 -> Ch_55
- U1 pad 65: Ch_59 -> GND
- U1 pad 75: Ch_69 -> GND
- U1 pad 81: Ch_75 -> GND
- U1 pad 83: Ch_77 -> GND
- U1 pad 85: Ch_79 -> GND
Routing:
- net Ch_2: track 0.00 -> 72.5 mm
- net Ch_49: track 46.6 -> 0.00 mm, vias 1 -> 0
- net Ch_51: track 45.1 -> 0.00 mm, vias 1 -> 0
- net Ch_53: track 44.2 -> 0.00 mm, vias 1 -> 0
- net Ch_77: track 44.1 -> 0.00 mm, vias 1 -> 0
- net Ch_79: track 40.8 -> 0.00 mm, vias 1 -> 0
- net Ch_75: track 37.2 -> 0.00 mm, vias 1 -> 0
- net Ch_73: track 46.4 -> 11.2 mm, vias 1 -> 2
- net Ch_55: track 43.2 -> 13.1 mm, vias 1 -> 2
- net Ch_116: track 0.00 -> 29.2 mm, vias 0 -> 1
- net Ch_120: track 0.00 -> 26.2 mm, vias 0 -> 1
- net Ch_118: track 0.00 -> 25.0 mm, vias 0 -> 2
- net Ch_124: track 0.00 -> 24.7 mm, vias 0 -> 1
- net Ch_122: track 0.00 -> 24.5 mm, vias 0 -> 2
- net Ch_126: track 0.00 -> 20.3 mm, vias 0 -> 2
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- added copper zone on In3.Cu, net GND
- removed copper zone on In3.Cu, net P1
Other:
- board size 105.3 x 61 mm -> 85.2 x 61 mm

Commit message: .
Parts:
- added J3: FPC_4pin, Custom_Footprints:CON_5034800440_MOL, B.Cu at (151.7, 128.8)
- C1, Temp_1: moved to F.Cu
- Temp_RX1, Temp_TX1: footprint IPEX:IPEX_20449-001E-03 -> Custom_Footprints:IPEX_20449-001E-03
- moved Temp_RX1 41.3 mm to (116.8, 85.0), turned to -90 degrees
- moved Temp_TX1 32.2 mm to (116.8, 88.9), turned to -90 degrees
- moved 3.3V_On1 8.94 mm to (115.6, 97.3), turned to -90 degrees
- moved 1.8_On1 8.92 mm to (115.7, 117.1), turned to 90 degrees
- moved R8 4.87 mm to (118.2, 116.2), turned to 180 degrees
- moved R7 4.83 mm to (118.1, 98.2), turned to 180 degrees
- moved C1 1.63 mm to (152.1, 101.4), turned to 90 degrees
- moved Temp_1 0.79 mm to (153.3, 101.1), turned to -90 degrees
Routing:
- net RX: track 22.3 -> 45.4 mm, vias 0 -> 2
- net TX: track 22.3 -> 45.4 mm, vias 0 -> 2
- net Heimtime: track 0.00 -> 8.60 mm
- net Master_Trigg: track 0.00 -> 8.28 mm
- net bit_2: track 0.00 -> 3.60 mm, vias 0 -> 1
- net bit_5: track 0.00 -> 3.27 mm, vias 0 -> 1
- net bit_4: track 0.00 -> 3.17 mm, vias 0 -> 1
- net bit_3: track 0.00 -> 3.14 mm, vias 0 -> 1
- net P2_Out: track 0.00 -> 2.98 mm
- net P1_Out: track 0.00 -> 2.57 mm
- net bit_0: track 0.00 -> 2.13 mm, vias 0 -> 1
- net bit_1: track 0.00 -> 2.07 mm, vias 0 -> 1
- net GND: track 8.68 -> 9.34 mm, vias 825 -> 862
- net P1: track 1.14 -> 1.45 mm, vias 85 -> 36
- net P2: vias 20 -> 89
- added copper zone on F.Cu, net P2
Other:
- outline, holes or cut-outs redrawn
- board text added: "0"
- board text added: "1"
- board text added: "2"
- board text added: "3"
- board text added: "4"
- board text added: "5"
- board text added: "Bit_nr:"

Commit message: .
Routing:
- net GND: vias 862 -> 919
