File: HYDRA_VMM3_card/HYDRA_VMM3_CARD_V3_Flex/HYDRA_VMM3_CARD_V3_Flex.kicad_pcb (KiCad board)
At the start: 8 copper layers, 85.2 x 61 mm, 57 parts, among them J1 ME1014010101011, J2 FPC: 68711714522, J3 FPC_4pin

Commit message: .
Parts:
- moved J3 3.11 mm to (151.5, 125.7), turned to 0 degrees
Connections:
- J3 pad 2: Heimtime -> Master_Trigg
- J3 pad 4: Master_Trigg -> Heimtime
Routing:
- net Ch_86: track 34.8 -> 34.0 mm
- net Ch_82: track 36.5 -> 35.9 mm
- net GND: vias 919 -> 1023
Other:
- board text added: "Edge Connector"

Commit message: .
Routing:
- net GND: track 9.34 -> 6.18 mm

Commit message: .
Connections:
- net Ch_50 renamed Ch_49
- net Ch_52 renamed Ch_51
- net Ch_76 renamed Ch_75
- net Ch_78 renamed Ch_77
- J1 pad A15: Ch_1 -> Ch_0
- J1 pad A16: Ch_3 -> Ch_2
- J1 pad A17: Ch_5 -> Ch_4
- J1 pad A18: Ch_7 -> Ch_6
- J1 pad A19: Ch_9 -> Ch_8
- J1 pad A20: Ch_11 -> Ch_10
- J1 pad A21: Ch_13 -> Ch_12
- J1 pad A22: Ch_15 -> Ch_14
- J1 pad A23: Ch_17 -> Ch_16
- J1 pad A24: Ch_19 -> Ch_18
- J1 pad A25: Ch_21 -> Ch_20
- J1 pad A26: Ch_23 -> Ch_22
- J1 pad A27: Ch_25 -> Ch_24
- J1 pad A28: Ch_27 -> Ch_26
- J1 pad A29: Ch_29 -> Ch_28
- J1 pad A30: Ch_31 -> Ch_30
- J1 pad A31: Ch_33 -> Ch_32
- J1 pad A32: Ch_35 -> Ch_34
- J1 pad A33: Ch_37 -> Ch_36
- J1 pad A34: Ch_39 -> Ch_38
- J1 pad A35: Ch_41 -> Ch_40
- J1 pad A36: Ch_114 -> Ch_113
- J1 pad A37: Ch_116 -> Ch_115
- J1 pad A38: Ch_118 -> Ch_117
- J1 pad A39: Ch_120 -> Ch_119
- J1 pad A40: Ch_122 -> Ch_121
- J1 pad A41: Ch_124 -> Ch_123
- J1 pad A42: Ch_126 -> Ch_125
- J1 pad A43: Ch_128 -> Ch_127
- J1 pad A44: Ch_43 -> Ch_42
- J1 pad A45: Ch_45 -> Ch_44
- J1 pad A46: Ch_47 -> Ch_46
- J1 pad A47: Ch_81 -> Ch_80
- J1 pad A48: Ch_83 -> Ch_82
- J1 pad A49: Ch_85 -> Ch_84
- J1 pad A50: Ch_87 -> Ch_86
- J1 pad A51: Ch_89 -> Ch_88
- J1 pad A52: Ch_91 -> Ch_90
- J1 pad A53: Ch_93 -> Ch_92
- J1 pad A54: Ch_95 -> Ch_94
- J1 pad A55: Ch_97 -> Ch_96
- J1 pad A56: Ch_99 -> Ch_98
- J1 pad A57: Ch_101 -> Ch_100
- J1 pad A58: Ch_103 -> Ch_102
- J1 pad A59: Ch_105 -> Ch_104
- J1 pad A60: Ch_107 -> Ch_106
- J1 pad A61: Ch_109 -> Ch_108
- J1 pad A62: Ch_111 -> Ch_110
- J1 pad A63: Ch_113 -> Ch_112
- J1 pad A64: Ch_115 -> Ch_114
- J1 pad A65: Ch_117 -> Ch_116
- J1 pad A66: Ch_119 -> Ch_118
- J1 pad A67: Ch_121 -> Ch_120
- J1 pad A68: Ch_123 -> Ch_122
- J1 pad A69: Ch_125 -> Ch_124
- J1 pad A70: Ch_127 -> Ch_126
- J1 pad B15: Ch_2 -> Ch_1
- J1 pad B16: Ch_4 -> Ch_3
- J1 pad B17: Ch_6 -> Ch_5
- J1 pad B18: Ch_8 -> Ch_7
- J1 pad B19: Ch_10 -> Ch_9
- J1 pad B20: Ch_12 -> Ch_11
- J1 pad B21: Ch_14 -> Ch_13
- J1 pad B22: Ch_16 -> Ch_15
- J1 pad B23: Ch_18 -> Ch_17
- J1 pad B24: Ch_20 -> Ch_19
- J1 pad B25: Ch_22 -> Ch_21
- J1 pad B26: Ch_24 -> Ch_23
- J1 pad B27: Ch_26 -> Ch_25
- J1 pad B28: Ch_28 -> Ch_27
- J1 pad B29: Ch_30 -> Ch_29
- J1 pad B30: Ch_32 -> Ch_31
- J1 pad B31: Ch_34 -> Ch_33
- J1 pad B32: Ch_36 -> Ch_35
- J1 pad B33: Ch_38 -> Ch_37
- J1 pad B34: Ch_40 -> Ch_39
- J1 pad B35: Ch_42 -> Ch_41
- J1 pad B36: Ch_44 -> Ch_43
- J1 pad B37: Ch_46 -> Ch_45
- J1 pad B38: Ch_48 -> Ch_47
- J1 pad B41: Ch_54 -> Ch_53
- J1 pad B42: Ch_56 -> Ch_55
- J1 pad B43: Ch_58 -> Ch_57
- J1 pad B44: Ch_60 -> Ch_59
- J1 pad B45: Ch_62 -> Ch_61
- J1 pad B46: Ch_64 -> Ch_63
- J1 pad B47: Ch_66 -> Ch_65
- J1 pad B48: Ch_68 -> Ch_67
- J1 pad B49: Ch_70 -> Ch_69
- J1 pad B50: Ch_72 -> Ch_71
- J1 pad B51: Ch_74 -> Ch_73
- J1 pad B54: Ch_80 -> Ch_79
- J1 pad B55: Ch_82 -> Ch_81
- J1 pad B56: Ch_84 -> Ch_83
- J1 pad B57: Ch_86 -> Ch_85
- J1 pad B58: Ch_88 -> Ch_87
- J1 pad B59: Ch_90 -> Ch_89
- J1 pad B60: Ch_92 -> Ch_91
- J1 pad B61: Ch_94 -> Ch_93
- J1 pad B62: Ch_112 -> Ch_111
- J1 pad B63: Ch_108 -> Ch_107
- J1 pad B64: Ch_102 -> Ch_101
- J1 pad B65: Ch_98 -> Ch_97
- J1 pad B66: Ch_110 -> Ch_109
- J1 pad B67: Ch_106 -> Ch_105
- J1 pad B68: Ch_104 -> Ch_103
- J1 pad B69: Ch_100 -> Ch_99
- J1 pad B70: Ch_96 -> Ch_95
- J2 pad 10: Ch_67 -> Ch_66
- J2 pad 12: Ch_65 -> Ch_64
- J2 pad 14: Ch_63 -> Ch_62
- J2 pad 16: Ch_61 -> Ch_60
- J2 pad 2: Ch_73 -> Ch_72
- J2 pad 4: Ch_71 -> Ch_70
- J2 pad 6: Ch_57 -> Ch_54
- J2 pad 8: Ch_55 -> Ch_56
- U1 pad 10: Ch_4 -> Ch_3
- U1 pad 100: Ch_94 -> Ch_93
- U1 pad 101: Ch_95 -> Ch_94
- U1 pad 102: Ch_96 -> Ch_95
- U1 pad 103: Ch_97 -> Ch_96
- U1 pad 104: Ch_98 -> Ch_97
- U1 pad 105: Ch_99 -> Ch_98
- U1 pad 106: Ch_100 -> Ch_99
- U1 pad 107: Ch_101 -> Ch_100
- U1 pad 108: Ch_102 -> Ch_101
- U1 pad 109: Ch_103 -> Ch_102
- U1 pad 11: Ch_5 -> Ch_4
- U1 pad 110: Ch_104 -> Ch_103
- U1 pad 111: Ch_105 -> Ch_104
- U1 pad 112: Ch_106 -> Ch_105
- U1 pad 113: Ch_107 -> Ch_106
- U1 pad 114: Ch_108 -> Ch_107
- U1 pad 115: Ch_109 -> Ch_108
- U1 pad 116: Ch_110 -> Ch_109
- U1 pad 117: Ch_111 -> Ch_110
- U1 pad 118: Ch_112 -> Ch_111
- U1 pad 119: Ch_113 -> Ch_112
- U1 pad 12: Ch_6 -> Ch_5
- U1 pad 120: Ch_114 -> Ch_113
- U1 pad 121: Ch_115 -> Ch_114
- U1 pad 122: Ch_116 -> Ch_115
- U1 pad 123: Ch_117 -> Ch_116
- U1 pad 124: Ch_118 -> Ch_117
- U1 pad 125: Ch_119 -> Ch_118
- U1 pad 126: Ch_120 -> Ch_119
- U1 pad 127: Ch_121 -> Ch_120
- U1 pad 128: Ch_122 -> Ch_121
- U1 pad 129: Ch_123 -> Ch_122
- U1 pad 13: Ch_7 -> Ch_6
- U1 pad 130: Ch_124 -> Ch_123
- U1 pad 131: Ch_125 -> Ch_124
- U1 pad 132: Ch_126 -> Ch_125
- U1 pad 133: Ch_127 -> Ch_126
- U1 pad 134: Ch_128 -> Ch_127
- U1 pad 14: Ch_8 -> Ch_7
- U1 pad 15: Ch_9 -> Ch_8
- U1 pad 16: Ch_10 -> Ch_9
- U1 pad 17: Ch_11 -> Ch_10
- U1 pad 18: Ch_12 -> Ch_11
- U1 pad 19: Ch_13 -> Ch_12
- U1 pad 20: Ch_14 -> Ch_13
- U1 pad 21: Ch_15 -> Ch_14
- U1 pad 22: Ch_16 -> Ch_15
- U1 pad 23: Ch_17 -> Ch_16
- U1 pad 24: Ch_18 -> Ch_17
- U1 pad 25: Ch_19 -> Ch_18
- U1 pad 26: Ch_20 -> Ch_19
- U1 pad 27: Ch_21 -> Ch_20
- U1 pad 28: Ch_22 -> Ch_21
- U1 pad 29: Ch_23 -> Ch_22
- U1 pad 30: Ch_24 -> Ch_23
- U1 pad 31: Ch_25 -> Ch_24
- U1 pad 32: Ch_26 -> Ch_25
- U1 pad 33: Ch_27 -> Ch_26
- U1 pad 34: Ch_28 -> Ch_27
- U1 pad 35: Ch_29 -> Ch_28
- U1 pad 36: Ch_30 -> Ch_29
- U1 pad 37: Ch_31 -> Ch_30
- U1 pad 38: Ch_32 -> Ch_31
- U1 pad 39: Ch_33 -> Ch_32
- U1 pad 40: Ch_34 -> Ch_33
- U1 pad 41: Ch_35 -> Ch_34
- U1 pad 42: Ch_36 -> Ch_35
- U1 pad 43: Ch_37 -> Ch_36
- U1 pad 44: Ch_38 -> Ch_37
- U1 pad 45: Ch_39 -> Ch_38
- U1 pad 46: Ch_40 -> Ch_39
- U1 pad 47: Ch_41 -> Ch_40
- U1 pad 48: Ch_42 -> Ch_41
- U1 pad 49: Ch_43 -> Ch_42
- U1 pad 50: Ch_44 -> Ch_43
- U1 pad 51: Ch_45 -> Ch_44
- U1 pad 52: Ch_46 -> Ch_45
- U1 pad 53: Ch_47 -> Ch_46
- U1 pad 54: Ch_48 -> Ch_47
- U1 pad 60: Ch_54 -> Ch_53
- U1 pad 61: Ch_57 -> Ch_54
- U1 pad 62: Ch_56 -> Ch_55
- U1 pad 63: Ch_55 -> Ch_56
- U1 pad 64: Ch_58 -> Ch_57
- U1 pad 66: Ch_60 -> Ch_59
- U1 pad 67: Ch_61 -> Ch_60
- U1 pad 68: Ch_62 -> Ch_61
- U1 pad 69: Ch_63 -> Ch_62
- U1 pad 7: Ch_1 -> Ch_0
- U1 pad 70: Ch_64 -> Ch_63
- U1 pad 71: Ch_65 -> Ch_64
- U1 pad 72: Ch_66 -> Ch_65
- U1 pad 73: Ch_67 -> Ch_66
- U1 pad 74: Ch_68 -> Ch_67
- U1 pad 76: Ch_70 -> Ch_69
- U1 pad 77: Ch_71 -> Ch_70
- U1 pad 78: Ch_72 -> Ch_71
- U1 pad 79: Ch_73 -> Ch_72
- U1 pad 8: Ch_2 -> Ch_1
- U1 pad 80: Ch_74 -> Ch_73
- U1 pad 86: Ch_80 -> Ch_79
- U1 pad 87: Ch_81 -> Ch_80
- U1 pad 88: Ch_82 -> Ch_81
- U1 pad 89: Ch_83 -> Ch_82
- U1 pad 9: Ch_3 -> Ch_2
- U1 pad 90: Ch_84 -> Ch_83
- U1 pad 91: Ch_85 -> Ch_84
- U1 pad 92: Ch_86 -> Ch_85
- U1 pad 93: Ch_87 -> Ch_86
- U1 pad 94: Ch_88 -> Ch_87
- U1 pad 95: Ch_89 -> Ch_88
- U1 pad 96: Ch_90 -> Ch_89
- U1 pad 97: Ch_91 -> Ch_90
- U1 pad 98: Ch_92 -> Ch_91
- U1 pad 99: Ch_93 -> Ch_92
Routing:
- net Ch_0: track 0.00 -> 74.0 mm, vias 0 -> 1
- net Ch_48: track 53.8 -> 0.00 mm, vias 2 -> 0
- net Ch_59: track 0.00 -> 48.6 mm, vias 0 -> 2
- net Ch_53: track 0.00 -> 47.0 mm
- net Ch_68: track 45.7 -> 0.00 mm, vias 2 -> 0
- net Ch_58: track 44.7 -> 0.00 mm
- net Ch_79: track 0.00 -> 40.9 mm, vias 0 -> 2
- net Ch_69: track 0.00 -> 40.3 mm
- net Ch_60: track 48.6 -> 8.39 mm, vias 2 -> 0
- net Ch_74: track 39.1 -> 0.00 mm
- net Ch_64: track 47.4 -> 8.39 mm, vias 2 -> 0
- net Ch_63: track 8.41 -> 47.4 mm, vias 0 -> 2
- net Ch_67: track 8.58 -> 45.7 mm, vias 0 -> 2
- net Ch_56: track 50.0 -> 13.1 mm
- net Ch_55: track 13.1 -> 50.0 mm
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