File: HYDRA_VMM3_card/HYDRA_VMM3_CARD_V3_Flex/HYDRA_VMM3_CARD_V3_Flex.kicad_sch (KiCad schematic)
At the start: 22 parts, among them J1 ME1014010101011

Commit message: .
Parts:
- added J2: FPC: 68711714522, Custom_Footprints:68711714522, symbol Connector:Conn_01x17_Socket
Connections:
- net Ch_59 is gone; now on net GND: U1.65
- net Ch_69 is gone; now on net GND: U1.75
- net Ch_10: now also J1.B19; no longer J1.B18
- net Ch_100: now also J1.B69; no longer J1.B64
- net Ch_102: now also J1.B64; no longer J1.B63
- net Ch_104: now also J1.B68; no longer J1.B62
- net Ch_106: now also J1.B67; no longer J1.B61
- net Ch_107: now also J1.A60; no longer J1.A70
- net Ch_108: now also J1.B63; no longer J1.B60
- net Ch_109: now also J1.A61; no longer J1.A69
- net Ch_110: now also J1.B66; no longer J1.B59
- net Ch_111: now also J1.A62; no longer J1.A68
- net Ch_112: now also J1.B62; no longer J1.B58
- net Ch_113: now also J1.A63; no longer J1.A67
- net Ch_114: now also J1.A36; no longer J1.B57
- net Ch_115: now also J1.A64; no longer J1.A66
- net Ch_116: now also J1.A37
- net Ch_118: now also J1.A38
- net Ch_119: now also J1.A66; no longer J1.A64
- net Ch_12: now also J1.B20; no longer J1.B19
- net Ch_120: now also J1.A39
- net Ch_121: now also J1.A67; no longer J1.A63
- net Ch_122: now also J1.A40
- net Ch_123: now also J1.A68; no longer J1.A62
- net Ch_124: now also J1.A41
- net Ch_125: now also J1.A69; no longer J1.A61
- net Ch_126: now also J1.A42
- net Ch_127: now also J1.A70; no longer J1.A60
- net Ch_128: now also J1.A43
- net Ch_14: now also J1.B21; no longer J1.B20
- net Ch_16: now also J1.B22; no longer J1.B21
- net Ch_18: now also J1.B23; no longer J1.B22
- net Ch_2: now also J1.B15
- net Ch_20: now also J1.B24; no longer J1.B23
- net Ch_22: now also J1.B25; no longer J1.B24
- net Ch_24: now also J1.B26; no longer J1.B25
- net Ch_26: now also J1.B27; no longer J1.B26
- net Ch_28: now also J1.B28; no longer J1.B27
- net Ch_30: now also J1.B29; no longer J1.B28
- net Ch_32: now also J1.B30; no longer J1.B29
- net Ch_34: now also J1.B31; no longer J1.B30
- net Ch_36: now also J1.B32; no longer J1.B31
- net Ch_38: now also J1.B33; no longer J1.B32
- net Ch_4: now also J1.B16; no longer J1.B15
- net Ch_40: now also J1.B34; no longer J1.B33
- net Ch_42: now also J1.B35; no longer J1.B34
- net Ch_43: now also J1.A44; no longer J1.A36
- net Ch_44: now also J1.B36; no longer J1.B35
- net Ch_45: now also J1.A45; no longer J1.A37
- net Ch_46: now also J1.B37; no longer J1.B36
- net Ch_47: now also J1.A46; no longer J1.A38
- net Ch_48: now also J1.B38; no longer J1.B37
- net Ch_50: now also J1.B39; no longer J1.B38
- net Ch_52: now also J1.B40; no longer J1.B39
- net Ch_54: now also J1.B41; no longer J1.B40
- net Ch_55: now also U1.63, J2.8 (Pin_8); no longer J1.A42, U1.61
- net Ch_56: now also J1.B42; no longer J1.B41
- net Ch_57: now also U1.61, J2.6 (Pin_6); no longer U1.63
- net Ch_58: now also J1.B43; no longer J1.B42
- net Ch_6: now also J1.B17; no longer J1.B16
- net Ch_60: now also J1.B44; no longer J1.B43
- net Ch_61: now also J2.16 (Pin_16)
- net Ch_62: now also J1.B45; no longer J1.B44
- net Ch_63: now also J2.14 (Pin_14)
- net Ch_64: now also J1.B46; no longer J1.B45
- net Ch_65: now also J2.12 (Pin_12)
- net Ch_66: now also J1.B47; no longer J1.B46
- net Ch_67: now also J2.10 (Pin_10)
- net Ch_68: now also J1.B48; no longer J1.B47
- net Ch_70: now also J1.B49; no longer J1.B48
- net Ch_71: now also J2.4 (Pin_4)
- net Ch_72: now also J1.B50; no longer J1.B49
- net Ch_73: now also J2.2 (Pin_2); no longer J1.A43
- net Ch_74: now also J1.B51; no longer J1.B50
- net Ch_76: now also J1.B52; no longer J1.B51
- net Ch_78: now also J1.B53; no longer J1.B52
- net Ch_8: now also J1.B18; no longer J1.B17
- net Ch_80: now also J1.B54; no longer J1.B53
- net Ch_82: now also J1.B55; no longer J1.B54
- net Ch_84: now also J1.B56; no longer J1.B55
- net Ch_86: now also J1.B57; no longer J1.B56
- net Ch_88: now also J1.B58; no longer J1.B70
- net Ch_90: now also J1.B59; no longer J1.B69
- net Ch_92: now also J1.B60; no longer J1.B68
- net Ch_94: now also J1.B61; no longer J1.B67
- net Ch_96: now also J1.B70; no longer J1.B66
- net GND: now also U1.55, U1.57, U1.59, U1.81, U1.83, U1.85, J2.1 (Pin_1), J2.11 (Pin_11), J2.13 (Pin_13), J2.15 (Pin_15), J2.17 (Pin_17), J2.3 (Pin_3), J2.5 (Pin_5), J2.7 (Pin_7), J2.9 (Pin_9)
- removed net Ch_49: J1.A39, U1.55
- removed net Ch_51: J1.A40, U1.57
- removed net Ch_53: J1.A41, U1.59
- removed net Ch_75: J1.A44, U1.81
- removed net Ch_77: J1.A45, U1.83
- removed net Ch_79: J1.A46, U1.85

Commit message: .
Parts:
- added J3: FPC_4pin, Custom_Footprints:CON_5034800440_MOL, symbol Connector:Conn_01x06_Socket
- Temp_RX1, Temp_TX1: footprint IPEX:IPEX_20449-001E-03 -> Custom_Footprints:IPEX_20449-001E-03
Connections:
- net +3V3: now also J3.1 (Pin_1)
- net GND: now also J3.3 (Pin_3), J3.P1 (Pin_5), J3.P2 (Pin_6)
- net Heimtime: now also J3.2 (Pin_2)
- net Master_Trigg: now also J3.4 (Pin_4)
Other:
- moved on the sheet: J2

Commit message: .
Connections:
- net Heimtime: now also J3.4 (Pin_4); no longer J3.2 (Pin_2)
- net Master_Trigg: now also J3.2 (Pin_2); no longer J3.4 (Pin_4)
Changed lines of the file:
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@@
 	(global_label "Heimtime"
 		(shape input)
-		(at 128.27 34.29 180)
+		(at 128.27 39.37 180)
 		(fields_autoplaced yes)
 		(effects
@@
 		)
 		(property "Intersheetrefs" "${INTERSHEET_REFS}"
-			(at 115.9792 34.29 0)
+			(at 115.9792 39.37 0)
 			(effects
 				(font
@@
 	(global_label "Master_Trigg"
 		(shape input)
-		(at 128.27 39.37 180)
+		(at 128.27 34.29 180)
 		(fields_autoplaced yes)
 		(effects
@@
 		)
 		(property "Intersheetrefs" "${INTERSHEET_REFS}"
-			(at 112.9556 39.37 0)
-			(effects
-				(font
+			(at 112.9556 34.29 0)
+			(effects
+				(font

Commit message: .
Changed lines of the file:
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@@
 (kicad_sch
-	(version 20231120)
+	(version 20250114)
 	(generator "eeschema")
-	(generator_version "8.0")
+	(generator_version "9.0")
 	(paper "A3")
+	(rectangle
+		(start 330.2 13.97)
+		(end 406.4 52.07)
+		(stroke
+			(width 0)
+			(type default)
+		)
+		(fill
+			(type color)
+			(color 198 220 255 1)
+		)
+	)
+	(rectangle
+		(start 29.21 57.15)
+		(end 55.88 113.03)
+		(stroke
+			(width 0)
+			(type default)
+			(color 39 255 15 1)
+		)
+		(fill
+			(type color)
+			(color 193 255 203 1)
+		)
+	)
+	(rectangle
+		(start 271.78 13.97)
+		(end 328.93 40.64)
+		(stroke
+			(width 0)
+			(type default)
+		)
+		(fill
+			(type color)
+			(color 255 224 219 1)
+		)
+	)
+	(rectangle
+		(start 243.84 13.97)
+		(end 270.51 36.83)
+		(stroke
+			(width 0)
+			(type solid)
+		)
+		(fill
+			(type color)
+			(color 255 246 107 1)
+		)
+	)
+	(text "6 bit geographical code\n"
+		(exclude_from_sim no)
+		(at 256.54 16.002 0)
+		(effects
+			(font
+				(size 1.27 1.27)
+				(thickness 0.254)
+				(bold yes)
+			)
+		)
+	)
+	(text "Decoupling capacitors\nNote! Add them near \npower pins"
+		(exclude_from_sim no)
+		(at 42.672 109.22 0)
+		(effects
+			(font
+				(size 1.27 1.27)
+			)
+		)
+	)
+	(text "Power LEDs"
+		(exclude_from_sim no)
+		(at 369.57 49.53 0)
+		(effects
+			(font
+				(size 1.27 1.27)
+				(thickness 0.254)
+				(bold yes)
+			)
+		)
+	)
+	(text "Temperature Readout"
+		(exclude_from_sim no)
+		(at 300.99 39.37 0)
+		(effects
+			(font
+				(size 1.27 1.27)
+				(thickness 0.254)
+				(bold yes)
+			)
+		)
+	)
 	(junction
 		(at 172.72 139.7)
@@
 		)
 	)
-	(rectangle
-		(start 330.2 13.97)
-		(end 406.4 52.07)
-		(stroke
-			(width 0)
-			(type default)
-		)
-		(fill
-			(type color)
-			(color 198 220 255 1)
-		)
-	)
-	(rectangle
-		(start 29.21 57.15)
-		(end 55.88 113.03)
-		(stroke
-			(width 0)
-			(type default)
-			(color 39 255 15 1)
-		)
-		(fill
-			(type color)
-			(color 193 255 203 1)
-		)
-	)
-	(rectangle
-		(start 271.78 13.97)
-		(end 328.93 40.64)
-		(stroke
-			(width 0)
-			(type default)
-		)
-		(fill
-			(type color)
-			(color 255 224 219 1)
-		)
-	)
-	(rectangle
-		(start 243.84 13.97)
-		(end 270.51 36.83)
-		(stroke
-			(width 0)
-			(type solid)
-		)
-		(fill
-			(type color)
-			(color 255 246 107 1)
-		)
-	)
-	(text "6 bit geographical code\n"
-		(exclude_from_sim no)
-		(at 256.54 16.002 0)
-		(effects
-			(font
-				(size 1.27 1.27)
-				(thickness 0.254)
-				(bold yes)
-			)
-		)
-	)
-	(text "Decoupling capacitors\nNote! Add them near \npower pins"
-		(exclude_from_sim no)
-		(at 42.672 109.22 0)
-		(effects
-			(font
-				(size 1.27 1.27)
-			)
-		)
-	)
-	(text "Power LEDs"
-		(exclude_from_sim no)
-		(at 369.57 49.53 0)
-		(effects
-			(font
-				(size 1.27 1.27)
-				(thickness 0.254)
-				(bold yes)
-			)
-		)
-	)
-	(text "Temperature Readout"
-		(exclude_from_sim no)
-		(at 300.99 39.37 0)
-		(effects
-			(font
-				(size 1.27 1.27)
-				(thickness 0.254)
-				(bold yes)
-			)
-		)
-	)
 	(global_label "Ch_21"
 		(shape input)
@@
 		)
 	)
+	(embedded_fonts no)
 )

Commit message: .
Connections:
- net Ch_1: now also U1.8; no longer U1.7
- net Ch_10: now also U1.17; no longer U1.16
- net Ch_100: now also U1.107; no longer U1.106
- net Ch_101: now also U1.108; no longer U1.107
- net Ch_102: now also U1.109; no longer U1.108
- net Ch_103: now also U1.110; no longer U1.109
- net Ch_104: now also U1.111; no longer U1.110
- net Ch_105: now also U1.112; no longer U1.111
- net Ch_106: now also U1.113; no longer U1.112
- net Ch_107: now also U1.114; no longer U1.113
- net Ch_108: now also U1.115; no longer U1.114
- net Ch_109: now also U1.116; no longer U1.115
- net Ch_11: now also U1.18; no longer U1.17
- net Ch_110: now also U1.117; no longer U1.116
- net Ch_111: now also U1.118; no longer U1.117
- net Ch_112: now also U1.119; no longer U1.118
- net Ch_113: now also U1.120; no longer U1.119
- net Ch_114: now also U1.121; no longer U1.120
- net Ch_115: now also U1.122; no longer U1.121
- net Ch_116: now also U1.123; no longer U1.122
- net Ch_117: now also U1.124; no longer U1.123
- net Ch_118: now also U1.125; no longer U1.124
- net Ch_119: now also U1.126; no longer U1.125
- net Ch_12: now also U1.19; no longer U1.18
- net Ch_120: now also U1.127; no longer U1.126
- net Ch_121: now also U1.128; no longer U1.127
- net Ch_122: now also U1.129; no longer U1.128
- net Ch_123: now also U1.130; no longer U1.129
- net Ch_124: now also U1.131; no longer U1.130
- net Ch_125: now also U1.132; no longer U1.131
- net Ch_126: now also U1.133; no longer U1.132
- net Ch_127: now also U1.134; no longer U1.133
- net Ch_128: no longer U1.134
- net Ch_13: now also U1.20; no longer U1.19
- net Ch_14: now also U1.21; no longer U1.20
- net Ch_15: now also U1.22; no longer U1.21
- net Ch_16: now also U1.23; no longer U1.22
- net Ch_17: now also U1.24; no longer U1.23
- net Ch_18: now also U1.25; no longer U1.24
- net Ch_19: now also U1.26; no longer U1.25
- net Ch_2: now also U1.9; no longer U1.8
- net Ch_20: now also U1.27; no longer U1.26
- net Ch_21: now also U1.28; no longer U1.27
- net Ch_22: now also U1.29; no longer U1.28
- net Ch_23: now also U1.30; no longer U1.29
- net Ch_24: now also U1.31; no longer U1.30
- net Ch_25: now also U1.32; no longer U1.31
- net Ch_26: now also U1.33; no longer U1.32
- net Ch_27: now also U1.34; no longer U1.33
- net Ch_28: now also U1.35; no longer U1.34
- net Ch_29: now also U1.36; no longer U1.35
- net Ch_3: now also U1.10; no longer U1.9
- net Ch_30: now also U1.37; no longer U1.36
- net Ch_31: now also U1.38; no longer U1.37
- net Ch_32: now also U1.39; no longer U1.38
- net Ch_33: now also U1.40; no longer U1.39
- net Ch_34: now also U1.41; no longer U1.40
- net Ch_35: now also U1.42; no longer U1.41
- net Ch_36: now also U1.43; no longer U1.42
- net Ch_37: now also U1.44; no longer U1.43
- net Ch_38: now also U1.45; no longer U1.44
- net Ch_39: now also U1.46; no longer U1.45
- net Ch_4: now also U1.11; no longer U1.10
- net Ch_40: now also U1.47; no longer U1.46
- net Ch_41: now also U1.48; no longer U1.47
- net Ch_42: now also U1.49; no longer U1.48
- net Ch_43: now also U1.50; no longer U1.49
- net Ch_44: now also U1.51; no longer U1.50
- net Ch_45: now also U1.52; no longer U1.51
- net Ch_46: now also U1.53; no longer U1.52
- net Ch_47: now also U1.54; no longer U1.53
- net Ch_48: no longer U1.54
- net Ch_5: now also U1.12; no longer U1.11
- net Ch_50: no longer U1.56
- net Ch_52: no longer U1.58
- net Ch_54: now also J2.6 (Pin_6), U1.61; no longer U1.60
- net Ch_55: now also U1.62; no longer J2.8 (Pin_8), U1.63
- net Ch_56: now also J2.8 (Pin_8), U1.63; no longer U1.62
- net Ch_57: now also U1.64; no longer J2.6 (Pin_6), U1.61
- net Ch_58: no longer U1.64
- net Ch_6: now also U1.13; no longer U1.12
- net Ch_60: now also J2.16 (Pin_16), U1.67; no longer U1.66
- net Ch_61: now also U1.68; no longer J2.16 (Pin_16), U1.67
- net Ch_62: now also J2.14 (Pin_14), U1.69; no longer U1.68
- net Ch_63: now also U1.70; no longer J2.14 (Pin_14), U1.69
- net Ch_64: now also J2.12 (Pin_12), U1.71; no longer U1.70
- net Ch_65: now also U1.72; no longer J2.12 (Pin_12), U1.71
- net Ch_66: now also J2.10 (Pin_10), U1.73; no longer U1.72
- net Ch_67: now also U1.74; no longer J2.10 (Pin_10), U1.73
- net Ch_68: no longer U1.74
- net Ch_7: now also U1.14; no longer U1.13
- net Ch_70: now also J2.4 (Pin_4), U1.77; no longer U1.76
- net Ch_71: now also U1.78; no longer J2.4 (Pin_4), U1.77
- net Ch_72: now also J2.2 (Pin_2), U1.79; no longer U1.78
- net Ch_73: now also U1.80; no longer J2.2 (Pin_2), U1.79
- net Ch_74: no longer U1.80
- net Ch_76: no longer U1.82
- net Ch_78: no longer U1.84
- net Ch_8: now also U1.15; no longer U1.14
- net Ch_80: now also U1.87; no longer U1.86
- net Ch_81: now also U1.88; no longer U1.87
- net Ch_82: now also U1.89; no longer U1.88
- net Ch_83: now also U1.90; no longer U1.89
- net Ch_84: now also U1.91; no longer U1.90
- net Ch_85: now also U1.92; no longer U1.91
- net Ch_86: now also U1.93; no longer U1.92
- net Ch_87: now also U1.94; no longer U1.93
- net Ch_88: now also U1.95; no longer U1.94
- net Ch_89: now also U1.96; no longer U1.95
- net Ch_9: now also U1.16; no longer U1.15
- net Ch_90: now also U1.97; no longer U1.96
- net Ch_91: now also U1.98; no longer U1.97
- net Ch_92: now also U1.99; no longer U1.98
- net Ch_93: now also U1.100; no longer U1.99
- net Ch_94: now also U1.101; no longer U1.100
- net Ch_95: now also U1.102; no longer U1.101
- net Ch_96: now also U1.103; no longer U1.102
- net Ch_97: now also U1.104; no longer U1.103
- net Ch_98: now also U1.105; no longer U1.104
- net Ch_99: now also U1.106; no longer U1.105
- new net Ch_0: U1.7
- new net Ch_49: U1.56
- new net Ch_51: U1.58
- new net Ch_53: U1.60
- new net Ch_59: U1.66
- new net Ch_69: U1.76
- new net Ch_75: U1.82
- new net Ch_77: U1.84
- new net Ch_79: U1.86

Commit message: .
Connections:
- net Ch_128 is gone; now on net Ch_127: J1.A43
- net Ch_48 is gone; now on net Ch_47: J1.B38
- net Ch_50 is gone; now on net Ch_49: J1.B39
- net Ch_52 is gone; now on net Ch_51: J1.B40
- net Ch_58 is gone; now on net Ch_57: J1.B43
- net Ch_68 is gone; now on net Ch_67: J1.B48
- net Ch_74 is gone; now on net Ch_73: J1.B51
- net Ch_76 is gone; now on net Ch_75: J1.B52
- net Ch_78 is gone; now on net Ch_77: J1.B53
- net Ch_0: now also J1.A15
- net Ch_1: now also J1.B15; no longer J1.A15
- net Ch_10: now also J1.A20; no longer J1.B19
- net Ch_100: now also J1.A57; no longer J1.B69
- net Ch_101: now also J1.B64; no longer J1.A57
- net Ch_102: now also J1.A58; no longer J1.B64
- net Ch_103: now also J1.B68; no longer J1.A58
- net Ch_104: now also J1.A59; no longer J1.B68
- net Ch_105: now also J1.B67; no longer J1.A59
- net Ch_106: now also J1.A60; no longer J1.B67
- net Ch_107: now also J1.B63; no longer J1.A60
- net Ch_108: now also J1.A61; no longer J1.B63
- net Ch_109: now also J1.B66; no longer J1.A61
- net Ch_11: now also J1.B20; no longer J1.A20
- net Ch_110: now also J1.A62; no longer J1.B66
- net Ch_111: now also J1.B62; no longer J1.A62
- net Ch_112: now also J1.A63; no longer J1.B62
- net Ch_113: now also J1.A36; no longer J1.A63
- net Ch_114: now also J1.A64; no longer J1.A36
- net Ch_115: now also J1.A37; no longer J1.A64
- net Ch_116: now also J1.A65; no longer J1.A37
- net Ch_117: now also J1.A38; no longer J1.A65
- net Ch_118: now also J1.A66; no longer J1.A38
- net Ch_119: now also J1.A39; no longer J1.A66
- net Ch_12: now also J1.A21; no longer J1.B20
- net Ch_120: now also J1.A67; no longer J1.A39
- net Ch_121: now also J1.A40; no longer J1.A67
- net Ch_122: now also J1.A68; no longer J1.A40
- net Ch_123: now also J1.A41; no longer J1.A68
- net Ch_124: now also J1.A69; no longer J1.A41
- net Ch_125: now also J1.A42; no longer J1.A69
- net Ch_126: now also J1.A70; no longer J1.A42
- net Ch_127: no longer J1.A70
- net Ch_13: now also J1.B21; no longer J1.A21
- net Ch_14: now also J1.A22; no longer J1.B21
- net Ch_15: now also J1.B22; no longer J1.A22
- net Ch_16: now also J1.A23; no longer J1.B22
- net Ch_17: now also J1.B23; no longer J1.A23
- net Ch_18: now also J1.A24; no longer J1.B23
- net Ch_19: now also J1.B24; no longer J1.A24
- net Ch_2: now also J1.A16; no longer J1.B15
- net Ch_20: now also J1.A25; no longer J1.B24
- net Ch_21: now also J1.B25; no longer J1.A25
- net Ch_22: now also J1.A26; no longer J1.B25
- net Ch_23: now also J1.B26; no longer J1.A26
- net Ch_24: now also J1.A27; no longer J1.B26
- net Ch_25: now also J1.B27; no longer J1.A27
- net Ch_26: now also J1.A28; no longer J1.B27
- net Ch_27: now also J1.B28; no longer J1.A28
- net Ch_28: now also J1.A29; no longer J1.B28
- net Ch_29: now also J1.B29; no longer J1.A29
- net Ch_3: now also J1.B16; no longer J1.A16
- net Ch_30: now also J1.A30; no longer J1.B29
- net Ch_31: now also J1.B30; no longer J1.A30
- net Ch_32: now also J1.A31; no longer J1.B30
- net Ch_33: now also J1.B31; no longer J1.A31
- net Ch_34: now also J1.A32; no longer J1.B31
- net Ch_35: now also J1.B32; no longer J1.A32
- net Ch_36: now also J1.A33; no longer J1.B32
- net Ch_37: now also J1.B33; no longer J1.A33
- net Ch_38: now also J1.A34; no longer J1.B33
- net Ch_39: now also J1.B34; no longer J1.A34
- net Ch_4: now also J1.A17; no longer J1.B16
- net Ch_40: now also J1.A35; no longer J1.B34
- net Ch_41: now also J1.B35; no longer J1.A35
- net Ch_42: now also J1.A44; no longer J1.B35
- net Ch_43: now also J1.B36; no longer J1.A44
- net Ch_44: now also J1.A45; no longer J1.B36
- net Ch_45: now also J1.B37; no longer J1.A45
- net Ch_46: now also J1.A46; no longer J1.B37
- net Ch_47: no longer J1.A46
- net Ch_5: now also J1.B17; no longer J1.A17
- net Ch_53: now also J1.B41
- net Ch_54: no longer J1.B41
- net Ch_55: now also J1.B42
- net Ch_56: no longer J1.B42
- net Ch_59: now also J1.B44
- net Ch_6: now also J1.A18; no longer J1.B17
- net Ch_60: no longer J1.B44
- net Ch_61: now also J1.B45
- net Ch_62: no longer J1.B45
- net Ch_63: now also J1.B46
- net Ch_64: no longer J1.B46
- net Ch_65: now also J1.B47
- net Ch_66: no longer J1.B47
- net Ch_69: now also J1.B49
- net Ch_7: now also J1.B18; no longer J1.A18
- net Ch_70: no longer J1.B49
- net Ch_71: now also J1.B50
- net Ch_72: no longer J1.B50
- net Ch_79: now also J1.B54
- net Ch_8: now also J1.A19; no longer J1.B18
- net Ch_80: now also J1.A47; no longer J1.B54
- net Ch_81: now also J1.B55; no longer J1.A47
- net Ch_82: now also J1.A48; no longer J1.B55
- net Ch_83: now also J1.B56; no longer J1.A48
- net Ch_84: now also J1.A49; no longer J1.B56
- net Ch_85: now also J1.B57; no longer J1.A49
- net Ch_86: now also J1.A50; no longer J1.B57
- net Ch_87: now also J1.B58; no longer J1.A50
- net Ch_88: now also J1.A51; no longer J1.B58
- net Ch_89: now also J1.B59; no longer J1.A51
- net Ch_9: now also J1.B19; no longer J1.A19
- net Ch_90: now also J1.A52; no longer J1.B59
- net Ch_91: now also J1.B60; no longer J1.A52
- net Ch_92: now also J1.A53; no longer J1.B60
- net Ch_93: now also J1.B61; no longer J1.A53
- net Ch_94: now also J1.A54; no longer J1.B61
- net Ch_95: now also J1.B70; no longer J1.A54
- net Ch_96: now also J1.A55; no longer J1.B70
- net Ch_97: now also J1.B65; no longer J1.A55
- net Ch_98: now also J1.A56; no longer J1.B65
- net Ch_99: now also J1.B69; no longer J1.A56
