File: HYDRA_VMM3_card/HYDRA_VMM3_CARD_V3_Flex/HYDRA_VMM3_CARD_V3_Flex.kicad_sch (KiCad schematic)
At the start: 24 parts, among them J1 ME1014010101011, J2 FPC: 68711714522, J3 FPC_4pin

Commit message: .
Connections:
- net Ch_0: now also J1.B15, U1.8; no longer J1.A15, U1.7
- net Ch_1: now also J1.A15, U1.7; no longer J1.B15, U1.8
- net Ch_10: now also J1.B20, U1.18; no longer J1.A20, U1.17
- net Ch_100: now also J1.B64, U1.108; no longer J1.A57, U1.107
- net Ch_101: now also J1.A57, U1.107; no longer J1.B64, U1.108
- net Ch_102: now also J1.B68, U1.110; no longer J1.A58, U1.109
- net Ch_103: now also J1.A58, U1.109; no longer J1.B68, U1.110
- net Ch_104: now also J1.B67, U1.112; no longer J1.A59, U1.111
- net Ch_105: now also J1.A59, U1.111; no longer J1.B67, U1.112
- net Ch_106: now also J1.B63, U1.114; no longer J1.A60, U1.113
- net Ch_107: now also J1.A60, U1.113; no longer J1.B63, U1.114
- net Ch_108: now also J1.B66, U1.116; no longer J1.A61, U1.115
- net Ch_109: now also J1.A61, U1.115; no longer J1.B66, U1.116
- net Ch_11: now also J1.A20, U1.17; no longer J1.B20, U1.18
- net Ch_110: now also J1.B62, U1.118; no longer J1.A62, U1.117
- net Ch_111: now also J1.A62, U1.117; no longer J1.B62, U1.118
- net Ch_112: now also U1.120; no longer J1.A63, U1.119
- net Ch_113: now also J1.A63, U1.119; no longer J1.A36, U1.120
- net Ch_114: now also J1.A36, U1.122; no longer J1.A64, U1.121
- net Ch_115: now also J1.A64, U1.121; no longer J1.A37, U1.122
- net Ch_116: now also J1.A37, U1.124; no longer J1.A65, U1.123
- net Ch_117: now also J1.A65, U1.123; no longer J1.A38, U1.124
- net Ch_118: now also J1.A38, U1.126; no longer J1.A66, U1.125
- net Ch_119: now also J1.A66, U1.125; no longer J1.A39, U1.126
- net Ch_12: now also J1.B21, U1.20; no longer J1.A21, U1.19
- net Ch_120: now also J1.A39, U1.128; no longer J1.A67, U1.127
- net Ch_121: now also J1.A67, U1.127; no longer J1.A40, U1.128
- net Ch_122: now also J1.A40, U1.130; no longer J1.A68, U1.129
- net Ch_123: now also J1.A68, U1.129; no longer J1.A41, U1.130
- net Ch_124: now also J1.A41, U1.132; no longer J1.A69, U1.131
- net Ch_125: now also J1.A69, U1.131; no longer J1.A42, U1.132
- net Ch_126: now also J1.A42, U1.134; no longer J1.A70, U1.133
- net Ch_127: now also J1.A70, U1.133; no longer J1.A43, U1.134
- net Ch_13: now also J1.A21, U1.19; no longer J1.B21, U1.20
- net Ch_14: now also J1.B22, U1.22; no longer J1.A22, U1.21
- net Ch_15: now also J1.A22, U1.21; no longer J1.B22, U1.22
- net Ch_16: now also J1.B23, U1.24; no longer J1.A23, U1.23
- net Ch_17: now also J1.A23, U1.23; no longer J1.B23, U1.24
- net Ch_18: now also J1.B24, U1.26; no longer J1.A24, U1.25
- net Ch_19: now also J1.A24, U1.25; no longer J1.B24, U1.26
- net Ch_2: now also J1.B16, U1.10; no longer J1.A16, U1.9
- net Ch_20: now also J1.B25, U1.28; no longer J1.A25, U1.27
- net Ch_21: now also J1.A25, U1.27; no longer J1.B25, U1.28
- net Ch_22: now also J1.B26, U1.30; no longer J1.A26, U1.29
- net Ch_23: now also J1.A26, U1.29; no longer J1.B26, U1.30
- net Ch_24: now also J1.B27, U1.32; no longer J1.A27, U1.31
- net Ch_25: now also J1.A27, U1.31; no longer J1.B27, U1.32
- net Ch_26: now also J1.B28, U1.34; no longer J1.A28, U1.33
- net Ch_27: now also J1.A28, U1.33; no longer J1.B28, U1.34
- net Ch_28: now also J1.B29, U1.36; no longer J1.A29, U1.35
- net Ch_29: now also J1.A29, U1.35; no longer J1.B29, U1.36
- net Ch_3: now also J1.A16, U1.9; no longer J1.B16, U1.10
- net Ch_30: now also J1.B30, U1.38; no longer J1.A30, U1.37
- net Ch_31: now also J1.A30, U1.37; no longer J1.B30, U1.38
- net Ch_32: now also J1.B31, U1.40; no longer J1.A31, U1.39
- net Ch_33: now also J1.A31, U1.39; no longer J1.B31, U1.40
- net Ch_34: now also J1.B32, U1.42; no longer J1.A32, U1.41
- net Ch_35: now also J1.A32, U1.41; no longer J1.B32, U1.42
- net Ch_36: now also J1.B33, U1.44; no longer J1.A33, U1.43
- net Ch_37: now also J1.A33, U1.43; no longer J1.B33, U1.44
- net Ch_38: now also J1.B34, U1.46; no longer J1.A34, U1.45
- net Ch_39: now also J1.A34, U1.45; no longer J1.B34, U1.46
- net Ch_4: now also J1.B17, U1.12; no longer J1.A17, U1.11
- net Ch_40: now also J1.B35, U1.48; no longer J1.A35, U1.47
- net Ch_41: now also J1.A35, U1.47; no longer J1.B35, U1.48
- net Ch_42: now also J1.B36, U1.50; no longer J1.A44, U1.49
- net Ch_43: now also J1.A44, U1.49; no longer J1.B36, U1.50
- net Ch_44: now also J1.B37, U1.52; no longer J1.A45, U1.51
- net Ch_45: now also J1.A45, U1.51; no longer J1.B37, U1.52
- net Ch_46: now also J1.B38, U1.54; no longer J1.A46, U1.53
- net Ch_47: now also J1.A46, U1.53; no longer J1.B38, U1.54
- net Ch_5: now also J1.A17, U1.11; no longer J1.B17, U1.12
- net Ch_54: now also J1.B42, U1.62; no longer J2.6 (Pin_6), U1.61
- net Ch_55: now also J2.6 (Pin_6), U1.61; no longer J1.B42, U1.62
- net Ch_56: now also J1.B43, U1.64; no longer J2.8 (Pin_8), U1.63
- net Ch_57: now also J2.8 (Pin_8), U1.63; no longer J1.B43, U1.64
- net Ch_6: now also J1.B18, U1.14; no longer J1.A18, U1.13
- net Ch_60: now also J1.B45, U1.68; no longer J2.16 (Pin_16), U1.67
- net Ch_61: now also J2.16 (Pin_16), U1.67; no longer J1.B45, U1.68
- net Ch_62: now also J1.B46, U1.70; no longer J2.14 (Pin_14), U1.69
- net Ch_63: now also J2.14 (Pin_14), U1.69; no longer J1.B46, U1.70
- net Ch_64: now also J1.B47, U1.72; no longer J2.12 (Pin_12), U1.71
- net Ch_65: now also J2.12 (Pin_12), U1.71; no longer J1.B47, U1.72
- net Ch_66: now also J1.B48, U1.74; no longer J2.10 (Pin_10), U1.73
- net Ch_67: now also J2.10 (Pin_10), U1.73; no longer J1.B48, U1.74
- net Ch_7: now also J1.A18, U1.13; no longer J1.B18, U1.14
- net Ch_70: now also J1.B50, U1.78; no longer J2.4 (Pin_4), U1.77
- net Ch_71: now also J2.4 (Pin_4), U1.77; no longer J1.B50, U1.78
- net Ch_72: now also J1.B51, U1.80; no longer J2.2 (Pin_2), U1.79
- net Ch_73: now also J2.2 (Pin_2), U1.79; no longer J1.B51, U1.80
- net Ch_8: now also J1.B19, U1.16; no longer J1.A19, U1.15
- net Ch_80: now also J1.B55, U1.88; no longer J1.A47, U1.87
- net Ch_81: now also J1.A47, U1.87; no longer J1.B55, U1.88
- net Ch_82: now also J1.B56, U1.90; no longer J1.A48, U1.89
- net Ch_83: now also J1.A48, U1.89; no longer J1.B56, U1.90
- net Ch_84: now also J1.B57, U1.92; no longer J1.A49, U1.91
- net Ch_85: now also J1.A49, U1.91; no longer J1.B57, U1.92
- net Ch_86: now also J1.B58, U1.94; no longer J1.A50, U1.93
- net Ch_87: now also J1.A50, U1.93; no longer J1.B58, U1.94
- net Ch_88: now also J1.B59, U1.96; no longer J1.A51, U1.95
- net Ch_89: now also J1.A51, U1.95; no longer J1.B59, U1.96
- net Ch_9: now also J1.A19, U1.15; no longer J1.B19, U1.16
- net Ch_90: now also J1.B60, U1.98; no longer J1.A52, U1.97
- net Ch_91: now also J1.A52, U1.97; no longer J1.B60, U1.98
- net Ch_92: now also J1.B61, U1.100; no longer J1.A53, U1.99
- net Ch_93: now also J1.A53, U1.99; no longer J1.B61, U1.100
- net Ch_94: now also J1.B70, U1.102; no longer J1.A54, U1.101
- net Ch_95: now also J1.A54, U1.101; no longer J1.B70, U1.102
- net Ch_96: now also J1.B65, U1.104; no longer J1.A55, U1.103
- net Ch_97: now also J1.A55, U1.103; no longer J1.B65, U1.104
- net Ch_98: now also J1.B69, U1.106; no longer J1.A56, U1.105
- net Ch_99: now also J1.A56, U1.105; no longer J1.B69, U1.106
- net Ch_49 renamed Ch_48
- net Ch_51 renamed Ch_50
- net Ch_53 renamed Ch_52
- net Ch_59 renamed Ch_58
- net Ch_69 renamed Ch_68
- net Ch_75 renamed Ch_74
- net Ch_77 renamed Ch_76
- net Ch_79 renamed Ch_78
- new net Ch_128: J1.A43

Commit message: .
Connections:
- net Ch_128 is gone; now on net Ch_126: J1.A43
- net Ch_112: now also J1.A36
- net Ch_114: now also J1.A37; no longer J1.A36
- net Ch_116: now also J1.A38; no longer J1.A37
- net Ch_118: now also J1.A39; no longer J1.A38
- net Ch_120: now also J1.A40; no longer J1.A39
- net Ch_122: now also J1.A41; no longer J1.A40
- net Ch_124: now also J1.A42; no longer J1.A41
- net Ch_126: no longer J1.A42
Changed lines of the file:
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@@
 	)
 	(junction
-		(at 172.72 134.62)
-		(diameter 0)
-		(color 0 0 0 0)
-	)
-	(junction
 		(at 73.66 60.96)
 		(diameter 0)
@@
 	(wire
 		(pts
-			(xy 172.72 134.62) (xy 176.53 134.62)
-		)
-		(stroke
-			(width 0)
-			(type default)
-		)
-	)
-	(wire
-		(pts
 			(xy 172.72 139.7) (xy 172.72 147.32)
 		)
@@
 	(wire
 		(pts
-			(xy 172.72 137.16) (xy 176.53 137.16)
-		)
-		(stroke
-			(width 0)
-			(type default)
-		)
-	)
-	(wire
-		(pts
 			(xy 172.72 173.99) (xy 172.72 172.72)
 		)
@@
 	(wire
 		(pts
-			(xy 172.72 139.7) (xy 176.53 139.7)
-		)
-		(stroke
-			(width 0)
-			(type default)
-		)
-	)
-	(wire
-		(pts
 			(xy 73.66 60.96) (xy 72.39 60.96)
 		)
@@
 	(wire
 		(pts
-			(xy 172.72 160.02) (xy 176.53 160.02)
-		)
-		(stroke
-			(width 0)
-			(type default)
-		)
-	)
-	(wire
-		(pts
 			(xy 111.76 41.91) (xy 111.76 44.45)
 		)
@@
 	(wire
 		(pts
-			(xy 172.72 147.32) (xy 176.53 147.32)
-		)
-		(stroke
-			(width 0)
-			(type default)
-		)
-	)
-	(wire
-		(pts
 			(xy 297.18 101.6) (xy 285.75 101.6)
 		)
@@
 		)
 	)
-	(global_label "Ch_118"
+	(global_label "Ch_116"
 		(shape input)
 		(at 101.6 161.29 0)
@@
 		)
 	)
-	(global_label "Ch_120"
+	(global_label "Ch_118"
 		(shape input)
 		(at 101.6 163.83 0)
@@
 	(global_label "Ch_53"
 		(shape input)
-		(at 176.53 139.7 0)
+		(at 184.15 139.7 0)
 		(fields_autoplaced yes)
 		(effects
@@
 		)
 		(property "Intersheetrefs" "${INTERSHEET_REFS}"
-			(at 185.3208 139.7 0)
+			(at 192.9408 139.7 0)
 			(effects
 				(font
@@
 	(global_label "Ch_49"
 		(shape input)
-		(at 176.53 134.62 0)
+		(at 184.15 134.62 0)
 		(fields_autoplaced yes)
 		(effects
@@
 		)
 		(property "Intersheetrefs" "${INTERSHEET_REFS}"
-			(at 185.3208 134.62 0)
+			(at 192.9408 134.62 0)
 			(effects
 				(font
@@
 	(global_label "Ch_51"
 		(shape input)
-		(at 176.53 137.16 0)
+		(at 184.15 137.16 0)
 		(fields_autoplaced yes)
 		(effects
@@
 		)
 		(property "Intersheetrefs" "${INTERSHEET_REFS}"
-			(at 185.3208 137.16 0)
+			(at 192.9408 137.16 0)
 			(effects
 				(font
@@
 		)
 	)
-	(global_label "Ch_128"
+	(global_label "Ch_126"
 		(shape input)
 		(at 101.6 173.99 0)
@@
 		)
 	)
-	(global_label "Ch_114"
+	(global_label "Ch_112"
 		(shape input)
 		(at 101.6 156.21 0)
@@
 		)
 	)
-	(global_label "Ch_116"
+	(global_label "Ch_114"
 		(shape input)
 		(at 101.6 158.75 0)
@@
 	(global_label "Ch_69"
 		(shape input)
-		(at 176.53 160.02 0)
+		(at 184.15 160.02 0)
 		(fields_autoplaced yes)
 		(effects
@@
 		)
 		(property "Intersheetrefs" "${INTERSHEET_REFS}"
-			(at 185.3208 160.02 0)
+			(at 192.9408 160.02 0)
 			(effects
 				(font
@@
 		)
 	)
-	(global_label "Ch_126"
+	(global_label "Ch_124"
 		(shape input)
 		(at 101.6 171.45 0)
@@
 		)
 	)
-	(global_label "Ch_122"
+	(global_label "Ch_120"
 		(shape input)
 		(at 101.6 166.37 0)
@@
 	(global_label "Ch_59"
 		(shape input)
-		(at 176.53 147.32 0)
+		(at 184.15 147.32 0)
 		(fields_autoplaced yes)
 		(effects
@@
 		)
 		(property "Intersheetrefs" "${INTERSHEET_REFS}"
-			(at 185.3208 147.32 0)
+			(at 192.9408 147.32 0)
 			(effects
 				(font
@@
 		)
 	)
-	(global_label "Ch_124"
+	(global_label "Ch_122"
 		(shape input)
 		(at 101.6 168.91 0)
