File: AddOns/2_In_6_Out/2_In_6_Out.kicad_pcb (KiCad board)
At the start: 4 copper layers, 20 x 20 mm, 23 parts, among them J1 Heimtime, J2 MasterTrigger, J3 Conn_01x13_Socket, J4 Conn_01x04_Socket, J5 Conn_01x04_Socket, U2 5PB1213NTGK8, U4 5PB1213NTGK8

Commit message: .
Parts:
- added D2: LED, LED_SMD:LED_0603_1608Metric, F.Cu at (99.9, 59.8)
- added D3: LED, LED_SMD:LED_0603_1608Metric, F.Cu at (99.9, 61.7)
- added R11: 680, Resistor_SMD:R_0402_1005Metric, F.Cu at (97.9, 58.0)
- added R12: 680, Resistor_SMD:R_0402_1005Metric, F.Cu at (97.9, 68.0)
- moved C1 25.1 mm to (97.8, 54.7)
- moved C11 25.1 mm to (97.8, 64.7)
- moved J1 25.1 mm to (93.1, 55.8)
- moved J2 25.1 mm to (93.1, 65.8)
- moved R1 25.1 mm to (99.9, 68.0)
- moved R2 25.1 mm to (100.9, 68.0)
- moved R3 25.1 mm to (98.9, 68.0)
- moved R4 25.1 mm to (99.9, 58.0)
- moved R8 25.1 mm to (100.9, 58.0)
- moved R9 25.1 mm to (98.9, 58.0)
- moved U2 25.1 mm to (99.9, 55.8)
- moved U4 25.1 mm to (99.9, 65.8)
- moved D1 25.1 mm to (91.1, 60.8)
- moved J4 25.1 mm to (97.0, 50.8)
- moved J5 25.1 mm to (97.0, 70.8)
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Routing:
- net Net-(D3-A): track 0.00 -> 9.35 mm, vias 0 -> 2
- net Net-(D2-A): track 0.00 -> 2.20 mm
- net /ClockBuffers/Heimtime_status: track 0.00 -> 2.14 mm
- net /ClockBuffers/MasterTrigger_status: track 0.00 -> 2.14 mm
- net 3V3: track 8.48 -> 9.69 mm, vias 9 -> 5
- net GND: vias 13 -> 96
- added copper zone on In1.Cu, net GND
Other:
- board text added: "H_t"
- board text added: "H_t_on"
- board text added: "M_t"
- board text added: "M_t_on"
- board text added: "Title: Clock Buffer AddOn Date/rev: 12.02.2025 REV_0 Author: Dr. Alexandru Enciu Institution: TU Darmstadt"

Commit message: .
Parts:
- added D10: SP1333-01UTG, Diode_SMD:D_0201_0603Metric, F.Cu at (103.4, 63.5)
- added D11: SP1333-01UTG, Diode_SMD:D_0201_0603Metric, F.Cu at (103.4, 53.1)
- added D13: SP1333-01UTG, Diode_SMD:D_0201_0603Metric, F.Cu at (103.6, 67.7)
- added D5: SP1333-01UTG, Diode_SMD:D_0201_0603Metric, F.Cu at (96.6, 56.1)
- added D6: SP1333-01UTG, Diode_SMD:D_0201_0603Metric, F.Cu at (96.6, 66.1)
- added D7: SP1333-01UTG, Diode_SMD:D_0201_0603Metric, F.Cu at (103.4, 57.2)
- added D8: SP1333-01UTG, Diode_SMD:D_0201_0603Metric, F.Cu at (104.5, 65.7)
- added D9: SP1333-01UTG, Diode_SMD:D_0201_0603Metric, F.Cu at (104.5, 55.0)
- D1: value LED -> LED_blue
- D2: value LED -> LED_yellow
- D3: value LED -> LED_red
Routing:
- net /ClockBuffers/Heimtime_out_2: track 11.0 -> 9.51 mm
- net GND: vias 96 -> 92

Commit message: .
Routing:
- net GND: vias 92 -> 91
Changed lines of the file:
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@@
 		(tags "diode")
 		(property "Reference" "D7"
-			(at 0 -1.05 360)
+			(at 0 -1.05 0)
 			(layer "F.SilkS")
 			(hide yes)
@@
 		)
 		(property "Value" "SP1333-01UTG"
-			(at 0 1.05 360)
+			(at 0 1.05 0)
 			(layer "F.Fab")
 			(effects
@@
 		)
 		(fp_text user "${REFERENCE}"
-			(at 0 -0.68 360)
+			(at 0 -0.68 0)
 			(layer "F.Fab")
 			(effects
@@
 		(tags "diode")
 		(property "Reference" "D10"
-			(at 0 -1.05 360)
+			(at 0 -1.05 0)
 			(layer "F.SilkS")
 			(hide yes)
@@
 		)
 		(property "Value" "SP1333-01UTG"
-			(at 0 1.05 360)
+			(at 0 1.05 0)
 			(layer "F.Fab")
 			(effects
@@
 		)
 		(fp_text user "${REFERENCE}"
-			(at 0 -0.68 360)
+			(at 0 -0.68 0)
 			(layer "F.Fab")
 			(effects
@@
 	)
 	(via
-		(at 92.45625 55.71)
-		(size 0.4)
-		(drill 0.25)
-		(layers "F.Cu" "B.Cu")
-		(free yes)
-		(net 1)
-	)
-	(via
 		(at 94.35625 57.02)
 		(size 0.4)
@@
 	)
 	(via
-		(at 92.45625 64.25)
+		(at 91.89625 64.75)
 		(size 0.4)
 		(drill 0.25)
@@
 	)
 	(zone
-		(net 4)
-		(net_name "/ClockBuffers/Heimtime_in")
+		(net 2)
+		(net_name "3V3")
 		(layer "F.Cu")
 		(name "$teardrop_padvia$")
 		(hatch full 0.1)
-		(priority 30001)
+		(priority 30004)
 		(attr
 			(teardrop
@@
 		(polygon
 			(pts
-				(xy 94.74625 65.6275) (xy 94.400061 65.5897) (xy 94.171907 65.489437) (xy 93.987462 65.346413) (xy 93.7724 65.180332)
-				(xy 93.452397 65.010896) (xy 93.14525 65.75) (xy 93.452397 66.489104) (xy 93.7724 66.319667) (xy 93.987462 66.153585)
-				(xy 94.171907 66.010562) (xy 94.400061 65.910299) (xy 94.74625 65.8725)
+				(xy 97.19625 55.07) (xy 97.19625 55.27) (xy 97.562674 55.439343) (xy 97.78725 55.17) (xy 97.562674 54.900657)
 			)
 		)
 	)
 	(zone
-		(net 3)
-		(net_name "/ClockBuffers/MasterTrigger_in")
+		(net 14)
+		(net_name "/ClockBuffers/Heimtime_out_2")
 		(layer "F.Cu")
 		(name "$teardrop_padvia$")
 		(hatch full 0.1)
-		(priority 30000)
+		(priority 30005)
 		(attr
 			(teardrop
@@
 		(polygon
 			(pts
-				(xy 94.74625 55.6275) (xy 94.400061 55.5897) (xy 94.171907 55.489437) (xy 93.987462 55.346413) (xy 93.7724 55.180332)
-				(xy 93.452397 55.010896) (xy 93.14525 55.75) (xy 93.452397 56.489104) (xy 93.7724 56.319667) (xy 93.987462 56.153585)
-				(xy 94.171907 56.010562) (xy 94.400061 55.910299) (xy 94.74625 55.8725)
+				(xy 104.73625 65.4725) (xy 104.885224 65.492592) (xy 104.987275 65.529907) (xy 105.13625 65.55)
+				(xy 105.13725 65.35) (xy 105.13625 65.15) (xy 104.987275 65.170092) (xy 104.885224 65.207407) (xy 104.73625 65.2275)
 			)
 		)
 	)
 	(zone
-		(net 2)
-		(net_name "3V3")
+		(net 4)
+		(net_name "/ClockBuffers/Heimtime_in")
 		(layer "F.Cu")
 		(name "$teardrop_padvia$")
 		(hatch full 0.1)
-		(priority 30003)
+		(priority 30001)
 		(attr
 			(teardrop
@@
 		(polygon
 			(pts
-				(xy 98.368293 65.45) (xy 98.368293 65.25) (xy 98.079918 64.967932) (xy 97.78525 65.17) (xy 97.743011 65.45)
+				(xy 94.74625 65.6275) (xy 94.400061 65.5897) (xy 94.171907 65.489437) (xy 93.987462 65.346413) (xy 93.7724 65.180332)
+				(xy 93.452397 65.010896) (xy 93.14525 65.75) (xy 93.452397 66.489104) (xy 93.7724 66.319667) (xy 93.987462 66.153585)
+				(xy 94.171907 66.010562) (xy 94.400061 65.910299) (xy 94.74625 65.8725)
 			)
 		)
@@
 		(name "$teardrop_padvia$")
 		(hatch full 0.1)
-		(priority 30002)
+		(priority 30007)
 		(attr
 			(teardrop
@@
 		(polygon
 			(pts
-				(xy 98.368293 55.45) (xy 98.368293 55.25) (xy 98.079918 54.967932) (xy 97.78525 55.17) (xy 97.743011 55.45)
+				(xy 97.48625 55.07) (xy 97.362406 55.062239) (xy 97.278145 55.035639) (xy 97.162787 54.985224) (xy 97.08525 55.17)
+				(xy 97.162787 55.354776) (xy 97.278145 55.30436) (xy 97.362406 55.27776) (xy 97.48625 55.27)
 			)
 		)
@@
 	)
 	(zone
-		(net 2)
-		(net_name "3V3")
+		(net 3)
+		(net_name "/ClockBuffers/MasterTrigger_in")
 		(layer "F.Cu")
 		(name "$teardrop_padvia$")
 		(hatch full 0.1)
-		(priority 30007)
+		(priority 30000)
 		(attr
 			(teardrop
@@
 		(polygon
 			(pts
-				(xy 97.48625 55.07) (xy 97.362406 55.062239) (xy 97.278145 55.035639) (xy 97.162787 54.985224) (xy 97.08525 55.17)
-				(xy 97.162787 55.354776) (xy 97.278145 55.30436) (xy 97.362406 55.27776) (xy 97.48625 55.27)
+				(xy 94.74625 55.6275) (xy 94.400061 55.5897) (xy 94.171907 55.489437) (xy 93.987462 55.346413) (xy 93.7724 55.180332)
+				(xy 93.452397 55.010896) (xy 93.14525 55.75) (xy 93.452397 56.489104) (xy 93.7724 56.319667) (xy 93.987462 56.153585)
+				(xy 94.171907 56.010562) (xy 94.400061 55.910299) (xy 94.74625 55.8725)
 			)
 		)
@@
 		(name "$teardrop_padvia$")
 		(hatch full 0.1)
-		(priority 30004)
+		(priority 30002)
 		(attr
 			(teardrop
@@
 		(polygon
 			(pts
-				(xy 97.19625 55.07) (xy 97.19625 55.27) (xy 97.562674 55.439343) (xy 97.78725 55.17) (xy 97.562674 54.900657)
+				(xy 98.368293 55.45) (xy 98.368293 55.25) (xy 98.079918 54.967932) (xy 97.78525 55.17) (xy 97.743011 55.45)
 			)
 		)
 	)
 	(zone
-		(net 14)
-		(net_name "/ClockBuffers/Heimtime_out_2")
+		(net 2)
+		(net_name "3V3")
 		(layer "F.Cu")
 		(name "$teardrop_padvia$")
 		(hatch full 0.1)
-		(priority 30005)
+		(priority 30003)
 		(attr
 			(teardrop
@@
 		(polygon
 			(pts
-				(xy 104.73625 65.4725) (xy 104.885224 65.492592) (xy 104.987275 65.529907) (xy 105.13625 65.55)
-				(xy 105.13725 65.35) (xy 105.13625 65.15) (xy 104.987275 65.170092) (xy 104.885224 65.207407) (xy 104.73625 65.2275)
+				(xy 98.368293 65.45) (xy 98.368293 65.25) (xy 98.079918 64.967932) (xy 97.78525 65.17) (xy 97.743011 65.45)
 			)
 		)

Commit message: .
Routing:
- net GND: vias 91 -> 101

Commit message: .
Parts:
- added REF**: KiCad-Logo2_5mm_SilkScreen, Symbol:KiCad-Logo2_5mm_SilkScreen, B.Cu at (101.4, 60.3)
Routing:
- net /ClockBuffers/Heimtime_out_2: track 9.51 -> 11.0 mm
- net GND: vias 101 -> 137
- added copper zone on In2.Cu, net GND
Other:
- board text added: "Title: Clock Buffer AddOn Date/rev: 25.02.2025 REV_1 Author: Dr. Alexandru Enciu Institution: TU Darmstadt"
- board text removed: "Title: Clock Buffer AddOn Date/rev: 12.02.2025 REV_0 Author: Dr. Alexandru Enciu Institution: TU Darmstadt"
