File: AddOns/Card_Adapter_Flex_AddOn/clock_buffer_4_outputs.kicad_sch (KiCad schematic)
At the start: 12 parts

Commit message: .
Parts:
- renumbered C to C1, C to C2, C to C3, R to R1, R to R2, R to R3, R to R4, U to U1
Changed lines of the file:
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@@
 		(on_board yes)
 		(dnp no)
-		(property "Reference" "R"
+		(property "Reference" "R4"
 			(at 172.212 94.488 90)
 			(effects
@@
 		(instances
 			(project "Card_Adapter_Flex_AddOn"
+				(path "/05374f14-0ccd-445f-8362-33aedd6aa709/88c7a278-827a-469b-946f-85b2017f4957"
+					(reference "R4")
+					(unit 1)
+				)
 				(path "/05374f14-0ccd-445f-8362-33aedd6aa709/c2fdd20f-7fee-47e0-99c8-8b435ae4c158"
 					(reference "R16")
@@
 		(on_board yes)
 		(dnp no)
-		(property "Reference" "R"
+		(property "Reference" "R2"
 			(at 160.782 100.33 90)
 			(effects
@@
 		(instances
 			(project "Card_Adapter_Flex_AddOn"
+				(path "/05374f14-0ccd-445f-8362-33aedd6aa709/88c7a278-827a-469b-946f-85b2017f4957"
+					(reference "R2")
+					(unit 1)
+				)
 				(path "/05374f14-0ccd-445f-8362-33aedd6aa709/c2fdd20f-7fee-47e0-99c8-8b435ae4c158"
 					(reference "R14")
@@
 		(on_board yes)
 		(dnp no)
-		(property "Reference" "R"
+		(property "Reference" "R3"
 			(at 165.862 96.266 90)
 			(effects
@@
 		(instances
 			(project "Card_Adapter_Flex_AddOn"
+				(path "/05374f14-0ccd-445f-8362-33aedd6aa709/88c7a278-827a-469b-946f-85b2017f4957"
+					(reference "R3")
+					(unit 1)
+				)
 				(path "/05374f14-0ccd-445f-8362-33aedd6aa709/c2fdd20f-7fee-47e0-99c8-8b435ae4c158"
 					(reference "R15")
@@
 		(on_board yes)
 		(dnp no)
-		(property "Reference" "C"
+		(property "Reference" "C1"
 			(at 76.962 91.694 0)
 			(effects
@@
 		(instances
 			(project "Card_Adapter_Flex_AddOn"
+				(path "/05374f14-0ccd-445f-8362-33aedd6aa709/88c7a278-827a-469b-946f-85b2017f4957"
+					(reference "C1")
+					(unit 1)
+				)
 				(path "/05374f14-0ccd-445f-8362-33aedd6aa709/c2fdd20f-7fee-47e0-99c8-8b435ae4c158"
 					(reference "C15")
@@
 		(on_board yes)
 		(dnp no)
-		(property "Reference" "U"
+		(property "Reference" "U1"
 			(at 142.24 80.518 0)
 			(effects
@@
 		(instances
 			(project "Card_Adapter_Flex_AddOn"
+				(path "/05374f14-0ccd-445f-8362-33aedd6aa709/88c7a278-827a-469b-946f-85b2017f4957"
+					(reference "U1")
+					(unit 1)
+				)
 				(path "/05374f14-0ccd-445f-8362-33aedd6aa709/c2fdd20f-7fee-47e0-99c8-8b435ae4c158"
 					(reference "U3")
@@
 		(on_board yes)
 		(dnp no)
-		(property "Reference" "R"
+		(property "Reference" "R1"
 			(at 154.432 101.346 90)
 			(effects
@@
 		(instances
 			(project "Card_Adapter_Flex_AddOn"
+				(path "/05374f14-0ccd-445f-8362-33aedd6aa709/88c7a278-827a-469b-946f-85b2017f4957"
+					(reference "R1")
+					(unit 1)
+				)
 				(path "/05374f14-0ccd-445f-8362-33aedd6aa709/c2fdd20f-7fee-47e0-99c8-8b435ae4c158"
 					(reference "R13")
@@
 		(on_board yes)
 		(dnp no)
-		(property "Reference" "C"
+		(property "Reference" "C3"
 			(at 94.742 91.694 0)
 			(effects
@@
 		(instances
 			(project "Card_Adapter_Flex_AddOn"
+				(path "/05374f14-0ccd-445f-8362-33aedd6aa709/88c7a278-827a-469b-946f-85b2017f4957"
+					(reference "C3")
+					(unit 1)
+				)
 				(path "/05374f14-0ccd-445f-8362-33aedd6aa709/c2fdd20f-7fee-47e0-99c8-8b435ae4c158"
 					(reference "C17")
@@
 		(on_board yes)
 		(dnp no)
-		(property "Reference" "C"
+		(property "Reference" "C2"
 			(at 85.852 91.694 0)
 			(effects
@@
 		(instances
 			(project "Card_Adapter_Flex_AddOn"
+				(path "/05374f14-0ccd-445f-8362-33aedd6aa709/88c7a278-827a-469b-946f-85b2017f4957"
+					(reference "C2")
+					(unit 1)
+				)
 				(path "/05374f14-0ccd-445f-8362-33aedd6aa709/c2fdd20f-7fee-47e0-99c8-8b435ae4c158"
 					(reference "C16")
