File: AddOns/Card_Adapter_Flex_AddOn/Card_Adapter_Flex_AddOn.kicad_pcb (KiCad board)
At the start: 4 copper layers, 57.4 x 27 mm, 28 parts, among them J1 17-pin-FPC, J2 4-pin-FPC, U2 5PB1214CMGK8, U3 5PB1214CMGK8

Commit message: .
Parts:
- renumbered C8 to C1, C10 to C2, C9 to C3, R10 to R1, R9 to R2, R8 to R3, R7 to R4, U2 to U1
Connections:
- C11 pad 2: unconnected-(C11-Pad2) -> Net-(U1-CLK_OUT1)
- C12 pad 2: unconnected-(C12-Pad2) -> Net-(U1-CLK_OUT2)
- C13 pad 2: unconnected-(C13-Pad2) -> Net-(U1-CLK_OUT3)
- C14 pad 2: unconnected-(C14-Pad2) -> Net-(U1-CLK_OUT4)
- J1 pad 3: unconnected-(J1-Pin_3-Pad3) -> GND
- R1 pad 2: unconnected-(C14-Pad2) -> Net-(U1-CLK_OUT4)
- R2 pad 2: unconnected-(C13-Pad2) -> Net-(U1-CLK_OUT3)
- R3 pad 2: unconnected-(C12-Pad2) -> Net-(U1-CLK_OUT2)
- R4 pad 2: unconnected-(C11-Pad2) -> Net-(U1-CLK_OUT1)
- U1 pad 10: unconnected-(C13-Pad2) -> Net-(U1-CLK_OUT3)
- U1 pad 11: unconnected-(C12-Pad2) -> Net-(U1-CLK_OUT2)
- U1 pad 13: unconnected-(C11-Pad2) -> Net-(U1-CLK_OUT1)
- U1 pad 8: unconnected-(C14-Pad2) -> Net-(U1-CLK_OUT4)
Routing:
- net unconnected-(C13-Pad2): track 3.25 -> 0.00 mm
- net Net-(U1-CLK_OUT3): track 0.00 -> 3.25 mm
- net unconnected-(C12-Pad2): track 3.23 -> 0.00 mm
- net Net-(U1-CLK_OUT2): track 0.00 -> 3.23 mm
- net unconnected-(C11-Pad2): track 2.38 -> 0.00 mm
- net Net-(U1-CLK_OUT1): track 0.00 -> 2.38 mm
- net unconnected-(C14-Pad2): track 2.34 -> 0.00 mm
- net Net-(U1-CLK_OUT4): track 0.00 -> 2.34 mm
- net unconnected-(J1-Pin_3-Pad3): track 1.47 -> 0.00 mm, vias 1 -> 0
- net GND: track 18.9 -> 20.1 mm, vias 30 -> 31
- net +3V3: vias 10 -> 11
Other:
- board text added: "3M 9077 Tape"
- board text added: "Title: Card Adapter Flex AddOn Rev_0 28.04.2025 Author: Alexandru Enciu Institution: TU Darmstadt"

Commit message: .
Routing:
- net GND: track 20.1 -> 16.2 mm, vias 31 -> 30
- net +3V3: track 5.44 -> 4.19 mm, vias 11 -> 10
- added copper zone on In1.Cu, net GND
