File: AddOns/2_In_6_Out_v2/FIFO.kicad_sch (KiCad schematic)
At the start: 12 parts, among them U2 5PB1213NTGK8, U4 5PB1213NTGK8

Commit message: .
Changed lines of the file:
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@@
 		(on_board yes)
 		(dnp no)
-		(fields_autoplaced yes)
 		(property "Reference" "C11"
-			(at 66.0399 60.96 0)
+			(at 67.818 60.96 90)
 			(effects
 				(font
@@
 		)
 		(property "Value" "10n"
-			(at 68.5799 60.96 0)
+			(at 72.136 63.754 90)
 			(effects
 				(font
@@
 		(dnp no)
 		(property "Reference" "C3"
-			(at 67.31 48.26 90)
-			(effects
-				(font
+			(at 67.31 51.816 90)
+			(effects
+				(font
