File: Spartan7_TriggerLogic/PSU_Stamp/Spartan7_PSU_Stamp_V0/TPS7A8801RTJT.kicad_sch (KiCad schematic)
At the start: 13 parts, among them U3 TPS7A8801RTJT

Commit message: Add status LEDs and update power nets
Added new 0402 LEDs (D1, D4) and supporting resistor (R12) for power-good status indication. Updated net assignments and replaced a capacitor footprint with an LED. Modified schematic and PCB files to reflect these changes.
Parts:
- R3: value R -> R_3
- R5: value R -> R_4
- R7: value R -> R_1
- R8: value R -> R_2
Other:
- note added: "For the feedback resistors: R_1, R_2, R_3, and R_4 see the TABLE_2"
Changed lines of the file:
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@@
 	(generator_version "9.0")
 	(paper "A4")
+	(rectangle
+		(start 176.53 40.64)
+		(end 187.96 105.41)
+		(stroke
+			(width 0.254)
+			(type dash)
+			(color 255 13 16 1)
+		)
+		(fill
+			(type none)
+		)
+	)
+	(text "For the feedback resistors:\nR_1, R_2, R_3, and R_4 see the TABLE_2"
+		(exclude_from_sim no)
+		(at 182.372 37.338 0)
+		(effects
+			(font
+				(size 1.27 1.27)
+				(thickness 0.254)
+				(bold yes)
+				(color 255 25 37 1)
+			)
+		)
+	)
 	(junction
 		(at 189.23 76.2)
@@
 		(on_board yes)
 		(dnp no)
-		(fields_autoplaced yes)
 		(property "Reference" "R8"
 			(at 184.15 67.3099 0)
@@
 			)
 		)
-		(property "Value" "R"
-			(at 184.15 69.8499 0)
+		(property "Value" "R_2"
+			(at 181.61 70.358 90)
 			(effects
 				(font
@@
 		(on_board yes)
 		(dnp no)
-		(fields_autoplaced yes)
 		(property "Reference" "R7"
 			(at 184.15 55.8799 0)
@@
 			)
 		)
-		(property "Value" "R"
-			(at 184.15 58.4199 0)
+		(property "Value" "R_1"
+			(at 181.61 58.928 90)
 			(effects
 				(font
@@
 		(on_board yes)
 		(dnp no)
-		(fields_autoplaced yes)
 		(property "Reference" "R5"
 			(at 184.15 96.5199 0)
@@
 			)
 		)
-		(property "Value" "R"
-			(at 184.15 99.0599 0)
+		(property "Value" "R_4"
+			(at 181.61 99.822 90)
 			(effects
 				(font
@@
 		(on_board yes)
 		(dnp no)
-		(fields_autoplaced yes)
 		(property "Reference" "R3"
 			(at 184.15 82.5499 0)
@@
 			)
 		)
-		(property "Value" "R"
-			(at 184.15 85.0899 0)
+		(property "Value" "R_3"
+			(at 181.61 85.598 90)
 			(effects
 				(font
