File: Spartan7_TriggerLogic/Spartan7_TriggerController/gnd.kicad_sch (KiCad schematic)
At the start: 1 part, among them U1 XC7S6-1FTGB196I

Commit message: .
Parts:
- U1: footprint (none) -> 0_lib:BGA196C100P14X14_1500X1500X155N
Changed lines of the file:
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@@
 			)
 		)
-		(property "Footprint" ""
+		(property "Footprint" "0_lib:BGA196C100P14X14_1500X1500X155N"
 			(at 140.97 58.42 0)
 			(effects
