File: Spartan7_TriggerLogic/Spartan7_TriggerController/Spartan7_TriggerController.kicad_pcb (KiCad board)
At the start: 2 copper layers, 5 parts

Commit message: m
Parts:
- removed REF** (x2): R_0201_0603Metric, Resistor_SMD:R_0201_0603Metric
- removed REF** (x2): C_0402_1005Metric, Capacitor_SMD:C_0402_1005Metric
Connections:
- U1 pad A10: unconnected-(U1D-IO_L3N_T0_DQS_EMCCLK_14-PadA10) -> (no net)
- U1 pad A12: unconnected-(U1D-IO_L4P_T0_D04_14-PadA12) -> (no net)
- U1 pad A13: unconnected-(U1D-IO_L4N_T0_D05_14-PadA13) -> (no net)
- U1 pad A2: unconnected-(U1E-IO_L3N_T0_DQS_34-PadA2) -> (no net)
- U1 pad A3: unconnected-(U1E-IO_L2N_T0_34-PadA3) -> (no net)
- U1 pad A4: unconnected-(U1E-IO_L2P_T0_34-PadA4) -> (no net)
- U1 pad A5: unconnected-(U1E-IO_L4N_T0_34-PadA5) -> (no net)
- U1 pad A7: unconnected-(U1C-TCK_0-PadA7) -> (no net)
- U1 pad A8: unconnected-(U1C-CCLK_0-PadA8) -> (no net)
- U1 pad B1: unconnected-(U1E-IO_L5N_T0_34-PadB1) -> (no net)
- U1 pad B10: unconnected-(U1D-IO_L3P_T0_DQS_PUDC_B_14-PadB10) -> (no net)
- U1 pad B11: unconnected-(U1D-IO_L1P_T0_D00_MOSI_14-PadB11) -> (no net)
- U1 pad B12: unconnected-(U1D-IO_L1N_T0_D01_DIN_14-PadB12) -> (no net)
- U1 pad B13: unconnected-(U1D-IO_L5P_T0_D06_14-PadB13) -> (no net)
- U1 pad B14: unconnected-(U1D-IO_L5N_T0_D07_14-PadB14) -> (no net)
- U1 pad B2: unconnected-(U1E-IO_L5P_T0_34-PadB2) -> (no net)
- U1 pad B3: unconnected-(U1E-IO_L3P_T0_DQS_34-PadB3) -> (no net)
- U1 pad B5: unconnected-(U1E-IO_L4P_T0_34-PadB5) -> (no net)
- U1 pad B6: unconnected-(U1E-IO_0_34-PadB6) -> (no net)
- U1 pad C1: unconnected-(U1E-IO_L11N_T1_SRCC_34-PadC1) -> (no net)
- U1 pad C10: unconnected-(U1D-IO_L2N_T0_D03_14-PadC10) -> (no net)
- U1 pad C11: unconnected-(U1D-IO_L6P_T0_FCS_B_14-PadC11) -> (no net)
- U1 pad C12: unconnected-(U1D-IO_L6N_T0_D08_VREF_14-PadC12) -> (no net)
- U1 pad C14: unconnected-(U1D-IO_L11N_T1_SRCC_14-PadC14) -> (no net)
- U1 pad C3: unconnected-(U1E-IO_L1N_T0_34-PadC3) -> (no net)
- U1 pad C4: unconnected-(U1E-IO_L6N_T0_VREF_34-PadC4) -> (no net)
- U1 pad C5: unconnected-(U1E-IO_L6P_T0_34-PadC5) -> (no net)
- U1 pad D1: unconnected-(U1E-IO_L11P_T1_SRCC_34-PadD1) -> (no net)
- U1 pad D10: unconnected-(U1D-IO_L2P_T0_D02_14-PadD10) -> (no net)
- U1 pad D12: unconnected-(U1D-IO_L8P_T1_D11_14-PadD12) -> (no net)
- U1 pad D13: unconnected-(U1D-IO_L8N_T1_D12_14-PadD13) -> (no net)
- U1 pad D14: unconnected-(U1D-IO_L11P_T1_SRCC_14-PadD14) -> (no net)
- U1 pad D2: unconnected-(U1E-IO_L10N_T1_34-PadD2) -> (no net)
- U1 pad D3: unconnected-(U1E-IO_L1P_T0_34-PadD3) -> (no net)
- U1 pad D4: unconnected-(U1E-IO_L7N_T1_34-PadD4) -> (no net)
- U1 pad D6: Net-(U1B-VCCINT-PadD6) -> unconnected-(U1B-VCCINT-PadD6)
- U1 pad D8: Net-(U1B-VCCINT-PadD6) -> unconnected-(U1B-VCCINT-PadD8)
- U1 pad E11: unconnected-(U1D-IO_0_14-PadE11) -> (no net)
- U1 pad E12: unconnected-(U1D-IO_L7N_T1_D10_14-PadE12) -> (no net)
- U1 pad E13: unconnected-(U1D-IO_L10N_T1_D15_14-PadE13) -> (no net)
- U1 pad E2: unconnected-(U1E-IO_L10P_T1_34-PadE2) -> (no net)
- U1 pad E4: unconnected-(U1E-IO_L7P_T1_34-PadE4) -> (no net)
- U1 pad E5: Net-(U1B-VCCBRAM-PadE5) -> unconnected-(U1B-VCCBRAM-PadE5)
- U1 pad E7: Net-(U1B-VCCINT-PadD6) -> unconnected-(U1B-VCCINT-PadE7)
- U1 pad E9: Net-(U1B-VCCINT-PadD6) -> unconnected-(U1B-VCCINT-PadE9)
- U1 pad F1: unconnected-(U1E-IO_L9N_T1_DQS_34-PadF1) -> (no net)
- U1 pad F10: Net-(U1B-VCCAUX-PadF10) -> unconnected-(U1B-VCCAUX-PadF10)
- U1 pad F11: unconnected-(U1D-IO_L12N_T1_MRCC_14-PadF11) -> (no net)
- U1 pad F12: unconnected-(U1D-IO_L7P_T1_D09_14-PadF12) -> (no net)
- U1 pad F13: unconnected-(U1D-IO_L10P_T1_D14_14-PadF13) -> (no net)
- U1 pad F14: unconnected-(U1D-IO_L9N_T1_DQS_D13_14-PadF14) -> (no net)
- U1 pad F2: unconnected-(U1E-IO_L8N_T1_34-PadF2) -> (no net)
- U1 pad F3: unconnected-(U1E-IO_L8P_T1_34-PadF3) -> (no net)
- U1 pad F4: unconnected-(U1E-IO_L12N_T1_MRCC_34-PadF4) -> (no net)
- U1 pad F6: Net-(U1B-VCCINT-PadD6) -> unconnected-(U1B-VCCINT-PadF6)
- U1 pad G1: unconnected-(U1E-IO_L9P_T1_DQS_34-PadG1) -> (no net)
- U1 pad G11: unconnected-(U1D-IO_L12P_T1_MRCC_14-PadG11) -> (no net)
- U1 pad G13: Net-(U1B-VCCO_14-PadG13) -> unconnected-(U1B-VCCO_14-PadG13)
- U1 pad G14: unconnected-(U1D-IO_L9P_T1_DQS_14-PadG14) -> (no net)
- U1 pad G2: Net-(U1B-VCCO_34-PadG2) -> unconnected-(U1B-VCCO_34-PadG2)
- U1 pad G4: unconnected-(U1E-IO_L12P_T1_MRCC_34-PadG4) -> (no net)
- U1 pad G5: Net-(U1B-VCCBRAM-PadE5) -> unconnected-(U1B-VCCBRAM-PadG5)
- U1 pad G9: Net-(U1B-VCCINT-PadD6) -> unconnected-(U1B-VCCINT-PadG9)
- U1 pad H1: unconnected-(U1E-IO_L14N_T2_SRCC_34-PadH1) -> (no net)
- U1 pad H10: Net-(U1B-VCCAUX-PadF10) -> unconnected-(U1B-VCCAUX-PadH10)
- U1 pad H11: unconnected-(U1D-IO_L13P_T2_MRCC_14-PadH11) -> (no net)
- U1 pad H12: unconnected-(U1D-IO_L13N_T2_MRCC_14-PadH12) -> (no net)
- U1 pad H13: unconnected-(U1D-IO_L14P_T2_SRCC_14-PadH13) -> (no net)
- U1 pad H14: unconnected-(U1D-IO_L14N_T2_SRCC_14-PadH14) -> (no net)
- U1 pad H2: unconnected-(U1E-IO_L14P_T2_SRCC_34-PadH2) -> (no net)
- U1 pad H3: unconnected-(U1E-IO_L13N_T2_MRCC_34-PadH3) -> (no net)
- U1 pad H4: unconnected-(U1E-IO_L13P_T2_MRCC_34-PadH4) -> (no net)
- U1 pad H6: Net-(U1B-VCCINT-PadD6) -> unconnected-(U1B-VCCINT-PadH6)
- U1 pad J1: unconnected-(U1E-IO_L15N_T2_DQS_34-PadJ1) -> (no net)
- U1 pad J11: unconnected-(U1D-IO_L17P_T2_D30_14-PadJ11) -> (no net)
- U1 pad J12: unconnected-(U1D-IO_L17N_T2_D29_14-PadJ12) -> (no net)
- U1 pad J13: unconnected-(U1D-IO_L18P_T2_D28_14-PadJ13) -> (no net)
- U1 pad J14: unconnected-(U1D-IO_L18N_T2_D27_14-PadJ14) -> (no net)
- U1 pad J2: unconnected-(U1E-IO_L15P_T2_DQS_34-PadJ2) -> (no net)
- U1 pad J3: unconnected-(U1E-IO_L17N_T2_34-PadJ3) -> (no net)
- U1 pad J4: unconnected-(U1E-IO_L17P_T2_34-PadJ4) -> (no net)
- U1 pad J5: Net-(U1B-VCCBRAM-PadE5) -> unconnected-(U1B-VCCBRAM-PadJ5)
- U1 pad J7: unconnected-(U1C-DXN_0-PadJ7) -> (no net)
- U1 pad J8: unconnected-(U1C-DXP_0-PadJ8) -> (no net)
- U1 pad J9: Net-(U1B-VCCINT-PadD6) -> unconnected-(U1B-VCCINT-PadJ9)
- U1 pad K10: Net-(U1B-VCCAUX-PadF10) -> unconnected-(U1B-VCCAUX-PadK10)
- U1 pad K11: unconnected-(U1D-IO_L19P_T3_D26_14-PadK11) -> (no net)
- U1 pad K12: unconnected-(U1D-IO_L19N_T3_D25_VREF_14-PadK12) -> (no net)
- U1 pad K13: Net-(U1B-VCCO_14-PadG13) -> unconnected-(U1B-VCCO_14-PadK13)
- U1 pad K2: Net-(U1B-VCCO_34-PadG2) -> unconnected-(U1B-VCCO_34-PadK2)
- U1 pad K3: unconnected-(U1E-IO_L16N_T2_34-PadK3) -> (no net)
- U1 pad K4: unconnected-(U1E-IO_L16P_T2_34-PadK4) -> (no net)
- U1 pad K6: Net-(U1B-VCCINT-PadD6) -> unconnected-(U1B-VCCINT-PadK6)
- U1 pad K8: Net-(U1B-VCCINT-PadD6) -> unconnected-(U1B-VCCINT-PadK8)
- U1 pad L1: unconnected-(U1E-IO_L18N_T2_34-PadL1) -> (no net)
- U1 pad L12: unconnected-(U1D-IO_L16P_T2_CSI_B_14-PadL12) -> (no net)
- U1 pad L13: unconnected-(U1D-IO_L16N_T2_D31_14-PadL13) -> (no net)
- U1 pad L14: unconnected-(U1D-IO_L15N_T2_DQS_DOUT_CSO_B_14-PadL14) -> (no net)
- U1 pad L2: unconnected-(U1E-IO_L22N_T3_34-PadL2) -> (no net)
- U1 pad L3: unconnected-(U1E-IO_L22P_T3_34-PadL3) -> (no net)
- U1 pad L5: unconnected-(U1E-IO_25_34-PadL5) -> (no net)
- U1 pad L7: unconnected-(U1C-PROGRAM_B_0-PadL7) -> (no net)
- U1 pad L9: Net-(U1B-VCCAUX-PadF10) -> unconnected-(U1B-VCCAUX-PadL9)
- U1 pad M1: unconnected-(U1E-IO_L18P_T2_34-PadM1) -> (no net)
- U1 pad M10: unconnected-(U1D-IO_25_14-PadM10) -> (no net)
- U1 pad M11: unconnected-(U1D-IO_L20P_T3_D24_14-PadM11) -> (no net)
- U1 pad M12: unconnected-(U1D-IO_L20N_T3_D23_14-PadM12) -> (no net)
- U1 pad M13: unconnected-(U1D-IO_L15P_T2_DQS_RDWR_B_14-PadM13) -> (no net)
- U1 pad M14: unconnected-(U1D-IO_L21N_T3_DQS_D22_14-PadM14) -> (no net)
- U1 pad M2: unconnected-(U1E-IO_L19N_T3_VREF_34-PadM2) -> (no net)
- U1 pad M3: unconnected-(U1E-IO_L19P_T3_34-PadM3) -> (no net)
- U1 pad M4: unconnected-(U1E-IO_L23N_T3_34-PadM4) -> (no net)
- U1 pad M5: unconnected-(U1E-IO_L23P_T3_34-PadM5) -> (no net)
- U1 pad M6: unconnected-(U1C-TMS_0-PadM6) -> (no net)
- U1 pad M7: unconnected-(U1C-M0_0-PadM7) -> (no net)
- U1 pad M8: unconnected-(U1C-M1_0-PadM8) -> (no net)
- U1 pad M9: unconnected-(U1C-M2_0-PadM9) -> (no net)
- U1 pad N1: unconnected-(U1E-IO_L20N_T3_34-PadN1) -> (no net)
- U1 pad N10: unconnected-(U1D-IO_L23P_T3_D19_14-PadN10) -> (no net)
- U1 pad N11: unconnected-(U1D-IO_L23N_T3_D18_14-PadN11) -> (no net)
- U1 pad N13: Net-(U1B-VCCO_14-PadG13) -> unconnected-(U1B-VCCO_14-PadN13)
- U1 pad N14: unconnected-(U1D-IO_L21P_T3_DQS_14-PadN14) -> (no net)
- U1 pad N2: Net-(U1B-VCCO_34-PadG2) -> unconnected-(U1B-VCCO_34-PadN2)
- U1 pad N4: unconnected-(U1E-IO_L24N_T3_34-PadN4) -> (no net)
- U1 pad N6: Net-(U1B-VCCO_0-PadN6) -> unconnected-(U1B-VCCO_0-PadN6)
- U1 pad N7: unconnected-(U1C-CFGBVS_0-PadN7) -> (no net)
- U1 pad N8: Net-(U1B-VCCO_0-PadN6) -> unconnected-(U1B-VCCO_0-PadN8)
- U1 pad P10: unconnected-(U1D-IO_L24P_T3_D17_14-PadP10) -> (no net)
- U1 pad P11: unconnected-(U1D-IO_L24N_T3_D16_14-PadP11) -> (no net)
- U1 pad P12: unconnected-(U1D-IO_L22P_T3_D21_14-PadP12) -> (no net)
- U1 pad P13: unconnected-(U1D-IO_L22N_T3_D20_14-PadP13) -> (no net)
- U1 pad P2: unconnected-(U1E-IO_L20P_T3_34-PadP2) -> (no net)
- U1 pad P3: unconnected-(U1E-IO_L21N_T3_DQS_34-PadP3) -> (no net)
- U1 pad P4: unconnected-(U1E-IO_L21P_T3_DQS_34-PadP4) -> (no net)
- U1 pad P5: unconnected-(U1E-IO_L24P_T3_34-PadP5) -> (no net)
- U1 pad P6: unconnected-(U1C-TDO_0-PadP6) -> (no net)
- U1 pad P7: unconnected-(U1C-TDI_0-PadP7) -> (no net)
- U1 pad P8: unconnected-(U1C-INIT_B_0-PadP8) -> (no net)
- U1 pad P9: unconnected-(U1C-DONE_0-PadP9) -> (no net)
Routing:
- net Net-(U1B-VCCO_34-PadG2): track 9.90 -> 0.00 mm
- net unconnected-(U1E-IO_L14P_T2_SRCC_34-PadH2): track 5.06 -> 0.00 mm
- net unconnected-(U1E-IO_L1N_T0_34-PadC3): track 4.89 -> 0.00 mm
- net unconnected-(U1E-IO_L8N_T1_34-PadF2): track 4.41 -> 0.00 mm
- net unconnected-(U1E-IO_L10P_T1_34-PadE2): track 4.06 -> 0.00 mm
- net unconnected-(U1E-IO_L5P_T0_34-PadB2): track 3.84 -> 0.00 mm
- net unconnected-(U1E-IO_L3N_T0_DQS_34-PadA2): track 3.80 -> 0.00 mm
- net unconnected-(U1E-IO_L19N_T3_VREF_34-PadM2): track 3.46 -> 0.00 mm
- net unconnected-(U1E-IO_L22N_T3_34-PadL2): track 3.32 -> 0.00 mm
- net unconnected-(U1E-IO_L20P_T3_34-PadP2): track 3.25 -> 0.00 mm
- net unconnected-(U1E-IO_L10N_T1_34-PadD2): track 3.15 -> 0.00 mm
- net unconnected-(U1E-IO_L14N_T2_SRCC_34-PadH1): track 3.10 -> 0.00 mm
- net unconnected-(U1E-IO_L11P_T1_SRCC_34-PadD1): track 2.77 -> 0.00 mm
- net unconnected-(U1E-IO_L15P_T2_DQS_34-PadJ2): track 2.64 -> 0.00 mm
- net unconnected-(U1E-IO_L11N_T1_SRCC_34-PadC1): track 2.58 -> 0.00 mm
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
Commit message: .
Parts:
- added J1: For_Catellated_holes, Connector_PinHeader_2.54mm:PinHeader_1x09_P2.54mm_Vertical, F.Cu at (131.5, 114.0)
- added J2: For_Catellated_holes, Connector_PinHeader_2.54mm:PinHeader_1x11_P2.54mm_Vertical, F.Cu at (129.6, 117.5)
- added J3: For_Catellated_holes, Connector_PinHeader_2.54mm:PinHeader_1x11_P2.54mm_Vertical, F.Cu at (153.6, 117.5)
- added REF**1: SAMTEC_MCX-J-P-X-RA-SM1, 0_lib:SAMTEC_MCX-J-P-X-RA-SM1, F.Cu at (124.7, 98.4)
- added REF**1: SAMTEC_MCX-J-P-X-RA-SM1, 0_lib:SAMTEC_MCX-J-P-X-RA-SM1, F.Cu at (156.9, 76.5)
- added REF**16: SAMTEC_MCX-J-P-X-RA-SM1, 0_lib:SAMTEC_MCX-J-P-X-RA-SM1, F.Cu at (103.1, 76.8)
- added REF**16: SAMTEC_MCX-J-P-X-RA-SM1, 0_lib:SAMTEC_MCX-J-P-X-RA-SM1, F.Cu at (178.4, 98.0)
- added REF**17: SAMTEC_MCX-J-P-X-RA-SM1, 0_lib:SAMTEC_MCX-J-P-X-RA-SM1, F.Cu at (110.3, 76.8)
- added REF**17: SAMTEC_MCX-J-P-X-RA-SM1, 0_lib:SAMTEC_MCX-J-P-X-RA-SM1, F.Cu at (171.2, 98.0)
- added REF**18: SAMTEC_MCX-J-P-X-RA-SM1, 0_lib:SAMTEC_MCX-J-P-X-RA-SM1, F.Cu at (164.0, 98.0)
- added REF**18: SAMTEC_MCX-J-P-X-RA-SM1, 0_lib:SAMTEC_MCX-J-P-X-RA-SM1, F.Cu at (117.5, 76.8)
- added REF**19: SAMTEC_MCX-J-P-X-RA-SM1, 0_lib:SAMTEC_MCX-J-P-X-RA-SM1, F.Cu at (156.9, 98.0)
- added REF**19: SAMTEC_MCX-J-P-X-RA-SM1, 0_lib:SAMTEC_MCX-J-P-X-RA-SM1, F.Cu at (124.7, 76.8)
- added REF**20: SAMTEC_MCX-J-P-X-RA-SM1, 0_lib:SAMTEC_MCX-J-P-X-RA-SM1, F.Cu at (178.4, 90.8)
- added REF**20: SAMTEC_MCX-J-P-X-RA-SM1, 0_lib:SAMTEC_MCX-J-P-X-RA-SM1, F.Cu at (103.1, 84.0)
- added REF**21: SAMTEC_MCX-J-P-X-RA-SM1, 0_lib:SAMTEC_MCX-J-P-X-RA-SM1, F.Cu at (110.3, 84.0)
- added REF**21: SAMTEC_MCX-J-P-X-RA-SM1, 0_lib:SAMTEC_MCX-J-P-X-RA-SM1, F.Cu at (171.2, 90.8)
- added REF**22: SAMTEC_MCX-J-P-X-RA-SM1, 0_lib:SAMTEC_MCX-J-P-X-RA-SM1, F.Cu at (117.5, 84.0)
- added REF**22: SAMTEC_MCX-J-P-X-RA-SM1, 0_lib:SAMTEC_MCX-J-P-X-RA-SM1, F.Cu at (164.0, 90.8)
- added REF**23: SAMTEC_MCX-J-P-X-RA-SM1, 0_lib:SAMTEC_MCX-J-P-X-RA-SM1, F.Cu at (124.7, 84.0)
- added REF**23: SAMTEC_MCX-J-P-X-RA-SM1, 0_lib:SAMTEC_MCX-J-P-X-RA-SM1, F.Cu at (156.9, 90.8)
- added REF**24: SAMTEC_MCX-J-P-X-RA-SM1, 0_lib:SAMTEC_MCX-J-P-X-RA-SM1, F.Cu at (178.4, 83.7)
- added REF**24: SAMTEC_MCX-J-P-X-RA-SM1, 0_lib:SAMTEC_MCX-J-P-X-RA-SM1, F.Cu at (103.1, 91.2)
- added REF**25: SAMTEC_MCX-J-P-X-RA-SM1, 0_lib:SAMTEC_MCX-J-P-X-RA-SM1, F.Cu at (110.3, 91.2)
- added REF**25: SAMTEC_MCX-J-P-X-RA-SM1, 0_lib:SAMTEC_MCX-J-P-X-RA-SM1, F.Cu at (171.2, 83.7)
- added REF**26: SAMTEC_MCX-J-P-X-RA-SM1, 0_lib:SAMTEC_MCX-J-P-X-RA-SM1, F.Cu at (117.5, 91.2)
- added REF**26: SAMTEC_MCX-J-P-X-RA-SM1, 0_lib:SAMTEC_MCX-J-P-X-RA-SM1, F.Cu at (164.0, 83.7)
- added REF**27: SAMTEC_MCX-J-P-X-RA-SM1, 0_lib:SAMTEC_MCX-J-P-X-RA-SM1, F.Cu at (156.9, 83.7)
- added REF**27: SAMTEC_MCX-J-P-X-RA-SM1, 0_lib:SAMTEC_MCX-J-P-X-RA-SM1, F.Cu at (124.7, 91.2)
- added REF**28: SAMTEC_MCX-J-P-X-RA-SM1, 0_lib:SAMTEC_MCX-J-P-X-RA-SM1, F.Cu at (178.4, 76.5)
- added REF**28: SAMTEC_MCX-J-P-X-RA-SM1, 0_lib:SAMTEC_MCX-J-P-X-RA-SM1, F.Cu at (103.1, 98.4)
- added REF**29: SAMTEC_MCX-J-P-X-RA-SM1, 0_lib:SAMTEC_MCX-J-P-X-RA-SM1, F.Cu at (171.2, 76.5)
- added REF**29: SAMTEC_MCX-J-P-X-RA-SM1, 0_lib:SAMTEC_MCX-J-P-X-RA-SM1, F.Cu at (110.3, 98.4)
- added REF**30: SAMTEC_MCX-J-P-X-RA-SM1, 0_lib:SAMTEC_MCX-J-P-X-RA-SM1, F.Cu at (164.0, 76.5)
- added REF**30: SAMTEC_MCX-J-P-X-RA-SM1, 0_lib:SAMTEC_MCX-J-P-X-RA-SM1, F.Cu at (117.5, 98.4)
- U1: value ~ -> XC7S6-1FTGB196I
Connections:
- U1 pad D6: unconnected-(U1B-VCCINT-PadD6) -> VCCINT&VCCBRAM
- U1 pad D8: unconnected-(U1B-VCCINT-PadD8) -> VCCINT&VCCBRAM
- U1 pad E5: unconnected-(U1B-VCCBRAM-PadE5) -> VCCINT&VCCBRAM
- U1 pad E7: unconnected-(U1B-VCCINT-PadE7) -> VCCINT&VCCBRAM
- U1 pad E9: unconnected-(U1B-VCCINT-PadE9) -> VCCINT&VCCBRAM
- U1 pad F10: unconnected-(U1B-VCCAUX-PadF10) -> VCCAUX
- U1 pad F6: unconnected-(U1B-VCCINT-PadF6) -> VCCINT&VCCBRAM
- U1 pad G13: unconnected-(U1B-VCCO_14-PadG13) -> VCCO_14&VCCO_34
- U1 pad G2: unconnected-(U1B-VCCO_34-PadG2) -> VCCO_14&VCCO_34
- U1 pad G5: unconnected-(U1B-VCCBRAM-PadG5) -> VCCINT&VCCBRAM
- U1 pad G9: unconnected-(U1B-VCCINT-PadG9) -> VCCINT&VCCBRAM
- U1 pad H10: unconnected-(U1B-VCCAUX-PadH10) -> VCCAUX
- U1 pad H6: unconnected-(U1B-VCCINT-PadH6) -> VCCINT&VCCBRAM
- U1 pad J5: unconnected-(U1B-VCCBRAM-PadJ5) -> VCCINT&VCCBRAM
- U1 pad J9: unconnected-(U1B-VCCINT-PadJ9) -> VCCINT&VCCBRAM
- U1 pad K10: unconnected-(U1B-VCCAUX-PadK10) -> VCCAUX
- U1 pad K13: unconnected-(U1B-VCCO_14-PadK13) -> VCCO_14&VCCO_34
- U1 pad K2: unconnected-(U1B-VCCO_34-PadK2) -> VCCO_14&VCCO_34
- U1 pad K6: unconnected-(U1B-VCCINT-PadK6) -> VCCINT&VCCBRAM
- U1 pad K8: unconnected-(U1B-VCCINT-PadK8) -> VCCINT&VCCBRAM
- U1 pad L9: unconnected-(U1B-VCCAUX-PadL9) -> VCCAUX
- U1 pad N13: unconnected-(U1B-VCCO_14-PadN13) -> VCCO_14&VCCO_34
- U1 pad N2: unconnected-(U1B-VCCO_34-PadN2) -> VCCO_14&VCCO_34
- U1 pad N6: unconnected-(U1B-VCCO_0-PadN6) -> VCCO_0
- U1 pad N8: unconnected-(U1B-VCCO_0-PadN8) -> VCCO_0
Routing:
- net VCCO_14&VCCO_34: vias 0 -> 6
- net VCCO_0: vias 0 -> 2
- added copper zone on F.Cu, net GND
Other:
- board outline added: 94 x 75.9 mm

Commit message: .
Parts:
- removed REF**1 (x2), REF**16 (x2), REF**17 (x2), REF**18 (x2), REF**19 (x2), REF**20 (x2), REF**21 (x2), REF**22 (x2), REF**23 (x2), REF**24 (x2), REF**25 (x2), REF**26 (x2), REF**27 (x2), REF**28 (x2), REF**29 (x2), REF**30 (x2): SAMTEC_MCX-J-P-X-RA-SM1, 0_lib:SAMTEC_MCX-J-P-X-RA-SM1
- added C1: 470nF, Capacitor_SMD:C_0402_1005Metric, B.Cu at (140.1, 92.1)
- added C10: 470nF, Capacitor_SMD:C_0402_1005Metric, B.Cu at (144.1, 88.0)
- added C11: 47uF, Capacitor_SMD:C_1210_3225Metric, B.Cu at (143.3, 108.5)
- added C12: 4.7uF, Capacitor_SMD:C_0603_1608Metric, B.Cu at (139.5, 100.1)
- added C13: 4.7uF, Capacitor_SMD:C_0603_1608Metric, B.Cu at (139.5, 98.6)
- added C14: 470nF, Capacitor_SMD:C_0402_1005Metric, B.Cu at (139.6, 94.5)
- added C15: 470nF, Capacitor_SMD:C_0402_1005Metric, B.Cu at (139.6, 96.2)
- added C16: 470nF, Capacitor_SMD:C_0402_1005Metric, B.Cu at (141.1, 95.2)
- added C17: 470nF, Capacitor_SMD:C_0402_1005Metric, B.Cu at (142.6, 94.6)
- added C18: 47uF, Capacitor_SMD:C_1210_3225Metric, B.Cu at (134.4, 109.7)
- added C19: 4.7uF, Capacitor_SMD:C_0603_1608Metric, B.Cu at (148.4, 93.0)
- added C2: 4.7uF, Capacitor_SMD:C_0603_1608Metric, B.Cu at (140.9, 90.4)
- added C20: 4.7uF, Capacitor_SMD:C_0603_1608Metric, B.Cu at (145.8, 85.5)
- added C21: 470nF, Capacitor_SMD:C_0402_1005Metric, B.Cu at (147.7, 95.0)
- added C22: 470nF, Capacitor_SMD:C_0402_1005Metric, B.Cu at (147.7, 91.5)
- added C23: 470nF, Capacitor_SMD:C_0402_1005Metric, B.Cu at (146.6, 88.5)
- added C24: 470nF, Capacitor_SMD:C_0402_1005Metric, B.Cu at (147.7, 86.8)
- added C25: 47uF, Capacitor_SMD:C_1210_3225Metric, B.Cu at (134.4, 106.5)
- added C26: 4.7uF, Capacitor_SMD:C_0603_1608Metric, B.Cu at (137.2, 93.6)
- added C27: 4.7uF, Capacitor_SMD:C_0603_1608Metric, B.Cu at (136.8, 84.5)
- added C28: 470nF, Capacitor_SMD:C_0402_1005Metric, B.Cu at (136.7, 86.5)
- added C29: 470nF, Capacitor_SMD:C_0402_1005Metric, B.Cu at (136.6, 88.5)
- added C3: 47uF, Capacitor_SMD:C_1210_3225Metric, B.Cu at (146.9, 104.8)
- added C30: 470nF, Capacitor_SMD:C_0402_1005Metric, B.Cu at (135.6, 91.5)
- added C31: 470nF, Capacitor_SMD:C_0402_1005Metric, B.Cu at (135.8, 94.8)
- added C4: 47uF, Capacitor_SMD:C_1210_3225Metric, B.Cu at (148.3, 109.4)
- added C5: 4.7uF, Capacitor_SMD:C_0603_1608Metric, B.Cu at (140.9, 88.5)
- added C6: 470nF, Capacitor_SMD:C_0402_1005Metric, B.Cu at (141.6, 86.5)
- added C7: 47uF, Capacitor_SMD:C_1210_3225Metric, B.Cu at (153.5, 106.1)
- added C8: 4.7uF, Capacitor_SMD:C_0603_1608Metric, B.Cu at (146.4, 96.6)
- added C9: 470nF, Capacitor_SMD:C_0402_1005Metric, B.Cu at (144.8, 92.1)
Routing:
- net GND: track 0.00 -> 0.94 mm, vias 49 -> 385
- net VCCO_14&VCCO_34: vias 6 -> 18
- net VCCO_0: vias 2 -> 14
- net VCCINT&VCCBRAM: vias 0 -> 25
- net VCCAUX: vias 0 -> 16
- added copper zone on In1.Cu, net GND
- added copper zone on In3.Cu, net GND
- added copper zone on In4.Cu, net GND
- added copper zone on B.Cu, net VCCAUX
- added copper zone on B.Cu, net VCCINT&VCCBRAM
- added copper zone on B.Cu, net VCCO_0
- added copper zone on B.Cu, net VCCO_14&VCCO_34
- removed copper zone on B.Cu, net GND
- removed copper zone on F.Cu, net GND
Other:
- board size 94 x 75.9 mm -> 93.2 x 75.9 mm
- copper layers 2 -> 6

Commit message: .
Parts:
- added C32: 470nF, Capacitor_SMD:C_0402_1005Metric, F.Cu at (140.5, 76.4)
- added C33: 100nF, Capacitor_SMD:C_0402_1005Metric, F.Cu at (139.5, 76.4)
- added C34: 470nF, Capacitor_SMD:C_0402_1005Metric, B.Cu at (136.7, 68.9)
- added C35: 4.7uF, Capacitor_SMD:C_0603_1608Metric, B.Cu at (138.5, 70.3)
- added C36: 470nF, Capacitor_SMD:C_0402_1005Metric, B.Cu at (136.7, 67.9)
- added D1: BAT54S, Package_TO_SOT_SMD:SOT-23, F.Cu at (137.1, 72.5)
- added D2: BAT54S, Package_TO_SOT_SMD:SOT-23, F.Cu at (133.5, 75.4)
- added D3: BAT54S, Package_TO_SOT_SMD:SOT-23, F.Cu at (127.7, 75.4)
- added D4: BAT54S, Package_TO_SOT_SMD:SOT-23, F.Cu at (124.2, 72.5)
- added J4: 878321422, 0_lib:CONN14_878321422_MOL, F.Cu at (129.6, 66.7)
- added R1: 0, Resistor_SMD:R_0402_1005Metric, F.Cu at (142.1, 79.5)
- added R10: 33, Resistor_SMD:R_0402_1005Metric, F.Cu at (129.6, 73.0)
- added R11: 33, Resistor_SMD:R_0402_1005Metric, F.Cu at (127.1, 72.5)
- added R12: 10k, Resistor_SMD:R_0402_1005Metric, F.Cu at (155.0, 93.1)
- added R13: 10k, Resistor_SMD:R_0402_1005Metric, F.Cu at (155.0, 95.7)
- added R14: 10k, Resistor_SMD:R_0402_1005Metric, F.Cu at (155.0, 98.2)
- added R15: 10k, Resistor_SMD:R_0402_1005Metric, F.Cu at (153.5, 93.6)
- added R16: 10k, Resistor_SMD:R_0402_1005Metric, F.Cu at (153.5, 96.2)
- added R17: 10k, Resistor_SMD:R_0402_1005Metric, F.Cu at (153.5, 98.7)
- added R2: 0, Resistor_SMD:R_0402_1005Metric, F.Cu at (149.6, 79.5)
- added R3: 10k, Resistor_SMD:R_0402_1005Metric, F.Cu at (148.7, 79.5)
- added R4: 0, Resistor_SMD:R_0402_1005Metric, F.Cu at (146.6, 79.5)
- added R5: 0, Resistor_SMD:R_0402_1005Metric, F.Cu at (145.6, 79.5)
- added R6: 0, Resistor_SMD:R_0402_1005Metric, F.Cu at (144.6, 79.5)
- added R7: 0, Resistor_SMD:R_0402_1005Metric, F.Cu at (143.6, 79.5)
- added R8: 33, Resistor_SMD:R_0402_1005Metric, F.Cu at (134.1, 72.5)
- added R9: 33, Resistor_SMD:R_0402_1005Metric, F.Cu at (131.6, 73.0)
- added REF**: CONN_EPY.00.250.NTN_LMO, 0_lib:CONN_EPY.00.250.NTN_LMO, F.Cu at (117.1, 139.0)
- added REF**: SAMTEC_MCX-J-P-X-RA-SM1, 0_lib:SAMTEC_MCX-J-P-X-RA-SM1, B.Cu at (82.2, 31.5)
- added REF**: CONN_EPY.00.250.NTN_LMO, 0_lib:CONN_EPY.00.250.NTN_LMO, F.Cu at (107.1, 139.0)
- added REF**: CONN_EPY.00.250.NTN_LMO, 0_lib:CONN_EPY.00.250.NTN_LMO, F.Cu at (162.4, 139.7)
- added REF**: CONN_EPY.00.250.NTN_LMO, 0_lib:CONN_EPY.00.250.NTN_LMO, F.Cu at (172.4, 139.7)
- added REF**: CONN_EPY.00.250.NTN_LMO, 0_lib:CONN_EPY.00.250.NTN_LMO, F.Cu at (87.3, 139.0)
- added REF**: CONN_EPY.00.250.NTN_LMO, 0_lib:CONN_EPY.00.250.NTN_LMO, F.Cu at (192.2, 139.7)
- added REF**: CONN_EPY.00.250.NTN_LMO, 0_lib:CONN_EPY.00.250.NTN_LMO, F.Cu at (97.2, 139.0)
- added REF**: SAMTEC_MCX-J-P-X-RA-SM1, 0_lib:SAMTEC_MCX-J-P-X-RA-SM1, F.Cu at (194.6, 31.6)
- added REF**: CONN_EPY.00.250.NTN_LMO, 0_lib:CONN_EPY.00.250.NTN_LMO, F.Cu at (182.3, 139.7)
- added REF**1: SAMTEC_MCX-J-P-X-RA-SM1, 0_lib:SAMTEC_MCX-J-P-X-RA-SM1, F.Cu at (82.1, 31.6)
- added REF**1: SAMTEC_MCX-J-P-X-RA-SM1, 0_lib:SAMTEC_MCX-J-P-X-RA-SM1, B.Cu at (194.7, 31.5)
- added REF**10: SAMTEC_MCX-J-P-X-RA-SM1, 0_lib:SAMTEC_MCX-J-P-X-RA-SM1, F.Cu at (149.6, 31.6)
- added REF**10: SAMTEC_MCX-J-P-X-RA-SM1, 0_lib:SAMTEC_MCX-J-P-X-RA-SM1, B.Cu at (127.2, 31.5)
- added REF**11: SAMTEC_MCX-J-P-X-RA-SM1, 0_lib:SAMTEC_MCX-J-P-X-RA-SM1, F.Cu at (157.1, 31.6)
- added REF**11: SAMTEC_MCX-J-P-X-RA-SM1, 0_lib:SAMTEC_MCX-J-P-X-RA-SM1, B.Cu at (119.7, 31.5)
- added REF**12: SAMTEC_MCX-J-P-X-RA-SM1, 0_lib:SAMTEC_MCX-J-P-X-RA-SM1, F.Cu at (164.6, 31.6)
- added REF**12: SAMTEC_MCX-J-P-X-RA-SM1, 0_lib:SAMTEC_MCX-J-P-X-RA-SM1, B.Cu at (112.2, 31.5)
- added REF**13: SAMTEC_MCX-J-P-X-RA-SM1, 0_lib:SAMTEC_MCX-J-P-X-RA-SM1, F.Cu at (172.1, 31.6)
- added REF**13: SAMTEC_MCX-J-P-X-RA-SM1, 0_lib:SAMTEC_MCX-J-P-X-RA-SM1, B.Cu at (104.7, 31.5)
- added REF**14: SAMTEC_MCX-J-P-X-RA-SM1, 0_lib:SAMTEC_MCX-J-P-X-RA-SM1, F.Cu at (179.6, 31.6)
- added REF**14: SAMTEC_MCX-J-P-X-RA-SM1, 0_lib:SAMTEC_MCX-J-P-X-RA-SM1, B.Cu at (97.2, 31.5)
- added REF**15: SAMTEC_MCX-J-P-X-RA-SM1, 0_lib:SAMTEC_MCX-J-P-X-RA-SM1, F.Cu at (187.1, 31.6)
- added REF**15: SAMTEC_MCX-J-P-X-RA-SM1, 0_lib:SAMTEC_MCX-J-P-X-RA-SM1, B.Cu at (89.7, 31.5)
- added REF**2: SAMTEC_MCX-J-P-X-RA-SM1, 0_lib:SAMTEC_MCX-J-P-X-RA-SM1, F.Cu at (89.6, 31.6)
- added REF**2: SAMTEC_MCX-J-P-X-RA-SM1, 0_lib:SAMTEC_MCX-J-P-X-RA-SM1, B.Cu at (187.2, 31.5)
- added REF**3: SAMTEC_MCX-J-P-X-RA-SM1, 0_lib:SAMTEC_MCX-J-P-X-RA-SM1, F.Cu at (97.1, 31.6)
- added REF**3: SAMTEC_MCX-J-P-X-RA-SM1, 0_lib:SAMTEC_MCX-J-P-X-RA-SM1, B.Cu at (179.7, 31.5)
- added REF**4: SAMTEC_MCX-J-P-X-RA-SM1, 0_lib:SAMTEC_MCX-J-P-X-RA-SM1, F.Cu at (104.6, 31.6)
- added REF**4: SAMTEC_MCX-J-P-X-RA-SM1, 0_lib:SAMTEC_MCX-J-P-X-RA-SM1, B.Cu at (172.2, 31.5)
- added REF**5: SAMTEC_MCX-J-P-X-RA-SM1, 0_lib:SAMTEC_MCX-J-P-X-RA-SM1, F.Cu at (112.1, 31.6)
- added REF**5: SAMTEC_MCX-J-P-X-RA-SM1, 0_lib:SAMTEC_MCX-J-P-X-RA-SM1, B.Cu at (164.7, 31.5)
- added REF**6: SAMTEC_MCX-J-P-X-RA-SM1, 0_lib:SAMTEC_MCX-J-P-X-RA-SM1, F.Cu at (119.6, 31.6)
- added REF**6: SAMTEC_MCX-J-P-X-RA-SM1, 0_lib:SAMTEC_MCX-J-P-X-RA-SM1, B.Cu at (157.2, 31.5)
- added REF**7: SAMTEC_MCX-J-P-X-RA-SM1, 0_lib:SAMTEC_MCX-J-P-X-RA-SM1, F.Cu at (127.1, 31.6)
- added REF**7: SAMTEC_MCX-J-P-X-RA-SM1, 0_lib:SAMTEC_MCX-J-P-X-RA-SM1, B.Cu at (149.7, 31.5)
- added REF**8: SAMTEC_MCX-J-P-X-RA-SM1, 0_lib:SAMTEC_MCX-J-P-X-RA-SM1, F.Cu at (134.6, 31.6)
- added REF**8: SAMTEC_MCX-J-P-X-RA-SM1, 0_lib:SAMTEC_MCX-J-P-X-RA-SM1, B.Cu at (142.2, 31.5)
- added REF**9: SAMTEC_MCX-J-P-X-RA-SM1, 0_lib:SAMTEC_MCX-J-P-X-RA-SM1, F.Cu at (142.1, 31.6)
- added REF**9: SAMTEC_MCX-J-P-X-RA-SM1, 0_lib:SAMTEC_MCX-J-P-X-RA-SM1, B.Cu at (134.7, 31.5)
- added SW1: SW_DIP_x03, Button_Switch_SMD:SW_DIP_SPSTx03_Slide_6.7x9.18mm_W6.73mm_P2.54mm_LowProfile_JPin, F.Cu at (160.3, 96.2)
- added U2: IS25LP256D-JLLE, 0_lib:WSON_6D-JLLE_ISI, F.Cu at (145.6, 74.0)
- moved C16 1.40 mm to (141.1, 96.6)
Connections:
- U1 pad A10: (no net) -> unconnected-(U1D-IO_L3N_T0_DQS_EMCCLK_14-PadA10)
- U1 pad A12: (no net) -> unconnected-(U1D-IO_L4P_T0_D04_14-PadA12)
- U1 pad A13: (no net) -> unconnected-(U1D-IO_L4N_T0_D05_14-PadA13)
- U1 pad A2: (no net) -> unconnected-(U1E-IO_L3N_T0_DQS_34-PadA2)
- U1 pad A3: (no net) -> unconnected-(U1E-IO_L2N_T0_34-PadA3)
- U1 pad A4: (no net) -> unconnected-(U1E-IO_L2P_T0_34-PadA4)
- U1 pad A5: (no net) -> unconnected-(U1E-IO_L4N_T0_34-PadA5)
- U1 pad A6: (no net) -> GND
- U1 pad A7: (no net) -> /JTAG/TCK
- U1 pad A8: (no net) -> /QSPI/QSPI_SCK
- U1 pad B1: (no net) -> unconnected-(U1E-IO_L5N_T0_34-PadB1)
- U1 pad B10: (no net) -> unconnected-(U1D-IO_L3P_T0_DQS_PUDC_B_14-PadB10)
- U1 pad B11: (no net) -> /QSPI/QSPI_IO_0
- U1 pad B12: (no net) -> /QSPI/QSPI_IO_1
- U1 pad B13: (no net) -> unconnected-(U1D-IO_L5P_T0_D06_14-PadB13)
- U1 pad B14: (no net) -> unconnected-(U1D-IO_L5N_T0_D07_14-PadB14)
- U1 pad B2: (no net) -> unconnected-(U1E-IO_L5P_T0_34-PadB2)
- U1 pad B3: (no net) -> unconnected-(U1E-IO_L3P_T0_DQS_34-PadB3)
- U1 pad B5: (no net) -> unconnected-(U1E-IO_L4P_T0_34-PadB5)
- U1 pad B6: (no net) -> unconnected-(U1E-IO_0_34-PadB6)
- U1 pad C1: (no net) -> unconnected-(U1E-IO_L11N_T1_SRCC_34-PadC1)
- U1 pad C10: (no net) -> /QSPI/QSPI_IO_3
- U1 pad C11: (no net) -> /QSPI/QSPI_CE_N
- U1 pad C12: (no net) -> unconnected-(U1D-IO_L6N_T0_D08_VREF_14-PadC12)
- U1 pad C14: (no net) -> unconnected-(U1D-IO_L11N_T1_SRCC_14-PadC14)
- U1 pad C3: (no net) -> unconnected-(U1E-IO_L1N_T0_34-PadC3)
- U1 pad C4: (no net) -> unconnected-(U1E-IO_L6N_T0_VREF_34-PadC4)
- U1 pad C5: (no net) -> unconnected-(U1E-IO_L6P_T0_34-PadC5)
- U1 pad D1: (no net) -> unconnected-(U1E-IO_L11P_T1_SRCC_34-PadD1)
- U1 pad D10: (no net) -> /QSPI/QSPI_IO_2
- U1 pad D12: (no net) -> unconnected-(U1D-IO_L8P_T1_D11_14-PadD12)
- U1 pad D13: (no net) -> unconnected-(U1D-IO_L8N_T1_D12_14-PadD13)
- U1 pad D14: (no net) -> unconnected-(U1D-IO_L11P_T1_SRCC_14-PadD14)
- U1 pad D2: (no net) -> unconnected-(U1E-IO_L10N_T1_34-PadD2)
- U1 pad D3: (no net) -> unconnected-(U1E-IO_L1P_T0_34-PadD3)
- U1 pad D4: (no net) -> unconnected-(U1E-IO_L7N_T1_34-PadD4)
- U1 pad E11: (no net) -> unconnected-(U1D-IO_0_14-PadE11)
- U1 pad E12: (no net) -> unconnected-(U1D-IO_L7N_T1_D10_14-PadE12)
- U1 pad E13: (no net) -> unconnected-(U1D-IO_L10N_T1_D15_14-PadE13)
- U1 pad E2: (no net) -> unconnected-(U1E-IO_L10P_T1_34-PadE2)
- U1 pad E4: (no net) -> unconnected-(U1E-IO_L7P_T1_34-PadE4)
- U1 pad F1: (no net) -> unconnected-(U1E-IO_L9N_T1_DQS_34-PadF1)
- U1 pad F11: (no net) -> unconnected-(U1D-IO_L12N_T1_MRCC_14-PadF11)
- U1 pad F12: (no net) -> unconnected-(U1D-IO_L7P_T1_D09_14-PadF12)
- U1 pad F13: (no net) -> unconnected-(U1D-IO_L10P_T1_D14_14-PadF13)
- U1 pad F14: (no net) -> unconnected-(U1D-IO_L9N_T1_DQS_D13_14-PadF14)
- U1 pad F2: (no net) -> unconnected-(U1E-IO_L8N_T1_34-PadF2)
- U1 pad F3: (no net) -> unconnected-(U1E-IO_L8P_T1_34-PadF3)
- U1 pad F4: (no net) -> unconnected-(U1E-IO_L12N_T1_MRCC_34-PadF4)
- U1 pad G1: (no net) -> unconnected-(U1E-IO_L9P_T1_DQS_34-PadG1)
- U1 pad G11: (no net) -> unconnected-(U1D-IO_L12P_T1_MRCC_14-PadG11)
- U1 pad G14: (no net) -> unconnected-(U1D-IO_L9P_T1_DQS_14-PadG14)
- U1 pad G4: (no net) -> unconnected-(U1E-IO_L12P_T1_MRCC_34-PadG4)
- U1 pad H1: (no net) -> unconnected-(U1E-IO_L14N_T2_SRCC_34-PadH1)
- U1 pad H11: (no net) -> unconnected-(U1D-IO_L13P_T2_MRCC_14-PadH11)
- U1 pad H12: (no net) -> unconnected-(U1D-IO_L13N_T2_MRCC_14-PadH12)
- U1 pad H13: (no net) -> unconnected-(U1D-IO_L14P_T2_SRCC_14-PadH13)
- U1 pad H14: (no net) -> unconnected-(U1D-IO_L14N_T2_SRCC_14-PadH14)
- U1 pad H2: (no net) -> unconnected-(U1E-IO_L14P_T2_SRCC_34-PadH2)
- U1 pad H3: (no net) -> unconnected-(U1E-IO_L13N_T2_MRCC_34-PadH3)
- U1 pad H4: (no net) -> unconnected-(U1E-IO_L13P_T2_MRCC_34-PadH4)
- U1 pad J1: (no net) -> unconnected-(U1E-IO_L15N_T2_DQS_34-PadJ1)
- U1 pad J11: (no net) -> unconnected-(U1D-IO_L17P_T2_D30_14-PadJ11)
- U1 pad J12: (no net) -> unconnected-(U1D-IO_L17N_T2_D29_14-PadJ12)
- U1 pad J13: (no net) -> unconnected-(U1D-IO_L18P_T2_D28_14-PadJ13)
- U1 pad J14: (no net) -> unconnected-(U1D-IO_L18N_T2_D27_14-PadJ14)
- U1 pad J2: (no net) -> unconnected-(U1E-IO_L15P_T2_DQS_34-PadJ2)
- U1 pad J3: (no net) -> unconnected-(U1E-IO_L17N_T2_34-PadJ3)
- U1 pad J4: (no net) -> unconnected-(U1E-IO_L17P_T2_34-PadJ4)
- U1 pad J7: (no net) -> unconnected-(U1C-DXN_0-PadJ7)
- U1 pad J8: (no net) -> unconnected-(U1C-DXP_0-PadJ8)
- U1 pad K11: (no net) -> unconnected-(U1D-IO_L19P_T3_D26_14-PadK11)
- U1 pad K12: (no net) -> unconnected-(U1D-IO_L19N_T3_D25_VREF_14-PadK12)
- U1 pad K3: (no net) -> unconnected-(U1E-IO_L16N_T2_34-PadK3)
- U1 pad K4: (no net) -> unconnected-(U1E-IO_L16P_T2_34-PadK4)
- U1 pad L1: (no net) -> unconnected-(U1E-IO_L18N_T2_34-PadL1)
- U1 pad L12: (no net) -> unconnected-(U1D-IO_L16P_T2_CSI_B_14-PadL12)
- U1 pad L13: (no net) -> unconnected-(U1D-IO_L16N_T2_D31_14-PadL13)
- U1 pad L14: (no net) -> unconnected-(U1D-IO_L15N_T2_DQS_DOUT_CSO_B_14-PadL14)
- U1 pad L2: (no net) -> unconnected-(U1E-IO_L22N_T3_34-PadL2)
- U1 pad L3: (no net) -> unconnected-(U1E-IO_L22P_T3_34-PadL3)
- U1 pad L5: (no net) -> unconnected-(U1E-IO_25_34-PadL5)
- U1 pad L7: (no net) -> unconnected-(U1C-PROGRAM_B_0-PadL7)
- U1 pad M1: (no net) -> unconnected-(U1E-IO_L18P_T2_34-PadM1)
- U1 pad M10: (no net) -> unconnected-(U1D-IO_25_14-PadM10)
- U1 pad M11: (no net) -> unconnected-(U1D-IO_L20P_T3_D24_14-PadM11)
- U1 pad M12: (no net) -> unconnected-(U1D-IO_L20N_T3_D23_14-PadM12)
- U1 pad M13: (no net) -> unconnected-(U1D-IO_L15P_T2_DQS_RDWR_B_14-PadM13)
- U1 pad M14: (no net) -> unconnected-(U1D-IO_L21N_T3_DQS_D22_14-PadM14)
- U1 pad M2: (no net) -> unconnected-(U1E-IO_L19N_T3_VREF_34-PadM2)
- U1 pad M3: (no net) -> unconnected-(U1E-IO_L19P_T3_34-PadM3)
- U1 pad M4: (no net) -> unconnected-(U1E-IO_L23N_T3_34-PadM4)
- U1 pad M5: (no net) -> unconnected-(U1E-IO_L23P_T3_34-PadM5)
- U1 pad M6: (no net) -> /JTAG/TMS
- U1 pad M7: (no net) -> /Boot_Mode/M0
- U1 pad M8: (no net) -> /Boot_Mode/M1
- U1 pad M9: (no net) -> /Boot_Mode/M2
- U1 pad N1: (no net) -> unconnected-(U1E-IO_L20N_T3_34-PadN1)
- U1 pad N10: (no net) -> unconnected-(U1D-IO_L23P_T3_D19_14-PadN10)
- U1 pad N11: (no net) -> unconnected-(U1D-IO_L23N_T3_D18_14-PadN11)
- U1 pad N14: (no net) -> unconnected-(U1D-IO_L21P_T3_DQS_14-PadN14)
- U1 pad N4: (no net) -> unconnected-(U1E-IO_L24N_T3_34-PadN4)
- U1 pad N7: (no net) -> unconnected-(U1C-CFGBVS_0-PadN7)
- U1 pad P10: (no net) -> unconnected-(U1D-IO_L24P_T3_D17_14-PadP10)
- U1 pad P11: (no net) -> unconnected-(U1D-IO_L24N_T3_D16_14-PadP11)
- U1 pad P12: (no net) -> unconnected-(U1D-IO_L22P_T3_D21_14-PadP12)
- U1 pad P13: (no net) -> unconnected-(U1D-IO_L22N_T3_D20_14-PadP13)
- U1 pad P2: (no net) -> unconnected-(U1E-IO_L20P_T3_34-PadP2)
- U1 pad P3: (no net) -> unconnected-(U1E-IO_L21N_T3_DQS_34-PadP3)
- U1 pad P4: (no net) -> unconnected-(U1E-IO_L21P_T3_DQS_34-PadP4)
- U1 pad P5: (no net) -> unconnected-(U1E-IO_L24P_T3_34-PadP5)
- U1 pad P6: (no net) -> /JTAG/TDO
- U1 pad P7: (no net) -> /JTAG/TDI
- U1 pad P8: (no net) -> unconnected-(U1C-INIT_B_0-PadP8)
- U1 pad P9: (no net) -> unconnected-(U1C-DONE_0-PadP9)
Routing:
- net /JTAG/TDI: track 0.00 -> 34.4 mm, vias 0 -> 1
- net /JTAG/TDO: track 0.00 -> 29.0 mm, vias 0 -> 1
- net /JTAG/TMS: track 0.00 -> 25.8 mm, vias 0 -> 1
- net /Boot_Mode/M0: track 0.00 -> 13.4 mm
- net /JTAG/TCK: track 0.00 -> 13.2 mm
- net /Boot_Mode/M1: track 0.00 -> 12.6 mm
- net /Boot_Mode/M2: track 0.00 -> 12.1 mm
- net Net-(U2-CE#): track 0.00 -> 10.9 mm
- net Net-(U2-SI_(IO0)): track 0.00 -> 8.62 mm, vias 0 -> 2
- net Net-(U2-WP#_(IO2)): track 0.00 -> 8.57 mm, vias 0 -> 2
- net Net-(U2-SCK): track 0.00 -> 8.56 mm, vias 0 -> 2
- net Net-(U2-HOLD#_or_RESET#_(IO3)): track 0.00 -> 8.55 mm, vias 0 -> 2
- net Net-(U2-SO_(IO1)): track 0.00 -> 8.53 mm, vias 0 -> 2
- net /QSPI/QSPI_CE_N: track 0.00 -> 7.54 mm
- net /QSPI/QSPI_IO_2: track 0.00 -> 7.00 mm
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Other:
- board size 93.2 x 75.9 mm -> 120.8 x 118.8 mm
