File: Spartan7_TriggerLogic/Spartan7_TriggerController/Spartan7_TriggerController.kicad_sch (KiCad schematic)
At the start: 0 parts

Commit message: Add initial Spartan7 TriggerController PCB files
Added KiCad project files, schematic, PCB layout, symbol and footprint libraries, backup archives, and supporting documentation for the Spartan7 TriggerController. This commit establishes the base hardware design files and resources for further development.
Parts:
- added U1: ~, 0_lib:BGA196C100P14X14_1500X1500X155N, symbol 0_lib:XC7S6-1FTGB196I
Connections:
- new net: U1.D6 (VCCINT), U1.D8 (VCCINT), U1.E7 (VCCINT), U1.E9 (VCCINT), U1.F6 (VCCINT), U1.G9 (VCCINT), U1.H6 (VCCINT), U1.J9 (VCCINT), U1.K6 (VCCINT), U1.K8 (VCCINT)
- new net: U1.E5 (VCCBRAM), U1.G5 (VCCBRAM), U1.J5 (VCCBRAM)
- new net: U1.F10 (VCCAUX), U1.H10 (VCCAUX), U1.K10 (VCCAUX), U1.L9 (VCCAUX)
- new net: U1.G13 (VCCO_14), U1.K13 (VCCO_14), U1.N13 (VCCO_14)
- new net: U1.G2 (VCCO_34), U1.K2 (VCCO_34), U1.N2 (VCCO_34)
- new net: U1.N6 (VCCO_0), U1.N8 (VCCO_0)
- new net GND: U1.A1 (GND), U1.A11 (GND), U1.A14 (GND), U1.A9 (GND), U1.B4 (GND), U1.B7 (GND), U1.B9 (GND), U1.C13 (GND), U1.C2 (GND), U1.C6 (GND), U1.C7 (GND), U1.C8 (GND), U1.C9 (GND), U1.D11 (GND), U1.D5 (GND), U1.D7 (GND), U1.D9 (GND), U1.E1 (GND), U1.E10 (GND), U1.E14 (GND), U1.E3 (GND), U1.E6 (GND), U1.E8 (GND), U1.F5 (GND), U1.F9 (GND), U1.G10 (GND), U1.G12 (GND), U1.G3 (GND), U1.G6 (GND), U1.H5 (GND), U1.H9 (GND), U1.J10 (GND), U1.J6 (GND), U1.K1 (GND), U1.K14 (GND), U1.K5 (GND), U1.K7 (GND), U1.K9 (GND), U1.L10 (GND), U1.L11 (GND), U1.L4 (GND), U1.L6 (GND), U1.L8 (GND), U1.N12 (GND), U1.N3 (GND), U1.N5 (GND), U1.N9 (GND), U1.P1 (GND), U1.P14 (GND)
Other:
- title: (none) -> HYDRA Clock Master

Commit message: m
Parts:
- removed U1: ~, 0_lib:BGA196C100P14X14_1500X1500X155N, symbol 0_lib:XC7S6-1FTGB196I
Other:
- added sheet Ground (gnd.kicad_sch)
- added sheet Power (power.kicad_sch)

Commit message: .
Changed lines of the file:
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@@
 	)
 	(sheet
-		(at 63.5 92.71)
-		(size 58.42 46.99)
+		(at 36.83 41.91)
+		(size 24.13 12.7)
 		(exclude_from_sim no)
 		(in_bom yes)
 		(on_board yes)
 		(dnp no)
-		(fields_autoplaced yes)
 		(stroke
 			(width 0.1524)
@@
 		)
 		(fill
-			(color 0 0 0 0.0000)
+			(color 255 198 108 1.0000)
 		)
 		(property "Sheetname" "Power"
-			(at 63.5 91.9984 0)
+			(at 36.83 51.816 0)
 			(effects
 				(font
-					(size 1.27 1.27)
+					(size 5 5)
+					(thickness 1)
+					(bold yes)
 				)
 				(justify left bottom)
@@
 		)
 		(property "Sheetfile" "power.kicad_sch"
-			(at 63.5 140.2846 0)
+			(at 36.83 89.4846 0)
 			(effects
 				(font
@@
 				)
 				(justify left top)
+				(hide yes)
 			)
 		)
@@
 	)
 	(sheet
-		(at 64.77 59.69)
+		(at 33.02 29.21)
 		(size 31.75 11.43)
 		(exclude_from_sim no)
@@
 		)
 		(property "Sheetname" "Ground"
-			(at 66.294 68.58 0)
+			(at 34.544 38.1 0)
 			(effects
 				(font
@@
 		)
 		(property "Sheetfile" "gnd.kicad_sch"
-			(at 64.77 126.3146 0)
+			(at 33.02 95.8346 0)
 			(effects
 				(font

Commit message: .
Other:
- removed sheet Ground
Changed lines of the file:
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@@
-		)
-	)
-	(sheet
-		(at 33.02 29.21)
-		(size 31.75 11.43)
-		(exclude_from_sim no)
-		(in_bom yes)
-		(on_board yes)
-		(dnp no)
-		(stroke
-			(width 0.1524)
-			(type solid)
-		)
-		(fill
-			(color 255 174 251 1.0000)
-		)
-		(property "Sheetname" "Ground"
-			(at 34.544 38.1 0)
-			(effects
-				(font
-					(size 5 5)
-					(thickness 1)
-					(bold yes)
-				)
-				(justify left bottom)
-			)
-		)
-		(property "Sheetfile" "gnd.kicad_sch"
-			(at 33.02 95.8346 0)
-			(effects
-				(font
-					(size 1.27 1.27)
-				)
-				(justify left top)
-				(hide yes)
-			)
-		)
-		(instances
-			(project "Spartan7_TriggerController"
-				(path "/4e8a1527-464a-4520-8845-f408be0bbc40"
-					(page "2")
-				)
-			)
 		)
 	)

Commit message: .
Connections:
- no-connect marks 0 -> 1
Other:
- added sheet Boot_Mode (Boot_Mode.kicad_sch)
- added sheet JTAG (JTAG.kicad_sch)
- added sheet QSPI (QSPI_IS25LP256D.kicad_sch)
- added sheet XC7S6 (XC7S6_FTGB196.kicad_sch)
