File: Spartan7_TriggerLogic/Spartan7_TriggerController/power.kicad_sch (KiCad schematic)
At the start: 32 parts, among them U1 XC7S6-1FTGB196I

Commit message: .
Parts:
- added J1: For_Catellated_holes, Connector_PinHeader_2.54mm:PinHeader_1x09_P2.54mm_Vertical, symbol Connector:Conn_01x09_Pin
- added J2, J3: For_Catellated_holes, Connector_PinHeader_2.54mm:PinHeader_1x11_P2.54mm_Vertical, symbol Connector:Conn_01x11_Pin
- U1: footprint (none) -> 0_lib:BGA196C100P14X14_1500X1500X155N
Connections:
- net VCCINT is gone; now on net VCCINT&VCCBRAM: C1.1, C2.1, C3.1, U1.D6 (VCCINT), U1.D8 (VCCINT), U1.E7 (VCCINT), U1.E9 (VCCINT), U1.F6 (VCCINT), U1.G9 (VCCINT), U1.H6 (VCCINT), U1.J9 (VCCINT), U1.K6 (VCCINT), U1.K8 (VCCINT)
- net VCCO_34 is gone; now on net VCCO_14&VCCO_34: C25.1, C26.1, C27.1, C28.1, C29.1, C30.1, C31.1, U1.G2 (VCCO_34), U1.K2 (VCCO_34), U1.N2 (VCCO_34)
- net GND: now also J1.2 (Pin_2), J1.4 (Pin_4), J1.6 (Pin_6), J1.8 (Pin_8), J2.1 (Pin_1), J2.10 (Pin_10), J2.11 (Pin_11), J2.2 (Pin_2), J2.3 (Pin_3), J2.4 (Pin_4), J2.5 (Pin_5), J2.6 (Pin_6), J2.7 (Pin_7), J2.8 (Pin_8), J2.9 (Pin_9), J3.1 (Pin_1), J3.10 (Pin_10), J3.11 (Pin_11), J3.2 (Pin_2), J3.3 (Pin_3), J3.4 (Pin_4), J3.5 (Pin_5), J3.6 (Pin_6), J3.7 (Pin_7), J3.8 (Pin_8), J3.9 (Pin_9)
- net VCCAUX: now also J1.9 (Pin_9)
- net VCCO_0: now also J1.5 (Pin_5)
- net VCCBRAM renamed VCCINT&VCCBRAM
- net VCCINT&VCCBRAM: now also J1.7 (Pin_7)
- net VCCO_14 renamed VCCO_14&VCCO_34
- net VCCO_14&VCCO_34: now also J1.3 (Pin_3)
- new net PowerGOOD_LDO3V3: J1.1 (Pin_1)
Other:
- moved on the sheet: C1, C10, C11, C12, C13, C14, C15, C16, C17, C18, C19, C2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

Commit message: .
Parts:
- added unit 1 of U1
- C1, C10, C14, C15, C16, C17, C21, C22, C23, C24, C28, C29, C30, C31, C6, C9: footprint (none) -> Capacitor_SMD:C_0402_1005Metric
- C11, C18, C25, C4, C7: footprint (none) -> Capacitor_SMD:C_1210_3225Metric
- C12, C13, C19, C2, C20, C26, C27, C5, C8: footprint (none) -> Capacitor_SMD:C_0603_1608Metric
- C3: value 100uF -> 47uF; footprint (none) -> Capacitor_SMD:C_1210_3225Metric
Connections:
- net GND: now also U1.A1 (GND), U1.A11 (GND), U1.A14 (GND), U1.A9 (GND), U1.B4 (GND), U1.B7 (GND), U1.B9 (GND), U1.C13 (GND), U1.C2 (GND), U1.C6 (GND), U1.C7 (GND), U1.C8 (GND), U1.C9 (GND), U1.D11 (GND), U1.D5 (GND), U1.D7 (GND), U1.D9 (GND), U1.E1 (GND), U1.E10 (GND), U1.E14 (GND), U1.E3 (GND), U1.E6 (GND), U1.E8 (GND), U1.F5 (GND), U1.F9 (GND), U1.G10 (GND), U1.G12 (GND), U1.G3 (GND), U1.G6 (GND), U1.H5 (GND), U1.H9 (GND), U1.J10 (GND), U1.J6 (GND), U1.K1 (GND), U1.K14 (GND), U1.K5 (GND), U1.K7 (GND), U1.K9 (GND), U1.L10 (GND), U1.L11 (GND), U1.L4 (GND), U1.L6 (GND), U1.L8 (GND), U1.N12 (GND), U1.N3 (GND), U1.N5 (GND), U1.N9 (GND), U1.P1 (GND), U1.P14 (GND)
Other:
- moved on the sheet: J1, J2, J3

Commit message: .
Connections:
- net GND: now also U1.A6 (GND)
- net VCCO_0 renamed +3.3V_0
- net VCCO_14&VCCO_34 renamed +3.3V_14_34
Changed lines of the file:
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@@
 	)
 	(junction
+		(at 54.61 152.4)
+		(diameter 0)
+		(color 0 0 0 0)
+	)
+	(junction
 		(at 90.17 83.82)
 		(diameter 0)
@@
 	)
 	(junction
+		(at 29.21 157.48)
+		(diameter 0)
+		(color 0 0 0 0)
+	)
+	(junction
 		(at 55.88 76.2)
 		(diameter 0)
@@
 	)
 	(junction
+		(at 207.01 22.86)
+		(diameter 0)
+		(color 0 0 0 0)
+	)
+	(junction
 		(at 81.28 99.06)
 		(diameter 0)
@@
 	(wire
 		(pts
+			(xy 207.01 20.32) (xy 207.01 22.86)
+		)
+		(stroke
+			(width 0)
+			(type default)
+		)
+	)
+	(wire
+		(pts
 			(xy 105.41 43.18) (xy 105.41 45.72)
 		)
@@
 	(wire
 		(pts
+			(xy 54.61 152.4) (xy 76.2 152.4)
+		)
+		(stroke
+			(width 0)
+			(type default)
+		)
+	)
+	(wire
+		(pts
 			(xy 207.01 88.9) (xy 207.01 91.44)
 		)
@@
 	(wire
 		(pts
-			(xy 53.34 157.48) (xy 76.2 157.48)
+			(xy 27.94 157.48) (xy 29.21 157.48)
 		)
 		(stroke
@@
 	(wire
 		(pts
+			(xy 29.21 157.48) (xy 76.2 157.48)
+		)
+		(stroke
+			(width 0)
+			(type default)
+		)
+	)
+	(wire
+		(pts
 			(xy 46.99 95.25) (xy 55.88 95.25)
 		)
@@
 	(wire
 		(pts
+			(xy 207.01 22.86) (xy 207.01 25.4)
+		)
+		(stroke
+			(width 0)
+			(type default)
+		)
+	)
+	(wire
+		(pts
 			(xy 207.01 25.4) (xy 207.01 27.94)
 		)
@@
 	(wire
 		(pts
-			(xy 53.34 152.4) (xy 76.2 152.4)
+			(xy 53.34 152.4) (xy 54.61 152.4)
 		)
 		(stroke
@@
 	(wire
 		(pts
-			(xy 105.41 53.34) (xy 105.41 55.88)
+			(xy 54.61 148.59) (xy 54.61 152.4)
 		)
 		(stroke
@@
 	(wire
 		(pts
-			(xy 120.65 157.48) (xy 120.65 160.02)
+			(xy 105.41 53.34) (xy 105.41 55.88)
 		)
 		(stroke
@@
 	(wire
 		(pts
-			(xy 81.28 99.06) (xy 90.17 99.06)
+			(xy 120.65 157.48) (xy 120.65 160.02)
 		)
 		(stroke
@@
 	(wire
 		(pts
-			(xy 207.01 66.04) (xy 207.01 68.58)
+			(xy 81.28 99.06) (xy 90.17 99.06)
 		)
 		(stroke
@@
 	(wire
 		(pts
-			(xy 207.01 22.86) (xy 207.01 25.4)
+			(xy 207.01 66.04) (xy 207.01 68.58)
 		)
 		(stroke
@@
 	(wire
 		(pts
+			(xy 29.21 148.59) (xy 29.21 157.48)
+		)
+		(stroke
+			(width 0)
+			(type default)
+		)
+	)
+	(wire
+		(pts
 			(xy 105.41 58.42) (xy 105.41 60.96)
 		)
@@
 	(global_label "VCCO_0"
 		(shape input)
-		(at 53.34 157.48 180)
+		(at 27.94 157.48 180)
 		(fields_autoplaced yes)
 		(effects
@@
 		)
 		(property "Intersheetrefs" "${INTERSHEET_REFS}"
-			(at 43.2186 157.48 0)
+			(at 17.8186 157.48 0)
 			(effects
 				(font
@@
 	)
 	(symbol
+		(lib_id "power:+3.3V")
+		(at 54.61 148.59 0)
+		(unit 1)
+		(exclude_from_sim no)
+		(in_bom yes)
+		(on_board yes)
+		(dnp no)
+		(fields_autoplaced yes)
+		(property "Reference" "#PWR010"
+			(at 54.61 152.4 0)
+			(effects
+				(font
+					(size 1.27 1.27)
+				)
+				(hide yes)
+			)
+		)
+		(property "Value" "+3.3V_14_34"
+			(at 54.61 143.51 0)
+			(effects
+				(font
+					(size 1.27 1.27)
+				)
+			)
+		)
+		(property "Footprint" ""
+			(at 54.61 148.59 0)
+			(effects
+				(font
+					(size 1.27 1.27)
+				)
+				(hide yes)
+			)
+		)
+		(property "Datasheet" ""
+			(at 54.61 148.59 0)
+			(effects
+				(font
+					(size 1.27 1.27)
+				)
+				(hide yes)
+			)
+		)
+		(property "Description" "Power symbol creates a global label with name \"+3.3V\""
+			(at 54.61 148.59 0)
+			(effects
+				(font
+					(size 1.27 1.27)
+				)
+				(hide yes)
+			)
+		)
+		(pin "1"
+		)
+		(instances
+			(project ""
+				(path "/4e8a1527-464a-4520-8845-f408be0bbc40/0e14c4f1-cc08-4711-a2cf-002e73f6382b"
+					(reference "#PWR010")
+					(unit 1)
+				)
+			)
+		)
+	)
+	(symbol
 		(lib_id "Device:C")
 		(at 55.88 91.44 0)
@@
 	)
 	(symbol
+		(lib_name "XC7S6-1FTGB196I_1")
 		(lib_id "0_lib:XC7S6-1FTGB196I")
 		(at 218.44 34.29 0)
@@
 		(pin "M2"
 		)
+		(pin "A6"
+		)
 		(instances
 			(project "Spartan7_TriggerController"
@@
 					(unit 1)
 				)
+			)
+		)
+	)
+	(symbol
+		(lib_id "power:+3.3V")
+		(at 29.21 148.59 0)
+		(unit 1)
+		(exclude_from_sim no)
+		(in_bom yes)
+		(on_board yes)
+		(dnp no)
+		(fields_autoplaced yes)
+		(property "Reference" "#PWR011"
+			(at 29.21 152.4 0)
+			(effects
+				(font
+					(size 1.27 1.27)
+				)
+				(hide yes)
+			)
+		)
+		(property "Value" "+3.3V_0"
+			(at 29.21 143.51 0)
+			(effects
+				(font
+					(size 1.27 1.27)
+				)
+			)
+		)
+		(property "Footprint" ""
+			(at 29.21 148.59 0)
+			(effects
+				(font
+					(size 1.27 1.27)
+				)
+				(hide yes)
+			)
+		)
+		(property "Datasheet" ""
+			(at 29.21 148.59 0)
+			(effects
+				(font
+					(size 1.27 1.27)
+				)
+				(hide yes)
+			)
+		)
+		(property "Description" "Power symbol creates a global label with name \"+3.3V\""
+			(at 29.21 148.59 0)
+			(effects
+				(font
+					(size 1.27 1.27)
+				)
+				(hide yes)
+			)
+		)
+		(pin "1"
+		)
+		(instances
+			(project "Spartan7_TriggerController"
+				(path "/4e8a1527-464a-4520-8845-f408be0bbc40/0e14c4f1-cc08-4711-a2cf-002e73f6382b"
+					(reference "#PWR011")
+					(unit 1)
+				)
