File: AddOns/Card_Adapter_Flex_AddOn_2Layers.kicad_pro/Card_Adapter_Flex_AddOn_2Layers.kicad_pro.kicad_sch (KiCad schematic)
At the start: 4 parts, among them J1 17-pin-FPC, J2 4-pin-FPC

Commit message: .
Parts:
- R11, R12: now not fitted
Changed lines of the file:
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@@
 		(in_bom yes)
 		(on_board yes)
-		(dnp no)
+		(dnp yes)
 		(property "Reference" "R12"
 			(at 116.078 114.3 90)
@@
 		(in_bom yes)
 		(on_board yes)
-		(dnp no)
+		(dnp yes)
 		(property "Reference" "R11"
 			(at 116.078 73.66 90)
@@
 		)
 		(instances
-			(project "Card_Adapter_Flex_AddOn"
+			(project "Card_Adapter_Flex_AddOn_2Layers.kicad_pro"
 				(path "/05374f14-0ccd-445f-8362-33aedd6aa709"
 					(page "2")
@@
 		)
 		(instances
-			(project "Card_Adapter_Flex_AddOn"
+			(project "Card_Adapter_Flex_AddOn_2Layers.kicad_pro"
 				(path "/05374f14-0ccd-445f-8362-33aedd6aa709"
 					(page "3")

Commit message: .
Parts:
- R11, R12: value 50 -> 10k; now fitted
Connections:
- no-connect marks 0 -> 2
Other:
- company: (none) -> TU Darmstadt
Changed lines of the file:
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@@
 		(title "Card Adapter Flex AddOn")
 		(date "2025-04-28")
-		(rev "0")
+		(rev "1")
+		(company "TU Darmstadt")
+		(comment 1 "Author: Dr. Alexandru Enciu")
 	)
 	(junction
@@
 		(color 0 0 0 0)
 	)
+	(no_connect
+		(at 120.65 73.66)
+	)
+	(no_connect
+		(at 120.65 114.3)
+	)
 	(wire
 		(pts
@@
 		(in_bom yes)
 		(on_board yes)
-		(dnp yes)
+		(dnp no)
 		(property "Reference" "R12"
 			(at 116.078 114.3 90)
@@
 			)
 		)
-		(property "Value" "50"
+		(property "Value" "10k"
 			(at 118.11 114.046 90)
 			(effects
@@
 		(in_bom yes)
 		(on_board yes)
-		(dnp yes)
+		(dnp no)
 		(property "Reference" "R11"
 			(at 116.078 73.66 90)
@@
 			)
 		)
-		(property "Value" "50"
+		(property "Value" "10k"
 			(at 118.11 73.406 90)
 			(effects
