File: Spartan7_TriggerLogic/Trigger_logic/Trigger_logic.kicad_sch (KiCad schematic)
At the start: 387 parts, among them U1 74LVC2G79

Commit message: .
Connections:
- net 2:8 Flex Clock Buffer0/Heimtime 0 is gone; now on net 2:8 Flex Clock Buffer0/Heimtime 0: C9.1
- net 2:8 Flex Clock Buffer0/Heimtime 1 is gone; now on net 2:8 Flex Clock Buffer0/Heimtime 1: C11.1
- net 2:8 Flex Clock Buffer0/Master Trigger 0 is gone; now on net 2:8 Flex Clock Buffer0/Master Trigger 0: C10.1
- net 2:8 Flex Clock Buffer0/Master Trigger 1 is gone; now on net 2:8 Flex Clock Buffer0/Master Trigger 1: C16.1
- net 2:8 Flex Clock Buffer1/Heimtime 0 is gone; now on net 2:8 Flex Clock Buffer1/Heimtime 0: C1.1
- net 2:8 Flex Clock Buffer1/Heimtime 1 is gone; now on net 2:8 Flex Clock Buffer1/Heimtime 1: C7.2
- net 2:8 Flex Clock Buffer1/Master Trigger 0 is gone; now on net 2:8 Flex Clock Buffer1/Master Trigger 0: C3.1
- net 2:8 Flex Clock Buffer1/Master Trigger 1 is gone; now on net 2:8 Flex Clock Buffer1/Master Trigger 1: C8.1
- net 2:8 Flex Clock Buffer10/Heimtime 0 is gone; now on net 2:8 Flex Clock Buffer10/Heimtime 0: C89.2
- net 2:8 Flex Clock Buffer10/Heimtime 1 is gone; now on net 2:8 Flex Clock Buffer10/Heimtime 1: C79.1
- net 2:8 Flex Clock Buffer10/Master Trigger 0 is gone; now on net 2:8 Flex Clock Buffer10/Master Trigger 0: C78.1
- net 2:8 Flex Clock Buffer10/Master Trigger 1 is gone; now on net 2:8 Flex Clock Buffer10/Master Trigger 1: C80.1
- net 2:8 Flex Clock Buffer11/Heimtime 0 is gone; now on net 2:8 Flex Clock Buffer11/Heimtime 0: C93.2
- net 2:8 Flex Clock Buffer11/Heimtime 1 is gone; now on net 2:8 Flex Clock Buffer11/Heimtime 1: C95.2
- net 2:8 Flex Clock Buffer11/Master Trigger 0 is gone; now on net 2:8 Flex Clock Buffer11/Master Trigger 0: C94.1
- net 2:8 Flex Clock Buffer11/Master Trigger 1 is gone; now on net 2:8 Flex Clock Buffer11/Master Trigger 1: C96.1
- net 2:8 Flex Clock Buffer12/Heimtime 0 is gone; now on net 2:8 Flex Clock Buffer12/Heimtime 0: C121.2
- net 2:8 Flex Clock Buffer12/Heimtime 1 is gone; now on net 2:8 Flex Clock Buffer12/Heimtime 1: C123.2
- net 2:8 Flex Clock Buffer12/Master Trigger 0 is gone; now on net 2:8 Flex Clock Buffer12/Master Trigger 0: C98.1
- net 2:8 Flex Clock Buffer12/Master Trigger 1 is gone; now on net 2:8 Flex Clock Buffer12/Master Trigger 1: C124.1
- net 2:8 Flex Clock Buffer13/Heimtime 0 is gone; now on net 2:8 Flex Clock Buffer13/Heimtime 0: C125.2
- net 2:8 Flex Clock Buffer13/Heimtime 1 is gone; now on net 2:8 Flex Clock Buffer13/Heimtime 1: C103.1
- net 2:8 Flex Clock Buffer13/Master Trigger 0 is gone; now on net 2:8 Flex Clock Buffer13/Master Trigger 0: C102.1
- net 2:8 Flex Clock Buffer13/Master Trigger 1 is gone; now on net 2:8 Flex Clock Buffer13/Master Trigger 1: C104.1
- net 2:8 Flex Clock Buffer14/Heimtime 0 is gone; now on net 2:8 Flex Clock Buffer14/Heimtime 0: C105.1
- net 2:8 Flex Clock Buffer14/Heimtime 1 is gone; now on net 2:8 Flex Clock Buffer14/Heimtime 1: C107.1
- net 2:8 Flex Clock Buffer14/Master Trigger 0 is gone; now on net 2:8 Flex Clock Buffer14/Master Trigger 0: C106.1
- net 2:8 Flex Clock Buffer14/Master Trigger 1 is gone; now on net 2:8 Flex Clock Buffer14/Master Trigger 1: C132.1
- net 2:8 Flex Clock Buffer15/Heimtime 0 is gone; now on net 2:8 Flex Clock Buffer15/Heimtime 0: C169.2
- net 2:8 Flex Clock Buffer15/Heimtime 1 is gone; now on net 2:8 Flex Clock Buffer15/Heimtime 1: C171.2
- net 2:8 Flex Clock Buffer15/Master Trigger 0 is gone; now on net 2:8 Flex Clock Buffer15/Master Trigger 0: C170.1
- net 2:8 Flex Clock Buffer15/Master Trigger 1 is gone; now on net 2:8 Flex Clock Buffer15/Master Trigger 1: C148.1
- net 2:8 Flex Clock Buffer16/Heimtime 0 is gone; now on net 2:8 Flex Clock Buffer16/Heimtime 0: C173.2
- net 2:8 Flex Clock Buffer16/Heimtime 1 is gone; now on net 2:8 Flex Clock Buffer16/Heimtime 1: C175.2
- net 2:8 Flex Clock Buffer16/Master Trigger 0 is gone; now on net 2:8 Flex Clock Buffer16/Master Trigger 0: C150.1
- net 2:8 Flex Clock Buffer16/Master Trigger 1 is gone; now on net 2:8 Flex Clock Buffer16/Master Trigger 1: C176.1
- net 2:8 Flex Clock Buffer17/Heimtime 0 is gone; now on net 2:8 Flex Clock Buffer17/Heimtime 0: C177.2
- net 2:8 Flex Clock Buffer17/Heimtime 1 is gone; now on net 2:8 Flex Clock Buffer17/Heimtime 1: C179.2
- net 2:8 Flex Clock Buffer17/Master Trigger 0 is gone; now on net 2:8 Flex Clock Buffer17/Master Trigger 0: C154.1
- net 2:8 Flex Clock Buffer17/Master Trigger 1 is gone; now on net 2:8 Flex Clock Buffer17/Master Trigger 1: C156.1
- net 2:8 Flex Clock Buffer18/Heimtime 0 is gone; now on net 2:8 Flex Clock Buffer18/Heimtime 0: C109.1
- net 2:8 Flex Clock Buffer18/Heimtime 1 is gone; now on net 2:8 Flex Clock Buffer18/Heimtime 1: C135.2
- net 2:8 Flex Clock Buffer18/Master Trigger 0 is gone; now on net 2:8 Flex Clock Buffer18/Master Trigger 0: C110.1
- net 2:8 Flex Clock Buffer18/Master Trigger 1 is gone; now on net 2:8 Flex Clock Buffer18/Master Trigger 1: C136.1
- net 2:8 Flex Clock Buffer19/Heimtime 0 is gone; now on net 2:8 Flex Clock Buffer19/Heimtime 0: C137.2
- net 2:8 Flex Clock Buffer19/Heimtime 1 is gone; now on net 2:8 Flex Clock Buffer19/Heimtime 1: C139.2
- net 2:8 Flex Clock Buffer19/Master Trigger 0 is gone; now on net 2:8 Flex Clock Buffer19/Master Trigger 0: C138.1
- net 2:8 Flex Clock Buffer19/Master Trigger 1 is gone; now on net 2:8 Flex Clock Buffer19/Master Trigger 1: C116.1
- net 2:8 Flex Clock Buffer2/Heimtime 0 is gone; now on net 2:8 Flex Clock Buffer2/Heimtime 0: C21.2
- net 2:8 Flex Clock Buffer2/Heimtime 1 is gone; now on net 2:8 Flex Clock Buffer2/Heimtime 1: C23.2
- net 2:8 Flex Clock Buffer2/Master Trigger 0 is gone; now on net 2:8 Flex Clock Buffer2/Master Trigger 0: C22.1
- net 2:8 Flex Clock Buffer2/Master Trigger 1 is gone; now on net 2:8 Flex Clock Buffer2/Master Trigger 1: C20.1
- net 2:8 Flex Clock Buffer20/Heimtime 0 is gone; now on net 2:8 Flex Clock Buffer20/Heimtime 0: C141.2
- net 2:8 Flex Clock Buffer20/Heimtime 1 is gone; now on net 2:8 Flex Clock Buffer20/Heimtime 1: C143.2
- net 2:8 Flex Clock Buffer20/Master Trigger 0 is gone; now on net 2:8 Flex Clock Buffer20/Master Trigger 0: C118.1
- net 2:8 Flex Clock Buffer20/Master Trigger 1 is gone; now on net 2:8 Flex Clock Buffer20/Master Trigger 1: C144.1
- net 2:8 Flex Clock Buffer21/Heimtime 0 is gone; now on net 2:8 Flex Clock Buffer21/Heimtime 0: C181.2
- net 2:8 Flex Clock Buffer21/Heimtime 1 is gone; now on net 2:8 Flex Clock Buffer21/Heimtime 1: C159.1
- net 2:8 Flex Clock Buffer21/Master Trigger 0 is gone; now on net 2:8 Flex Clock Buffer21/Master Trigger 0: C158.1
- net 2:8 Flex Clock Buffer21/Master Trigger 1 is gone; now on net 2:8 Flex Clock Buffer21/Master Trigger 1: C184.1
- net 2:8 Flex Clock Buffer22/Heimtime 0 is gone; now on net 2:8 Flex Clock Buffer22/Heimtime 0: C161.1
- net 2:8 Flex Clock Buffer22/Heimtime 1 is gone; now on net 2:8 Flex Clock Buffer22/Heimtime 1: C163.1
- net 2:8 Flex Clock Buffer22/Master Trigger 0 is gone; now on net 2:8 Flex Clock Buffer22/Master Trigger 0: C162.1
- net 2:8 Flex Clock Buffer22/Master Trigger 1 is gone; now on net 2:8 Flex Clock Buffer22/Master Trigger 1: C164.1
- net 2:8 Flex Clock Buffer23/Heimtime 0 is gone; now on net 2:8 Flex Clock Buffer23/Heimtime 0: C165.1
- net 2:8 Flex Clock Buffer23/Heimtime 1 is gone; now on net 2:8 Flex Clock Buffer23/Heimtime 1: C167.1
- net 2:8 Flex Clock Buffer23/Master Trigger 0 is gone; now on net 2:8 Flex Clock Buffer23/Master Trigger 0: C166.1
- net 2:8 Flex Clock Buffer23/Master Trigger 1 is gone; now on net 2:8 Flex Clock Buffer23/Master Trigger 1: C192.1
- net 2:8 Flex Clock Buffer24/Heimtime 0 is gone; now on net 2:8 Flex Clock Buffer24/Heimtime 0: C217.1
- net 2:8 Flex Clock Buffer24/Heimtime 1 is gone; now on net 2:8 Flex Clock Buffer24/Heimtime 1: C219.1
- net 2:8 Flex Clock Buffer24/Master Trigger 0 is gone; now on net 2:8 Flex Clock Buffer24/Master Trigger 0: C218.1
- net 2:8 Flex Clock Buffer24/Master Trigger 1 is gone; now on net 2:8 Flex Clock Buffer24/Master Trigger 1: C268.1
- net 2:8 Flex Clock Buffer25/Heimtime 0 is gone; now on net 2:8 Flex Clock Buffer25/Heimtime 0: C269.2
- net 2:8 Flex Clock Buffer25/Heimtime 1 is gone; now on net 2:8 Flex Clock Buffer25/Heimtime 1: C271.2
- net 2:8 Flex Clock Buffer25/Master Trigger 0 is gone; now on net 2:8 Flex Clock Buffer25/Master Trigger 0: C270.1
- net 2:8 Flex Clock Buffer25/Master Trigger 1 is gone; now on net 2:8 Flex Clock Buffer25/Master Trigger 1: C272.1
- net 2:8 Flex Clock Buffer26/Heimtime 0 is gone; now on net 2:8 Flex Clock Buffer26/Heimtime 0: C273.2
- net 2:8 Flex Clock Buffer26/Heimtime 1 is gone; now on net 2:8 Flex Clock Buffer26/Heimtime 1: C275.2
- net 2:8 Flex Clock Buffer26/Master Trigger 0 is gone; now on net 2:8 Flex Clock Buffer26/Master Trigger 0: C274.1
- net 2:8 Flex Clock Buffer26/Master Trigger 1 is gone; now on net 2:8 Flex Clock Buffer26/Master Trigger 1: C228.1
- net 2:8 Flex Clock Buffer27/Heimtime 0 is gone; now on net 2:8 Flex Clock Buffer27/Heimtime 0: C361.2
- net 2:8 Flex Clock Buffer27/Heimtime 1 is gone; now on net 2:8 Flex Clock Buffer27/Heimtime 1: C315.1
- net 2:8 Flex Clock Buffer27/Master Trigger 0 is gone; now on net 2:8 Flex Clock Buffer27/Master Trigger 0: C314.1
- net 2:8 Flex Clock Buffer27/Master Trigger 1 is gone; now on net 2:8 Flex Clock Buffer27/Master Trigger 1: C364.1
- net 2:8 Flex Clock Buffer28/Heimtime 0 is gone; now on net 2:8 Flex Clock Buffer28/Heimtime 0: C365.2
- net 2:8 Flex Clock Buffer28/Heimtime 1 is gone; now on net 2:8 Flex Clock Buffer28/Heimtime 1: C367.2
- net 2:8 Flex Clock Buffer28/Master Trigger 0 is gone; now on net 2:8 Flex Clock Buffer28/Master Trigger 0: C366.1
- net 2:8 Flex Clock Buffer28/Master Trigger 1 is gone; now on net 2:8 Flex Clock Buffer28/Master Trigger 1: C368.1
- net 2:8 Flex Clock Buffer29/Heimtime 0 is gone; now on net 2:8 Flex Clock Buffer29/Heimtime 0: C369.2
- net 2:8 Flex Clock Buffer29/Heimtime 1 is gone; now on net 2:8 Flex Clock Buffer29/Heimtime 1: C323.1
- net 2:8 Flex Clock Buffer29/Master Trigger 0 is gone; now on net 2:8 Flex Clock Buffer29/Master Trigger 0: C322.1
- net 2:8 Flex Clock Buffer29/Master Trigger 1 is gone; now on net 2:8 Flex Clock Buffer29/Master Trigger 1: C324.1
- net 2:8 Flex Clock Buffer3/Heimtime 0 is gone; now on net 2:8 Flex Clock Buffer3/Heimtime 0: C25.1
- net 2:8 Flex Clock Buffer3/Heimtime 1 is gone; now on net 2:8 Flex Clock Buffer3/Heimtime 1: C39.2
- net 2:8 Flex Clock Buffer3/Master Trigger 0 is gone; now on net 2:8 Flex Clock Buffer3/Master Trigger 0: C38.1
- net 2:8 Flex Clock Buffer3/Master Trigger 1 is gone; now on net 2:8 Flex Clock Buffer3/Master Trigger 1: C28.1
- net 2:8 Flex Clock Buffer30/Heimtime 0 is gone; now on net 2:8 Flex Clock Buffer30/Heimtime 0: C277.2
- net 2:8 Flex Clock Buffer30/Heimtime 1 is gone; now on net 2:8 Flex Clock Buffer30/Heimtime 1: C279.2
- net 2:8 Flex Clock Buffer30/Master Trigger 0 is gone; now on net 2:8 Flex Clock Buffer30/Master Trigger 0: C230.1
- net 2:8 Flex Clock Buffer30/Master Trigger 1 is gone; now on net 2:8 Flex Clock Buffer30/Master Trigger 1: C280.1
- net 2:8 Flex Clock Buffer31/Heimtime 0 is gone; now on net 2:8 Flex Clock Buffer31/Heimtime 0: C233.1
- net 2:8 Flex Clock Buffer31/Heimtime 1 is gone; now on net 2:8 Flex Clock Buffer31/Heimtime 1: C235.1
- net 2:8 Flex Clock Buffer31/Master Trigger 0 is gone; now on net 2:8 Flex Clock Buffer31/Master Trigger 0: C234.1
- net 2:8 Flex Clock Buffer31/Master Trigger 1 is gone; now on net 2:8 Flex Clock Buffer31/Master Trigger 1: C284.1
- net 2:8 Flex Clock Buffer32/Heimtime 0 is gone; now on net 2:8 Flex Clock Buffer32/Heimtime 0: C237.1
- net 2:8 Flex Clock Buffer32/Heimtime 1 is gone; now on net 2:8 Flex Clock Buffer32/Heimtime 1: C239.1
- net 2:8 Flex Clock Buffer32/Master Trigger 0 is gone; now on net 2:8 Flex Clock Buffer32/Master Trigger 0: C286.1
- net 2:8 Flex Clock Buffer32/Master Trigger 1 is gone; now on net 2:8 Flex Clock Buffer32/Master Trigger 1: C240.1
- net 2:8 Flex Clock Buffer33/Heimtime 0 is gone; now on net 2:8 Flex Clock Buffer33/Heimtime 0: C373.2
- net 2:8 Flex Clock Buffer33/Heimtime 1 is gone; now on net 2:8 Flex Clock Buffer33/Heimtime 1: C327.1
- net 2:8 Flex Clock Buffer33/Master Trigger 0 is gone; now on net 2:8 Flex Clock Buffer33/Master Trigger 0: C326.1
- net 2:8 Flex Clock Buffer33/Master Trigger 1 is gone; now on net 2:8 Flex Clock Buffer33/Master Trigger 1: C376.1
- net 2:8 Flex Clock Buffer34/Heimtime 0 is gone; now on net 2:8 Flex Clock Buffer34/Heimtime 0: C329.1
- net 2:8 Flex Clock Buffer34/Heimtime 1 is gone; now on net 2:8 Flex Clock Buffer34/Heimtime 1: C379.2
- net 2:8 Flex Clock Buffer34/Master Trigger 0 is gone; now on net 2:8 Flex Clock Buffer34/Master Trigger 0: C378.1
- net 2:8 Flex Clock Buffer34/Master Trigger 1 is gone; now on net 2:8 Flex Clock Buffer34/Master Trigger 1: C380.1
- net 2:8 Flex Clock Buffer35/Heimtime 0 is gone; now on net 2:8 Flex Clock Buffer35/Heimtime 0: C333.1
- net 2:8 Flex Clock Buffer35/Heimtime 1 is gone; now on net 2:8 Flex Clock Buffer35/Heimtime 1: C335.1
- net 2:8 Flex Clock Buffer35/Master Trigger 0 is gone; now on net 2:8 Flex Clock Buffer35/Master Trigger 0: C334.1
- net 2:8 Flex Clock Buffer35/Master Trigger 1 is gone; now on net 2:8 Flex Clock Buffer35/Master Trigger 1: C336.1
- net 2:8 Flex Clock Buffer36/Heimtime 0 is gone; now on net 2:8 Flex Clock Buffer36/Heimtime 0: C241.2
- net 2:8 Flex Clock Buffer36/Heimtime 1 is gone; now on net 2:8 Flex Clock Buffer36/Heimtime 1: C243.2
- net 2:8 Flex Clock Buffer36/Master Trigger 0 is gone; now on net 2:8 Flex Clock Buffer36/Master Trigger 0: C194.1
- net 2:8 Flex Clock Buffer36/Master Trigger 1 is gone; now on net 2:8 Flex Clock Buffer36/Master Trigger 1: C196.1
- net 2:8 Flex Clock Buffer37/Heimtime 0 is gone; now on net 2:8 Flex Clock Buffer37/Heimtime 0: C197.1
- net 2:8 Flex Clock Buffer37/Heimtime 1 is gone; now on net 2:8 Flex Clock Buffer37/Heimtime 1: C247.2
- net 2:8 Flex Clock Buffer37/Master Trigger 0 is gone; now on net 2:8 Flex Clock Buffer37/Master Trigger 0: C198.1
- net 2:8 Flex Clock Buffer37/Master Trigger 1 is gone; now on net 2:8 Flex Clock Buffer37/Master Trigger 1: C200.1
- net 2:8 Flex Clock Buffer38/Heimtime 0 is gone; now on net 2:8 Flex Clock Buffer38/Heimtime 0: C249.2
- net 2:8 Flex Clock Buffer38/Heimtime 1 is gone; now on net 2:8 Flex Clock Buffer38/Heimtime 1: C203.1
- net 2:8 Flex Clock Buffer38/Master Trigger 0 is gone; now on net 2:8 Flex Clock Buffer38/Master Trigger 0: C202.1
- net 2:8 Flex Clock Buffer38/Master Trigger 1 is gone; now on net 2:8 Flex Clock Buffer38/Master Trigger 1: C252.1
- net 2:8 Flex Clock Buffer39/Heimtime 0 is gone; now on net 2:8 Flex Clock Buffer39/Heimtime 0: C337.2
- net 2:8 Flex Clock Buffer39/Heimtime 1 is gone; now on net 2:8 Flex Clock Buffer39/Heimtime 1: C291.1
- net 2:8 Flex Clock Buffer39/Master Trigger 0 is gone; now on net 2:8 Flex Clock Buffer39/Master Trigger 0: C290.1
- net 2:8 Flex Clock Buffer39/Master Trigger 1 is gone; now on net 2:8 Flex Clock Buffer39/Master Trigger 1: C292.1
- net 2:8 Flex Clock Buffer4/Heimtime 0 is gone; now on net 2:8 Flex Clock Buffer4/Heimtime 0: C29.1
- net 2:8 Flex Clock Buffer4/Heimtime 1 is gone; now on net 2:8 Flex Clock Buffer4/Heimtime 1: C43.2
- net 2:8 Flex Clock Buffer4/Master Trigger 0 is gone; now on net 2:8 Flex Clock Buffer4/Master Trigger 0: C30.1
- net 2:8 Flex Clock Buffer4/Master Trigger 1 is gone; now on net 2:8 Flex Clock Buffer4/Master Trigger 1: C32.1
- net 2:8 Flex Clock Buffer40/Heimtime 0 is gone; now on net 2:8 Flex Clock Buffer40/Heimtime 0: C341.2
- net 2:8 Flex Clock Buffer40/Heimtime 1 is gone; now on net 2:8 Flex Clock Buffer40/Heimtime 1: C343.2
- net 2:8 Flex Clock Buffer40/Master Trigger 0 is gone; now on net 2:8 Flex Clock Buffer40/Master Trigger 0: C342.1
- net 2:8 Flex Clock Buffer40/Master Trigger 1 is gone; now on net 2:8 Flex Clock Buffer40/Master Trigger 1: C344.1
- net 2:8 Flex Clock Buffer41/Heimtime 0 is gone; now on net 2:8 Flex Clock Buffer41/Heimtime 0: C345.2
- net 2:8 Flex Clock Buffer41/Heimtime 1 is gone; now on net 2:8 Flex Clock Buffer41/Heimtime 1: C299.1
- net 2:8 Flex Clock Buffer41/Master Trigger 0 is gone; now on net 2:8 Flex Clock Buffer41/Master Trigger 0: C346.1
- net 2:8 Flex Clock Buffer41/Master Trigger 1 is gone; now on net 2:8 Flex Clock Buffer41/Master Trigger 1: C348.1
- net 2:8 Flex Clock Buffer42/Heimtime 0 is gone; now on net 2:8 Flex Clock Buffer42/Heimtime 0: C253.2
- net 2:8 Flex Clock Buffer42/Heimtime 1 is gone; now on net 2:8 Flex Clock Buffer42/Heimtime 1: C207.1
- net 2:8 Flex Clock Buffer42/Master Trigger 0 is gone; now on net 2:8 Flex Clock Buffer42/Master Trigger 0: C254.1
- net 2:8 Flex Clock Buffer42/Master Trigger 1 is gone; now on net 2:8 Flex Clock Buffer42/Master Trigger 1: C208.1
- net 2:8 Flex Clock Buffer43/Heimtime 0 is gone; now on net 2:8 Flex Clock Buffer43/Heimtime 0: C257.2
- net 2:8 Flex Clock Buffer43/Heimtime 1 is gone; now on net 2:8 Flex Clock Buffer43/Heimtime 1: C211.1
- net 2:8 Flex Clock Buffer43/Master Trigger 0 is gone; now on net 2:8 Flex Clock Buffer43/Master Trigger 0: C258.1
- net 2:8 Flex Clock Buffer43/Master Trigger 1 is gone; now on net 2:8 Flex Clock Buffer43/Master Trigger 1: C212.1
- net 2:8 Flex Clock Buffer44/Heimtime 0 is gone; now on net 2:8 Flex Clock Buffer44/Heimtime 0: C213.1
- net 2:8 Flex Clock Buffer44/Heimtime 1 is gone; now on net 2:8 Flex Clock Buffer44/Heimtime 1: C263.2
- net 2:8 Flex Clock Buffer44/Master Trigger 0 is gone; now on net 2:8 Flex Clock Buffer44/Master Trigger 0: C214.1
- net 2:8 Flex Clock Buffer44/Master Trigger 1 is gone; now on net 2:8 Flex Clock Buffer44/Master Trigger 1: C216.1
- net 2:8 Flex Clock Buffer45/Heimtime 0 is gone; now on net 2:8 Flex Clock Buffer45/Heimtime 0: C349.2
- net 2:8 Flex Clock Buffer45/Heimtime 1 is gone; now on net 2:8 Flex Clock Buffer45/Heimtime 1: C351.2
- net 2:8 Flex Clock Buffer45/Master Trigger 0 is gone; now on net 2:8 Flex Clock Buffer45/Master Trigger 0: C302.1
- net 2:8 Flex Clock Buffer45/Master Trigger 1 is gone; now on net 2:8 Flex Clock Buffer45/Master Trigger 1: C352.1
- net 2:8 Flex Clock Buffer46/Heimtime 0 is gone; now on net 2:8 Flex Clock Buffer46/Heimtime 0: C305.1
- net 2:8 Flex Clock Buffer46/Heimtime 1 is gone; now on net 2:8 Flex Clock Buffer46/Heimtime 1: C307.1
- net 2:8 Flex Clock Buffer46/Master Trigger 0 is gone; now on net 2:8 Flex Clock Buffer46/Master Trigger 0: C306.1
- net 2:8 Flex Clock Buffer46/Master Trigger 1 is gone; now on net 2:8 Flex Clock Buffer46/Master Trigger 1: C308.1
- net 2:8 Flex Clock Buffer47/Heimtime 0 is gone; now on net 2:8 Flex Clock Buffer47/Heimtime 0: C357.2
- net 2:8 Flex Clock Buffer47/Heimtime 1 is gone; now on net 2:8 Flex Clock Buffer47/Heimtime 1: C359.2
- net 2:8 Flex Clock Buffer47/Master Trigger 0 is gone; now on net 2:8 Flex Clock Buffer47/Master Trigger 0: C310.1
- net 2:8 Flex Clock Buffer47/Master Trigger 1 is gone; now on net 2:8 Flex Clock Buffer47/Master Trigger 1: C360.1
- net 2:8 Flex Clock Buffer5/Heimtime 0 is gone; now on net 2:8 Flex Clock Buffer5/Heimtime 0: C33.1
- net 2:8 Flex Clock Buffer5/Heimtime 1 is gone; now on net 2:8 Flex Clock Buffer5/Heimtime 1: C47.2
- net 2:8 Flex Clock Buffer5/Master Trigger 0 is gone; now on net 2:8 Flex Clock Buffer5/Master Trigger 0: C34.1
- net 2:8 Flex Clock Buffer5/Master Trigger 1 is gone; now on net 2:8 Flex Clock Buffer5/Master Trigger 1: C36.1
- net 2:8 Flex Clock Buffer6/Heimtime 0 is gone; now on net 2:8 Flex Clock Buffer6/Heimtime 0: C61.2
- net 2:8 Flex Clock Buffer6/Heimtime 1 is gone; now on net 2:8 Flex Clock Buffer6/Heimtime 1: C63.2
- net 2:8 Flex Clock Buffer6/Master Trigger 0 is gone; now on net 2:8 Flex Clock Buffer6/Master Trigger 0: C62.1
- net 2:8 Flex Clock Buffer6/Master Trigger 1 is gone; now on net 2:8 Flex Clock Buffer6/Master Trigger 1: C64.1
- net 2:8 Flex Clock Buffer7/Heimtime 0 is gone; now on net 2:8 Flex Clock Buffer7/Heimtime 0: C65.2
- net 2:8 Flex Clock Buffer7/Heimtime 1 is gone; now on net 2:8 Flex Clock Buffer7/Heimtime 1: C67.2
- net 2:8 Flex Clock Buffer7/Master Trigger 0 is gone; now on net 2:8 Flex Clock Buffer7/Master Trigger 0: C66.1
- net 2:8 Flex Clock Buffer7/Master Trigger 1 is gone; now on net 2:8 Flex Clock Buffer7/Master Trigger 1: C68.1
- net 2:8 Flex Clock Buffer8/Heimtime 0 is gone; now on net 2:8 Flex Clock Buffer8/Heimtime 0: C57.1
- net 2:8 Flex Clock Buffer8/Heimtime 1 is gone; now on net 2:8 Flex Clock Buffer8/Heimtime 1: C59.1
- net 2:8 Flex Clock Buffer8/Master Trigger 0 is gone; now on net 2:8 Flex Clock Buffer8/Master Trigger 0: C58.1
- net 2:8 Flex Clock Buffer8/Master Trigger 1 is gone; now on net 2:8 Flex Clock Buffer8/Master Trigger 1: C60.1
- net 2:8 Flex Clock Buffer9/Heimtime 0 is gone; now on net 2:8 Flex Clock Buffer9/Heimtime 0: C73.1
- net 2:8 Flex Clock Buffer9/Heimtime 1 is gone; now on net 2:8 Flex Clock Buffer9/Heimtime 1: C75.1
- net 2:8 Flex Clock Buffer9/Master Trigger 0 is gone; now on net 2:8 Flex Clock Buffer9/Master Trigger 0: C86.1
- net 2:8 Flex Clock Buffer9/Master Trigger 1 is gone; now on net 2:8 Flex Clock Buffer9/Master Trigger 1: C76.1
- net VMM3a_ASIC_0/Hybrid Ch.55 is gone; now on net VMM3a_ASIC_0/Hybrid Ch.55: C77.2
- net VMM3a_ASIC_0/Hybrid Ch.57 is gone; now on net VMM3a_ASIC_0/Hybrid Ch.57: C89.1
- net VMM3a_ASIC_0/Hybrid Ch.61 is gone; now on net VMM3a_ASIC_0/Hybrid Ch.61: C322.2
- net VMM3a_ASIC_0/Hybrid Ch.63 is gone; now on net VMM3a_ASIC_0/Hybrid Ch.63: C342.2
- net VMM3a_ASIC_1/Hybrid Ch.65 is gone; now on net VMM3a_ASIC_1/Hybrid Ch.65: C211.2
- net VMM3a_ASIC_1/Hybrid Ch.67 is gone; now on net VMM3a_ASIC_1/Hybrid Ch.67: C243.1
- net VMM3a_ASIC_1/Hybrid Ch.71 is gone; now on net VMM3a_ASIC_1/Hybrid Ch.71: C32.2
- net VMM3a_ASIC_1/Hybrid Ch.73 is gone; now on net VMM3a_ASIC_1/Hybrid Ch.73: C176.2
- net 2:8 Flex Clock Buffer0/Heimtime 0: no longer C13.2
- net 2:8 Flex Clock Buffer0/Heimtime 1: no longer C15.2
- net 2:8 Flex Clock Buffer0/Master Trigger 0: no longer C14.1
- net 2:8 Flex Clock Buffer0/Master Trigger 1: no longer C12.1
- net 2:8 Flex Clock Buffer1/Heimtime 0: no longer C2.2
- net 2:8 Flex Clock Buffer1/Heimtime 1: no longer C5.1
- net 2:8 Flex Clock Buffer1/Master Trigger 0: no longer C4.1
- net 2:8 Flex Clock Buffer1/Master Trigger 1: no longer C6.1
- net 2:8 Flex Clock Buffer10/Heimtime 0: no longer C77.1
- net 2:8 Flex Clock Buffer10/Heimtime 1: no longer C91.2
- net 2:8 Flex Clock Buffer10/Master Trigger 0: no longer C90.1
- net 2:8 Flex Clock Buffer10/Master Trigger 1: no longer C92.1
- net 2:8 Flex Clock Buffer11/Heimtime 0: no longer C81.1
- net 2:8 Flex Clock Buffer11/Heimtime 1: no longer C83.1
- net 2:8 Flex Clock Buffer11/Master Trigger 0: no longer C82.1
- net 2:8 Flex Clock Buffer11/Master Trigger 1: no longer C84.1
- net 2:8 Flex Clock Buffer12/Heimtime 0: no longer C97.1
- net 2:8 Flex Clock Buffer12/Heimtime 1: no longer C99.1
- net 2:8 Flex Clock Buffer12/Master Trigger 0: no longer C122.1
- net 2:8 Flex Clock Buffer12/Master Trigger 1: no longer C100.1
- net 2:8 Flex Clock Buffer13/Heimtime 0: no longer C101.1
- net 2:8 Flex Clock Buffer13/Heimtime 1: no longer C127.2
- net 2:8 Flex Clock Buffer13/Master Trigger 0: no longer C126.1
- net 2:8 Flex Clock Buffer13/Master Trigger 1: no longer C128.1
- net 2:8 Flex Clock Buffer14/Heimtime 0: no longer C129.2
- net 2:8 Flex Clock Buffer14/Heimtime 1: no longer C131.2
- net 2:8 Flex Clock Buffer14/Master Trigger 0: no longer C130.1
- net 2:8 Flex Clock Buffer14/Master Trigger 1: no longer C108.1
- net 2:8 Flex Clock Buffer15/Heimtime 0: no longer C145.1
- net 2:8 Flex Clock Buffer15/Heimtime 1: no longer C147.1
- net 2:8 Flex Clock Buffer15/Master Trigger 0: no longer C146.1
- net 2:8 Flex Clock Buffer15/Master Trigger 1: no longer C172.1
- net 2:8 Flex Clock Buffer16/Heimtime 0: no longer C149.1
- net 2:8 Flex Clock Buffer16/Heimtime 1: no longer C151.1
- net 2:8 Flex Clock Buffer16/Master Trigger 0: no longer C174.1
- net 2:8 Flex Clock Buffer16/Master Trigger 1: no longer C152.1
- net 2:8 Flex Clock Buffer17/Heimtime 0: no longer C153.1
- net 2:8 Flex Clock Buffer17/Heimtime 1: no longer C155.1
- net 2:8 Flex Clock Buffer17/Master Trigger 0: no longer C178.1
- net 2:8 Flex Clock Buffer17/Master Trigger 1: no longer C180.1
- net 2:8 Flex Clock Buffer18/Heimtime 0: no longer C133.2
- net 2:8 Flex Clock Buffer18/Heimtime 1: no longer C111.1
- net 2:8 Flex Clock Buffer18/Master Trigger 0: no longer C134.1
- net 2:8 Flex Clock Buffer18/Master Trigger 1: no longer C112.1
- net 2:8 Flex Clock Buffer19/Heimtime 0: no longer C113.1
- net 2:8 Flex Clock Buffer19/Heimtime 1: no longer C115.1
- net 2:8 Flex Clock Buffer19/Master Trigger 0: no longer C114.1
- net 2:8 Flex Clock Buffer19/Master Trigger 1: no longer C140.1
- net 2:8 Flex Clock Buffer2/Heimtime 0: no longer C17.1
- net 2:8 Flex Clock Buffer2/Heimtime 1: no longer C19.1
- net 2:8 Flex Clock Buffer2/Master Trigger 0: no longer C18.1
- net 2:8 Flex Clock Buffer2/Master Trigger 1: no longer C24.1
- net 2:8 Flex Clock Buffer20/Heimtime 0: no longer C117.1
- net 2:8 Flex Clock Buffer20/Heimtime 1: no longer C119.1
- net 2:8 Flex Clock Buffer20/Master Trigger 0: no longer C142.1
- net 2:8 Flex Clock Buffer20/Master Trigger 1: no longer C120.1
- net 2:8 Flex Clock Buffer21/Heimtime 0: no longer C157.1
- net 2:8 Flex Clock Buffer21/Heimtime 1: no longer C183.2
- net 2:8 Flex Clock Buffer21/Master Trigger 0: no longer C182.1
- net 2:8 Flex Clock Buffer21/Master Trigger 1: no longer C160.1
- net 2:8 Flex Clock Buffer22/Heimtime 0: no longer C185.2
- net 2:8 Flex Clock Buffer22/Heimtime 1: no longer C187.2
- net 2:8 Flex Clock Buffer22/Master Trigger 0: no longer C186.1
- net 2:8 Flex Clock Buffer22/Master Trigger 1: no longer C188.1
- net 2:8 Flex Clock Buffer23/Heimtime 0: no longer C189.2
- net 2:8 Flex Clock Buffer23/Heimtime 1: no longer C191.2
- net 2:8 Flex Clock Buffer23/Master Trigger 0: no longer C190.1
- net 2:8 Flex Clock Buffer23/Master Trigger 1: no longer C168.1
- net 2:8 Flex Clock Buffer24/Heimtime 0: no longer C265.2
- net 2:8 Flex Clock Buffer24/Heimtime 1: no longer C267.2
- net 2:8 Flex Clock Buffer24/Master Trigger 0: no longer C266.1
- net 2:8 Flex Clock Buffer24/Master Trigger 1: no longer C220.1
- net 2:8 Flex Clock Buffer25/Heimtime 0: no longer C221.1
- net 2:8 Flex Clock Buffer25/Heimtime 1: no longer C223.1
- net 2:8 Flex Clock Buffer25/Master Trigger 0: no longer C222.1
- net 2:8 Flex Clock Buffer25/Master Trigger 1: no longer C224.1
- net 2:8 Flex Clock Buffer26/Heimtime 0: no longer C225.1
- net 2:8 Flex Clock Buffer26/Heimtime 1: no longer C227.1
- net 2:8 Flex Clock Buffer26/Master Trigger 0: no longer C226.1
- net 2:8 Flex Clock Buffer26/Master Trigger 1: no longer C276.1
- net 2:8 Flex Clock Buffer27/Heimtime 0: no longer C313.1
- net 2:8 Flex Clock Buffer27/Heimtime 1: no longer C363.2
- net 2:8 Flex Clock Buffer27/Master Trigger 0: no longer C362.1
- net 2:8 Flex Clock Buffer27/Master Trigger 1: no longer C316.1
- net 2:8 Flex Clock Buffer28/Heimtime 0: no longer C317.1
- net 2:8 Flex Clock Buffer28/Heimtime 1: no longer C319.1
- net 2:8 Flex Clock Buffer28/Master Trigger 0: no longer C318.1
- net 2:8 Flex Clock Buffer28/Master Trigger 1: no longer C320.1
- net 2:8 Flex Clock Buffer29/Heimtime 0: no longer C321.1
- net 2:8 Flex Clock Buffer29/Heimtime 1: no longer C371.2
- net 2:8 Flex Clock Buffer29/Master Trigger 0: no longer C370.1
- net 2:8 Flex Clock Buffer29/Master Trigger 1: no longer C372.1
- net 2:8 Flex Clock Buffer3/Heimtime 0: no longer C37.2
- net 2:8 Flex Clock Buffer3/Heimtime 1: no longer C27.1
- net 2:8 Flex Clock Buffer3/Master Trigger 0: no longer C26.1
- net 2:8 Flex Clock Buffer3/Master Trigger 1: no longer C40.1
- net 2:8 Flex Clock Buffer30/Heimtime 0: no longer C229.1
- net 2:8 Flex Clock Buffer30/Heimtime 1: no longer C231.1
- net 2:8 Flex Clock Buffer30/Master Trigger 0: no longer C278.1
- net 2:8 Flex Clock Buffer30/Master Trigger 1: no longer C232.1
- net 2:8 Flex Clock Buffer31/Heimtime 0: no longer C281.2
- net 2:8 Flex Clock Buffer31/Heimtime 1: no longer C283.2
- net 2:8 Flex Clock Buffer31/Master Trigger 0: no longer C282.1
- net 2:8 Flex Clock Buffer31/Master Trigger 1: no longer C236.1
- net 2:8 Flex Clock Buffer32/Heimtime 0: no longer C285.2
- net 2:8 Flex Clock Buffer32/Heimtime 1: no longer C287.2
- net 2:8 Flex Clock Buffer32/Master Trigger 0: no longer C238.1
- net 2:8 Flex Clock Buffer32/Master Trigger 1: no longer C288.1
- net 2:8 Flex Clock Buffer33/Heimtime 0: no longer C325.1
- net 2:8 Flex Clock Buffer33/Heimtime 1: no longer C375.2
- net 2:8 Flex Clock Buffer33/Master Trigger 0: no longer C374.1
- net 2:8 Flex Clock Buffer33/Master Trigger 1: no longer C328.1
- net 2:8 Flex Clock Buffer34/Heimtime 0: no longer C377.2
- net 2:8 Flex Clock Buffer34/Heimtime 1: no longer C331.1
- net 2:8 Flex Clock Buffer34/Master Trigger 0: no longer C330.1
- net 2:8 Flex Clock Buffer34/Master Trigger 1: no longer C332.1
- net 2:8 Flex Clock Buffer35/Heimtime 0: no longer C381.2
- net 2:8 Flex Clock Buffer35/Heimtime 1: no longer C383.2
- net 2:8 Flex Clock Buffer35/Master Trigger 0: no longer C382.1
- net 2:8 Flex Clock Buffer35/Master Trigger 1: no longer C384.1
- net 2:8 Flex Clock Buffer36/Heimtime 0: no longer C193.1
- net 2:8 Flex Clock Buffer36/Heimtime 1: no longer C195.1
- net 2:8 Flex Clock Buffer36/Master Trigger 0: no longer C242.1
- net 2:8 Flex Clock Buffer36/Master Trigger 1: no longer C244.1
- net 2:8 Flex Clock Buffer37/Heimtime 0: no longer C245.2
- net 2:8 Flex Clock Buffer37/Heimtime 1: no longer C199.1
- net 2:8 Flex Clock Buffer37/Master Trigger 0: no longer C246.1
- net 2:8 Flex Clock Buffer37/Master Trigger 1: no longer C248.1
- net 2:8 Flex Clock Buffer38/Heimtime 0: no longer C201.1
- net 2:8 Flex Clock Buffer38/Heimtime 1: no longer C251.2
- new net: U1.7 (Q), U2. (Out), U3. (Out)
- new net 2:8 Flex Clock Buffer0/Heimtime 0: C13.2
- new net 2:8 Flex Clock Buffer0/Heimtime 1: C15.2
- new net 2:8 Flex Clock Buffer0/Master Trigger 0: C14.1
- new net 2:8 Flex Clock Buffer0/Master Trigger 1: C12.1
- new net 2:8 Flex Clock Buffer1/Heimtime 0: C2.2
- new net 2:8 Flex Clock Buffer1/Heimtime 1: C5.1
- new net 2:8 Flex Clock Buffer1/Master Trigger 0: C4.1
- new net 2:8 Flex Clock Buffer1/Master Trigger 1: C6.1
- new net 2:8 Flex Clock Buffer10/Heimtime 0: C77.1
- new net 2:8 Flex Clock Buffer10/Heimtime 1: C91.2
- new net 2:8 Flex Clock Buffer10/Master Trigger 0: C90.1
- new net 2:8 Flex Clock Buffer10/Master Trigger 1: C92.1
- new net 2:8 Flex Clock Buffer11/Heimtime 0: C81.1
- new net 2:8 Flex Clock Buffer11/Heimtime 1: C83.1
- new net 2:8 Flex Clock Buffer11/Master Trigger 0: C82.1
- new net 2:8 Flex Clock Buffer11/Master Trigger 1: C84.1
- new net 2:8 Flex Clock Buffer12/Heimtime 0: C97.1
- new net 2:8 Flex Clock Buffer12/Heimtime 1: C99.1
- new net 2:8 Flex Clock Buffer12/Master Trigger 0: C122.1
- new net 2:8 Flex Clock Buffer12/Master Trigger 1: C100.1
- new net 2:8 Flex Clock Buffer13/Heimtime 0: C101.1
- new net 2:8 Flex Clock Buffer13/Heimtime 1: C127.2
- new net 2:8 Flex Clock Buffer13/Master Trigger 0: C126.1
- new net 2:8 Flex Clock Buffer13/Master Trigger 1: C128.1
- new net 2:8 Flex Clock Buffer14/Heimtime 0: C129.2
- new net 2:8 Flex Clock Buffer14/Heimtime 1: C131.2
- new net 2:8 Flex Clock Buffer14/Master Trigger 0: C130.1
- new net 2:8 Flex Clock Buffer14/Master Trigger 1: C108.1
- new net 2:8 Flex Clock Buffer15/Heimtime 0: C145.1
- new net 2:8 Flex Clock Buffer15/Heimtime 1: C147.1
- new net 2:8 Flex Clock Buffer15/Master Trigger 0: C146.1
- new net 2:8 Flex Clock Buffer15/Master Trigger 1: C172.1
- new net 2:8 Flex Clock Buffer16/Heimtime 0: C149.1
- new net 2:8 Flex Clock Buffer16/Heimtime 1: C151.1
- new net 2:8 Flex Clock Buffer16/Master Trigger 0: C174.1
- new net 2:8 Flex Clock Buffer16/Master Trigger 1: C152.1
- new net 2:8 Flex Clock Buffer17/Heimtime 0: C153.1
- new net 2:8 Flex Clock Buffer17/Heimtime 1: C155.1
- new net 2:8 Flex Clock Buffer17/Master Trigger 0: C178.1
- new net 2:8 Flex Clock Buffer17/Master Trigger 1: C180.1
- new net 2:8 Flex Clock Buffer18/Heimtime 0: C133.2
- new net 2:8 Flex Clock Buffer18/Heimtime 1: C111.1
- new net 2:8 Flex Clock Buffer18/Master Trigger 0: C134.1
- new net 2:8 Flex Clock Buffer18/Master Trigger 1: C112.1
- new net 2:8 Flex Clock Buffer19/Heimtime 0: C113.1
- new net 2:8 Flex Clock Buffer19/Heimtime 1: C115.1
- new net 2:8 Flex Clock Buffer19/Master Trigger 0: C114.1
- new net 2:8 Flex Clock Buffer19/Master Trigger 1: C140.1
- new net 2:8 Flex Clock Buffer2/Heimtime 0: C17.1
- new net 2:8 Flex Clock Buffer2/Heimtime 1: C19.1
- new net 2:8 Flex Clock Buffer2/Master Trigger 0: C18.1
- new net 2:8 Flex Clock Buffer2/Master Trigger 1: C24.1
- new net 2:8 Flex Clock Buffer20/Heimtime 0: C117.1
- new net 2:8 Flex Clock Buffer20/Heimtime 1: C119.1
- new net 2:8 Flex Clock Buffer20/Master Trigger 0: C142.1
- new net 2:8 Flex Clock Buffer20/Master Trigger 1: C120.1
- new net 2:8 Flex Clock Buffer21/Heimtime 0: C157.1
- new net 2:8 Flex Clock Buffer21/Heimtime 1: C183.2
- new net 2:8 Flex Clock Buffer21/Master Trigger 0: C182.1
- new net 2:8 Flex Clock Buffer21/Master Trigger 1: C160.1
- new net 2:8 Flex Clock Buffer22/Heimtime 0: C185.2
- new net 2:8 Flex Clock Buffer22/Heimtime 1: C187.2
- new net 2:8 Flex Clock Buffer22/Master Trigger 0: C186.1
- new net 2:8 Flex Clock Buffer22/Master Trigger 1: C188.1
- new net 2:8 Flex Clock Buffer23/Heimtime 0: C189.2
- new net 2:8 Flex Clock Buffer23/Heimtime 1: C191.2
- new net 2:8 Flex Clock Buffer23/Master Trigger 0: C190.1
- new net 2:8 Flex Clock Buffer23/Master Trigger 1: C168.1
- new net 2:8 Flex Clock Buffer24/Heimtime 0: C265.2
- new net 2:8 Flex Clock Buffer24/Heimtime 1: C267.2
- new net 2:8 Flex Clock Buffer24/Master Trigger 0: C266.1
- new net 2:8 Flex Clock Buffer24/Master Trigger 1: C220.1
- new net 2:8 Flex Clock Buffer25/Heimtime 0: C221.1
- new net 2:8 Flex Clock Buffer25/Heimtime 1: C223.1
- new net 2:8 Flex Clock Buffer25/Master Trigger 0: C222.1
- new net 2:8 Flex Clock Buffer25/Master Trigger 1: C224.1
- new net 2:8 Flex Clock Buffer26/Heimtime 0: C225.1
- new net 2:8 Flex Clock Buffer26/Heimtime 1: C227.1
- new net 2:8 Flex Clock Buffer26/Master Trigger 0: C226.1
- new net 2:8 Flex Clock Buffer26/Master Trigger 1: C276.1
- new net 2:8 Flex Clock Buffer27/Heimtime 0: C313.1
- new net 2:8 Flex Clock Buffer27/Heimtime 1: C363.2
- new net 2:8 Flex Clock Buffer27/Master Trigger 0: C362.1
- new net 2:8 Flex Clock Buffer27/Master Trigger 1: C316.1
- new net 2:8 Flex Clock Buffer28/Heimtime 0: C317.1
- new net 2:8 Flex Clock Buffer28/Heimtime 1: C319.1
- new net 2:8 Flex Clock Buffer28/Master Trigger 0: C318.1
- new net 2:8 Flex Clock Buffer28/Master Trigger 1: C320.1
- new net 2:8 Flex Clock Buffer29/Heimtime 0: C321.1
- new net 2:8 Flex Clock Buffer29/Heimtime 1: C371.2
- new net 2:8 Flex Clock Buffer29/Master Trigger 0: C370.1
- new net 2:8 Flex Clock Buffer29/Master Trigger 1: C372.1
- new net 2:8 Flex Clock Buffer3/Heimtime 0: C37.2
- new net 2:8 Flex Clock Buffer3/Heimtime 1: C27.1
- new net 2:8 Flex Clock Buffer3/Master Trigger 0: C26.1
- new net 2:8 Flex Clock Buffer3/Master Trigger 1: C40.1
- new net 2:8 Flex Clock Buffer30/Heimtime 0: C229.1
- new net 2:8 Flex Clock Buffer30/Heimtime 1: C231.1
- new net 2:8 Flex Clock Buffer30/Master Trigger 0: C278.1
- new net 2:8 Flex Clock Buffer30/Master Trigger 1: C232.1
- new net 2:8 Flex Clock Buffer31/Heimtime 0: C281.2
- new net 2:8 Flex Clock Buffer31/Heimtime 1: C283.2
- new net 2:8 Flex Clock Buffer31/Master Trigger 0: C282.1
- new net 2:8 Flex Clock Buffer31/Master Trigger 1: C236.1
- new net 2:8 Flex Clock Buffer32/Heimtime 0: C285.2
- new net 2:8 Flex Clock Buffer32/Heimtime 1: C287.2
- new net 2:8 Flex Clock Buffer32/Master Trigger 0: C238.1
- new net 2:8 Flex Clock Buffer32/Master Trigger 1: C288.1
- new net 2:8 Flex Clock Buffer33/Heimtime 0: C325.1
- new net 2:8 Flex Clock Buffer33/Heimtime 1: C375.2
- new net 2:8 Flex Clock Buffer33/Master Trigger 0: C374.1
- new net 2:8 Flex Clock Buffer33/Master Trigger 1: C328.1
- new net 2:8 Flex Clock Buffer34/Heimtime 0: C377.2
- new net 2:8 Flex Clock Buffer34/Heimtime 1: C331.1
- new net 2:8 Flex Clock Buffer34/Master Trigger 0: C330.1
- new net 2:8 Flex Clock Buffer34/Master Trigger 1: C332.1
- new net 2:8 Flex Clock Buffer35/Heimtime 0: C381.2
- new net 2:8 Flex Clock Buffer35/Heimtime 1: C383.2
- new net 2:8 Flex Clock Buffer35/Master Trigger 0: C382.1
- new net 2:8 Flex Clock Buffer35/Master Trigger 1: C384.1
- new net 2:8 Flex Clock Buffer36/Heimtime 0: C193.1
- new net 2:8 Flex Clock Buffer36/Heimtime 1: C195.1
- new net 2:8 Flex Clock Buffer36/Master Trigger 0: C242.1
- new net 2:8 Flex Clock Buffer36/Master Trigger 1: C244.1
- new net 2:8 Flex Clock Buffer37/Heimtime 0: C245.2
- new net 2:8 Flex Clock Buffer37/Heimtime 1: C199.1
- new net 2:8 Flex Clock Buffer37/Master Trigger 0: C246.1
- new net 2:8 Flex Clock Buffer37/Master Trigger 1: C248.1
- new net 2:8 Flex Clock Buffer38/Heimtime 0: C201.1
- new net 2:8 Flex Clock Buffer38/Heimtime 1: C251.2
- new net 2:8 Flex Clock Buffer38/Master Trigger 0: C250.1
- new net 2:8 Flex Clock Buffer38/Master Trigger 1: C204.1
- new net 2:8 Flex Clock Buffer39/Heimtime 0: C289.1
- new net 2:8 Flex Clock Buffer39/Heimtime 1: C339.2
- new net 2:8 Flex Clock Buffer39/Master Trigger 0: C338.1
- new net 2:8 Flex Clock Buffer39/Master Trigger 1: C340.1
- new net 2:8 Flex Clock Buffer4/Heimtime 0: C41.2
- new net 2:8 Flex Clock Buffer4/Heimtime 1: C31.1
- new net 2:8 Flex Clock Buffer4/Master Trigger 0: C42.1
- new net 2:8 Flex Clock Buffer4/Master Trigger 1: C44.1
- new net 2:8 Flex Clock Buffer40/Heimtime 0: C293.1
- new net 2:8 Flex Clock Buffer40/Heimtime 1: C295.1
- new net 2:8 Flex Clock Buffer40/Master Trigger 0: C294.1
- new net 2:8 Flex Clock Buffer40/Master Trigger 1: C296.1
- new net 2:8 Flex Clock Buffer41/Heimtime 0: C297.1
- new net 2:8 Flex Clock Buffer41/Heimtime 1: C347.2
- new net 2:8 Flex Clock Buffer41/Master Trigger 0: C298.1
- new net 2:8 Flex Clock Buffer41/Master Trigger 1: C300.1
- new net 2:8 Flex Clock Buffer42/Heimtime 0: C205.1
- new net 2:8 Flex Clock Buffer42/Heimtime 1: C255.2
- new net 2:8 Flex Clock Buffer42/Master Trigger 0: C206.1
- new net 2:8 Flex Clock Buffer42/Master Trigger 1: C256.1
- new net 2:8 Flex Clock Buffer43/Heimtime 0: C209.1
- new net 2:8 Flex Clock Buffer43/Heimtime 1: C259.2
- new net 2:8 Flex Clock Buffer43/Master Trigger 0: C210.1
- new net 2:8 Flex Clock Buffer43/Master Trigger 1: C260.1
- new net 2:8 Flex Clock Buffer44/Heimtime 0: C261.2
- new net 2:8 Flex Clock Buffer44/Heimtime 1: C215.1
- new net 2:8 Flex Clock Buffer44/Master Trigger 0: C262.1
- new net 2:8 Flex Clock Buffer44/Master Trigger 1: C264.1
- new net 2:8 Flex Clock Buffer45/Heimtime 0: C301.1
- new net 2:8 Flex Clock Buffer45/Heimtime 1: C303.1
- new net 2:8 Flex Clock Buffer45/Master Trigger 0: C350.1
- new net 2:8 Flex Clock Buffer45/Master Trigger 1: C304.1
- new net 2:8 Flex Clock Buffer46/Heimtime 0: C353.2
- new net 2:8 Flex Clock Buffer46/Heimtime 1: C355.2
- new net 2:8 Flex Clock Buffer46/Master Trigger 0: C354.1
- new net 2:8 Flex Clock Buffer46/Master Trigger 1: C356.1
- new net 2:8 Flex Clock Buffer47/Heimtime 0: C309.1
- new net 2:8 Flex Clock Buffer47/Heimtime 1: C311.1
- new net 2:8 Flex Clock Buffer47/Master Trigger 0: C358.1
- new net 2:8 Flex Clock Buffer47/Master Trigger 1: C312.1
- new net 2:8 Flex Clock Buffer5/Heimtime 0: C45.2
- new net 2:8 Flex Clock Buffer5/Heimtime 1: C35.1
- new net 2:8 Flex Clock Buffer5/Master Trigger 0: C46.1
- new net 2:8 Flex Clock Buffer5/Master Trigger 1: C48.1
- new net 2:8 Flex Clock Buffer6/Heimtime 0: C49.1
- new net 2:8 Flex Clock Buffer6/Heimtime 1: C51.1
- new net 2:8 Flex Clock Buffer6/Master Trigger 0: C50.1
- new net 2:8 Flex Clock Buffer6/Master Trigger 1: C52.1
- new net 2:8 Flex Clock Buffer7/Heimtime 0: C53.1
- new net 2:8 Flex Clock Buffer7/Heimtime 1: C55.1
- new net 2:8 Flex Clock Buffer7/Master Trigger 0: C54.1
- new net 2:8 Flex Clock Buffer7/Master Trigger 1: C56.1
- new net 2:8 Flex Clock Buffer8/Heimtime 0: C69.2
- new net 2:8 Flex Clock Buffer8/Heimtime 1: C71.2
- new net 2:8 Flex Clock Buffer8/Master Trigger 0: C70.1
- new net 2:8 Flex Clock Buffer8/Master Trigger 1: C72.1
- new net 2:8 Flex Clock Buffer9/Heimtime 0: C85.2
- new net 2:8 Flex Clock Buffer9/Heimtime 1: C87.2
- new net 2:8 Flex Clock Buffer9/Master Trigger 0: C74.1
- new net 2:8 Flex Clock Buffer9/Master Trigger 1: C88.1
- new net VMM3a_ASIC_0/Hybrid Ch.55: C81.2
- new net VMM3a_ASIC_0/Hybrid Ch.57: C353.1
- new net VMM3a_ASIC_0/Hybrid Ch.61: C74.2
- new net VMM3a_ASIC_0/Hybrid Ch.63: C282.2
- new net VMM3a_ASIC_1/Hybrid Ch.65: C311.2
- new net VMM3a_ASIC_1/Hybrid Ch.67: C355.1
- new net VMM3a_ASIC_1/Hybrid Ch.71: C12.2
- new net VMM3a_ASIC_1/Hybrid Ch.73: C180.2
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Other:
- note added: "Clock Distribution Unit"
- note removed: "Clock Distribution BOX"
Changed lines of the file:
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@@
 		)
 	)
-	(text "Clock Distribution BOX"
+	(text "Clock Distribution Unit"
 		(exclude_from_sim no)
 		(at 202.692 539.496 0)
