File: Spartan7_TriggerLogic/OpticalTransreciver_2layers/OpticalTransreciver_2layers/OpticalTransreciver_2layers.kicad_sch (KiCad schematic)
At the start: 24 parts, among them J1 Conn_01x05_Pin, U1 DS90LV011A, U2 DS90LV012ATMF

Commit message: .
Parts:
- removed C12, C13, C14, C15, C16, C17: 10u, Capacitor_SMD:C_0603_1608Metric, symbol Device:C
