File: Spartan7_TriggerLogic/trigger_scheme/trigger_scheme.kicad_sch (KiCad schematic)
At the start: 8 parts

Commit message: .
Connections:
- net 2:8 Flex AddOn/Heimtime 1 is gone; now on net VMM3a_ASIC_1/Hybrid Ch.67: C7.2
- net 2:8 Flex AddOn/Heimtime 0: now also C2.1; no longer C2.2
- net 2:8 Flex AddOn/Heimtime 1: now also C7.1; no longer C5.1
- net VMM3a_ASIC_0/Hybrid Ch.57: now also C2.2; no longer C2.1
- net VMM3a_ASIC_1/Hybrid Ch.67: no longer C7.1
- net 2:8 Flex AddOn/Master Trigger 0 renamed 2:8 Flex AddOn/Master Start 0 (x2)
- net 2:8 Flex AddOn/Master Trigger 1 renamed 2:8 Flex AddOn/Master Start 1 (x2)
- new net 2:8 Flex AddOn/Heimtime 1: C5.1
Other:
- sheet 2:6 Clock Buffer Pad Plane Adapter renamed 2:6 AddOn
- sheet 2:8 Flex Clock Buffer renamed 2:8 Flex AddOn
- sheet 2:6 AddOn ports: added Master Start, Master Start 1, Master Start 2, Master Start 3; removed Master Trigger, Master Trigger 1, Master Trigger 2, Master Trigger 3
- sheet 2:8 Flex AddOn ports: added Master Start, Master Start 0, Master Start 1; removed Master Trigger, Master Trigger 0, Master Trigger 1
- sheet HYDRA Clock Distribution Box ports: added Master Start 1, Master Start 16; removed Master Trigger 1, Master Trigger 16
- note added: "2:8 Flex AddOn"
- note removed: "500 fF"
