File: HYDRA_VMM3_Adapter_V3/HYDRA_VMM3_Adapter_V3.kicad_sch (KiCad schematic)
At the start: 32 parts, among them J1 ME1014010101011, J10 MCX-J-P-X-RA-SM1, J12 MCX-J-P-X-RA-SM1, J13 Conn_01x01_Socket, J14 Conn_01x01_Socket, J15 Conn_01x01_Socket, J16 Conn_01x01_Socket, J2 ME1014010101011, J3 ME1014010101011, J4 ME1014010101011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

Commit message: .
Parts:
- removed J10, J12, J8, J9: MCX-J-P-X-RA-SM1, PCI-E_SMD:SAMTEC_MCX-J-P-X-RA-SM1, symbol MCX_Coax:MCX-J-P-X-RA-SM1
- added J7, J8: Conn_01x08_Socket, Components:2_in_6_out_module, symbol Connector:Conn_01x08_Socket
Connections:
- net GND: now also J7.2 (Pin_2), J8.2 (Pin_2)
- net Heimtime_A: now also J8.4 (Pin_4), J8.6 (Pin_6), J8.8 (Pin_8)
- net Heimtime_B: now also J7.4 (Pin_4), J7.6 (Pin_6), J7.8 (Pin_8)
- net Master_Trigg_A: now also J8.3 (Pin_3), J8.5 (Pin_5), J8.7 (Pin_7)
- net Master_Trigg_B: now also J7.3 (Pin_3), J7.5 (Pin_5), J7.7 (Pin_7)
- net P1A: now also J8.1 (Pin_1)
- net P1B: now also J7.1 (Pin_1)
Other:
- removed sheet FIFO

Commit message: .
Other:
- note added: "NOTE: The 16x88 connector is build by using 2x5x88 and 1x6x88 connectors with serial numbers ESQT-144-03-F-5-375 and ESQT-144-03-F-6-375."
Changed lines of the file:
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@@
 (kicad_sch
-	(version 20231120)
+	(version 20250114)
 	(generator "eeschema")
-	(generator_version "8.0")
+	(generator_version "9.0")
 	(paper "A3")
 	(title_block
@@
 		(comment 1 "AUTOR: Alexandru Enciu")
 	)
+	(text "NOTE: The 16x88 connector is build by using 2x5x88 and 1x6x88 connectors with \nserial numbers ESQT-144-03-F-5-375 and ESQT-144-03-F-6-375."
+		(exclude_from_sim no)
+		(at 364.236 246.634 0)
+		(effects
+			(font
+				(size 1.27 1.27)
+				(thickness 0.254)
+				(bold yes)
+			)
+		)
+	)
 	(junction
 		(at 68.58 224.79)
@@
 	)
 	(sheet
-		(at 374.65 220.98)
+		(at 347.98 222.25)
 		(size 25.4 17.78)
+		(exclude_from_sim no)
+		(in_bom yes)
+		(on_board yes)
+		(dnp no)
 		(fields_autoplaced yes)
 		(stroke
@@
 		)
 		(property "Sheetname" "TPC_Adapter"
-			(at 374.65 220.2446 0)
+			(at 347.98 221.5146 0)
 			(effects
 				(font
@@
 		)
 		(property "Sheetfile" "TPC_Adapter.kicad_sch"
-			(at 374.65 239.3684 0)
+			(at 347.98 240.6384 0)
 			(effects
 				(font
@@
 		)
 	)
+	(embedded_fonts no)
 )
